File: hardware/AEL2005.sch (KiCad schematic (older format))
At the start: 0 parts

Commit message: Fill in 10GE interface (WIP)
Parts:
- added C? (x20): C_Small, symbol C_Small
- added D? (x2): LED, symbol LED
- added P?: CONN_01X05 (DNP), symbol CONN_01X05
- added P?: CONN_01X06 (DNP), symbol CONN_01X06
- added R? (x13): DNP, symbol R
- added R? (x6): 0, symbol R
- added R?: 820, symbol R
- added R?: 300, symbol R
- added R?: 11k8, symbol R
- added R? (x8): 10k, symbol R
- added R? (x5): R, symbol R
- added U?: AEL2005, symbol AEL2005
- added W? (x4): TEST_1P, symbol TEST_1P
Connections:
- net labels added: +1V2, +3V3, AEL_CLK_N, AEL_CLK_P, AEL_RESET, GND, HSRXDATA_N, HSRXDATA_P, HSTXDATA_N, HSTXDATA_P, MDC, MDIO, MODDET, RXDATA[0]_N, RXDATA[0]_P, RXDATA[1]_N, RXDATA[1]_P, RXDATA[2]_N, RXDATA[2]_P, RXDATA[3]_N, RXDATA[3]_P, RX_LOS, SFP_GPIO, SFP_SCL, SFP_SDA, TXDATA[0]_N, TXDATA[0]_P, TXDATA[1]_N, TXDATA[1]_P, TXDATA[2]_N, TXDATA[2]_P, TXDATA[3]_N, TXDATA[3]_P, TX_DISABLE, TX_FAULT
- wire segments 0 -> 131
