File: hardware/AEL2005.sch (KiCad schematic (older format))
At the start: 64 parts

Commit message: Change 10GE interface phy to TLK10031
Low speed signals are still missing. Low speed signals from sfp+ part now need to be connected to the fpga. The new Phy does not support i2c etc..

Also changed KiCad Version to 4.0.7
Parts:
- P?: symbol CONN_01X05 -> Conn_01x05
- P?: symbol CONN_01X06 -> Conn_01x06
Changed lines of the file:
@@
 EESchema Schematic File Version 2
+LIBS:zynq_board-rescue
 LIBS:power
 LIBS:device
@@
 $Descr A4 11693 8268
 encoding utf-8
-Sheet 9 18
+Sheet 9 20
 Title ""
 Date ""
@@
 $EndComp
 $Comp
-L CONN_01X05 P?
+L Conn_01x05 P?
 U 1 1 59742E43
 P 9450 5600
+AR Path="/59742E43" Ref="P?"  Part="1"
+AR Path="/596E816C/59742E43" Ref="P?"  Part="1"
 F 0 "P?" H 9450 5900 50  0000 C CNN
 F 1 "CONN_01X05 (DNP)" V 9550 5600 50  0000 C CNN
@@
 $EndComp
 $Comp
-L CONN_01X06 P?
+L Conn_01x06 P?
 U 1 1 59744178
 P 10000 3850
+AR Path="/59744178" Ref="P?"  Part="1"
+AR Path="/596E816C/59744178" Ref="P?"  Part="1"
 F 0 "P?" H 10000 4200 50  0000 C CNN
 F 1 "CONN_01X06 (DNP)" V 10100 3850 50  0000 C CNN
