File: hardware/cam_conn.sch (KiCad schematic (older format))
At the start: 0 parts

Commit message: Added lshm-150 symbol
Parts:
- added J?: LSHM-150-xxx-x-DV-A-S, symbol LSHM-150-xxx-x-DV-A-S
Changed lines of the file:
@@
 LIBS:misc
 LIBS:tlk10031
+LIBS:lshm-150-xxx-x-dv-a-s
 LIBS:zynq_board-cache
 EELAYER 25 0
@@
 Text Notes 950  4750 0    60   ~ 0
 Open questions\n* LVDS clock input to camera needed?\n* Two separate clocks for two cameras needed?\n\nMissing\n* I2C\n* GPIO
+$Comp
+L LSHM-150-xxx-x-DV-A-S J?
+U 1 1 5ACC34F1
+P 7700 3550
+F 0 "J?" H 7700 1000 60  0000 C CNN
+F 1 "LSHM-150-xxx-x-DV-A-S" V 7700 3550 60  0000 C CNN
+F 2 "" H 7700 4700 60  0001 C CNN
+F 3 "" H 7700 4700 60  0001 C CNN
+	1    7700 3550
+	1    0    0    -1
+$EndComp
 $EndSCHEMATC

Commit message: Almost drew 3,3 V lowspeed signals. Added Levelshifter Subschematic
1,8 V Lowspeed Singals from 10 G Phy to FPGA are still missing.

CAM_REF_CLK is not really low speed, maybe we should consider to use the lvds clock instead. I think it will work, since the signal should be realtive short(FPGA->Connector->Camerasensor[->Camerasensor2]). The levelshifter should also be fast enough.

The i2c signals use simple N-Channel MOSTFET Transistors for Levelshifting
Connections:
- net labels added: SCL, SDA
Other:
- note added: "Afaik is LVDS Clock optional"
- note added: "Open questions\n* LVDS clock input to camera needed?\n* Two separate clocks for two cameras needed?\n\nMissing\n!* I2C\n* GPIO"
- note removed: "Open questions\n* LVDS clock input to camera needed?\n* Two separate clocks for two cameras needed?\n\nMissing\n* I2C\n* GPIO"
Changed lines of the file:
@@
 LIBS:tlk10031
 LIBS:lshm-150-xxx-x-dv-a-s
+LIBS:sn74axc8t245
 LIBS:zynq_board-cache
 EELAYER 25 0
@@
 $Descr A4 11693 8268
 encoding utf-8
-Sheet 8 18
+Sheet 18 19
 Title ""
 Date ""
@@
 Comment4 ""
 $EndDescr
-Text HLabel 1550 2200 0    60   Output ~ 0
+Text HLabel 1550 1600 0    60   Output ~ 0
 CAM_CLK_1_N
-Text HLabel 1550 1850 0    60   Output ~ 0
+Text HLabel 1550 1250 0    60   Output ~ 0
 CAM_CLK_0_P
-Text HLabel 1550 1950 0    60   Output ~ 0
+Text HLabel 1550 1350 0    60   Output ~ 0
 CAM_CLK_0_N
-Text HLabel 1550 2100 0    60   Output ~ 0
+Text HLabel 1550 1500 0    60   Output ~ 0
 CAM_CLK_1_P
-Text HLabel 1550 1200 0    60   Output ~ 0
+Text HLabel 1550 600  0    60   Output ~ 0
 CAM_DATA
 Entry Wire Line
+	5600 2500 5700 2600
+Entry Wire Line
+	5600 1100 5700 1200
+Entry Wire Line
+	5600 1200 5700 1300
+Entry Wire Line
+	5600 1300 5700 1400
+Entry Wire Line
+	5600 1400 5700 1500
+Entry Wire Line
+	5600 1500 5700 1600
+Entry Wire Line
+	5600 1600 5700 1700
+Entry Wire Line
+	5600 1700 5700 1800
+Entry Wire Line
+	5600 1800 5700 1900
+Entry Wire Line
+	5600 1900 5700 2000
+Entry Wire Line
+	5600 2000 5700 2100
+Entry Wire Line
+	5600 2100 5700 2200
+Entry Wire Line
+	5600 2200 5700 2300
+Entry Wire Line
+	5600 2300 5700 2400
+Entry Wire Line
+	5600 2400 5700 2500
+Text Label 5800 1300 0    60   ~ 0
+D0_N
+Text Label 5800 1200 0    60   ~ 0
+D0_P
+Text Label 5800 1500 0    60   ~ 0
+D1_N
+Text Label 5800 1400 0    60   ~ 0
+D1_P
+Text Label 5800 1700 0    60   ~ 0
+D2_N
+Text Label 5800 1600 0    60   ~ 0
+D2_P
+Text Label 5800 1900 0    60   ~ 0
+D3_N
+Text Label 5800 1800 0    60   ~ 0
+D3_P
+Text Label 5800 2100 0    60   ~ 0
+D4_N
+Text Label 5800 2000 0    60   ~ 0
+D4_P
+Text Label 5800 2300 0    60   ~ 0
+D5_N
+Text Label 5800 2200 0    60   ~ 0
+D5_P
+Text Label 5800 2500 0    60   ~ 0
+D6_N
+Text Label 5800 2400 0    60   ~ 0
+D6_P
+Text Label 5800 2700 0    60   ~ 0
+D7_N
+Text Label 5800 2600 0    60   ~ 0
+D7_P
+Text Label 5800 2900 0    60   ~ 0
+D8_N
+Text Label 5800 2800 0    60   ~ 0
+D8_P
+Text Label 5800 3100 0    60   ~ 0
+D9_N
+Text Label 5800 3000 0    60   ~ 0
+D9_P
+Text Label 5800 3300 0    60   ~ 0
+D10_N
+Text Label 5800 3200 0    60   ~ 0
+D10_P
+Text Label 5800 3500 0    60   ~ 0
+D11_N
+Text Label 5800 3400 0    60   ~ 0
+D11_P
+Text Label 5800 3700 0    60   ~ 0
+D12_N
+Text Label 5800 3600 0    60   ~ 0
+D12_P
+Text Label 5800 3900 0    60   ~ 0
+D13_N
+Text Label 5800 3800 0    60   ~ 0
+D13_P
+Text Label 5800 4100 0    60   ~ 0
+D14_N
+Text Label 5800 4000 0    60   ~ 0
+D14_P
+Text Label 5800 4300 0    60   ~ 0
+D15_N
+Text Label 5800 4200 0    60   ~ 0
+D15_P
+Entry Wire Line
+	5600 2600 5700 2700
+Entry Wire Line
+	5600 2700 5700 2800
+Entry Wire Line
+	5600 2800 5700 2900
+Entry Wire Line
+	5600 2900 5700 3000
+Entry Wire Line
+	5600 3000 5700 3100
+Entry Wire Line
 	5600 3100 5700 3200
 Entry Wire Line
-	5600 1700 5700 1800
-Entry Wire Line
-	5600 1800 5700 1900
-Entry Wire Line
-	5600 1900 5700 2000
-Entry Wire Line
-	5600 2000 5700 2100
-Entry Wire Line
-	5600 2100 5700 2200
-Entry Wire Line
-	5600 2200 5700 2300
-Entry Wire Line
-	5600 2300 5700 2400
-Entry Wire Line
-	5600 2400 5700 2500
-Entry Wire Line
-	5600 2500 5700 2600
-Entry Wire Line
-	5600 2600 5700 2700
-Entry Wire Line
-	5600 2700 5700 2800
-Entry Wire Line
-	5600 2800 5700 2900
-Entry Wire Line
-	5600 2900 5700 3000
-Entry Wire Line
-	5600 3000 5700 3100
-Text Label 5800 1900 0    60   ~ 0
-D0_N
-Text Label 5800 1800 0    60   ~ 0
-D0_P
-Text Label 5800 2100 0    60   ~ 0
-D1_N
-Text Label 5800 2000 0    60   ~ 0
-D1_P
-Text Label 5800 2300 0    60   ~ 0
-D2_N
-Text Label 5800 2200 0    60   ~ 0
-D2_P
-Text Label 5800 2500 0    60   ~ 0
-D3_N
-Text Label 5800 2400 0    60   ~ 0
-D3_P
-Text Label 5800 2700 0    60   ~ 0
-D4_N
-Text Label 5800 2600 0    60   ~ 0
-D4_P
-Text Label 5800 2900 0    60   ~ 0
-D5_N
-Text Label 5800 2800 0    60   ~ 0
-D5_P
-Text Label 5800 3100 0    60   ~ 0
-D6_N
-Text Label 5800 3000 0    60   ~ 0
-D6_P
-Text Label 5800 3300 0    60   ~ 0
-D7_N
-Text Label 5800 3200 0    60   ~ 0
-D7_P
-Text Label 5800 3500 0    60   ~ 0
-D8_N
-Text Label 5800 3400 0    60   ~ 0
-D8_P
-Text Label 5800 3700 0    60   ~ 0
-D9_N
-Text Label 5800 3600 0    60   ~ 0
-D9_P
-Text Label 5800 3900 0    60   ~ 0
-D10_N
-Text Label 5800 3800 0    60   ~ 0
-D10_P
-Text Label 5800 4100 0    60   ~ 0
-D11_N
-Text Label 5800 4000 0    60   ~ 0
-D11_P
-Text Label 5800 4300 0    60   ~ 0
-D12_N
-Text Label 5800 4200 0    60   ~ 0
-D12_P
-Text Label 5800 4500 0    60   ~ 0
-D13_N
-Text Label 5800 4400 0    60   ~ 0
-D13_P
-Text Label 5800 4700 0    60   ~ 0
-D14_N
-Text Label 5800 4600 0    60   ~ 0
-D14_P
-Text Label 5800 4900 0    60   ~ 0
-D15_N
-Text Label 5800 4800 0    60   ~ 0
-D15_P
-Entry Wire Line
 	5600 3200 5700 3300
 Entry Wire Line
@@
 Entry Wire Line
 	5600 4200 5700 4300
-Entry Wire Line
-	5600 4300 5700 4400
-Entry Wire Line
-	5600 4400 5700 4500
-Entry Wire Line
-	5600 4500 5700 4600
-Entry Wire Line
-	5600 4600 5700 4700
-Entry Wire Line
-	5600 4700 5700 4800
-Entry Wire Line
-	5600 4800 5700 4900
+Wire Wire Line
+	5700 1200 5800 1200
+Wire Wire Line
+	5700 1300 5800 1300
+Wire Wire Line
+	5700 1400 5800 1400
+Wire Wire Line
+	5800 1500 5700 1500
+Wire Wire Line
+	5700 1600 5800 1600
+Wire Wire Line
+	5800 1700 5700 1700
 Wire Wire Line
 	5700 1800 5800 1800
 Wire Wire Line
-	5700 1900 5800 1900
+	5800 1900 5700 1900
 Wire Wire Line
 	5700 2000 5800 2000
 Wire Wire Line
-	5800 2100 5700 2100
-Wire Wire Line
-	5700 2200 5800 2200
-Wire Wire Line
-	5800 2300 5700 2300
-Wire Wire Line
-	5700 2400 5800 2400
-Wire Wire Line
-	5800 2500 5700 2500
-Wire Wire Line
-	5700 2600 5800 2600
+	5700 2100 5800 2100
+Wire Wire Line
+	5800 2200 5700 2200
+Wire Wire Line
+	5700 2300 5800 2300
+Wire Wire Line
+	5800 2400 5700 2400
+Wire Wire Line
+	5700 2500 5800 2500
+Wire Wire Line
+	5800 2600 5700 2600
 Wire Wire Line
 	5700 2700 5800 2700
@@
 	5800 3400 5700 3400
 Wire Wire Line
-	5700 3500 5800 3500
-Wire Wire Line
-	5800 3600 5700 3600
-Wire Wire Line
-	5700 3700 5800 3700
-Wire Wire Line
-	5800 3800 5700 3800
-Wire Wire Line
-	5700 3900 5800 3900
-Wire Wire Line
-	5800 4000 5700 4000
+	5800 3500 5700 3500
+Wire Wire Line
+	5700 3600 5800 3600
+Wire Wire Line
+	5800 3700 5700 3700
+Wire Wire Line
+	5700 3800 5800 3800
+Wire Wire Line
+	5800 3900 5700 3900
+Wire Wire Line
+	5700 4000 5800 4000
 Wire Wire Line
 	5800 4100 5700 4100
@@
 Wire Wire Line
 	5800 4300 5700 4300
-Wire Wire Line
-	5700 4400 5800 4400
-Wire Wire Line
-	5800 4500 5700 4500
-Wire Wire Line
-	5700 4600 5800 4600
-Wire Wire Line
-	5800 4700 5700 4700
-Wire Wire Line
-	5700 4800 5800 4800
-Wire Wire Line
-	5800 4900 5700 4900
 Wire Bus Line
-	5600 4800 5600 1200
+	5600 4200 5600 600
 Wire Bus Line
-	5600 1200 1550 1200
-Text HLabel 1550 2500 0    60   Input ~ 0
+	5600 600  1550 600
+Text HLabel 1550 1900 0    60   Input ~ 0
 FRAME_REQ_0
-Text HLabel 1550 2850 0    60   Input ~ 0
+Text HLabel 1550 2250 0    60   Input ~ 0
 FRAME_REQ_1
-Text HLabel 1550 2600 0    60   Input ~ 0
+Text HLabel 1550 2000 0    60   Input ~ 0
 T_EXP1_0
+Text HLabel 1550 2100 0    60   Input ~ 0
+T_EXP2_0
+Text HLabel 1550 2350 0    60   Input ~ 0
+T_EXP1_1
+Text HLabel 1550 2450 0    60   Input ~ 0
+T_EXP2_1
+Text HLabel 1550 750  0    60   Output ~ 0
+CAM_CTRL_0_P
+Text HLabel 1550 850  0    60   Output ~ 0
+CAM_CTRL_0_N
+Text HLabel 1550 1000 0    60   Output ~ 0
+CAM_CTRL_1_P
+Text HLabel 1550 1100 0    60   Output ~ 0
+CAM_CTRL_1_N
+Text HLabel 1550 2600 0    60   Output ~ 0
+SPI_MISO
 Text HLabel 1550 2700 0    60   Input ~ 0
-T_EXP2_0
+SPI_MOSI
+Text HLabel 1550 2800 0    60   Input ~ 0
+SPI_CLK
 Text HLabel 1550 2950 0    60   Input ~ 0
-T_EXP1_1
+SPI_EN_0
 Text HLabel 1550 3050 0    60   Input ~ 0
-T_EXP2_1
-Text HLabel 1550 1350 0    60   Output ~ 0
-CAM_CTRL_0_P
-Text HLabel 1550 1450 0    60   Output ~ 0
-CAM_CTRL_0_N
-Text HLabel 1550 1600 0    60   Output ~ 0
-CAM_CTRL_1_P
-Text HLabel 1550 1700 0    60   Output ~ 0
-CAM_CTRL_1_N
-Text HLabel 1550 3200 0    60   Output ~ 0
-SPI_MISO
-Text HLabel 1550 3300 0    60   Input ~ 0
-SPI_MOSI
-Text HLabel 1550 3400 0    60   Input ~ 0
-SPI_CLK
-Text HLabel 1550 3550 0    60   Input ~ 0
-SPI_EN_0
-Text HLabel 1550 3650 0    60   Input ~ 0
 SPI_EN_1
-Text HLabel 1550 3800 0    60   Input ~ 0
+Text HLabel 1550 3200 0    60   Input ~ 0
 ~CAM_RESET~
-Text HLabel 1550 2350 0    60   Input ~ 0
+Text HLabel 1550 1750 0    60   Input ~ 0
 CAM_CLK_REF
-Text Notes 950  4750 0    60   ~ 0
-Open questions\n* LVDS clock input to camera needed?\n* Two separate clocks for two cameras needed?\n\nMissing\n* I2C\n* GPIO
+Text Notes 900  6900 0    60   ~ 0
+Open questions\n* LVDS clock input to camera needed?\n* Two separate clocks for two cameras needed?\n\nMissing\n!* I2C\n* GPIO
 $Comp
 L LSHM-150-xxx-x-DV-A-S J?
@@
 	1    0    0    -1
 $EndComp
+Text HLabel 1550 3400 0    60   BiDi ~ 0
+SDA
+Text HLabel 1550 3500 0    60   BiDi ~ 0
+SCL
+Text Notes 3350 6450 0    60   ~ 0
+Afaik is LVDS Clock optional
 $EndSCHEMATC

Commit message: Drew Camera Connector part.
There is some space left on the connector. So it is still possible to add two lvds clocks for the Cameras
Connections:
- net labels added: +5V, GND
- wire segments 32 -> 99

Commit message: KiCad does not support differential Busses yet. See https://bugs.launchpad.net/kicad/+bug/1419146. Fixed Data Lanes for Camera Connector.
Parts:
- J?: footprint (none) -> Connectors_Samtec:LSHM-150-xxx-x-DV-A-S
Connections:
- net labels removed: CAM_DATA
Changed lines of the file:
@@
 Text HLabel 7450 3950 0    60   Output ~ 0
 CAM_CLK_1_P
-Text HLabel 1600 950  0    60   Output ~ 0
-CAM_DATA
-Entry Wire Line
-	5650 3550 5750 3650
-Entry Wire Line
-	5650 1450 5750 1550
-Entry Wire Line
-	5650 1550 5750 1650
-Entry Wire Line
-	5650 1750 5750 1850
-Entry Wire Line
-	5650 1850 5750 1950
-Entry Wire Line
-	5650 2050 5750 2150
-Entry Wire Line
-	5650 2150 5750 2250
-Entry Wire Line
-	5650 2350 5750 2450
-Entry Wire Line
-	5650 2450 5750 2550
-Entry Wire Line
-	5650 2650 5750 2750
-Entry Wire Line
-	5650 2750 5750 2850
-Entry Wire Line
-	5650 2950 5750 3050
-Entry Wire Line
-	5650 3050 5750 3150
-Entry Wire Line
-	5650 3250 5750 3350
-Entry Wire Line
-	5650 3350 5750 3450
-Text Label 5850 1650 0    60   ~ 0
-D0_N
-Text Label 5850 1550 0    60   ~ 0
-D0_P
-Text Label 5850 1950 0    60   ~ 0
-D1_N
-Text Label 5850 1850 0    60   ~ 0
-D1_P
-Text Label 5850 2250 0    60   ~ 0
-D2_N
-Text Label 5850 2150 0    60   ~ 0
-D2_P
-Text Label 5850 2550 0    60   ~ 0
-D3_N
-Text Label 5850 2450 0    60   ~ 0
-D3_P
-Text Label 5850 2850 0    60   ~ 0
-D4_N
-Text Label 5850 2750 0    60   ~ 0
-D4_P
-Text Label 5850 3150 0    60   ~ 0
-D5_N
-Text Label 5850 3050 0    60   ~ 0
-D5_P
-Text Label 5850 3450 0    60   ~ 0
-D6_N
-Text Label 5850 3350 0    60   ~ 0
-D6_P
-Text Label 5850 3750 0    60   ~ 0
-D7_N
-Text Label 5850 3650 0    60   ~ 0
-D7_P
-Text Label 5850 4650 0    60   ~ 0
-D8_N
-Text Label 5850 4550 0    60   ~ 0
-D8_P
-Text Label 5850 4950 0    60   ~ 0
-D9_N
-Text Label 5850 4850 0    60   ~ 0
-D9_P
-Text Label 5850 5250 0    60   ~ 0
-D10_N
-Text Label 5850 5150 0    60   ~ 0
-D10_P
-Text Label 5850 5550 0    60   ~ 0
-D11_N
-Text Label 5850 5450 0    60   ~ 0
-D11_P
-Text Label 5850 5850 0    60   ~ 0
-D12_N
-Text Label 5850 5750 0    60   ~ 0
-D12_P
-Text Label 9900 5750 0    60   ~ 0
-D13_N
-Text Label 9900 5850 0    60   ~ 0
-D13_P
-Text Label 9900 5450 0    60   ~ 0
-D14_N
-Text Label 9900 5550 0    60   ~ 0
-D14_P
-Text Label 9900 5150 0    60   ~ 0
-D15_N
-Text Label 9900 5250 0    60   ~ 0
-D15_P
-Entry Wire Line
-	5650 3650 5750 3750
-Entry Wire Line
-	5650 4450 5750 4550
-Entry Wire Line
-	5650 4550 5750 4650
-Entry Wire Line
-	5650 4750 5750 4850
-Entry Wire Line
-	5650 4850 5750 4950
-Entry Wire Line
-	5650 5050 5750 5150
-Entry Wire Line
-	5650 5150 5750 5250
-Entry Wire Line
-	5650 5350 5750 5450
-Entry Wire Line
-	5650 5450 5750 5550
-Entry Wire Line
-	5650 5650 5750 5750
-Entry Wire Line
-	5650 5750 5750 5850
-Entry Wire Line
-	10250 5550 10350 5650
-Entry Wire Line
-	10250 5450 10350 5550
-Entry Wire Line
-	10250 5250 10350 5350
-Entry Wire Line
-	10250 5150 10350 5250
 Text HLabel 9350 4750 2    60   Input ~ 0
 FRAME_REQ_0
@@
 F 0 "J?" H 8350 850 60  0000 C CNN
 F 1 "LSHM-150-xxx-x-DV-A-S" V 8350 3400 60  0000 C CNN
-F 2 "" H 8350 4550 60  0001 C CNN
+F 2 "Connectors_Samtec:LSHM-150-xxx-x-DV-A-S" H 8350 4550 60  0001 C CNN
 F 3 "" H 8350 4550 60  0001 C CNN
 	1    8350 3400
@@
 Text HLabel 9400 2650 2    60   BiDi ~ 0
 SCL
-Text Notes 3350 6450 0    60   ~ 0
+Text Notes 3250 6400 0    60   ~ 0
 Afaik is LVDS Clock optional
-Entry Wire Line
-	10250 5850 10350 5950
-Entry Wire Line
-	10250 5750 10350 5850
-Wire Wire Line
-	5750 1550 8050 1550
-Wire Bus Line
-	5650 950  5650 6300
-Wire Bus Line
-	5650 950  1600 950
 Wire Wire Line
 	8050 950  7450 950
@@
 	8050 1350 7450 1350
 Wire Wire Line
-	5750 1650 8050 1650
-Wire Wire Line
-	5750 1850 8050 1850
-Wire Wire Line
-	5750 1950 8050 1950
-Wire Wire Line
-	5750 2150 8050 2150
-Wire Wire Line
-	5750 2250 8050 2250
-Wire Wire Line
-	5750 2450 8050 2450
-Wire Wire Line
-	5750 2550 8050 2550
-Wire Wire Line
-	5750 2750 8050 2750
-Wire Wire Line
-	5750 2850 8050 2850
-Wire Wire Line
-	5750 3050 8050 3050
-Wire Wire Line
-	5750 3150 8050 3150
-Wire Wire Line
-	5750 3350 8050 3350
-Wire Wire Line
-	5750 3450 8050 3450
-Wire Wire Line
-	5750 3650 8050 3650
-Wire Wire Line
-	5750 3750 8050 3750
-Wire Wire Line
 	7450 3950 8050 3950
 Wire Wire Line
@@
 Wire Wire Line
 	7450 4350 8050 4350
-Wire Wire Line
-	5750 4550 8050 4550
-Wire Wire Line
-	5750 4650 8050 4650
-Wire Wire Line
-	5750 4850 8050 4850
-Wire Wire Line
-	8050 4950 5750 4950
-Wire Wire Line
-	5750 5150 8050 5150
-Wire Wire Line
-	8050 5250 5750 5250
-Wire Wire Line
-	5750 5450 8050 5450
-Wire Wire Line
-	5750 5550 8050 5550
-Wire Wire Line
-	5750 5750 8050 5750
-Wire Wire Line
-	5750 5850 8050 5850
-Wire Wire Line
-	8650 5850 10250 5850
-Wire Wire Line
-	10250 5750 8650 5750
-Wire Wire Line
-	10250 5550 8650 5550
-Wire Wire Line
-	8650 5450 10250 5450
-Wire Wire Line
-	8650 5250 10250 5250
-Wire Wire Line
-	10250 5150 8650 5150
-Wire Bus Line
-	10350 5250 10350 6300
 Wire Wire Line
 	9350 4950 8650 4950
@@
 	8650 2750 8850 2750
 Connection ~ 8850 2750
-Wire Bus Line
-	10350 6300 5650 6300
 $Comp
 L GND #PWR?
@@
 $EndComp
 Connection ~ 8850 950
+Text HLabel 7450 1550 0    60   Output ~ 0
+D0_N
+Text HLabel 7450 1650 0    60   Output ~ 0
+D0_P
+Text HLabel 7450 1850 0    60   Output ~ 0
+D1_N
+Text HLabel 7450 1950 0    60   Output ~ 0
+D1_P
+Text HLabel 7450 2150 0    60   Output ~ 0
+D2_N
+Text HLabel 7450 2250 0    60   Output ~ 0
+D2_P
+Text HLabel 7450 2450 0    60   Output ~ 0
+D3_N
+Text HLabel 7450 2550 0    60   Output ~ 0
+D3_P
+Text HLabel 7450 2750 0    60   Output ~ 0
+D4_N
+Text HLabel 7450 2850 0    60   Output ~ 0
+D4_P
+Text HLabel 7450 3050 0    60   Output ~ 0
+D5_N
+Text HLabel 7450 3150 0    60   Output ~ 0
+D5_P
+Text HLabel 7450 3350 0    60   Output ~ 0
+D6_N
+Text HLabel 7450 3450 0    60   Output ~ 0
+D6_P
+Text HLabel 7450 3650 0    60   Output ~ 0
+D7_N
+Text HLabel 7450 3750 0    60   Output ~ 0
+D7_P
+Text HLabel 7450 4550 0    60   Output ~ 0
+D8_N
+Text HLabel 7450 4650 0    60   Output ~ 0
+D8_P
+Text HLabel 7450 4850 0    60   Output ~ 0
+D9_N
+Text HLabel 7450 4950 0    60   Output ~ 0
+D9_P
+Text HLabel 7450 5150 0    60   Output ~ 0
+D10_N
+Text HLabel 7450 5250 0    60   Output ~ 0
+D10_P
+Text HLabel 7450 5450 0    60   Output ~ 0
+D11_N
+Text HLabel 7450 5550 0    60   Output ~ 0
+D11_P
+Text HLabel 7450 5750 0    60   Output ~ 0
+D12_N
+Text HLabel 7450 5850 0    60   Output ~ 0
+D12_P
+Text HLabel 9400 5850 2    60   Output ~ 0
+D13_N
+Text HLabel 9400 5750 2    60   Output ~ 0
+D13_P
+Text HLabel 9400 5550 2    60   Output ~ 0
+D14_N
+Text HLabel 9400 5450 2    60   Output ~ 0
+D14_P
+Text HLabel 9400 5250 2    60   Output ~ 0
+D15_N
+Text HLabel 9400 5150 2    60   Output ~ 0
+D15_P
+Wire Wire Line
+	7450 1550 8050 1550
+Wire Wire Line
+	8050 1650 7450 1650
+Wire Wire Line
+	7450 1850 8050 1850
+Wire Wire Line
+	8050 1950 7450 1950
+Wire Wire Line
+	7450 2150 8050 2150
+Wire Wire Line
+	8050 2250 7450 2250
+Wire Wire Line
+	7450 2450 8050 2450
+Wire Wire Line
+	8050 2550 7450 2550
+Wire Wire Line
+	7450 2750 8050 2750
+Wire Wire Line
+	8050 2850 7450 2850
+Wire Wire Line
+	8050 3050 7450 3050
+Wire Wire Line
+	7450 3150 8050 3150
+Wire Wire Line
+	8050 3350 7450 3350
+Wire Wire Line
+	7450 3450 8050 3450
+Wire Wire Line
+	8050 3650 7450 3650
+Wire Wire Line
+	7450 3750 8050 3750
+Wire Wire Line
+	8050 4550 7450 4550
+Wire Wire Line
+	7450 4650 8050 4650
+Wire Wire Line
+	8050 4850 7450 4850
+Wire Wire Line
+	7450 4950 8050 4950
+Wire Wire Line
+	8050 5150 7450 5150
+Wire Wire Line
+	7450 5250 8050 5250
+Wire Wire Line
+	8050 5450 7450 5450
+Wire Wire Line
+	7450 5550 8050 5550
+Wire Wire Line
+	8050 5750 7450 5750
+Wire Wire Line
+	7450 5850 8050 5850
+Wire Wire Line
+	8650 5850 9400 5850
+Wire Wire Line
+	9400 5750 8650 5750
+Wire Wire Line
+	8650 5550 9400 5550
+Wire Wire Line
+	9400 5450 8650 5450
+Wire Wire Line
+	8650 5250 9400 5250
+Wire Wire Line
+	9400 5150 8650 5150
 $EndSCHEMATC
