File: hardware/cam_conn.sch (KiCad schematic (older format))
At the start: 1 part

Commit message: Added Second SPI Bus for IMUs to Cam Connector
This SPI works on 1.8 V, don't confuse them. If this second SPI Bus shall be used for the Cam Chips, add Levelshifters on the Cam Board.

Also reorderd some stuff around this connector, to ease routing
Connections:
- net labels added: IMU_SPI_CLK, IMU_SPI_EN_0, IMU_SPI_EN_1, IMU_SPI_MISO, IMU_SPI_MOSI
- wire segments 99 -> 104
Other:
- note added: "1.8 V only"
Changed lines of the file:
@@
 LIBS:lshm-150-xxx-x-dv-a-s
 LIBS:sn74axc8t245
+LIBS:sn74lvc2t45
 LIBS:zynq_board-cache
 EELAYER 25 0
@@
 $Descr A4 11693 8268
 encoding utf-8
-Sheet 18 19
+Sheet 20 20
 Title ""
 Date ""
@@
 Text HLabel 7450 3950 0    60   Output ~ 0
 CAM_CLK_1_P
-Text HLabel 9350 4750 2    60   Input ~ 0
+Text HLabel 9400 4950 2    60   Input ~ 0
 FRAME_REQ_0
-Text HLabel 9350 4350 2    60   Input ~ 0
+Text HLabel 9400 4550 2    60   Input ~ 0
 FRAME_REQ_1
-Text HLabel 9350 4650 2    60   Input ~ 0
+Text HLabel 9400 4850 2    60   Input ~ 0
 T_EXP1_0
-Text HLabel 9350 4550 2    60   Input ~ 0
+Text HLabel 9400 4750 2    60   Input ~ 0
 T_EXP2_0
-Text HLabel 9350 4250 2    60   Input ~ 0
+Text HLabel 9400 4450 2    60   Input ~ 0
 T_EXP1_1
-Text HLabel 9350 4150 2    60   Input ~ 0
+Text HLabel 9400 4350 2    60   Input ~ 0
 T_EXP2_1
 Text HLabel 7450 1250 0    60   Output ~ 0
@@
 Text HLabel 7450 4350 0    60   Output ~ 0
 CAM_CTRL_1_N
-Text HLabel 9400 3950 2    60   Output ~ 0
+Text HLabel 9400 4150 2    60   Output ~ 0
 SPI_MISO
+Text HLabel 9400 3950 2    60   Input ~ 0
+SPI_MOSI
 Text HLabel 9400 3750 2    60   Input ~ 0
-SPI_MOSI
+SPI_CLK
 Text HLabel 9400 3550 2    60   Input ~ 0
-SPI_CLK
-Text HLabel 9400 3350 2    60   Input ~ 0
 SPI_EN_0
+Text HLabel 9400 3450 2    60   Input ~ 0
+SPI_EN_1
 Text HLabel 9400 3250 2    60   Input ~ 0
-SPI_EN_1
-Text HLabel 9400 3050 2    60   Input ~ 0
 ~CAM_RESET~
-Text HLabel 9350 4950 2    60   Input ~ 0
+Text HLabel 9400 2750 2    60   Input ~ 0
 CAM_CLK_REF
 Text Notes 900  6900 0    60   ~ 0
@@
 	1    0    0    -1
 $EndComp
-Text HLabel 9400 2850 2    60   BiDi ~ 0
+Text HLabel 9400 3050 2    60   BiDi ~ 0
 SDA
-Text HLabel 9400 2650 2    60   BiDi ~ 0
+Text HLabel 9400 2950 2    60   BiDi ~ 0
 SCL
 Text Notes 3250 6400 0    60   ~ 0
@@
 	7450 4350 8050 4350
 Wire Wire Line
-	9350 4950 8650 4950
-Wire Wire Line
-	9350 4750 8650 4750
-Wire Wire Line
-	8650 4650 9350 4650
-Wire Wire Line
-	9350 4550 8650 4550
-Wire Wire Line
-	9350 4350 8650 4350
-Wire Wire Line
-	8650 4250 9350 4250
-Wire Wire Line
-	9350 4150 8650 4150
+	8650 4950 9400 4950
+Wire Wire Line
+	8650 4850 9400 4850
+Wire Wire Line
+	8650 4750 9400 4750
+Wire Wire Line
+	8650 4550 9400 4550
+Wire Wire Line
+	8650 4450 9400 4450
+Wire Wire Line
+	8650 4350 9400 4350
+Wire Wire Line
+	9400 4150 8650 4150
 Wire Wire Line
 	9400 3950 8650 3950
@@
 	9400 3550 8650 3550
 Wire Wire Line
-	9400 3350 8650 3350
-Wire Wire Line
-	8650 3250 9400 3250
+	8650 3450 9400 3450
+Wire Wire Line
+	9400 3250 8650 3250
 Wire Wire Line
 	9400 3050 8650 3050
 Wire Wire Line
-	9400 2850 8650 2850
-Wire Wire Line
-	9400 2650 8650 2650
-Wire Wire Line
 	8050 1150 7800 1150
 Wire Wire Line
@@
 Wire Wire Line
 	7800 6050 8850 6050
-Wire Wire Line
-	8850 6050 8850 2550
-Wire Wire Line
-	8850 2550 8650 2550
 Wire Wire Line
 	8050 1450 7800 1450
@@
 Wire Wire Line
 	8650 5650 8850 5650
-Connection ~ 8850 5650
 Wire Wire Line
 	8650 5350 8850 5350
-Connection ~ 8850 5350
 Wire Wire Line
 	8650 5050 8850 5050
-Connection ~ 8850 5050
-Wire Wire Line
-	8650 4850 8850 4850
-Connection ~ 8850 4850
-Wire Wire Line
-	8650 4450 8850 4450
-Connection ~ 8850 4450
-Wire Wire Line
-	8650 4050 8850 4050
-Connection ~ 8850 4050
-Wire Wire Line
-	8650 3850 8850 3850
-Connection ~ 8850 3850
-Wire Wire Line
-	8650 3650 8850 3650
-Connection ~ 8850 3650
-Wire Wire Line
-	8650 3450 8850 3450
-Connection ~ 8850 3450
-Wire Wire Line
-	8650 3150 8850 3150
-Connection ~ 8850 3150
-Wire Wire Line
-	8650 2950 8850 2950
-Connection ~ 8850 2950
-Wire Wire Line
-	8650 2750 8850 2750
-Connection ~ 8850 2750
 $Comp
 L GND #PWR?
@@
 Connection ~ 8350 6050
 Wire Wire Line
-	8650 1850 8850 1850
-Wire Wire Line
-	8850 1850 8850 800
-Wire Wire Line
 	8650 950  8850 950
 Wire Wire Line
@@
 Wire Wire Line
 	8650 1750 8850 1750
-Connection ~ 8850 1750
 $Comp
 L +5V #PWR?
@@
 Wire Wire Line
 	9400 5150 8650 5150
+Text HLabel 9400 2550 2    60   Output ~ 0
+IMU_SPI_MISO
+Text HLabel 9400 2350 2    60   Input ~ 0
+IMU_SPI_MOSI
+Text HLabel 9400 2150 2    60   Input ~ 0
+IMU_SPI_CLK
+Wire Wire Line
+	9400 2950 8650 2950
+Wire Wire Line
+	8850 1750 8850 800
+Text HLabel 9400 1950 2    60   Input ~ 0
+IMU_SPI_EN_0
+Text HLabel 9400 1850 2    60   Input ~ 0
+IMU_SPI_EN_1
+Wire Wire Line
+	9400 1850 8650 1850
+Wire Wire Line
+	8650 1950 9400 1950
+Wire Wire Line
+	8650 2050 8850 2050
+Connection ~ 8850 2250
+Wire Notes Line
+	9200 1750 9200 2700
+Wire Notes Line
+	9200 2700 10200 2700
+Wire Notes Line
+	10200 2700 10200 1750
+Wire Notes Line
+	10200 1750 9200 1750
+Text Notes 9900 1700 2    60   ~ 0
+1.8 V only
+Wire Wire Line
+	9400 2150 8650 2150
+Wire Wire Line
+	8650 2350 9400 2350
+Wire Wire Line
+	8650 2550 9400 2550
+Wire Wire Line
+	9400 2750 8650 2750
+Wire Wire Line
+	8850 2050 8850 6050
+Connection ~ 8850 5650
+Connection ~ 8850 5350
+Connection ~ 8850 5050
+Wire Wire Line
+	8650 4650 8850 4650
+Connection ~ 8850 4650
+Wire Wire Line
+	8650 4250 8850 4250
+Connection ~ 8850 4250
+Wire Wire Line
+	8650 4050 8850 4050
+Connection ~ 8850 4050
+Wire Wire Line
+	8650 3850 8850 3850
+Connection ~ 8850 3850
+Wire Wire Line
+	8650 3650 8850 3650
+Connection ~ 8850 3650
+Wire Wire Line
+	8650 3350 8850 3350
+Connection ~ 8850 3350
+Wire Wire Line
+	8650 3150 8850 3150
+Connection ~ 8850 3150
+Wire Wire Line
+	8650 2850 8850 2850
+Connection ~ 8850 2850
+Wire Wire Line
+	8650 2650 8850 2650
+Connection ~ 8850 2650
+Wire Wire Line
+	8650 2450 8850 2450
+Connection ~ 8850 2450
 $EndSCHEMATC

Commit message: Triggerbus WIP.
Also added more production data
Parts:
- J?: Digikey (none) -> SAM9033CT-ND; MFG Name (none) -> Samtech; MFG Part Num (none) -> LSHM-150-04.0-L-DV-A-S-K-TR; Populated (none) -> 1; Source (none) -> SPEC
Changed lines of the file:
@@
 LIBS:sn74axc8t245
 LIBS:sn74lvc2t45
+LIBS:dmf05lcflp
+LIBS:txs02612
+LIBS:bss138ps
 LIBS:zynq_board-cache
 EELAYER 25 0
@@
 F 1 "LSHM-150-xxx-x-DV-A-S" V 8350 3400 60  0000 C CNN
 F 2 "Connectors_Samtec:LSHM-150-xxx-x-DV-A-S" H 8350 4550 60  0001 C CNN
-F 3 "" H 8350 4550 60  0001 C CNN
+F 3 "http://suddendocs.samtec.com/catalog_english/lshm_dv.pdf" H 8350 4550 60  0001 C CNN
+F 4 "Samtech" H 8350 3400 60  0001 C CNN "MFG Name"
+F 5 "LSHM-150-04.0-L-DV-A-S-K-TR" H 8350 3400 60  0001 C CNN "MFG Part Num"
+F 6 "SAM9033CT-ND" H 8350 3400 60  0001 C CNN "Digikey"
+F 7 "1" H 8350 3400 60  0001 C CNN "Populated"
+F 8 "SPEC" H 8350 3400 60  0001 C CNN "Source"
 	1    8350 3400
 	1    0    0    -1
@@
 	8650 5050 8850 5050
 $Comp
-L GND #PWR?
+L GND #PWR0128
 U 1 1 5AFB9A6C
 P 8350 6100
-F 0 "#PWR?" H 8350 5850 50  0001 C CNN
+F 0 "#PWR0128" H 8350 5850 50  0001 C CNN
 F 1 "GND" H 8350 5950 50  0000 C CNN
 F 2 "" H 8350 6100 50  0001 C CNN
@@
 	8650 1750 8850 1750
 $Comp
-L +5V #PWR?
+L +5V #PWR0129
 U 1 1 5AFBA51B
 P 8850 800
-F 0 "#PWR?" H 8850 650 50  0001 C CNN
+F 0 "#PWR0129" H 8850 650 50  0001 C CNN
 F 1 "+5V" H 8850 940 50  0000 C CNN
 F 2 "" H 8850 800 50  0001 C CNN
