File: hardware/usb.sch (KiCad schematic (older format))
At the start: 17 parts

Commit message: Repaired USB OTG Connector
Parts:
- removed P?: USB_OTG, symbol USB_OTG
- added J?: USB_OTG, symbol USB_OTG
Connections:
- wire segments 65 -> 70
Changed lines of the file:
@@
 $Descr A4 11693 8268
 encoding utf-8
-Sheet 15 18
+Sheet 13 18
 Title ""
 Date ""
@@
 	1    7100 3800
 	1    0    0    -1
-$EndComp
-$Comp
-L USB_OTG P?
-U 1 1 599150DC
-P 1200 4000
-F 0 "P?" H 1525 3875 50  0000 C CNN
-F 1 "USB_OTG" H 1200 4200 50  0000 C CNN
-F 2 "" V 1150 3900 50  0000 C CNN
-F 3 "" V 1150 3900 50  0000 C CNN
-	1    1200 4000
-	0    -1   1    0
 $EndComp
 Text HLabel 8100 3000 2    60   BiDi ~ 0
@@
 Text HLabel 8100 4200 2    60   Output ~ 0
 CLK
-Wire Wire Line
-	1500 3900 6100 3900
-Wire Wire Line
-	1500 4000 6100 4000
-Wire Wire Line
-	1500 4100 6100 4100
 $Comp
 L GND #PWR?
@@
 L GND #PWR?
 U 1 1 59921F43
-P 1600 4700
-F 0 "#PWR?" H 1600 4450 50  0001 C CNN
-F 1 "GND" H 1600 4550 50  0000 C CNN
-F 2 "" H 1600 4700 50  0000 C CNN
-F 3 "" H 1600 4700 50  0000 C CNN
-	1    1600 4700
-	1    0    0    -1
-$EndComp
-Wire Wire Line
-	1500 4200 1600 4200
+P 1200 4700
+F 0 "#PWR?" H 1200 4450 50  0001 C CNN
+F 1 "GND" H 1200 4550 50  0000 C CNN
+F 2 "" H 1200 4700 50  0000 C CNN
+F 3 "" H 1200 4700 50  0000 C CNN
+	1    1200 4700
+	1    0    0    -1
+$EndComp
 $Comp
 L R R?
 U 1 1 59922379
-P 1100 4550
-F 0 "R?" V 1180 4550 50  0000 C CNN
-F 1 "0" V 1100 4550 50  0000 C CNN
-F 2 "" V 1030 4550 50  0000 C CNN
-F 3 "" H 1100 4550 50  0000 C CNN
-	1    1100 4550
+P 1000 4550
+F 0 "R?" V 1080 4550 50  0000 C CNN
+F 1 "0" V 1000 4550 50  0000 C CNN
+F 2 "" V 930 4550 50  0000 C CNN
+F 3 "" H 1000 4550 50  0000 C CNN
+	1    1000 4550
 	1    0    0    -1
 $EndComp
@@
 L GND #PWR?
 U 1 1 599223A7
-P 1100 4700
-F 0 "#PWR?" H 1100 4450 50  0001 C CNN
-F 1 "GND" H 1100 4550 50  0000 C CNN
-F 2 "" H 1100 4700 50  0000 C CNN
-F 3 "" H 1100 4700 50  0000 C CNN
-	1    1100 4700
+P 1000 4700
+F 0 "#PWR?" H 1000 4450 50  0001 C CNN
+F 1 "GND" H 1000 4550 50  0000 C CNN
+F 2 "" H 1000 4700 50  0000 C CNN
+F 3 "" H 1000 4700 50  0000 C CNN
+	1    1000 4700
 	1    0    0    -1
 $EndComp
@@
 	0    1    1    0
 $EndComp
-Wire Wire Line
-	1500 3800 1500 3600
-Wire Wire Line
-	1500 3600 5600 3600
 $Comp
 L C C?
@@
 Connection ~ 1850 3600
 Wire Wire Line
-	1600 4200 1600 4700
+	1200 4200 1200 4700
 $Comp
 L GND #PWR?
@@
 	3000 4500 2900 4500
 Wire Wire Line
-	2900 4500 2900 4000
-Connection ~ 2900 4000
-Wire Wire Line
 	3000 4600 2800 4600
 Wire Wire Line
-	2800 4600 2800 3900
-Connection ~ 2800 3900
-Wire Wire Line
 	3000 4700 2700 4700
-Wire Wire Line
-	2700 4700 2700 4100
-Connection ~ 2700 4100
 Wire Wire Line
 	2700 3600 2700 3000
@@
 Text Notes 9000 4750 0    60   ~ 0
 Oscillator: DSC6003CI2A-012.0000\n(12 MHz)
+$Comp
+L USB_OTG J?
+U 1 1 5ACE0B3C
+P 1200 3800
+F 0 "J?" H 1000 4250 50  0000 L CNN
+F 1 "USB_OTG" H 1000 4150 50  0000 L CNN
+F 2 "" H 1350 3750 50  0001 C CNN
+F 3 "" H 1350 3750 50  0001 C CNN
+	1    1200 3800
+	1    0    0    -1
+$EndComp
+Wire Wire Line
+	1500 3600 5600 3600
+Wire Wire Line
+	6100 4000 5950 4000
+Wire Wire Line
+	5950 4000 5950 3800
+Wire Wire Line
+	5950 3800 1500 3800
+Wire Wire Line
+	6100 3900 1500 3900
+Wire Wire Line
+	1500 4000 5850 4000
+Wire Wire Line
+	5850 4000 5850 4100
+Wire Wire Line
+	5850 4100 6100 4100
+Wire Wire Line
+	2900 4500 2900 3800
+Connection ~ 2900 3800
+Wire Wire Line
+	2800 4600 2800 3900
+Connection ~ 2800 3900
+Wire Wire Line
+	2700 4700 2700 4000
+Connection ~ 2700 4000
+Wire Wire Line
+	1000 4400 1000 4300
+Wire Wire Line
+	1000 4300 1100 4300
+Wire Wire Line
+	1100 4300 1100 4200
 $EndSCHEMATC

Commit message: KiCad does not support differential Busses yet. See https://bugs.launchpad.net/kicad/+bug/1419146. Fixed Data Lanes for Camera Connector.
Parts:
- C? (x7): footprint (none) -> Capacitors_SMD:C_0402
- J?: footprint (none) -> Connectors:USB_Micro-B
- R? (x5): footprint (none) -> Resistors_SMD:R_0402
Changed lines of the file:
@@
 $Descr A4 11693 8268
 encoding utf-8
-Sheet 12 19
+Sheet 11 19
 Title ""
 Date ""
@@
 F 0 "R?" V 8330 4700 50  0000 C CNN
 F 1 "8.06k" V 8250 4700 50  0000 C CNN
-F 2 "" V 8180 4700 50  0001 C CNN
+F 2 "Resistors_SMD:R_0402" V 8180 4700 50  0001 C CNN
 F 3 "" H 8250 4700 50  0000 C CNN
 	1    8250 4700
@@
 F 0 "R?" V 1080 4550 50  0000 C CNN
 F 1 "0" V 1000 4550 50  0000 C CNN
-F 2 "" V 930 4550 50  0001 C CNN
+F 2 "Resistors_SMD:R_0402" V 930 4550 50  0001 C CNN
 F 3 "" H 1000 4550 50  0000 C CNN
 	1    1000 4550
@@
 F 0 "R?" V 5830 3600 50  0000 C CNN
 F 1 "1k" V 5750 3600 50  0000 C CNN
-F 2 "" V 5680 3600 50  0001 C CNN
+F 2 "Resistors_SMD:R_0402" V 5680 3600 50  0001 C CNN
 F 3 "" H 5750 3600 50  0000 C CNN
 	1    5750 3600
@@
 F 0 "C?" H 1875 4450 50  0000 L CNN
 F 1 "2u2" H 1875 4250 50  0000 L CNN
-F 2 "" H 1888 4200 50  0001 C CNN
+F 2 "Capacitors_SMD:C_0402" H 1888 4200 50  0001 C CNN
 F 3 "" H 1850 4350 50  0000 C CNN
 	1    1850 4350
@@
 F 0 "C?" H 6875 1950 50  0000 L CNN
 F 1 "100n" H 6875 1750 50  0000 L CNN
-F 2 "" H 6888 1700 50  0001 C CNN
+F 2 "Capacitors_SMD:C_0402" H 6888 1700 50  0001 C CNN
 F 3 "" H 6850 1850 50  0000 C CNN
 	1    6850 1850
@@
 F 0 "C?" H 7375 1950 50  0000 L CNN
 F 1 "100n" H 7375 1750 50  0000 L CNN
-F 2 "" H 7388 1700 50  0001 C CNN
+F 2 "Capacitors_SMD:C_0402" H 7388 1700 50  0001 C CNN
 F 3 "" H 7350 1850 50  0000 C CNN
 	1    7350 1850
@@
 F 0 "C?" H 6425 1950 50  0000 L CNN
 F 1 "2u2" H 6425 1750 50  0000 L CNN
-F 2 "" H 6438 1700 50  0001 C CNN
+F 2 "Capacitors_SMD:C_0402" H 6438 1700 50  0001 C CNN
 F 3 "" H 6400 1850 50  0000 C CNN
 	1    6400 1850
@@
 F 0 "C?" H 4725 2850 50  0000 L CNN
 F 1 "100n" H 4725 2650 50  0000 L CNN
-F 2 "" H 4738 2600 50  0001 C CNN
+F 2 "Capacitors_SMD:C_0402" H 4738 2600 50  0001 C CNN
 F 3 "" H 4700 2750 50  0000 C CNN
 	1    4700 2750
@@
 F 0 "R?" V 4730 3200 50  0000 C CNN
 F 1 "100k" V 4650 3200 50  0000 C CNN
-F 2 "" V 4580 3200 50  0001 C CNN
+F 2 "Resistors_SMD:R_0402" V 4580 3200 50  0001 C CNN
 F 3 "" H 4650 3200 50  0000 C CNN
 	1    4650 3200
@@
 F 0 "R?" V 5230 3100 50  0000 C CNN
 F 1 "10k" V 5150 3100 50  0000 C CNN
-F 2 "" V 5080 3100 50  0001 C CNN
+F 2 "Resistors_SMD:R_0402" V 5080 3100 50  0001 C CNN
 F 3 "" H 5150 3100 50  0000 C CNN
 	1    5150 3100
@@
 F 0 "C?" H 10375 4200 50  0000 L CNN
 F 1 "100n" H 10375 4000 50  0000 L CNN
-F 2 "" H 10388 3950 50  0001 C CNN
+F 2 "Capacitors_SMD:C_0402" H 10388 3950 50  0001 C CNN
 F 3 "" H 10350 4100 50  0000 C CNN
 	1    10350 4100
@@
 F 0 "C?" H 7825 1950 50  0000 L CNN
 F 1 "100n" H 7825 1750 50  0000 L CNN
-F 2 "" H 7838 1700 50  0001 C CNN
+F 2 "Capacitors_SMD:C_0402" H 7838 1700 50  0001 C CNN
 F 3 "" H 7800 1850 50  0000 C CNN
 	1    7800 1850
@@
 F 0 "J?" H 1000 4250 50  0000 L CNN
 F 1 "USB_OTG" H 1000 4150 50  0000 L CNN
-F 2 "" H 1350 3750 50  0001 C CNN
+F 2 "Connectors:USB_Micro-B" H 1350 3750 50  0001 C CNN
 F 3 "" H 1350 3750 50  0001 C CNN
 	1    1200 3800

Commit message: Added Second SPI Bus for IMUs to Cam Connector
This SPI works on 1.8 V, don't confuse them. If this second SPI Bus shall be used for the Cam Chips, add Levelshifters on the Cam Board.

Also reorderd some stuff around this connector, to ease routing
Parts:
- U?: footprint (none) -> Housings_DFN_QFN:QFN-32-1EP_5x5mm_Pitch0.5mm
- U?: footprint (none) -> footprints:WLCSP12_3x4_1.35x1.65mm_Pitch0.4mm
Changed lines of the file:
@@
 LIBS:lshm-150-xxx-x-dv-a-s
 LIBS:sn74axc8t245
+LIBS:sn74lvc2t45
 LIBS:zynq_board-cache
 EELAYER 25 0
@@
 $Descr A4 11693 8268
 encoding utf-8
-Sheet 11 19
+Sheet 11 20
 Title ""
 Date ""
@@
 F 0 "U?" H 7100 3750 60  0000 C CNN
 F 1 "USB3320" H 7100 3850 60  0000 C CNN
-F 2 "" H 7100 3800 60  0001 C CNN
+F 2 "Housings_DFN_QFN:QFN-32-1EP_5x5mm_Pitch0.5mm" H 7100 3800 60  0001 C CNN
 F 3 "" H 7100 3800 60  0001 C CNN
 	1    7100 3800
@@
 F 0 "U?" H 3800 3150 60  0000 C CNN
 F 1 "NX5P3090" H 3800 3250 60  0000 C CNN
-F 2 "" H 3800 3200 60  0001 C CNN
+F 2 "footprints:WLCSP12_3x4_1.35x1.65mm_Pitch0.4mm" H 3800 3200 60  0001 C CNN
 F 3 "" H 3800 3200 60  0001 C CNN
 	1    3800 3200

Commit message: Added Reset Button, Power LED, 2 Status LEDs and an external Button.
Other:
- note removed: "VDDIO: TBD"
Changed lines of the file:
@@
 LIBS:bss138ps
 LIBS:max14854
+LIBS:switches
 LIBS:zynq_board-cache
 EELAYER 25 0
@@
 $EndComp
 Connection ~ 7800 1650
-Text Notes 7550 1500 0    60   ~ 0
-VDDIO: TBD
 Text Notes 5150 2400 0    60   ~ 0
 REFSEL[2:0] = 010\nto select 12 MHz\nREFCLK input
@@
 Wire Wire Line
 	1100 4300 1100 4200
+$Comp
+L +3V3 #PWR?
+U 1 1 5B1F6406
+P 7800 1600
+F 0 "#PWR?" H 7800 1450 50  0001 C CNN
+F 1 "+3V3" H 7800 1740 50  0000 C CNN
+F 2 "" H 7800 1600 50  0000 C CNN
+F 3 "" H 7800 1600 50  0000 C CNN
+	1    7800 1600
+	1    0    0    -1
+$EndComp
 $EndSCHEMATC
