File: hardware/zynq_memory.sch (KiCad schematic (older format))
At the start: 1 part

Commit message: Change 10GE interface phy to TLK10031
Low speed signals are still missing. Low speed signals from sfp+ part now need to be connected to the fpga. The new Phy does not support i2c etc..

Also changed KiCad Version to 4.0.7
Changed lines of the file:
@@
 EESchema Schematic File Version 2
+LIBS:zynq_board-rescue
 LIBS:power
 LIBS:device
@@
 Text Notes 3950 9750 0    60   ~ 0
 TODO: VREFx, VRx, VCCO_DDR
+Connection ~ 4900 3750
 $EndSCHEMATC

Commit message: KiCad does not support differential Busses yet. See https://bugs.launchpad.net/kicad/+bug/1419146. Fixed Data Lanes for Camera Connector.
Parts:
- U?: footprint (none) -> footprints:SBG485_22x22_19.0x19.0mm_Pitch0.8mm
Changed lines of the file:
@@
 F 0 "U?" H 5350 2200 60  0000 L CNN
 F 1 "xc7z030sbg485" H 5350 2100 60  0000 L CNN
-F 2 "" H 5150 1950 60  0001 C CNN
+F 2 "footprints:SBG485_22x22_19.0x19.0mm_Pitch0.8mm" H 5150 1950 60  0001 C CNN
 F 3 "" H 5150 1950 60  0001 C CNN
 	8    5150 1950

Commit message: Moved the FPGAs Memory Port to the DDR Sheet due KiCad 4.0.7 does not support Busses through hiearchical Labels
Parts:
- removed U?: xc7z030sbg485, footprints:SBG485_22x22_19.0x19.0mm_Pitch0.8mm, symbol xc7z030sbg485
Connections:
- net labels removed: A0, A1, A10, A11, A12, A13, A14, A2, A3, A4, A5, A6, A7, A8, A9, DDR_A[0..14], DDR_BA0, DDR_BA1, DDR_BA2, DDR_CKE, DDR_CLK_N, DDR_CLK_P, DDR_DM0, DDR_DM1, DDR_DM2, DDR_DM3, DDR_DQS0_N, DDR_DQS0_P, DDR_DQS1_N, DDR_DQS1_P, DDR_DQS2_N, DDR_DQS2_P, DDR_DQS3_N, DDR_DQS3_P, DDR_DQ[0..31], DDR_ODT, DQ0, DQ1, DQ10, DQ11, DQ12, DQ13, DQ14, DQ15, DQ16, DQ17, DQ18, DQ19, DQ2, DQ20, DQ21, DQ22, DQ23, DQ24, DQ25, DQ26, DQ27, DQ28, DQ29, DQ3, DQ30, DQ31, DQ4, DQ5, DQ6, DQ7, DQ8, DQ9, ~DDR_CAS~, ~DDR_CS~, ~DDR_RAS~, ~DDR_RESET~, ~DDR_WE~
- wire segments 79 -> 0
Other:
- note added: "Moved to DDR3 RAM Sheet, because KiCad 4.0.7 does not support Busses through Hiearchical Labels"
