File: hardware/zynq_pl_34.sch (KiCad schematic (older format))
At the start: 1 part

Commit message: Almost drew 3,3 V lowspeed signals. Added Levelshifter Subschematic
1,8 V Lowspeed Singals from 10 G Phy to FPGA are still missing.

CAM_REF_CLK is not really low speed, maybe we should consider to use the lvds clock instead. I think it will work, since the signal should be realtive short(FPGA->Connector->Camerasensor[->Camerasensor2]). The levelshifter should also be fast enough.

The i2c signals use simple N-Channel MOSTFET Transistors for Levelshifting
Connections:
- net labels added: MODDET_18, RX_LOS_18, SFP_GPIO_18, SFP_SCL_18, SFP_SDA_18, TX_DISABLE_18, TX_FAULT_18
- wire segments 0 -> 7
Changed lines of the file:
@@
 LIBS:misc
 LIBS:tlk10031
+LIBS:lshm-150-xxx-x-dv-a-s
+LIBS:sn74axc8t245
 LIBS:zynq_board-cache
 EELAYER 25 0
@@
 $Descr A4 11693 8268
 encoding utf-8
-Sheet 6 18
+Sheet 6 19
 Title ""
 Date ""
@@
 	1    0    0    -1
 $EndComp
+Text HLabel 4800 2400 0    60   Output ~ 0
+SFP_GPIO_18
+Text HLabel 4800 2800 0    60   Input ~ 0
+RX_LOS_18
+Text HLabel 4800 3400 0    60   Input ~ 0
+MODDET_18
+Text HLabel 4800 3800 0    60   BiDi ~ 0
+SFP_SDA_18
+Text HLabel 4800 4000 0    60   BiDi ~ 0
+SFP_SCL_18
+Text HLabel 4800 4100 0    60   Input ~ 0
+TX_FAULT_18
+Text HLabel 4800 3600 0    60   Output ~ 0
+TX_DISABLE_18
+Wire Wire Line
+	4800 2400 5250 2400
+Wire Wire Line
+	4800 2800 5250 2800
+Wire Wire Line
+	4800 3400 5250 3400
+Wire Wire Line
+	5250 3600 4800 3600
+Wire Wire Line
+	4800 3800 5250 3800
+Wire Wire Line
+	5250 4000 4800 4000
+Wire Wire Line
+	4800 4100 5250 4100
 $EndSCHEMATC

Commit message: Drew missing 10 G Phy Lowspeed Signals.
Also moved the SFP+ Lowspeedsignals a bit to ease routing
Connections:
- net labels added: LS_OK_IN_A, LS_OK_OUT_A, MDC, MDIO, PRBSEN, ST, TLK_RESET
- wire segments 7 -> 14
Changed lines of the file:
@@
 Text HLabel 4800 2400 0    60   Output ~ 0
 SFP_GPIO_18
-Text HLabel 4800 2800 0    60   Input ~ 0
+Text HLabel 4800 2500 0    60   Input ~ 0
 RX_LOS_18
-Text HLabel 4800 3400 0    60   Input ~ 0
+Text HLabel 4800 2600 0    60   Input ~ 0
 MODDET_18
-Text HLabel 4800 3800 0    60   BiDi ~ 0
+Text HLabel 4800 2900 0    60   BiDi ~ 0
 SFP_SDA_18
-Text HLabel 4800 4000 0    60   BiDi ~ 0
+Text HLabel 4800 2800 0    60   BiDi ~ 0
 SFP_SCL_18
-Text HLabel 4800 4100 0    60   Input ~ 0
+Text HLabel 4800 3900 0    60   Input ~ 0
 TX_FAULT_18
+Text HLabel 4800 3800 0    60   Output ~ 0
+TX_DISABLE_18
+Text HLabel 4800 4200 0    60   Output ~ 0
+ST
+Text HLabel 4800 4100 0    60   Output ~ 0
+LS_OK_IN_A
+Text HLabel 4800 4000 0    60   Input ~ 0
+LS_OK_OUT_A
+Text HLabel 4800 4400 0    60   Output ~ 0
+PRBSEN
+Text HLabel 4800 3400 0    60   Output ~ 0
+MDC
+Text HLabel 4800 3500 0    60   BiDi ~ 0
+MDIO
 Text HLabel 4800 3600 0    60   Output ~ 0
-TX_DISABLE_18
+TLK_RESET
+Wire Wire Line
+	4800 2800 5250 2800
+Wire Wire Line
+	5250 2900 4800 2900
 Wire Wire Line
 	4800 2400 5250 2400
 Wire Wire Line
-	4800 2800 5250 2800
+	4800 2500 5250 2500
 Wire Wire Line
-	4800 3400 5250 3400
-Wire Wire Line
-	5250 3600 4800 3600
+	4800 2600 5250 2600
 Wire Wire Line
 	4800 3800 5250 3800
 Wire Wire Line
-	5250 4000 4800 4000
+	5250 3900 4800 3900
 Wire Wire Line
-	4800 4100 5250 4100
+	5250 4100 4800 4100
+Wire Wire Line
+	4800 4000 5250 4000
+Wire Wire Line
+	5250 4400 4800 4400
+Wire Wire Line
+	4800 4200 5250 4200
+Wire Wire Line
+	5250 3400 4800 3400
+Wire Wire Line
+	4800 3500 5250 3500
+Wire Wire Line
+	4800 3600 5250 3600
 $EndSCHEMATC

Commit message: KiCad does not support differential Busses yet. See https://bugs.launchpad.net/kicad/+bug/1419146. Fixed Data Lanes for Camera Connector.
Parts:
- U?: footprint (none) -> footprints:SBG485_22x22_19.0x19.0mm_Pitch0.8mm
Changed lines of the file:
@@
 F 0 "U?" H 5450 1050 60  0000 L CNN
 F 1 "xc7z030sbg485" H 5450 950 60  0000 L CNN
-F 2 "" H 5250 800 60  0001 C CNN
+F 2 "footprints:SBG485_22x22_19.0x19.0mm_Pitch0.8mm" H 5250 800 60  0001 C CNN
 F 3 "" H 5250 800 60  0001 C CNN
 	3    5250 800

Commit message: Finished Triggerbus and added GPIO Header to schematic.
Also moved some Connections to the FPGA around to hopefully ease routing.
Connections:
- net labels added: DE, GPIO_10, GPIO_11, GPIO_12, GPIO_13, GPIO_14, GPIO_15, GPIO_9, RXD, TXD, ~RE~, ~SBA~, ~TLK_RESET~
- net labels removed: TLK_RESET
- wire segments 14 -> 26
Changed lines of the file:
@@
 LIBS:sn74lvc2t45
 LIBS:dmf05lcflp
-LIBS:txs02612
 LIBS:bss138ps
+LIBS:max14854
 LIBS:zynq_board-cache
 EELAYER 25 0
@@
 $Descr A4 11693 8268
 encoding utf-8
-Sheet 6 20
+Sheet 6 21
 Title ""
 Date ""
@@
 MDIO
 Text HLabel 4800 3600 0    60   Output ~ 0
-TLK_RESET
+~TLK_RESET~
 Wire Wire Line
 	4800 2800 5250 2800
@@
 Wire Wire Line
 	4800 3600 5250 3600
+Text HLabel 4800 4500 0    60   Input ~ 0
+RXD
+Text HLabel 4800 5000 0    60   Output ~ 0
+~RE~
+Text HLabel 4800 5200 0    60   Output ~ 0
+DE
+Text HLabel 4800 3000 0    60   Output ~ 0
+TXD
+Text HLabel 4800 2700 0    60   Output ~ 0
+~SBA~
+Wire Wire Line
+	4800 2700 5250 2700
+Wire Wire Line
+	5250 3000 4800 3000
+Wire Wire Line
+	4800 4500 5250 4500
+Wire Wire Line
+	4800 5000 5250 5000
+Wire Wire Line
+	4800 5200 5250 5200
+Text HLabel 4800 3100 0    60   BiDi ~ 0
+GPIO_9
+Text HLabel 4800 3200 0    60   BiDi ~ 0
+GPIO_10
+Text HLabel 4800 5300 0    60   BiDi ~ 0
+GPIO_11
+Text HLabel 4800 5100 0    60   BiDi ~ 0
+GPIO_12
+Text HLabel 4800 5400 0    60   BiDi ~ 0
+GPIO_13
+Text HLabel 4800 4300 0    60   BiDi ~ 0
+GPIO_14
+Text HLabel 4800 3700 0    60   BiDi ~ 0
+GPIO_15
+Wire Wire Line
+	4800 3100 5250 3100
+Wire Wire Line
+	5250 3200 4800 3200
+Wire Wire Line
+	4800 3700 5250 3700
+Wire Wire Line
+	4800 5100 5250 5100
+Wire Wire Line
+	5250 5300 4800 5300
+Wire Wire Line
+	4800 5400 5250 5400
+Wire Wire Line
+	4800 4300 5250 4300
 $EndSCHEMATC
