File: hardware/zynq_config.sch (KiCad schematic (older format))
At the start: 1 part

Commit message: KiCad does not support differential Busses yet. See https://bugs.launchpad.net/kicad/+bug/1419146. Fixed Data Lanes for Camera Connector.
Parts:
- U?: footprint (none) -> footprints:SBG485_22x22_19.0x19.0mm_Pitch0.8mm
Changed lines of the file:
@@
 $Descr A4 11693 8268
 encoding utf-8
-Sheet 16 19
+Sheet 14 19
 Title ""
 Date ""
@@
 F 0 "U?" H 8300 2250 60  0000 L CNN
 F 1 "xc7z030sbg485" H 8300 2150 60  0000 L CNN
-F 2 "" H 8100 2000 60  0001 C CNN
+F 2 "footprints:SBG485_22x22_19.0x19.0mm_Pitch0.8mm" H 8100 2000 60  0001 C CNN
 F 3 "" H 8100 2000 60  0001 C CNN
 	1    8100 2000

Commit message: Added Sdcard Slot.
Parts:
- gave numbers to parts that had none: 1
Changed lines of the file:
@@
 $Descr A4 11693 8268
 encoding utf-8
-Sheet 14 21
+Sheet 14 20
 Title ""
 Date ""
@@
 $EndDescr
 $Comp
-L xc7z030sbg485 U?
+L xc7z030sbg485 U1
 U 1 1 5AC336D4
 P 8100 2000
-F 0 "U?" H 8300 2250 60  0000 L CNN
+F 0 "U1" H 8300 2250 60  0000 L CNN
 F 1 "xc7z030sbg485" H 8300 2150 60  0000 L CNN
 F 2 "footprints:SBG485_22x22_19.0x19.0mm_Pitch0.8mm" H 8100 2000 60  0001 C CNN
