File: hardware/zynq_config.sch (KiCad schematic (older format))
At the start: 4 parts, among them J2 Conn_01x05, U1 xc7z030sbg485

Commit message: Added Power/Protection Circuit
Parts:
- renumbered J2 to J1101, R78 to R1101, R79 to R1102, U1 to U201
Changed lines of the file:
@@
 $EndDescr
 $Comp
-L xc7z030sbg485 U1
+L xc7z030sbg485 U201
 U 1 1 5AC336D4
 P 4550 2450
-F 0 "U1" H 4750 2700 60  0000 L CNN
+F 0 "U201" H 4750 2700 60  0000 L CNN
 F 1 "xc7z030sbg485" H 4750 2600 60  0000 L CNN
 F 2 "footprints:SBG485_22x22_19.0x19.0mm_Pitch0.8mm" H 4550 2450 60  0001 C CNN
@@
 $EndComp
 $Comp
-L Conn_01x05 J2
+L Conn_01x05 J1101
 U 1 1 5AE1C32D
 P 3100 3750
-F 0 "J2" H 3100 4050 50  0000 C CNN
+F 0 "J1101" H 3100 4050 50  0000 C CNN
 F 1 "Conn_01x05" H 3100 3450 50  0000 C CNN
 F 2 "" H 3100 3750 50  0001 C CNN
@@
 CFGBVS is connected to GND if VCCO is 1,8 V or lower. If VCCO is 2,5 or\n3,3 V, connect CFGBVS to VCCO.\n\nDONE is open-drain. Singals High if configuration sequence is completed.\n\nDXN and DXP are the Temperature-sensing diode. When not used, tie to GND.\nTemperature Monitoring can use the temperature Sensore inside the XADC Block.\n\nGNDADC is the ground reference for the XADC. Tie to GND even if not used.\n\nINIT_B is open-drain. Hold low to delay pl configuration. Will signal low if an\nconfiguration error has been occured.\n\nPROGRAMM_B is the active low Reset for PL.\n\nRSVDGND - Tie to GND\n\nRSVDVCC[1-3] - Tie to VCCO\n\nVCCADC is the analog supply for the XADCs. Tie to VCCAUX even if the XADCs are not used.\n\nVCCBATT is Backup Power for AES Key. Is not related to VCCO. Connect to GND or VCCAUX.\n\nVN and VP are the dedicated differential Analog Input to the XADC. Tie to GND if them are not used.\n\nVREFN and VREFP are the differential reference voltage input for the XADC.\nConnect to GND if not used.
 $Comp
-L R_Small R79
+L R_Small R1102
 U 1 1 5AE1E0D7
 P 4350 3050
-F 0 "R79" V 4400 3150 50  0000 L CNN
+F 0 "R1102" V 4400 3150 50  0000 L CNN
 F 1 "4k7" V 4350 3050 50  0000 C CNN
 F 2 "Resistors_SMD:R_0402" H 4350 3050 50  0001 C CNN
@@
 	4450 3050 4550 3050
 $Comp
-L R_Small R78
+L R_Small R1101
 U 1 1 5AE1E489
 P 4350 2950
-F 0 "R78" V 4400 3050 50  0000 L CNN
+F 0 "R1101" V 4400 3050 50  0000 L CNN
 F 1 "4k7" V 4350 2950 50  0000 C CNN
 F 2 "Resistors_SMD:R_0402" H 4350 2950 50  0001 C CNN

Commit message: Length matched DDR3 Memory again.
Forgot to keep enough space between the traces and between the meander waves.

Also, I switched to Kicad 5.0 RC2.

Swaped a few ddr signals.
Parts:
- J1101: symbol Conn_01x05 -> conn:Conn_01x05
- R1101, R1102: symbol R_Small -> device:R_Small
- U201: symbol xc7z030sbg485 -> xilinx_zynq_clg485:xc7z030sbg485
Changed lines of the file:
@@
-EESchema Schematic File Version 2
-LIBS:zynq_board-rescue
-LIBS:power
-LIBS:device
-LIBS:transistors
-LIBS:conn
-LIBS:linear
-LIBS:regul
-LIBS:74xx
-LIBS:cmos4000
-LIBS:adc-dac
-LIBS:memory
-LIBS:xilinx
-LIBS:microcontrollers
-LIBS:dsp
-LIBS:microchip
-LIBS:analog_switches
-LIBS:motorola
-LIBS:texas
-LIBS:intel
-LIBS:audio
-LIBS:interface
-LIBS:digital-audio
-LIBS:philips
-LIBS:display
-LIBS:cypress
-LIBS:siliconi
-LIBS:opto
-LIBS:atmel
-LIBS:contrib
-LIBS:valves
-LIBS:xilinx_zynq_clg485
-LIBS:SFP_plus
-LIBS:ael2005
-LIBS:diff_osc
-LIBS:si53340
-LIBS:usb3320
-LIBS:nx5p3090
-LIBS:smp1255putg
-LIBS:osc
-LIBS:ddr
-LIBS:misc
-LIBS:tlk10031
-LIBS:lshm-150-xxx-x-dv-a-s
-LIBS:sn74axc8t245
-LIBS:sn74lvc2t45
-LIBS:dmf05lcflp
-LIBS:bss138ps
-LIBS:max14854
-LIBS:switches
-LIBS:ft234xd
-LIBS:sn74lv1t126
-LIBS:emif06-msd02n16
-LIBS:cat24c02tdi-gt3
-LIBS:power_symbols
-LIBS:ti_power_modules
-LIBS:mdr20
-LIBS:dm3cs
-LIBS:lsf0102
-LIBS:dmp3056l
+EESchema Schematic File Version 4
 LIBS:zynq_board-cache
-EELAYER 25 0
+EELAYER 26 0
 EELAYER END
 $Descr A4 11693 8268
@@
 $EndDescr
 $Comp
-L xc7z030sbg485 U201
+L xilinx_zynq_clg485:xc7z030sbg485 U201
 U 1 1 5AC336D4
 P 4550 2450
@@
 $EndComp
 $Comp
-L Conn_01x05 J1101
+L conn:Conn_01x05 J1101
 U 1 1 5AE1C32D
 P 3100 3750
@@
 	4550 3850 3300 3850
 $Comp
-L GND #PWR0120
+L power1:GND #PWR0120
 U 1 1 5AE1DF94
 P 3400 4050
@@
 VCCO
 $Comp
-L GND #PWR0121
+L power1:GND #PWR0121
 U 1 1 5AE1E08B
 P 3850 2450
@@
 CFGBVS is connected to GND if VCCO is 1,8 V or lower. If VCCO is 2,5 or\n3,3 V, connect CFGBVS to VCCO.\n\nDONE is open-drain. Singals High if configuration sequence is completed.\n\nDXN and DXP are the Temperature-sensing diode. When not used, tie to GND.\nTemperature Monitoring can use the temperature Sensore inside the XADC Block.\n\nGNDADC is the ground reference for the XADC. Tie to GND even if not used.\n\nINIT_B is open-drain. Hold low to delay pl configuration. Will signal low if an\nconfiguration error has been occured.\n\nPROGRAMM_B is the active low Reset for PL.\n\nRSVDGND - Tie to GND\n\nRSVDVCC[1-3] - Tie to VCCO\n\nVCCADC is the analog supply for the XADCs. Tie to VCCAUX even if the XADCs are not used.\n\nVCCBATT is Backup Power for AES Key. Is not related to VCCO. Connect to GND or VCCAUX.\n\nVN and VP are the dedicated differential Analog Input to the XADC. Tie to GND if them are not used.\n\nVREFN and VREFP are the differential reference voltage input for the XADC.\nConnect to GND if not used.
 $Comp
-L R_Small R1102
+L device:R_Small R1102
 U 1 1 5AE1E0D7
 P 4350 3050
@@
 	4450 3050 4550 3050
 $Comp
-L R_Small R1101
+L device:R_Small R1101
 U 1 1 5AE1E489
 P 4350 2950
@@
 NoConn ~ 4550 2550
 $Comp
-L GND #PWR0122
+L power1:GND #PWR0122
 U 1 1 5ADFC840
 P 3850 4050
@@
 	3850 4050 4550 4050
 $Comp
-L GND #PWR0123
+L power1:GND #PWR0123
 U 1 1 5ADFC883
 P 3850 2650
@@
 	3850 2650 4550 2650
 $Comp
-L GND #PWR0124
+L power1:GND #PWR0124
 U 1 1 5ADFC8A4
 P 3850 2750
@@
 	3850 2750 4550 2750
 $Comp
-L GND #PWR0125
+L power1:GND #PWR0125
 U 1 1 5ADFC914
 P 3850 2850
@@
 	3850 2850 4550 2850
 $Comp
-L GND #PWR0126
+L power1:GND #PWR0126
 U 1 1 5ADFC9B4
 P 3850 4250
@@
 	3850 4250 4550 4250
 $Comp
-L GND #PWR0127
+L power1:GND #PWR0127
 U 1 1 5ADFC9BB
 P 3850 4350
@@
 	3850 4350 4550 4350
 $Comp
-L GND #PWR0128
+L power1:GND #PWR0128
 U 1 1 5ADFC9D4
 P 3850 4450
@@
 	3850 4450 4550 4450
 $Comp
-L GND #PWR0129
+L power1:GND #PWR0129
 U 1 1 5ADFC9DB
 P 3850 4550
@@
 VCCO
 $Comp
-L GND #PWR0130
+L power1:GND #PWR0130
 U 1 1 5ADFCAC7
 P 3850 3150

Commit message: Layouted USB-UART.
Also moved USB-OTG to the right Side of the Board. To get there
some free Space, i moved the DDR3/Memory and the FPGA a few
Millimeters down.
Parts:
- R1101, R1102: footprint Resistors_SMD:R_0402 -> Resistor_SMD:R_0402_1005Metric
Changed lines of the file:
@@
 F 0 "R1102" V 4400 3150 50  0000 L CNN
 F 1 "4k7" V 4350 3050 50  0000 C CNN
-F 2 "Resistors_SMD:R_0402" H 4350 3050 50  0001 C CNN
+F 2 "Resistor_SMD:R_0402_1005Metric" H 4350 3050 50  0001 C CNN
 F 3 "" H 4350 3050 50  0001 C CNN
 F 4 "1" H 4350 3050 60  0001 C CNN "Populated"
@@
 F 0 "R1101" V 4400 3050 50  0000 L CNN
 F 1 "4k7" V 4350 2950 50  0000 C CNN
-F 2 "Resistors_SMD:R_0402" H 4350 2950 50  0001 C CNN
+F 2 "Resistor_SMD:R_0402_1005Metric" H 4350 2950 50  0001 C CNN
 F 3 "" H 4350 2950 50  0001 C CNN
 F 4 "1" H 4350 2950 60  0001 C CNN "Populated"

Commit message: Improved Powerdistribution Network of the FPGA.
Also started to layout USB.
Parts:
- removed J1101: Conn_01x05, symbol conn:Conn_01x05
- added J?: Conn_01x06, Connector_PinHeader_2.54mm:PinHeader_1x06_P2.54mm_Vertical, symbol Connector_Generic:Conn_01x06
Connections:
- net labels added: JTAG_TCK, JTAG_TDI, JTAG_TDO, JTAG_TMS, JTAG_VDD
- wire segments 27 -> 34
Changed lines of the file:
@@
 $EndComp
-$Comp
-L conn:Conn_01x05 J1101
-U 1 1 5AE1C32D
-P 3100 3750
-F 0 "J1101" H 3100 4050 50  0000 C CNN
-F 1 "Conn_01x05" H 3100 3450 50  0000 C CNN
-F 2 "" H 3100 3750 50  0001 C CNN
-F 3 "" H 3100 3750 50  0001 C CNN
-	1    3100 3750
-	-1   0    0    -1
-$EndComp
-Wire Wire Line
-	3300 3550 4550 3550
-Wire Wire Line
-	4550 3650 3300 3650
-Wire Wire Line
-	3300 3750 4550 3750
-Wire Wire Line
-	4550 3850 3300 3850
 $Comp
 L power1:GND #PWR0120
 U 1 1 5AE1DF94
-P 3400 4050
-F 0 "#PWR0120" H 3400 3800 50  0001 C CNN
-F 1 "GND" H 3400 3900 50  0000 C CNN
-F 2 "" H 3400 4050 50  0001 C CNN
-F 3 "" H 3400 4050 50  0001 C CNN
-	1    3400 4050
+P 3000 3650
+F 0 "#PWR0120" H 3000 3400 50  0001 C CNN
+F 1 "GND" H 3000 3500 50  0000 C CNN
+F 2 "" H 3000 3650 50  0001 C CNN
+F 3 "" H 3000 3650 50  0001 C CNN
+	1    3000 3650
 	1    0    0    -1
 $EndComp
 Wire Wire Line
-	3400 4050 3400 3950
-Wire Wire Line
-	3400 3950 3300 3950
+	3000 3650 3000 3550
 Wire Wire Line
 	3850 4150 4550 4150
@@
 Wire Wire Line
 	1650 1500 1650 1600
+$Comp
+L Connector_Generic:Conn_01x06 J?
+U 1 1 5B586617
+P 2200 3350
+F 0 "J?" H 2120 3767 50  0000 C CNN
+F 1 "Conn_01x06" H 2120 3676 50  0000 C CNN
+F 2 "Connector_PinHeader_2.54mm:PinHeader_1x06_P2.54mm_Vertical" H 2200 3350 50  0001 C CNN
+F 3 "~" H 2200 3350 50  0001 C CNN
+F 4 "1" H 2200 3350 50  0001 C CNN "Populated"
+F 5 "SPEC" H 2200 3350 50  0001 C CNN "Source"
+F 6 "1" H 2200 3350 50  0001 C CNN "Populate for SBGA485(Z-7030)"
+F 7 "1" H 2200 3350 50  0001 C CNN "Populate for CLG484(Z-7012s/Z-7015)"
+	1    2200 3350
+	-1   0    0    -1
+$EndComp
+Text Label 2800 3150 2    50   ~ 0
+JTAG_TMS
+Text Label 2800 3250 2    50   ~ 0
+JTAG_TDI
+Text Label 2800 3350 2    50   ~ 0
+JTAG_TDO
+Text Label 2800 3450 2    50   ~ 0
+JTAG_TCK
+Text Label 2800 3650 2    50   ~ 0
+JTAG_VDD
+Wire Wire Line
+	2800 3650 2400 3650
+Wire Wire Line
+	2400 3450 2800 3450
+Wire Wire Line
+	2800 3350 2400 3350
+Wire Wire Line
+	2400 3250 2800 3250
+Wire Wire Line
+	2800 3150 2400 3150
+Text Label 3850 3850 0    50   ~ 0
+JTAG_TMS
+Text Label 3850 3650 0    50   ~ 0
+JTAG_TDI
+Text Label 3850 3750 0    50   ~ 0
+JTAG_TDO
+Text Label 3850 3550 0    50   ~ 0
+JTAG_TCK
+Wire Wire Line
+	3850 3850 4550 3850
+Wire Wire Line
+	4550 3750 3850 3750
+Wire Wire Line
+	3850 3650 4550 3650
+Wire Wire Line
+	4550 3550 3850 3550
+Wire Wire Line
+	2400 3550 3000 3550
+Text Label 2100 1750 2    50   ~ 0
+JTAG_VDD
+Wire Wire Line
+	2100 1750 1650 1750
+Wire Wire Line
+	1650 1750 1650 1600
+Connection ~ 1650 1600
 $EndSCHEMATC

Commit message: Fixed Schematic Symbols
Parts:
- R1101, R1102: symbol device:R_Small -> Device:R_Small
Changed lines of the file:
@@
 $Descr A4 11693 8268
 encoding utf-8
-Sheet 11 22
+Sheet 11 21
 Title ""
 Date ""
@@
 $EndComp
 $Comp
-L power1:GND #PWR0120
+L power:GND #PWR0120
 U 1 1 5AE1DF94
 P 3000 3650
@@
 VCCO
 $Comp
-L power1:GND #PWR0121
+L power:GND #PWR0121
 U 1 1 5AE1E08B
 P 3850 2450
@@
 CFGBVS is connected to GND if VCCO is 1,8 V or lower. If VCCO is 2,5 or\n3,3 V, connect CFGBVS to VCCO.\n\nDONE is open-drain. Singals High if configuration sequence is completed.\n\nDXN and DXP are the Temperature-sensing diode. When not used, tie to GND.\nTemperature Monitoring can use the temperature Sensore inside the XADC Block.\n\nGNDADC is the ground reference for the XADC. Tie to GND even if not used.\n\nINIT_B is open-drain. Hold low to delay pl configuration. Will signal low if an\nconfiguration error has been occured.\n\nPROGRAMM_B is the active low Reset for PL.\n\nRSVDGND - Tie to GND\n\nRSVDVCC[1-3] - Tie to VCCO\n\nVCCADC is the analog supply for the XADCs. Tie to VCCAUX even if the XADCs are not used.\n\nVCCBATT is Backup Power for AES Key. Is not related to VCCO. Connect to GND or VCCAUX.\n\nVN and VP are the dedicated differential Analog Input to the XADC. Tie to GND if them are not used.\n\nVREFN and VREFP are the differential reference voltage input for the XADC.\nConnect to GND if not used.
 $Comp
-L device:R_Small R1102
+L Device:R_Small R1102
 U 1 1 5AE1E0D7
 P 4350 3050
@@
 	4450 3050 4550 3050
 $Comp
-L device:R_Small R1101
+L Device:R_Small R1101
 U 1 1 5AE1E489
 P 4350 2950
@@
 NoConn ~ 4550 2550
 $Comp
-L power1:GND #PWR0122
+L power:GND #PWR0122
 U 1 1 5ADFC840
 P 3850 4050
@@
 	3850 4050 4550 4050
 $Comp
-L power1:GND #PWR0123
+L power:GND #PWR0123
 U 1 1 5ADFC883
 P 3850 2650
@@
 	3850 2650 4550 2650
 $Comp
-L power1:GND #PWR0124
+L power:GND #PWR0124
 U 1 1 5ADFC8A4
 P 3850 2750
@@
 	3850 2750 4550 2750
 $Comp
-L power1:GND #PWR0125
+L power:GND #PWR0125
 U 1 1 5ADFC914
 P 3850 2850
@@
 	3850 2850 4550 2850
 $Comp
-L power1:GND #PWR0126
+L power:GND #PWR0126
 U 1 1 5ADFC9B4
 P 3850 4250
@@
 	3850 4250 4550 4250
 $Comp
-L power1:GND #PWR0127
+L power:GND #PWR0127
 U 1 1 5ADFC9BB
 P 3850 4350
@@
 	3850 4350 4550 4350
 $Comp
-L power1:GND #PWR0128
+L power:GND #PWR0128
 U 1 1 5ADFC9D4
 P 3850 4450
@@
 	3850 4450 4550 4450
 $Comp
-L power1:GND #PWR0129
+L power:GND #PWR0129
 U 1 1 5ADFC9DB
 P 3850 4550
@@
 VCCO
 $Comp
-L power1:GND #PWR0130
+L power:GND #PWR0130
 U 1 1 5ADFCAC7
 P 3850 3150

Commit message: WIP: TLK Powerdistribution
Parts:
- gave numbers to parts that had none: 1
Changed lines of the file:
@@
 EESchema Schematic File Version 4
-LIBS:zynq_board-cache
 EELAYER 26 0
 EELAYER END
@@
 	1650 1500 1650 1600
 $Comp
-L Connector_Generic:Conn_01x06 J?
+L Connector_Generic:Conn_01x06 J1001
 U 1 1 5B586617
 P 2200 3350
-F 0 "J?" H 2120 3767 50  0000 C CNN
+F 0 "J1001" H 2120 3767 50  0000 C CNN
 F 1 "Conn_01x06" H 2120 3676 50  0000 C CNN
 F 2 "Connector_PinHeader_2.54mm:PinHeader_1x06_P2.54mm_Vertical" H 2200 3350 50  0001 C CNN
