File: hardware/zynq_power.sch (KiCad schematic (older format))
At the start: 16 parts

Commit message: Connected the Configuration Bank(0).
Connections:
- net labels added: VCCAUX
Changed lines of the file:
@@
 L +1V0 #PWR?
 U 1 1 5ADF2035
-P 8400 950
-F 0 "#PWR?" H 8400 800 50  0001 C CNN
-F 1 "+1V0" H 8400 1090 50  0000 C CNN
-F 2 "" H 8400 950 50  0001 C CNN
-F 3 "" H 8400 950 50  0001 C CNN
-	1    8400 950
+P 7900 950
+F 0 "#PWR?" H 7900 800 50  0001 C CNN
+F 1 "+1V0" H 7900 1090 50  0000 C CNN
+F 2 "" H 7900 950 50  0001 C CNN
+F 3 "" H 7900 950 50  0001 C CNN
+	1    7900 950
 	1    0    0    -1
 $EndComp
@@
 	8950 1250 8850 1250
 Connection ~ 8850 1250
-Wire Wire Line
-	8850 1650 9900 1650
 Connection ~ 8850 1550
 Wire Wire Line
@@
 Connection ~ 8850 1650
 Wire Wire Line
-	8400 1850 9900 1850
+	7900 1850 9900 1850
 Wire Wire Line
-	8400 950  8400 2050
+	7900 950  7900 2050
 Wire Wire Line
-	8400 2050 9900 2050
-Connection ~ 8400 1850
+	7900 2050 9900 2050
+Connection ~ 7900 1850
 Wire Wire Line
-	9900 1750 8400 1750
-Connection ~ 8400 1750
+	7900 1750 9900 1750
+Connection ~ 7900 1750
 Wire Wire Line
 	9900 1350 9800 1350
@@
 	1    0    0    -1
 $EndComp
+Text GLabel 8450 1650 0    60   Output ~ 0
+VCCAUX
+Wire Wire Line
+	8450 1650 9900 1650
 $EndSCHEMATC

Commit message: Added decoupling Capacitors for the Zynq. Also added the 2,5 V Power supply.
The 2,5 V supply was implemented as LDO and is sourced by the 3,3 V Line.
Parts:
- removed C?: 4.7µF, Capacitors_SMD:C_0805, symbol C_Small
- removed C?: 47µF, Capacitors_SMD:C_1210, symbol C_Small
- removed C?: 100µF, Capacitors_SMD:C_1210, symbol CP_Small
- removed C?: 330µF, C_2917, symbol CP_Small
- removed C? (x3): 0.47µF, Capacitors_SMD:C_0603, symbol C_Small
- added C? (x6): 100µF, Capacitors_SMD:C_1210, symbol CP_Small
- added C? (x29): 0.47µF, Capacitors_SMD:C_0603, symbol C_Small
- added C? (x13): 4.7µF, Capacitors_SMD:C_0805, symbol C_Small
- added C? (x4): 47µF, Capacitors_SMD:C_1210, symbol C_Small
- C?: Description CAP CER 0.47UF 6.3V X7R 0603,1 mΩ < ESR < 20 mΩ, ESL 0.5 nH -> CAP CER 0.47UF 6.3V X5R 0603; Digikey 490-6416-1-ND -> 490-3266-1-ND; MFG Part Num GRM188R70J474KA01 -> GRM155R60J474KE19D
- C? (x2): Populate for CLG484(Z-7012s/Z-7015) (none) -> Populate; Populate for SBGA485(Z-7030) (none) -> DNP
- L?: value 100 Ohm @ 1Mhz -> 120 Ohm @ 1Mhz; footprint (none) -> Inductors_SMD:L_0603; Digikey (none) -> 490-3996-1-ND; MFG Name (none) -> Murata Electronics North America; MFG Part Num (none) -> BLM18SG121TN1D; Populated (none) -> 1; Source (none) -> SPEC
Connections:
- net labels added: +2V5, +3V3, +V_DDR, VCCO_13, VCCO_34, VCCO_35, VCCO_DDR, VCCO_MIO0, VCCO_MIO1, VCC_AUX, VCC_BRAM, VCC_INT, VCC_PAUX, VCC_PINT, VCC_PLL, V_BANK0
- net labels removed: VCCAUX
- wire segments 17 -> 184
Other:
- note added: "1,8 V"
- note added: "2,5 V"
- note added: "Only needed for\nCLG484 Package\n(Z-7012S/Z-7015)"
- note added: "Only needed for\nSBG485 Package\n(Z-7030)"
- note added: "Only one 47 µF Cap\nneeded per 4 Banks\nof the same Type(HP/HR)\nat the same Voltage"
- note added: "VCCO_MIO0"
- note added: "VCCO_MIO1"
- note added: "VCC_PLL"
- note removed: "VCC_MIO1"

Commit message: Enhanced Power Connector and Filtering.
Also added a few more production informations.
Parts:
- C?: Populate for CLG484(Z-7012s/Z-7015) (none) -> 1; Populate for SBGA485(Z-7030) (none) -> 1
Changed lines of the file:
@@
 F 8 "CAP CER 10UF 4V X5R 0603" H 9100 5450 60  0001 C CNN "Description"
 F 9 "SPEC" H 9100 5450 60  0001 C CNN "Source"
+F 10 "1" H 9100 5450 60  0001 C CNN "Populate for SBGA485(Z-7030)"
+F 11 "1" H 9100 5450 60  0001 C CNN "Populate for CLG484(Z-7012s/Z-7015)"
 	1    9100 5450
 	1    0    0    -1

Commit message: Started to route DDR3 Memory.
At first added missing Footprint for Reference- and Terminationvoltage Regulator. Added Powerplanes for GND and VCCO. Added decoupling Network to both DDR3 Memory Chips. There are more small caps, to support Memory from other Manufactors.
Parts:
- gave numbers to parts that had none: 61
