File: hardware/Levelshifters.sch (KiCad schematic (older format))
At the start: 30 parts

Commit message: Failed to save Levelshifter Symbol correctly...
Parts:
- C? (x6): footprint (none) -> Capacitors_SMD:C_0201
- R? (x17): footprint (none) -> Resistors_SMD:R_0402
- U? (x3): footprint (none) -> Housings_SSOP:TSSOP-24_4.4x7.8mm_Pitch0.65mm
Changed lines of the file:
@@
 LIBS:lshm-150-xxx-x-dv-a-s
 LIBS:sn74axc8t245
-LIBS:zynq_board-cache
 EELAYER 25 0
 EELAYER END
@@
 F 0 "U?" H 4100 5250 60  0000 C CNN
 F 1 "SN74AXC8T245" V 4100 6250 60  0000 C CNN
-F 2 "" H 4050 6300 60  0001 C CNN
+F 2 "Housings_SSOP:TSSOP-24_4.4x7.8mm_Pitch0.65mm" H 4050 6300 60  0001 C CNN
 F 3 "" H 4050 6300 60  0001 C CNN
 	1    4100 6300
@@
 F 0 "R?" H 3430 5820 50  0000 L CNN
 F 1 "10k" H 3430 5760 50  0000 L CNN
-F 2 "" H 3400 5800 50  0001 C CNN
+F 2 "Resistors_SMD:R_0402" H 3400 5800 50  0001 C CNN
 F 3 "" H 3400 5800 50  0001 C CNN
 	1    3400 5800
@@
 F 0 "R?" H 3430 6820 50  0000 L CNN
 F 1 "10k" H 3430 6760 50  0000 L CNN
-F 2 "" H 3400 6800 50  0001 C CNN
+F 2 "Resistors_SMD:R_0402" H 3400 6800 50  0001 C CNN
 F 3 "" H 3400 6800 50  0001 C CNN
 	1    3400 6800
@@
 F 0 "U?" H 4050 650 60  0000 C CNN
 F 1 "SN74AXC8T245" V 4050 1650 60  0000 C CNN
-F 2 "" H 4000 1700 60  0001 C CNN
+F 2 "Housings_SSOP:TSSOP-24_4.4x7.8mm_Pitch0.65mm" H 4000 1700 60  0001 C CNN
 F 3 "" H 4000 1700 60  0001 C CNN
 	1    4050 1700
@@
 F 0 "R?" H 3380 1220 50  0000 L CNN
 F 1 "10k" H 3380 1160 50  0000 L CNN
-F 2 "" H 3350 1200 50  0001 C CNN
+F 2 "Resistors_SMD:R_0402" H 3350 1200 50  0001 C CNN
 F 3 "" H 3350 1200 50  0001 C CNN
 	1    3350 1200
@@
 F 0 "R?" H 3380 2220 50  0000 L CNN
 F 1 "10k" H 3380 2160 50  0000 L CNN
-F 2 "" H 3350 2200 50  0001 C CNN
+F 2 "Resistors_SMD:R_0402" H 3350 2200 50  0001 C CNN
 F 3 "" H 3350 2200 50  0001 C CNN
 	1    3350 2200
@@
 F 0 "U?" H 4050 3000 60  0000 C CNN
 F 1 "SN74AXC8T245" V 4050 3950 60  0000 C CNN
-F 2 "" H 4000 4000 60  0001 C CNN
+F 2 "Housings_SSOP:TSSOP-24_4.4x7.8mm_Pitch0.65mm" H 4000 4000 60  0001 C CNN
 F 3 "" H 4000 4000 60  0001 C CNN
 	1    4050 4000
@@
 F 0 "R?" H 3380 3520 50  0000 L CNN
 F 1 "10k" H 3380 3460 50  0000 L CNN
-F 2 "" H 3350 3500 50  0001 C CNN
+F 2 "Resistors_SMD:R_0402" H 3350 3500 50  0001 C CNN
 F 3 "" H 3350 3500 50  0001 C CNN
 	1    3350 3500
@@
 F 0 "R?" H 3380 4520 50  0000 L CNN
 F 1 "10k" H 3380 4460 50  0000 L CNN
-F 2 "" H 3350 4500 50  0001 C CNN
+F 2 "Resistors_SMD:R_0402" H 3350 4500 50  0001 C CNN
 F 3 "" H 3350 4500 50  0001 C CNN
 	1    3350 4500
@@
 F 0 "R?" H 9630 1220 50  0000 L CNN
 F 1 "10k" H 9630 1160 50  0000 L CNN
-F 2 "" H 9600 1200 50  0001 C CNN
+F 2 "Resistors_SMD:R_0402" H 9600 1200 50  0001 C CNN
 F 3 "" H 9600 1200 50  0001 C CNN
 	1    9600 1200
@@
 F 0 "R?" H 10230 1220 50  0000 L CNN
 F 1 "10k" H 10230 1160 50  0000 L CNN
-F 2 "" H 10200 1200 50  0001 C CNN
+F 2 "Resistors_SMD:R_0402" H 10200 1200 50  0001 C CNN
 F 3 "" H 10200 1200 50  0001 C CNN
 	1    10200 1200
@@
 F 0 "R?" H 9630 2370 50  0000 L CNN
 F 1 "10k" H 9630 2310 50  0000 L CNN
-F 2 "" H 9600 2350 50  0001 C CNN
+F 2 "Resistors_SMD:R_0402" H 9600 2350 50  0001 C CNN
 F 3 "" H 9600 2350 50  0001 C CNN
 	1    9600 2350
@@
 F 0 "R?" H 10230 2370 50  0000 L CNN
 F 1 "10k" H 10230 2310 50  0000 L CNN
-F 2 "" H 10200 2350 50  0001 C CNN
+F 2 "Resistors_SMD:R_0402" H 10200 2350 50  0001 C CNN
 F 3 "" H 10200 2350 50  0001 C CNN
 	1    10200 2350
@@
 F 0 "R?" H 9630 3520 50  0000 L CNN
 F 1 "10k" H 9630 3460 50  0000 L CNN
-F 2 "" H 9600 3500 50  0001 C CNN
+F 2 "Resistors_SMD:R_0402" H 9600 3500 50  0001 C CNN
 F 3 "" H 9600 3500 50  0001 C CNN
 	1    9600 3500
@@
 F 0 "R?" H 10230 3520 50  0000 L CNN
 F 1 "10k" H 10230 3460 50  0000 L CNN
-F 2 "" H 10200 3500 50  0001 C CNN
+F 2 "Resistors_SMD:R_0402" H 10200 3500 50  0001 C CNN
 F 3 "" H 10200 3500 50  0001 C CNN
 	1    10200 3500
@@
 F 0 "R?" H 9630 4670 50  0000 L CNN
 F 1 "10k" H 9630 4610 50  0000 L CNN
-F 2 "" H 9600 4650 50  0001 C CNN
+F 2 "Resistors_SMD:R_0402" H 9600 4650 50  0001 C CNN
 F 3 "" H 9600 4650 50  0001 C CNN
 	1    9600 4650
@@
 F 0 "R?" H 10230 4670 50  0000 L CNN
 F 1 "10k" H 10230 4610 50  0000 L CNN
-F 2 "" H 10200 4650 50  0001 C CNN
+F 2 "Resistors_SMD:R_0402" H 10200 4650 50  0001 C CNN
 F 3 "" H 10200 4650 50  0001 C CNN
 	1    10200 4650
@@
 F 0 "C?" H 660 4220 50  0000 L CNN
 F 1 "100 nF" H 660 4070 50  0000 L CNN
-F 2 "" H 650 4150 50  0001 C CNN
+F 2 "Capacitors_SMD:C_0201" H 650 4150 50  0001 C CNN
 F 3 "" H 650 4150 50  0001 C CNN
 	1    650  4150
@@
 F 0 "C?" H 960 4220 50  0000 L CNN
 F 1 "100 nF" H 960 4070 50  0000 L CNN
-F 2 "" H 950 4150 50  0001 C CNN
+F 2 "Capacitors_SMD:C_0201" H 950 4150 50  0001 C CNN
 F 3 "" H 950 4150 50  0001 C CNN
 	1    950  4150
@@
 F 0 "C?" H 1260 4220 50  0000 L CNN
 F 1 "100 nF" H 1260 4070 50  0000 L CNN
-F 2 "" H 1250 4150 50  0001 C CNN
+F 2 "Capacitors_SMD:C_0201" H 1250 4150 50  0001 C CNN
 F 3 "" H 1250 4150 50  0001 C CNN
 	1    1250 4150
@@
 F 0 "C?" H 1610 4220 50  0000 L CNN
 F 1 "100 nF" H 1610 4070 50  0000 L CNN
-F 2 "" H 1600 4150 50  0001 C CNN
+F 2 "Capacitors_SMD:C_0201" H 1600 4150 50  0001 C CNN
 F 3 "" H 1600 4150 50  0001 C CNN
 	1    1600 4150
@@
 F 0 "C?" H 1910 4220 50  0000 L CNN
 F 1 "100 nF" H 1910 4070 50  0000 L CNN
-F 2 "" H 1900 4150 50  0001 C CNN
+F 2 "Capacitors_SMD:C_0201" H 1900 4150 50  0001 C CNN
 F 3 "" H 1900 4150 50  0001 C CNN
 	1    1900 4150
@@
 F 0 "C?" H 2210 4220 50  0000 L CNN
 F 1 "100 nF" H 2210 4070 50  0000 L CNN
-F 2 "" H 2200 4150 50  0001 C CNN
+F 2 "Capacitors_SMD:C_0201" H 2200 4150 50  0001 C CNN
 F 3 "" H 2200 4150 50  0001 C CNN
 	1    2200 4150
@@
 F 0 "R?" H 3380 2420 50  0000 L CNN
 F 1 "10k" H 3380 2360 50  0000 L CNN
-F 2 "" H 3350 2400 50  0001 C CNN
+F 2 "Resistors_SMD:R_0402" H 3350 2400 50  0001 C CNN
 F 3 "" H 3350 2400 50  0001 C CNN
 	1    3350 2400
@@
 F 0 "R?" H 3380 4720 50  0000 L CNN
 F 1 "10k" H 3380 4660 50  0000 L CNN
-F 2 "" H 3350 4700 50  0001 C CNN
+F 2 "Resistors_SMD:R_0402" H 3350 4700 50  0001 C CNN
 F 3 "" H 3350 4700 50  0001 C CNN
 	1    3350 4700
@@
 F 0 "R?" H 3430 7020 50  0000 L CNN
 F 1 "10k" H 3430 6960 50  0000 L CNN
-F 2 "" H 3400 7000 50  0001 C CNN
+F 2 "Resistors_SMD:R_0402" H 3400 7000 50  0001 C CNN
 F 3 "" H 3400 7000 50  0001 C CNN
 	1    3400 7000

Commit message: Added Second SPI Bus for IMUs to Cam Connector
This SPI works on 1.8 V, don't confuse them. If this second SPI Bus shall be used for the Cam Chips, add Levelshifters on the Cam Board.

Also reorderd some stuff around this connector, to ease routing
Parts:
- U? (x3): footprint Housings_SSOP:TSSOP-24_4.4x7.8mm_Pitch0.65mm -> footprints:VQFN-24
Connections:
- no-connect marks 6 -> 3

Commit message: Triggerbus WIP.
Also added more production data
Parts:
- removed Q? (x4): BSS138, TO_SOT_Packages_SMD:SOT-23, symbol BSS138
- added Q? (x4): BSS138PS, TO_SOT_Packages_SMD:SOT-363_SC-70-6, symbol BSS138PS
- R? (x2): Populated (none) -> 1; Source (none) -> SPEC
- U? (x3): Digikey (none) -> 296-48832-1-ND; MFG Name (none) -> Texas Instruments; MFG Part Num (none) -> SN74AXC8T245; Mouser (none) -> 595-SN74AXC8T245RHLR; Populated (none) -> 1; Source (none) -> SPEC

Commit message: Added Sdcard Slot.
Parts:
- gave numbers to parts that had none: 28

Commit message: Added USB-Uart subschematic. WIP
USB-Uart will be bus powered. Buffer between FTDI and FPGA is missing.
Parts:
- renumbered C71 to C?, C72 to C?, C73 to C?, C74 to C?, C75 to C?, C76 to C?, Q1 to Q?, Q2 to Q?, R88 to R?, R89 to R?, R82 to R?, R83 to R?, R85 to R?, R86 to R?, R91 to R?, R95 to R?, R92 to R?, R96 to R?, R93 to R?, R97 to R?, R94 to R?, R98 to R?, R84 to R?, R87 to R?, R90 to R?, U16 to U?, U14 to U?, U15 to U?
