File: hardware/TLK10031_Power.sch (KiCad schematic (older format))
At the start: 1 part

Commit message: Almost drew 3,3 V lowspeed signals. Added Levelshifter Subschematic
1,8 V Lowspeed Singals from 10 G Phy to FPGA are still missing.

CAM_REF_CLK is not really low speed, maybe we should consider to use the lvds clock instead. I think it will work, since the signal should be realtive short(FPGA->Connector->Camerasensor[->Camerasensor2]). The levelshifter should also be fast enough.

The i2c signals use simple N-Channel MOSTFET Transistors for Levelshifting
Connections:
- net labels added: +1V8
- net labels removed: +1V5
Changed lines of the file:
@@
 LIBS:misc
 LIBS:tlk10031
+LIBS:lshm-150-xxx-x-dv-a-s
+LIBS:sn74axc8t245
 LIBS:zynq_board-cache
 EELAYER 25 0
@@
 $Descr A4 11693 8268
 encoding utf-8
-Sheet 18 18
+Sheet 16 19
 Title ""
 Date ""
@@
 Connection ~ 6650 2950
 Connection ~ 6750 2950
-$Comp
-L +1V5 #PWR?
-U 1 1 5ACA62F0
-P 6650 2850
-F 0 "#PWR?" H 6650 2700 50  0001 C CNN
-F 1 "+1V5" H 6650 2990 50  0000 C CNN
-F 2 "" H 6650 2850 50  0001 C CNN
-F 3 "" H 6650 2850 50  0001 C CNN
-	1    6650 2850
-	1    0    0    -1
-$EndComp
 Wire Wire Line
 	6650 2850 6650 2950
-Text Notes 6450 2650 0    60   ~ 0
-1V5 or 1V8
 Wire Wire Line
 	7350 2950 7450 2950
-$Comp
-L +1V5 #PWR?
-U 1 1 5ACA694F
-P 7350 2850
-F 0 "#PWR?" H 7350 2700 50  0001 C CNN
-F 1 "+1V5" H 7350 2990 50  0000 C CNN
-F 2 "" H 7350 2850 50  0001 C CNN
-F 3 "" H 7350 2850 50  0001 C CNN
-	1    7350 2850
-	1    0    0    -1
-$EndComp
 Wire Wire Line
 	7350 2850 7350 2950
@@
 Text Notes 3450 5450 0    60   ~ 0
 Note: Decoupling Cpacitors may missing!
+Text Notes 6450 2650 0    60   ~ 0
+1V5 or 1V8
+$Comp
+L +1V8 #PWR?
+U 1 1 5AC913A1
+P 6650 2850
+F 0 "#PWR?" H 6650 2700 50  0001 C CNN
+F 1 "+1V8" H 6650 2990 50  0000 C CNN
+F 2 "" H 6650 2850 50  0001 C CNN
+F 3 "" H 6650 2850 50  0001 C CNN
+	1    6650 2850
+	1    0    0    -1
+$EndComp
+$Comp
+L +1V8 #PWR?
+U 1 1 5AC913B6
+P 7350 2850
+F 0 "#PWR?" H 7350 2700 50  0001 C CNN
+F 1 "+1V8" H 7350 2990 50  0000 C CNN
+F 2 "" H 7350 2850 50  0001 C CNN
+F 3 "" H 7350 2850 50  0001 C CNN
+	1    7350 2850
+	1    0    0    -1
+$EndComp
 $EndSCHEMATC

Commit message: KiCad does not support differential Busses yet. See https://bugs.launchpad.net/kicad/+bug/1419146. Fixed Data Lanes for Camera Connector.
Parts:
- U?: footprint (none) -> footprints:TI-CTR_FCBGA_N144_12x12_13x13mm_Pitch1.0mm
Changed lines of the file:
@@
 $Descr A4 11693 8268
 encoding utf-8
-Sheet 16 19
+Sheet 15 19
 Title ""
 Date ""
@@
 F 0 "U?" H 5550 3600 60  0000 C CNN
 F 1 "TLK10031" H 5550 3700 60  0000 C CNN
-F 2 "" H 5250 3150 60  0001 C CNN
+F 2 "footprints:TI-CTR_FCBGA_N144_12x12_13x13mm_Pitch1.0mm" H 5250 3150 60  0001 C CNN
 F 3 "" H 5250 3150 60  0001 C CNN
 	2    5550 3650

Commit message: Added Sdcard Slot.
Parts:
- gave numbers to parts that had none: 1
Changed lines of the file:
@@
 $Descr A4 11693 8268
 encoding utf-8
-Sheet 15 21
+Sheet 15 20
 Title ""
 Date ""
@@
 $EndDescr
 $Comp
-L TLK10031 U?
+L TLK10031 U13
 U 2 1 5ACA3B74
 P 5550 3650
-F 0 "U?" H 5550 3600 60  0000 C CNN
+F 0 "U13" H 5550 3600 60  0000 C CNN
 F 1 "TLK10031" H 5550 3700 60  0000 C CNN
 F 2 "footprints:TI-CTR_FCBGA_N144_12x12_13x13mm_Pitch1.0mm" H 5250 3150 60  0001 C CNN
@@
 $EndComp
 $Comp
-L GND #PWR060
+L GND #PWR068
 U 1 1 5ACA4579
 P 5450 4500
-F 0 "#PWR060" H 5450 4250 50  0001 C CNN
+F 0 "#PWR068" H 5450 4250 50  0001 C CNN
 F 1 "GND" H 5450 4350 50  0000 C CNN
 F 2 "" H 5450 4500 50  0001 C CNN
@@
 Connection ~ 3450 2950
 $Comp
-L +1V0 #PWR061
+L +1V0 #PWR069
 U 1 1 5ACA5A88
 P 3250 2850
-F 0 "#PWR061" H 3250 2700 50  0001 C CNN
+F 0 "#PWR069" H 3250 2700 50  0001 C CNN
 F 1 "+1V0" H 3250 2990 50  0000 C CNN
 F 2 "" H 3250 2850 50  0001 C CNN
@@
 Connection ~ 4150 2950
 $Comp
-L +1V0 #PWR062
+L +1V0 #PWR070
 U 1 1 5ACA60C7
 P 4150 2850
-F 0 "#PWR062" H 4150 2700 50  0001 C CNN
+F 0 "#PWR070" H 4150 2700 50  0001 C CNN
 F 1 "+1V0" H 4150 2990 50  0000 C CNN
 F 2 "" H 4150 2850 50  0001 C CNN
@@
 Connection ~ 5050 2950
 $Comp
-L +1V0 #PWR063
+L +1V0 #PWR071
 U 1 1 5ACA6173
 P 4950 2850
-F 0 "#PWR063" H 4950 2700 50  0001 C CNN
+F 0 "#PWR071" H 4950 2700 50  0001 C CNN
 F 1 "+1V0" H 4950 2990 50  0000 C CNN
 F 2 "" H 4950 2850 50  0001 C CNN
@@
 Connection ~ 5950 2950
 $Comp
-L +1V0 #PWR064
+L +1V0 #PWR072
 U 1 1 5ACA6227
 P 5850 2850
-F 0 "#PWR064" H 5850 2700 50  0001 C CNN
+F 0 "#PWR072" H 5850 2700 50  0001 C CNN
 F 1 "+1V0" H 5850 2990 50  0000 C CNN
 F 2 "" H 5850 2850 50  0001 C CNN
@@
 1V5 or 1V8
 $Comp
-L +1V8 #PWR065
+L +1V8 #PWR073
 U 1 1 5AC913A1
 P 6650 2850
-F 0 "#PWR065" H 6650 2700 50  0001 C CNN
+F 0 "#PWR073" H 6650 2700 50  0001 C CNN
 F 1 "+1V8" H 6650 2990 50  0000 C CNN
 F 2 "" H 6650 2850 50  0001 C CNN
@@
 $EndComp
 $Comp
-L +1V8 #PWR066
+L +1V8 #PWR074
 U 1 1 5AC913B6
 P 7350 2850
-F 0 "#PWR066" H 7350 2700 50  0001 C CNN
+F 0 "#PWR074" H 7350 2700 50  0001 C CNN
 F 1 "+1V8" H 7350 2990 50  0000 C CNN
 F 2 "" H 7350 2850 50  0001 C CNN

Commit message: Added USB-Uart subschematic. WIP
USB-Uart will be bus powered. Buffer between FTDI and FPGA is missing.
Parts:
- renumbered U13 to U?
Changed lines of the file:
@@
 LIBS:max14854
 LIBS:switches
+LIBS:ft234xd
 LIBS:zynq_board-cache
 EELAYER 25 0
@@
 $Descr A4 11693 8268
 encoding utf-8
-Sheet 15 20
+Sheet 15 21
 Title ""
 Date ""
@@
 $EndDescr
 $Comp
-L TLK10031 U13
+L TLK10031 U?
 U 2 1 5ACA3B74
 P 5550 3650
-F 0 "U13" H 5550 3600 60  0000 C CNN
+F 0 "U?" H 5550 3600 60  0000 C CNN
 F 1 "TLK10031" H 5550 3700 60  0000 C CNN
 F 2 "footprints:TI-CTR_FCBGA_N144_12x12_13x13mm_Pitch1.0mm" H 5250 3150 60  0001 C CNN
@@
 $EndComp
 $Comp
-L GND #PWR068
+L GND #PWR?
 U 1 1 5ACA4579
 P 5450 4500
-F 0 "#PWR068" H 5450 4250 50  0001 C CNN
+F 0 "#PWR?" H 5450 4250 50  0001 C CNN
 F 1 "GND" H 5450 4350 50  0000 C CNN
 F 2 "" H 5450 4500 50  0001 C CNN
@@
 Connection ~ 3450 2950
 $Comp
-L +1V0 #PWR069
+L +1V0 #PWR?
 U 1 1 5ACA5A88
 P 3250 2850
-F 0 "#PWR069" H 3250 2700 50  0001 C CNN
+F 0 "#PWR?" H 3250 2700 50  0001 C CNN
 F 1 "+1V0" H 3250 2990 50  0000 C CNN
 F 2 "" H 3250 2850 50  0001 C CNN
@@
 Connection ~ 4150 2950
 $Comp
-L +1V0 #PWR070
+L +1V0 #PWR?
 U 1 1 5ACA60C7
 P 4150 2850
-F 0 "#PWR070" H 4150 2700 50  0001 C CNN
+F 0 "#PWR?" H 4150 2700 50  0001 C CNN
 F 1 "+1V0" H 4150 2990 50  0000 C CNN
 F 2 "" H 4150 2850 50  0001 C CNN
@@
 Connection ~ 5050 2950
 $Comp
-L +1V0 #PWR071
+L +1V0 #PWR?
 U 1 1 5ACA6173
 P 4950 2850
-F 0 "#PWR071" H 4950 2700 50  0001 C CNN
+F 0 "#PWR?" H 4950 2700 50  0001 C CNN
 F 1 "+1V0" H 4950 2990 50  0000 C CNN
 F 2 "" H 4950 2850 50  0001 C CNN
@@
 Connection ~ 5950 2950
 $Comp
-L +1V0 #PWR072
+L +1V0 #PWR?
 U 1 1 5ACA6227
 P 5850 2850
-F 0 "#PWR072" H 5850 2700 50  0001 C CNN
+F 0 "#PWR?" H 5850 2700 50  0001 C CNN
 F 1 "+1V0" H 5850 2990 50  0000 C CNN
 F 2 "" H 5850 2850 50  0001 C CNN
@@
 1V5 or 1V8
 $Comp
-L +1V8 #PWR073
+L +1V8 #PWR?
 U 1 1 5AC913A1
 P 6650 2850
-F 0 "#PWR073" H 6650 2700 50  0001 C CNN
+F 0 "#PWR?" H 6650 2700 50  0001 C CNN
 F 1 "+1V8" H 6650 2990 50  0000 C CNN
 F 2 "" H 6650 2850 50  0001 C CNN
@@
 $EndComp
 $Comp
-L +1V8 #PWR074
+L +1V8 #PWR?
 U 1 1 5AC913B6
 P 7350 2850
-F 0 "#PWR074" H 7350 2700 50  0001 C CNN
+F 0 "#PWR?" H 7350 2700 50  0001 C CNN
 F 1 "+1V8" H 7350 2990 50  0000 C CNN
 F 2 "" H 7350 2850 50  0001 C CNN
