File: hardware/triggerbus.sch (KiCad schematic (older format))
At the start: 6 parts

Commit message: Triggerbus WIP.
Also added more production data
Parts:
- added 10k, R? (x3): DNP, symbol R_Small
- added R? (x2): 10k, symbol R_Small
- added R? (x6): 270, symbol R_Small
- added U? (x3): SN74LVC2T45, footprints:DSBGA_2x4_0.918x1.918mm_Pitch0.5mm, symbol SN74LVC2T45
- added U? (x2): DMF05LCFLP, Housings_DFN_QFN:DFN-6-1EP_2x2mm_Pitch0.5mm, symbol DMF05LCFLP
- U?: Digikey (none) -> 296-17036-1-ND; MFG Name (none) -> Texas Instruments; MFG Part Num (none) -> SN74LVC2T45YZP; Populated (none) -> 1; Source (none) -> SPEC
Connections:
- net labels added: TRIG_IN_2, TRIG_IN_3, TRIG_OUT_0, TRIG_OUT_1, TRIG_OUT_2, TRIG_OUT_3
- wire segments 14 -> 74

Commit message: Finished Triggerbus and added GPIO Header to schematic.
Also moved some Connections to the FPGA around to hopefully ease routing.
Parts:
- removed J?: DB15_Male, symbol DB15_Male
- added C? (x11): 100 nF, symbol C_Small
- added C? (x3): 1 µF, symbol C_Small
- added J?: DB15_Female, symbol DB15_Female
- added U?: MAX14854, Housings_SOIC:SOIC-16W_7.5x10.3mm_Pitch1.27mm, symbol MAX14854
Connections:
- net labels added: +5V, A, B, DE, EXT_TRIG_IN_0, EXT_TRIG_IN_1, EXT_TRIG_IN_2, EXT_TRIG_IN_3, EXT_TRIG_OUT_0, EXT_TRIG_OUT_1, EXT_TRIG_OUT_2, EXT_TRIG_OUT_3, RXD, TXD, Y, Z, ~RE~, ~SBA~
- wire segments 74 -> 149
Other:
- note added: "Bypass Capacitors for MAX14854.\nPlace as close as possible to it"
- note added: "Bypass Capacitors for the Triggerbus Levelshifters.\nPlace them as close as possible to their power inputs."
- note added: "Ideas:\nTriggerbus should be as robust as possible. That means 5 V tolerant,\nidiot Diodes at Poweroutputs, ESD protection Diodes, current limiting Resistors."
- note added: "TODO: Select Connector and connect it"
- note removed: "Ideas:\nTriggerbus should be as robust as possible. That means 5 V tolerant,\nidiot Diodes at Poweroutputs, ESD protection Diodes, current limiting Resistors.\n\nAdditional Ideas:\nMaybe allow to switch between input and output Operation, thats not much overhead."

Commit message: Added Sdcard Slot.
Parts:
- gave numbers to parts that had none: 37
- renumbered 10k to 10k1

Commit message: Added USB-Uart subschematic. WIP
USB-Uart will be bus powered. Buffer between FTDI and FPGA is missing.
Parts:
- renumbered 10k1 to 10k?, C88 to C?, C87 to C?, C86 to C?, C85 to C?, C89 to C?, C90 to C?, C77 to C?, C78 to C?, C79 to C?, C80 to C?, C81 to C?, C82 to C?, C83 to C?, C84 to C?, J6 to J?, R100 to R?, R106 to R?, R107 to R?, R99 to R?, R101 to R?, R102 to R?, R108 to R?, R109 to R?, R103 to R?, R104 to R?, R110 to R?, R111 to R?, R105 to R?, R112 to R?, R113 to R?, U23 to U?, U18 to U?, U19 to U?, U20 to U?, U22 to U?, U21 to U?, U17 to U?

Commit message: Added decoupling Caps for TLK
Parts:
- added D? (x2): D, symbol D
Connections:
- wire segments 149 -> 151
Other:
- note added: "So called Idiot Diodes.\nThey protect the Board from reverse Current,\nbut consume 0,5 to 0,7 V."
- note removed: "TODO: Select Connector and connect it"
Changed lines of the file:
@@
 Text HLabel 8350 2700 0    60   Input ~ 0
 TXD
-Text Notes 6100 6250 0    60   ~ 0
-TODO: Select Connector and connect it
 Connection ~ 4350 1400
 Connection ~ 4450 1500
@@
 EXT_TRIG_OUT_0
 Wire Wire Line
-	10050 5250 9200 5250
-Wire Wire Line
-	10050 5350 9200 5350
-Wire Wire Line
 	10050 5450 9950 5450
 Wire Wire Line
@@
 	0    -1   -1   0
 $EndComp
+$Comp
+L D D?
+U 1 1 5ADD1C0F
+P 9700 5250
+F 0 "D?" H 9700 5350 50  0000 C CNN
+F 1 "D" H 9700 5150 50  0000 C CNN
+F 2 "" H 9700 5250 50  0001 C CNN
+F 3 "" H 9700 5250 50  0001 C CNN
+	1    9700 5250
+	-1   0    0    1
+$EndComp
+$Comp
+L D D?
+U 1 1 5ADD1CFF
+P 9700 5350
+F 0 "D?" H 9700 5450 50  0000 C CNN
+F 1 "D" H 9700 5250 50  0000 C CNN
+F 2 "" H 9700 5350 50  0001 C CNN
+F 3 "" H 9700 5350 50  0001 C CNN
+	1    9700 5350
+	-1   0    0    1
+$EndComp
+Wire Wire Line
+	9850 5250 10050 5250
+Wire Wire Line
+	10050 5350 9850 5350
+Wire Wire Line
+	9550 5350 9200 5350
+Wire Wire Line
+	9200 5250 9550 5250
+Wire Notes Line
+	9500 5150 9500 5550
+Wire Notes Line
+	9500 5550 9850 5550
+Wire Notes Line
+	9850 5550 9850 5150
+Wire Notes Line
+	9850 5150 9500 5150
+Text Notes 9000 6050 0    60   ~ 0
+So called Idiot Diodes.\nThey protect the Board from reverse Current,\nbut consume 0,5 to 0,7 V.
 $EndSCHEMATC

Commit message: Added LDO for Triggerbus.
Parts:
- removed D? (x2): D, symbol D
- added C? (x2): 1 µF, Capacitors_SMD:C_0603, symbol C_Small
- added D?: D_Schottky, symbol D_Schottky
- added U?: TC1262-33, TO_SOT_Packages_SMD:SOT-223, symbol TC1262-33
Connections:
- net labels added: 3.3V_OUT, 5V_OUT
- wire segments 151 -> 159
Other:
- note removed: "So called Idiot Diodes.\nThey protect the Board from reverse Current,\nbut consume 0,5 to 0,7 V."
