File: hardware/triggerbus.sch (KiCad schematic (older format))
At the start: 42 parts, among them J6 MDR20, U28 SN74LVC2T45, U29 SN74LVC2T45, U30 SN74LVC2T45, U31 SN74LVC2T45, U32 DMF05LCFLP, U33 DMF05LCFLP, U34 TC1262-33, U35 MAX14854

Commit message: Added Power/Protection Circuit
Parts:
- renumbered 10k1 to 10k1501, C223 to C1501, C224 to C1502, C225 to C1503, C226 to C1504, C227 to C1505, C228 to C1506, C229 to C1507, C230 to C1508, C231 to C1509, C232 to C1510, C233 to C1511, C234 to C1512, C235 to C1513, C236 to C1514, C237 to C1515, C238 to C1516, D3 to D1501, J6 to J1501, R127 to R1501, R128 to R1502, R129 to R1503, R130 to R1504, R131 to R1505, R132 to R1506, R133 to R1507, R134 to R1508, R135 to R1509, R136 to R1510, R137 to R1511, R138 to R1512, R139 to R1513, R140 to R1514, R141 to R1515, U28 to U1501, U29 to U1502, U30 to U1503, U31 to U1504, U32 to U1505, U33 to U1506, U34 to U1507, U35 to U1508

Commit message: Length matched DDR3 Memory again.
Forgot to keep enough space between the traces and between the meander waves.

Also, I switched to Kicad 5.0 RC2.

Swaped a few ddr signals.
Parts:
- 10k1501, R1501, R1502, R1503, R1504, R1505, R1506, R1507, R1508, R1509, R1510, R1511, R1512, R1513, R1514, R1515: symbol R_Small -> device:R_Small
- C1501, C1502, C1503, C1504, C1505, C1506, C1507, C1508, C1509, C1510, C1511, C1512, C1513, C1514, C1515, C1516: symbol C_Small -> device:C_Small
- D1501: symbol D_Schottky -> device:D_Schottky
- J1501: symbol MDR20 -> mdr20:MDR20
- U1501, U1502, U1503, U1504: symbol SN74LVC2T45 -> sn74lvc2t45:SN74LVC2T45
- U1505, U1506: symbol DMF05LCFLP -> dmf05lcflp:DMF05LCFLP
- U1507: symbol TC1262-33 -> regul:TC1262-33
- U1508: symbol MAX14854 -> dmf05lcflp:MAX14854

Commit message: Layouted most of the Power Circuit and Triggerbus Levelshifters.
Added Footprint for Tantal Caps. Modified Footprint for MDR20 Connector, SD-Card.

Fixed Symbol and Circuit for Power Supervisor/Delay IC.

Also fixed some smaller things in the schematics.
Parts:
- C1501, C1502, C1503, C1504, C1505, C1506, C1507, C1508, C1512, C1514, C1515: footprint (none) -> Capacitor_SMD:C_0201_0603Metric; Description (none) -> CAP CER 0.1UF 6.3V X5R 0201; Digikey (none) -> 490-3167-1-ND; MFG Name (none) -> Murata Electronics North America; MFG Part Num (none) -> GRM033R60J104KE19D; Populate for CLG484(Z-7012s/Z-7015) (none) -> 1; Populate for SBGA485(Z-7030) (none) -> 1; Populated (none) -> 1; Source (none) -> SPEC
- C1509, C1510: footprint Capacitors_SMD:C_0402 -> Capacitor_SMD:C_0402_1005Metric; Populate for CLG484(Z-7012s/Z-7015) (none) -> 1; Populate for SBGA485(Z-7030) (none) -> 1
- C1511, C1513, C1516: value 1 µF -> 1 µF 6,3 V; footprint (none) -> Capacitor_SMD:C_0402_1005Metric; Description (none) -> CAP CER 1UF 6.3V X5R 0402; Digikey (none) -> 490-10006-1-ND; MFG Name (none) -> Murata Electronics North America; MFG Part Num (none) -> GRM152R60J105ME15D; Populate for CLG484(Z-7012s/Z-7015) (none) -> 1; Populate for SBGA485(Z-7030) (none) -> 1; Populated (none) -> 1; Source (none) -> SPEC
- D1501: value D_Schottky -> PMEG3020EGWX; footprint (none) -> Diode_SMD:D_SOD-123; Description (none) -> DIODE SCHOTTKY 30V 2A SOD123; Digikey (none) -> 1727-7331-1-ND; MFG Name (none) -> Nexperia USA Inc.; MFG Part Num (none) -> PMEG3020EGWX; Populate for CLG484(Z-7012s/Z-7015) (none) -> 1; Populate for SBGA485(Z-7030) (none) -> 1; Populated (none) -> 1; Source (none) -> SPEC
- R1501, R1502, R1503, R1504, R1505, R1506, R1507, R1508, R1509, R1510, R1511, R1512, R1513, R1514, R1515: footprint (none) -> Resistor_SMD:R_0402_1005Metric; Populate for CLG484(Z-7012s/Z-7015) (none) -> 1; Populate for SBGA485(Z-7030) (none) -> 1; Populated (none) -> 1; Source (none) -> SPEC
- R1516: renamed from 10k1501; value DNP -> 10k; footprint (none) -> Resistor_SMD:R_0402_1005Metric; Populate for CLG484(Z-7012s/Z-7015) (none) -> 1; Populate for SBGA485(Z-7030) (none) -> 1; Populated (none) -> 1; Source (none) -> SPEC
- U1506: Populate for CLG484(Z-7012s/Z-7015) (none) -> 1; Populate for SBGA485(Z-7030) (none) -> 1
- U1507: symbol regul:TC1262-33 -> TC1262:TC1262-33; Populate for CLG484(Z-7012s/Z-7015) (none) -> 1; Populate for SBGA485(Z-7030) (none) -> 1
Connections:
- wire segments 164 -> 206
Other:
- moved on the sheet: U1505, U1506

Commit message: Layouted USB-UART.
Also moved USB-OTG to the right Side of the Board. To get there
some free Space, i moved the DDR3/Memory and the FPGA a few
Millimeters down.
Parts:
- added F1501: Fuse, Fuse:Fuse_1206_3216Metric, symbol device:Fuse
Connections:
- net labels removed: +3V3
- wire segments 206 -> 214
Changed lines of the file:
@@
 TRIG_IN_1
-$Comp
-L power1:+3V3 #PWR0188
-U 1 1 5AD03794
-P 3300 1150
-F 0 "#PWR0188" H 3300 1000 50  0001 C CNN
-F 1 "+3V3" H 3300 1290 50  0000 C CNN
-F 2 "" H 3300 1150 50  0001 C CNN
-F 3 "" H 3300 1150 50  0001 C CNN
-	1    3300 1150
-	1    0    0    -1
-$EndComp
 $Comp
 L device:R_Small R1508
@@
 TRIG_IN_3
 $Comp
-L power1:+3V3 #PWR0193
-U 1 1 5AE68070
-P 3300 2400
-F 0 "#PWR0193" H 3300 2250 50  0001 C CNN
-F 1 "+3V3" H 3300 2540 50  0000 C CNN
-F 2 "" H 3300 2400 50  0001 C CNN
-F 3 "" H 3300 2400 50  0001 C CNN
-	1    3300 2400
-	1    0    0    -1
-$EndComp
-$Comp
 L device:R_Small R1510
 U 1 1 5AE68076
@@
 TRIG_OUT_1
 $Comp
-L power1:+3V3 #PWR0198
-U 1 1 5AE683CD
-P 3300 3650
-F 0 "#PWR0198" H 3300 3500 50  0001 C CNN
-F 1 "+3V3" H 3300 3790 50  0000 C CNN
-F 2 "" H 3300 3650 50  0001 C CNN
-F 3 "" H 3300 3650 50  0001 C CNN
-	1    3300 3650
-	1    0    0    -1
-$EndComp
-$Comp
 L device:R_Small R1512
 U 1 1 5AE683D3
@@
 Text HLabel 1950 5250 0    60   Input ~ 0
 TRIG_OUT_3
-$Comp
-L power1:+3V3 #PWR0203
-U 1 1 5AE6841A
-P 3400 6350
-F 0 "#PWR0203" H 3400 6200 50  0001 C CNN
-F 1 "+3V3" H 3400 6490 50  0000 C CNN
-F 2 "" H 3400 6350 50  0001 C CNN
-F 3 "" H 3400 6350 50  0001 C CNN
-	1    3400 6350
-	1    0    0    -1
-$EndComp
 $Comp
 L device:R_Small R1514
@@
 	1    9500 800
 	1    0    0    1
-$EndComp
-$Comp
-L power1:+3V3 #PWR0211
-U 1 1 5AD9904E
-P 9050 1650
-F 0 "#PWR0211" H 9050 1500 50  0001 C CNN
-F 1 "+3V3" H 9050 1790 50  0000 C CNN
-F 2 "" H 9050 1650 50  0001 C CNN
-F 3 "" H 9050 1650 50  0001 C CNN
-	1    9050 1650
-	1    0    0    -1
 $EndComp
 Text Notes 5850 800  0    60   ~ 0
@@
 L power1:+5V #PWR0216
 U 1 1 5B11913A
-P 5850 4300
-F 0 "#PWR0216" H 5850 4150 50  0001 C CNN
-F 1 "+5V" V 5850 4550 50  0000 C CNN
-F 2 "" H 5850 4300 50  0001 C CNN
-F 3 "" H 5850 4300 50  0001 C CNN
-	1    5850 4300
-	0    -1   -1   0
+P 5850 3750
+F 0 "#PWR0216" H 5850 3600 50  0001 C CNN
+F 1 "+5V" V 5850 4000 50  0000 C CNN
+F 2 "" H 5850 3750 50  0001 C CNN
+F 3 "" H 5850 3750 50  0001 C CNN
+	1    5850 3750
+	1    0    0    -1
 $EndComp
 $Comp
@@
 	2100 1250 2200 1250
 Wire Wire Line
-	3300 1150 3300 1250
-Wire Wire Line
 	3300 1250 3200 1250
 Wire Wire Line
@@
 	2100 2500 2200 2500
 Wire Wire Line
-	3300 2400 3300 2500
-Wire Wire Line
 	3300 2500 3200 2500
 Wire Wire Line
@@
 	2100 3750 2200 3750
 Wire Wire Line
-	3300 3650 3300 3750
-Wire Wire Line
 	3300 3750 3200 3750
 Wire Wire Line
@@
 	2100 5000 2200 5000
 Wire Wire Line
-	3300 4900 3300 5000
-Wire Wire Line
 	3300 5000 3200 5000
 Wire Wire Line
@@
 	9500 800  9500 900
 Connection ~ 9500 900
-Wire Wire Line
-	9050 1650 9050 1700
 Wire Wire Line
 	9350 1200 9350 1300
@@
 	2050 6350 2050 6450
 Connection ~ 2050 6450
-Wire Wire Line
-	3400 6350 3400 6450
 Connection ~ 3400 6450
 Wire Notes Line
@@
 	10300 5250 10650 5250
 Wire Wire Line
-	5850 4300 6000 4300
-Wire Wire Line
 	6300 4300 6600 4300
 $Comp
@@
 	-1   0    0    1
 $EndComp
-$Comp
-L power1:+3V3 #PWR0264
-U 1 1 5B2BC772
-P 3300 4900
-F 0 "#PWR0264" H 3300 4750 50  0001 C CNN
-F 1 "+3V3" H 3300 5040 50  0000 C CNN
-F 2 "" H 3300 4900 50  0001 C CNN
-F 3 "" H 3300 4900 50  0001 C CNN
-	1    3300 4900
-	1    0    0    -1
-$EndComp
+Text Label 3900 700  3    60   ~ 0
+5V_OUT
+Wire Wire Line
+	3900 700  3900 1300
+Wire Wire Line
+	3900 1300 4250 1300
+Wire Wire Line
+	4250 1300 4250 1200
+Wire Wire Line
+	3900 3700 4150 3700
+Wire Wire Line
+	4150 3700 4150 3600
+Text Label 3900 3200 3    60   ~ 0
+3.3V_OUT
+Wire Wire Line
+	3900 3200 3900 3700
+Text Label 3300 800  3    60   ~ 0
+3.3V_OUT
+Text Label 3300 2050 3    60   ~ 0
+3.3V_OUT
+Text Label 3300 3300 3    60   ~ 0
+3.3V_OUT
+Text Label 3300 4550 3    60   ~ 0
+3.3V_OUT
+Wire Wire Line
+	3300 4550 3300 5000
+Wire Wire Line
+	3300 2050 3300 2500
+Wire Wire Line
+	3300 800  3300 1250
+Text Label 9050 1250 3    60   ~ 0
+3.3V_OUT
+Wire Wire Line
+	9050 1250 9050 1700
+Text Label 3400 6250 0    60   ~ 0
+3.3V_OUT
+Wire Wire Line
+	3400 6250 3400 6450
+Wire Wire Line
+	3300 3300 3300 3750
+$Comp
+L device:Fuse F1501
+U 1 1 5B4B93EE
+P 5850 4000
+F 0 "F1501" V 5930 4000 50  0000 C CNN
+F 1 "Fuse" V 5775 4000 50  0000 C CNN
+F 2 "Fuse:Fuse_1206_3216Metric" V 5780 4000 50  0001 C CNN
+F 3 "https://industrial.panasonic.com/cdbs/www-data/pdf/AFA0000/AFA0000C7.pdf" H 5850 4000 50  0001 C CNN
+F 4 "Panasonic Electronic Components" H 5850 4000 60  0001 C CNN "MFG Name"
+F 5 "ERB-RG2R50V" H 5850 4000 60  0001 C CNN "MFG Part Num"
+F 6 "P16740CT-ND" H 5850 4000 60  0001 C CNN "Digikey"
+F 7 "1" H 5850 4000 60  0001 C CNN "Populated"
+F 8 "FUSE BOARD MOUNT 2.5A 32VDC 1206 " H 5850 4000 60  0001 C CNN "Description"
+F 9 "SPEC" H 5850 4000 60  0001 C CNN "Source"
+F 10 "1" H 5850 4000 60  0001 C CNN "Populate for SBGA485(Z-7030)"
+F 11 "1" H 5850 4000 60  0001 C CNN "Populate for CLG484(Z-7012s/Z-7015)"
+	1    5850 4000
+	-1   0    0    1
+$EndComp
+Wire Wire Line
+	5850 3850 5850 3750
+Wire Wire Line
+	5850 4150 5850 4300
+Wire Wire Line
+	5850 4300 6000 4300
 $EndSCHEMATC

Commit message: Fixed Schematic Symbols
Parts:
- C1501, C1502, C1503, C1504, C1505, C1506, C1507, C1508, C1509, C1510, C1511, C1512, C1513, C1514, C1515, C1516: symbol device:C_Small -> Device:C_Small
- D1501: symbol device:D_Schottky -> Device:D_Schottky
- F1501: symbol device:Fuse -> Device:Fuse
- R1501, R1502, R1503, R1504, R1505, R1506, R1507, R1508, R1509, R1510, R1511, R1512, R1513, R1514, R1515, R1516: symbol device:R_Small -> Device:R_Small
Changed lines of the file:
@@
 $Descr A4 11693 8268
 encoding utf-8
-Sheet 15 22
+Sheet 15 21
 Title ""
 Date ""
@@
 $EndComp
 $Comp
-L power1:+1V8 #PWR0184
+L power:+1V8 #PWR0184
 U 1 1 5AD1622E
 P 2100 1150
@@
 $EndComp
 $Comp
-L power1:GND #PWR0185
+L power:GND #PWR0185
 U 1 1 5AD1628E
 P 2100 1900
@@
 $EndComp
 $Comp
-L device:R_Small R1501
+L Device:R_Small R1501
 U 1 1 5AD162EE
 P 1150 1450
@@
 $EndComp
 $Comp
-L power1:+1V8 #PWR0186
+L power:+1V8 #PWR0186
 U 1 1 5AD163D6
 P 1150 1250
@@
 $EndComp
 $Comp
-L device:R_Small R1502
+L Device:R_Small R1502
 U 1 1 5AD035E9
 P 1150 1850
@@
 $EndComp
 $Comp
-L power1:GND #PWR0187
+L power:GND #PWR0187
 U 1 1 5AD0367E
 P 1150 2050
@@
 TRIG_IN_1
 $Comp
-L device:R_Small R1508
+L Device:R_Small R1508
 U 1 1 5AD0382A
 P 3400 1400
@@
 $EndComp
 $Comp
-L device:R_Small R1509
+L Device:R_Small R1509
 U 1 1 5AD039C8
 P 3400 1500
@@
 $EndComp
 $Comp
-L power1:+1V8 #PWR0189
+L power:+1V8 #PWR0189
 U 1 1 5AE6803D
 P 2100 2400
@@
 $EndComp
 $Comp
-L power1:GND #PWR0190
+L power:GND #PWR0190
 U 1 1 5AE68043
 P 2100 3150
@@
 $EndComp
 $Comp
-L device:R_Small R1503
+L Device:R_Small R1503
 U 1 1 5AE68049
 P 1150 2700
@@
 $EndComp
 $Comp
-L power1:+1V8 #PWR0191
+L power:+1V8 #PWR0191
 U 1 1 5AE6804F
 P 1150 2500
@@
 $EndComp
 $Comp
-L device:R_Small R1504
+L Device:R_Small R1504
 U 1 1 5AE6805E
 P 1150 3100
@@
 $EndComp
 $Comp
-L power1:GND #PWR0192
+L power:GND #PWR0192
 U 1 1 5AE68065
 P 1150 3300
@@
 TRIG_IN_3
 $Comp
-L device:R_Small R1510
+L Device:R_Small R1510
 U 1 1 5AE68076
 P 3400 2650
@@
 $EndComp
 $Comp
-L device:R_Small R1511
+L Device:R_Small R1511
 U 1 1 5AE6807D
 P 3400 2750
@@
 $EndComp
 $Comp
-L power1:+1V8 #PWR0194
+L power:+1V8 #PWR0194
 U 1 1 5AE6839A
 P 2100 3650
@@
 $EndComp
 $Comp
-L power1:GND #PWR0195
+L power:GND #PWR0195
 U 1 1 5AE683A0
 P 2100 4400
@@
 $EndComp
 $Comp
-L device:R_Small R1505
+L Device:R_Small R1505
 U 1 1 5AE683A6
 P 1150 3950
@@
 $EndComp
 $Comp
-L power1:+1V8 #PWR0196
+L power:+1V8 #PWR0196
 U 1 1 5AE683AC
 P 1150 3750
@@
 $EndComp
 $Comp
-L device:R_Small R1506
+L Device:R_Small R1506
 U 1 1 5AE683BB
 P 1150 4350
@@
 $EndComp
 $Comp
-L power1:GND #PWR0197
+L power:GND #PWR0197
 U 1 1 5AE683C2
 P 1150 4550
@@
 TRIG_OUT_1
 $Comp
-L device:R_Small R1512
+L Device:R_Small R1512
 U 1 1 5AE683D3
 P 3400 3900
@@
 $EndComp
 $Comp
-L device:R_Small R1513
+L Device:R_Small R1513
 U 1 1 5AE683DA
 P 3400 4000
@@
 $EndComp
 $Comp
-L power1:+1V8 #PWR0199
+L power:+1V8 #PWR0199
 U 1 1 5AE683E7
 P 2100 4900
@@
 $EndComp
 $Comp
-L power1:GND #PWR0200
+L power:GND #PWR0200
 U 1 1 5AE683ED
 P 2100 5650
@@
 $EndComp
 $Comp
-L device:R_Small R1507
+L Device:R_Small R1507
 U 1 1 5AE683F3
 P 1150 5200
@@
 $EndComp
 $Comp
-L power1:+1V8 #PWR0201
+L power:+1V8 #PWR0201
 U 1 1 5AE683F9
 P 1150 5000
@@
 $EndComp
 $Comp
-L device:R_Small R1516
+L Device:R_Small R1516
 U 1 1 5AE68408
 P 1150 5600
@@
 $EndComp
 $Comp
-L power1:GND #PWR0202
+L power:GND #PWR0202
 U 1 1 5AE6840F
 P 1150 5800
@@
 TRIG_OUT_3
 $Comp
-L device:R_Small R1514
+L Device:R_Small R1514
 U 1 1 5AE68420
 P 3400 5150
@@
 $EndComp
 $Comp
-L device:R_Small R1515
+L Device:R_Small R1515
 U 1 1 5AE68427
 P 3400 5250
@@
 $EndComp
 $Comp
-L power1:GND #PWR0204
+L power:GND #PWR0204
 U 1 1 5AE694D8
 P 4950 750
@@
 $EndComp
 $Comp
-L power1:GND #PWR0205
+L power:GND #PWR0205
 U 1 1 5AE69964
 P 4950 3150
@@
 $EndComp
 $Comp
-L power1:GND #PWR0206
+L power:GND #PWR0206
 U 1 1 5AD980A9
 P 8850 3450
@@
 $EndComp
 $Comp
-L power1:+1V8 #PWR0207
+L power:+1V8 #PWR0207
 U 1 1 5AD981B6
 P 8650 1650
@@
 $EndComp
 $Comp
-L power1:GND #PWR0208
+L power:GND #PWR0208
 U 1 1 5AD98A40
 P 8800 800
@@
 $EndComp
 $Comp
-L power1:GND #PWR0209
+L power:GND #PWR0209
 U 1 1 5AD98C8A
 P 8200 800
@@
 $EndComp
 $Comp
-L power1:GND #PWR0210
+L power:GND #PWR0210
 U 1 1 5AD98EEA
 P 9500 800
@@
 Bypass Capacitors for MAX14854.\nPlace as close as possible to it
 $Comp
-L device:C_Small C1501
+L Device:C_Small C1501
 U 1 1 5AD9AF72
 P 1600 6650
@@
 $EndComp
 $Comp
-L power1:GND #PWR0212
+L power:GND #PWR0212
 U 1 1 5AD9BAB3
 P 2050 6950
@@
 $EndComp
 $Comp
-L power1:GND #PWR0213
+L power:GND #PWR0213
 U 1 1 5AD9BEC4
 P 3400 6950
@@
 $EndComp
 $Comp
-L power1:+1V8 #PWR0214
+L power:+1V8 #PWR0214
 U 1 1 5AD9BF16
 P 2050 6350
@@
 EXT_TRIG_OUT_0
 $Comp
-L power1:GND #PWR0215
+L power:GND #PWR0215
 U 1 1 5B119013
 P 10200 4300
@@
 $EndComp
 $Comp
-L power1:+5V #PWR0216
+L power:+5V #PWR0216
 U 1 1 5B11913A
 P 5850 3750
@@
 $EndComp
 $Comp
-L device:D_Schottky D1501
+L Device:D_Schottky D1501
 U 1 1 5AE9D86E
 P 6150 4300
@@
 	6300 4300 6600 4300
 $Comp
-L device:C_Small C1509
+L Device:C_Small C1509
 U 1 1 5AE9E531
 P 6600 4500
@@
 Connection ~ 7200 4700
 $Comp
-L power1:GND #PWR0217
+L power:GND #PWR0217
 U 1 1 5AE9EE3D
 P 7050 4800
@@
 	4150 2750 5350 2750
 $Comp
-L device:C_Small C1510
+L Device:C_Small C1510
 U 1 1 5B2592FD
 P 7650 4500
@@
 $EndComp
 $Comp
-L device:C_Small C1511
+L Device:C_Small C1511
 U 1 1 5B259397
 P 8050 1100
@@
 $EndComp
 $Comp
-L device:C_Small C1513
+L Device:C_Small C1513
 U 1 1 5B259673
 P 8650 1100
@@
 $EndComp
 $Comp
-L device:C_Small C1516
+L Device:C_Small C1516
 U 1 1 5B25979C
 P 9650 1100
@@
 $EndComp
 $Comp
-L device:C_Small C1502
+L Device:C_Small C1502
 U 1 1 5B26F36E
 P 1900 6650
@@
 $EndComp
 $Comp
-L device:C_Small C1503
+L Device:C_Small C1503
 U 1 1 5B284332
 P 2200 6650
@@
 $EndComp
 $Comp
-L device:C_Small C1504
+L Device:C_Small C1504
 U 1 1 5B284341
 P 2500 6650
@@
 $EndComp
 $Comp
-L device:C_Small C1505
+L Device:C_Small C1505
 U 1 1 5B2AE1C0
 P 2950 6650
@@
 $EndComp
 $Comp
-L device:C_Small C1506
+L Device:C_Small C1506
 U 1 1 5B2AE1CF
 P 3250 6650
@@
 $EndComp
 $Comp
-L device:C_Small C1507
+L Device:C_Small C1507
 U 1 1 5B2AE1DE
 P 3550 6650
@@
 $EndComp
 $Comp
-L device:C_Small C1508
+L Device:C_Small C1508
 U 1 1 5B2AE1ED
 P 3850 6650
@@
 $EndComp
 $Comp
-L device:C_Small C1512
+L Device:C_Small C1512
 U 1 1 5B2B88DF
 P 8350 1100
@@
 $EndComp
 $Comp
-L device:C_Small C1514
+L Device:C_Small C1514
 U 1 1 5B2B8CBD
 P 8950 1100
@@
 $EndComp
 $Comp
-L device:C_Small C1515
+L Device:C_Small C1515
 U 1 1 5B2B8D61
 P 9350 1100
@@
 	3300 3300 3300 3750
 $Comp
-L device:Fuse F1501
+L Device:Fuse F1501
 U 1 1 5B4B93EE
 P 5850 4000

Commit message: SFP+ Power Filter, Levelshifter and MGT/TLK Clock Distribution.
Parts:
- added TP1401, TP1402: Test_Point, footprints:TestPoint_SMD_0.5mm, symbol Connector:Test_Point
Connections:
- wire segments 214 -> 216
Changed lines of the file:
@@
 	4550 5250 5300 5250
 Wire Wire Line
-	6600 4300 6900 4300
+	6600 4300 6800 4300
 Wire Wire Line
 	7200 4700 7650 4700
@@
 	7050 4700 7200 4700
 Wire Wire Line
-	7650 4300 7900 4300
+	7650 4300 7750 4300
 Wire Wire Line
 	10200 4450 10200 4550
@@
 Wire Wire Line
 	5850 4300 6000 4300
+$Comp
+L Connector:Test_Point TP1401
+U 1 1 5BA6BB84
+P 6800 4300
+F 0 "TP1401" H 6858 4420 50  0000 L CNN
+F 1 "Test_Point" H 6858 4329 50  0000 L CNN
+F 2 "footprints:TestPoint_SMD_0.5mm" H 7000 4300 50  0001 C CNN
+F 3 "~" H 7000 4300 50  0001 C CNN
+F 4 "1" H 6800 4300 50  0001 C CNN "Populated"
+F 5 "SPEC" H 6800 4300 50  0001 C CNN "Source"
+F 6 "1" H 6800 4300 50  0001 C CNN "Populate for SBGA485(Z-7030)"
+F 7 "1" H 6800 4300 50  0001 C CNN "Populate for CLG484(Z-7012s/Z-7015)"
+	1    6800 4300
+	1    0    0    -1
+$EndComp
+Connection ~ 6800 4300
+Wire Wire Line
+	6800 4300 6900 4300
+$Comp
+L Connector:Test_Point TP1402
+U 1 1 5BA77261
+P 7750 4300
+F 0 "TP1402" H 7808 4420 50  0000 L CNN
+F 1 "Test_Point" H 7808 4329 50  0000 L CNN
+F 2 "footprints:TestPoint_SMD_0.5mm" H 7950 4300 50  0001 C CNN
+F 3 "~" H 7950 4300 50  0001 C CNN
+F 4 "1" H 7750 4300 50  0001 C CNN "Populated"
+F 5 "SPEC" H 7750 4300 50  0001 C CNN "Source"
+F 6 "1" H 7750 4300 50  0001 C CNN "Populate for SBGA485(Z-7030)"
+F 7 "1" H 7750 4300 50  0001 C CNN "Populate for CLG484(Z-7012s/Z-7015)"
+	1    7750 4300
+	1    0    0    -1
+$EndComp
+Connection ~ 7750 4300
+Wire Wire Line
+	7750 4300 7900 4300
 $EndSCHEMATC
