File: hardware/triggerbus.sch (KiCad schematic (older format))
At the start: 45 parts, among them J1501 MDR20, U1501 SN74LVC2T45, U1502 SN74LVC2T45, U1503 SN74LVC2T45, U1504 SN74LVC2T45, U1505 DMF05LCFLP, U1506 DMF05LCFLP, U1507 TC1262-33, U1508 MAX14854

Commit message: PS Clock, Reset Button, Cam Levelshifters and big 1.0 V Cap placed.
Improved some Footprints and library Symbols.

Also though about Chassis Ground.
Parts:
- added L1401: L_Core_Ferrite, Inductor_SMD:L_0805_2012Metric, symbol Device:L_Core_Ferrite
- added R1422: 0, Resistor_SMD:R_0402_1005Metric, symbol Device:R
Connections:
- wire segments 216 -> 225
Changed lines of the file:
@@
 Wire Wire Line
 	7750 4300 7900 4300
+$Comp
+L Device:R R1422
+U 1 1 5BC69B8D
+P 8750 5700
+F 0 "R1422" V 8830 5700 50  0000 C CNN
+F 1 "0" V 8750 5700 50  0000 C CNN
+F 2 "Resistor_SMD:R_0402_1005Metric" V 8680 5700 50  0001 C CNN
+F 3 "" H 8750 5700 50  0000 C CNN
+F 4 "1" H 8850 5850 50  0001 C CNN "Populated"
+F 5 "SPEC" H 8750 5700 50  0001 C CNN "Source"
+F 6 "1" H 8750 5700 50  0001 C CNN "Populate for SBGA485(Z-7030)"
+F 7 "1" H 8750 5700 50  0001 C CNN "Populate for CLG484(Z-7012s/Z-7015)"
+	1    8750 5700
+	1    0    0    -1
+$EndComp
+Wire Wire Line
+	8750 5850 8750 5950
+Wire Wire Line
+	8750 5950 8900 5950
+Wire Wire Line
+	9050 5950 9050 5850
+$Comp
+L power:GND #PWR01401
+U 1 1 5BC69B97
+P 8900 6050
+F 0 "#PWR01401" H 8900 5800 50  0001 C CNN
+F 1 "GND" H 8900 5900 50  0000 C CNN
+F 2 "" H 8900 6050 50  0000 C CNN
+F 3 "" H 8900 6050 50  0000 C CNN
+	1    8900 6050
+	1    0    0    -1
+$EndComp
+Wire Wire Line
+	8900 6050 8900 5950
+Connection ~ 8900 5950
+Wire Wire Line
+	8900 5950 9050 5950
+$Comp
+L Device:L_Core_Ferrite L1401
+U 1 1 5BC69BA4
+P 9050 5700
+F 0 "L1401" H 9138 5746 50  0000 L CNN
+F 1 "L_Core_Ferrite" H 9138 5655 50  0000 L CNN
+F 2 "Inductor_SMD:L_0805_2012Metric" H 9050 5700 50  0001 C CNN
+F 3 "~" H 9050 5700 50  0001 C CNN
+F 4 "1" H 9050 5700 50  0001 C CNN "Populated"
+F 5 "SPEC" H 9050 5700 50  0001 C CNN "Source"
+F 6 "1" H 9050 5700 50  0001 C CNN "Populate for SBGA485(Z-7030)"
+F 7 "1" H 9050 5700 50  0001 C CNN "Populate for CLG484(Z-7012s/Z-7015)"
+	1    9050 5700
+	1    0    0    -1
+$EndComp
+Wire Wire Line
+	8750 5550 8750 5450
+Wire Wire Line
+	8750 5450 9050 5450
+Wire Wire Line
+	9050 5550 9050 5450
+Connection ~ 9050 5450
+Wire Wire Line
+	9050 5450 9150 5450
 $EndSCHEMATC

Commit message: Routed a first Version of the High Speed Part of the Camera Connector. The optional LVDS Clocks are left unconnected. I couldn't keep the Connectors Pin Assignment because it was just impossible to route.
WIP: general Routing

Fixed: DDR3 Trace Length Matching
Connections:
- wire segments 225 -> 226
Changed lines of the file:
@@
 $Descr A4 11693 8268
 encoding utf-8
-Sheet 14 21
+Sheet 13 21
 Title ""
 Date ""
@@
 	10300 5250 10650 5250
 Wire Wire Line
-	6300 4300 6600 4300
+	6300 4300 6350 4300
 $Comp
 L Device:C_Small C1509
@@
 Wire Wire Line
 	9050 5450 9150 5450
+$Comp
+L power:PWR_FLAG #FLG0113
+U 1 1 5C1F0DDD
+P 6350 4300
+F 0 "#FLG0113" H 6350 4375 50  0001 C CNN
+F 1 "PWR_FLAG" H 6350 4474 50  0000 C CNN
+F 2 "" H 6350 4300 50  0001 C CNN
+F 3 "~" H 6350 4300 50  0001 C CNN
+	1    6350 4300
+	1    0    0    -1
+$EndComp
+Connection ~ 6350 4300
+Wire Wire Line
+	6350 4300 6600 4300
 $EndSCHEMATC

Commit message: Added Courtyard to selfmade Footprints. Also general Routing WIP.
Connections:
- net labels added: RS485_DE, RS485_RXD, RS485_TXD, ~RS485_RE~, ~RS485_SBA~
- net labels removed: DE, RXD, TXD, ~RE~, ~SBA~
- wire segments 226 -> 231
Other:
- note added: "BANK 35"
Changed lines of the file:
@@
 EESchema Schematic File Version 4
+LIBS:zynq_board-cache
 EELAYER 26 0
 EELAYER END
@@
 Text Notes 1450 6050 0    60   ~ 0
 Bypass Capacitors for the Triggerbus Levelshifters.\nPlace them as close as possible to their power inputs.
-Text HLabel 8350 2400 0    60   Output ~ 0
-RXD
-Text HLabel 8350 2300 0    60   Output ~ 0
-~SBA~
-Text HLabel 8350 2500 0    60   Input ~ 0
-~RE~
-Text HLabel 8350 2600 0    60   Input ~ 0
-DE
-Text HLabel 8350 2700 0    60   Input ~ 0
-TXD
 Text Label 5350 1400 2    60   ~ 0
 EXT_TRIG_IN_0
@@
 Wire Wire Line
 	6350 4300 6600 4300
+Text GLabel 8200 2300 0    50   Output ~ 0
+~RS485_SBA~
+Text GLabel 8200 2400 0    50   Output ~ 0
+RS485_RXD
+Text GLabel 8200 2500 0    50   Input ~ 0
+~RS485_RE~
+Text GLabel 8200 2700 0    50   Input ~ 0
+RS485_DE
+Text GLabel 8200 2600 0    50   Input ~ 0
+RS485_TXD
+Wire Wire Line
+	8350 2300 8200 2300
+Wire Wire Line
+	8200 2400 8350 2400
+Wire Wire Line
+	8350 2500 8200 2500
+Wire Wire Line
+	8200 2600 8350 2600
+Wire Wire Line
+	8350 2700 8200 2700
+Text Notes 7700 2650 1    50   ~ 0
+BANK 35
 $EndSCHEMATC

Commit message: Routed extra GPIO Solder Pads, reannotated the whole schematic to make it consistent.
Power Distribution routing WIP
Parts:
- renumbered C1501 to C1301, C1502 to C1302, C1503 to C1303, C1504 to C1304, C1505 to C1305, C1506 to C1306, C1507 to C1307, C1508 to C1308, C1509 to C1309, C1510 to C1310, C1511 to C1311, C1512 to C1312, C1513 to C1313, C1514 to C1314, C1515 to C1315, C1516 to C1316, D1501 to D1301, F1501 to F1301, J1501 to J1301, L1401 to L1301, R1501 to R1301, R1502 to R1302, R1503 to R1303, R1504 to R1304, R1505 to R1305, R1506 to R1306, R1507 to R1307, R1516 to R1308, R1508 to R1309, R1509 to R1310, R1510 to R1311, R1511 to R1312, R1512 to R1313, R1513 to R1314, R1514 to R1315, R1515 to R1316, R1422 to R1317, TP1401 to TP1301, TP1402 to TP1302, U1501 to U1301, U1502 to U1302, U1503 to U1303, U1504 to U1304, U1506 to U1305, U1505 to U1306, U1507 to U1307, U1508 to U1308

Commit message: general routing mainly power distribution, fixed some footprints
Parts:
- U1307: footprint TO_SOT_Packages_SMD:SOT-223 -> Package_TO_SOT_SMD:SOT-223
Changed lines of the file:
@@
 F 0 "U1307" H 7050 4425 50  0000 C CNN
 F 1 "TC1262-33" H 7200 4425 50  0000 L CNN
-F 2 "TO_SOT_Packages_SMD:SOT-223" H 7200 4525 50  0001 C CIN
+F 2 "Package_TO_SOT_SMD:SOT-223" H 7200 4525 50  0001 C CIN
 F 3 "http://ww1.microchip.com/downloads/en/DeviceDoc/21373C.pdf" H 7200 4000 50  0001 C CNN
 F 4 "Microchip Technology" H 7200 4300 60  0001 C CNN "MFG Name"

Commit message: First Version without any Net not routed.
Parts:
- L1301: Populated 1 -> DNP
- R1302, R1304, R1305, R1307: value DNP -> 10k; Populated 1 -> DNP
- U1305, U1306: footprint Housings_DFN_QFN:DFN-6-1EP_2x2mm_Pitch0.5mm -> Package_DFN_QFN:DFN-6-1EP_2x2mm_P0.5mm_EP0.61x1.42mm
- U1308: footprint Housings_SOIC:SOIC-16W_7.5x10.3mm_Pitch1.27mm -> Package_SO:SOIC-16W_7.5x10.3mm_P1.27mm; symbol dmf05lcflp:MAX14854 -> max14854:MAX14854; Populate for CLG484(Z-7012s/Z-7015) (none) -> 1; Populate for SBGA485(Z-7030) (none) -> 1
Connections:
- wire segments 231 -> 239
Other:
- note added: "Ideas:\nTriggerbus should be as robust as possible. That means 5 V tolerant,\nidiot Diodes at Poweroutputs, ESD protection Diodes, current limiting \nseries Resistors. But: Triggerbus is not galvanic isolated."
- note added: "If internal LDO is used,\nVDDB is connected to a decoupling and\na bulk capacitor."
- note added: "This RS485 Transceiver is\nmaybe overkill. Also it takes\na lot of space from the PCB.\nBut:\nIt works directly with 1,8 V signal level\nand is really robust."
- note removed: "Ideas:\nTriggerbus should be as robust as possible. That means 5 V tolerant,\nidiot Diodes at Poweroutputs, ESD protection Diodes, current limiting Resistors."
- note removed: "This RS485 Transceiver is\nmaybe overkill. Also it takes\na lot of space from the PCB."
- moved on the sheet: C1309, C1310, C1311, C1312, C1313, C1314, C1315, C1316, D1301, F1301, J1301, L1301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

Commit message: Add sym-lib-table and fp-lib-table, fixes for KiCad 5
Parts:
- TP1301, TP1302: symbol Connector:Test_Point -> Connector:TestPoint
Changed lines of the file:
@@
 	5750 5400 5900 5400
 $Comp
-L Connector:Test_Point TP1301
+L Connector:TestPoint TP1301
 U 1 1 5BA6BB84
 P 6700 5400
@@
 	6700 5400 6800 5400
 $Comp
-L Connector:Test_Point TP1302
+L Connector:TestPoint TP1302
 U 1 1 5BA77261
 P 7650 5400
