File: hardware/gpio.sch (KiCad schematic (older format))
At the start: 1 part

Commit message: Added Reset Button, Power LED, 2 Status LEDs and an external Button.
Parts:
- added D? (x3): LED, LEDs:LED_0402, symbol LED
- added J?: Conn_01x02, Pin_Headers:Pin_Header_Angled_1x02_Pitch2.54mm, symbol Conn_01x02
- added Q? (x2): BSS138PS, TO_SOT_Packages_SMD:SOT-363_SC-70-6, symbol BSS138PS
- added R? (x3): 430, Resistors_SMD:R_0402, symbol R_Small
- added R? (x2): 100k, Resistors_SMD:R_0402, symbol R_Small
- added R?: DNP, Resistors_SMD:R_0402, symbol R_Small
Connections:
- net labels added: +1V8, BUTTON1, LED1, LED2
- wire segments 0 -> 24
Other:
- note added: "GPIOs are 1,8 V only.\n!!!Not 3,3 V or 5 V tolerant!!!"
- note added: "Power Led"
- note added: "User LEDs"

Commit message: Added Sdcard Slot.
Parts:
- gave numbers to parts that had none: 12
Changed lines of the file:
@@
 $Descr A4 11693 8268
 encoding utf-8
-Sheet 21 21
+Sheet 19 20
 Title ""
 Date ""
@@
 $EndDescr
 $Comp
-L Conn_02x09_Counter_Clockwise J?
+L Conn_02x09_Counter_Clockwise J8
 U 1 1 5B0F5739
 P 5150 3350
-F 0 "J?" H 5200 3850 50  0000 C CNN
+F 0 "J8" H 5200 3850 50  0000 C CNN
 F 1 "Conn_02x09_Counter_Clockwise" H 5200 2850 50  0000 C CNN
 F 2 "" H 5150 3350 50  0001 C CNN
@@
 GPIO_15
 $Comp
-L GND #PWR?
+L GND #PWR0150
 U 1 1 5B0F584E
 P 4950 3750
-F 0 "#PWR?" H 4950 3500 50  0001 C CNN
+F 0 "#PWR0150" H 4950 3500 50  0001 C CNN
 F 1 "GND" V 4950 3550 50  0000 C CNN
 F 2 "" H 4950 3750 50  0001 C CNN
@@
 $EndComp
 $Comp
-L +3V3 #PWR?
+L +3V3 #PWR0151
 U 1 1 5B0F5864
 P 5450 3750
-F 0 "#PWR?" H 5450 3600 50  0001 C CNN
+F 0 "#PWR0151" H 5450 3600 50  0001 C CNN
 F 1 "+3V3" V 5450 4000 50  0000 C CNN
 F 2 "" H 5450 3750 50  0001 C CNN
@@
 $EndComp
 $Comp
-L LED D?
+L LED D1
 U 1 1 5B1B21E2
 P 8000 3150
-F 0 "D?" H 8000 3250 50  0000 C CNN
+F 0 "D1" H 8000 3250 50  0000 C CNN
 F 1 "LED" H 8000 3050 50  0000 C CNN
 F 2 "LEDs:LED_0402" H 8000 3150 50  0001 C CNN
@@
 $EndComp
 $Comp
-L R_Small R?
+L R_Small R114
 U 1 1 5B1B2374
 P 8000 2800
-F 0 "R?" H 8030 2820 50  0000 L CNN
+F 0 "R114" H 8030 2820 50  0000 L CNN
 F 1 "430" H 8030 2760 50  0000 L CNN
 F 2 "Resistors_SMD:R_0402" H 8000 2800 50  0001 C CNN
@@
 GPIOs are 1,8 V only.\n!!!Not 3,3 V or 5 V tolerant!!!
 $Comp
-L +3V3 #PWR?
+L +3V3 #PWR0152
 U 1 1 5B1B2AD0
 P 8000 2550
-F 0 "#PWR?" H 8000 2400 50  0001 C CNN
+F 0 "#PWR0152" H 8000 2400 50  0001 C CNN
 F 1 "+3V3" H 8000 2690 50  0000 C CNN
 F 2 "" H 8000 2550 50  0001 C CNN
@@
 	8000 2550 8000 2700
 $Comp
-L GND #PWR?
+L GND #PWR0153
 U 1 1 5B1B2B0C
 P 8000 3400
-F 0 "#PWR?" H 8000 3150 50  0001 C CNN
+F 0 "#PWR0153" H 8000 3150 50  0001 C CNN
 F 1 "GND" H 8000 3250 50  0000 C CNN
 F 2 "" H 8000 3400 50  0001 C CNN
@@
 	8000 3300 8000 3400
 $Comp
-L BSS138PS Q?
+L BSS138PS Q3
 U 1 1 5B1B2B60
 P 9100 3150
-F 0 "Q?" H 9300 3225 50  0000 L CNN
+F 0 "Q3" H 9300 3225 50  0000 L CNN
 F 1 "BSS138PS" H 9300 3150 50  0000 L CNN
 F 2 "TO_SOT_Packages_SMD:SOT-363_SC-70-6" H 9300 3075 50  0001 L CIN
@@
 $EndComp
 $Comp
-L LED D?
+L LED D2
 U 1 1 5B1B2C38
 P 9200 2700
-F 0 "D?" H 9200 2800 50  0000 C CNN
+F 0 "D2" H 9200 2800 50  0000 C CNN
 F 1 "LED" H 9200 2600 50  0000 C CNN
 F 2 "LEDs:LED_0402" H 9200 2700 50  0001 C CNN
@@
 $EndComp
 $Comp
-L R_Small R?
+L R_Small R116
 U 1 1 5B1B2C8F
 P 9200 2350
-F 0 "R?" H 9230 2370 50  0000 L CNN
+F 0 "R116" H 9230 2370 50  0000 L CNN
 F 1 "430" H 9230 2310 50  0000 L CNN
 F 2 "Resistors_SMD:R_0402" H 9200 2350 50  0001 C CNN
@@
 	9200 2850 9200 2950
 $Comp
-L GND #PWR?
+L GND #PWR0154
 U 1 1 5B1B2D14
 P 9200 3700
-F 0 "#PWR?" H 9200 3450 50  0001 C CNN
+F 0 "#PWR0154" H 9200 3450 50  0001 C CNN
 F 1 "GND" H 9200 3550 50  0000 C CNN
 F 2 "" H 9200 3700 50  0001 C CNN
@@
 	9200 3350 9200 3700
 $Comp
-L +3V3 #PWR?
+L +3V3 #PWR0155
 U 1 1 5B1B2D42
 P 9200 2150
-F 0 "#PWR?" H 9200 2000 50  0001 C CNN
+F 0 "#PWR0155" H 9200 2000 50  0001 C CNN
 F 1 "+3V3" H 9200 2290 50  0000 C CNN
 F 2 "" H 9200 2150 50  0001 C CNN
@@
 LED1
 $Comp
-L BSS138PS Q?
+L BSS138PS Q3
 U 2 1 5B1B2E27
 P 10600 3150
-F 0 "Q?" H 10800 3225 50  0000 L CNN
+F 0 "Q3" H 10800 3225 50  0000 L CNN
 F 1 "BSS138PS" H 10800 3150 50  0000 L CNN
 F 2 "TO_SOT_Packages_SMD:SOT-363_SC-70-6" H 10800 3075 50  0001 L CIN
@@
 $EndComp
 $Comp
-L LED D?
+L LED D3
 U 1 1 5B1B2E2D
 P 10700 2700
-F 0 "D?" H 10700 2800 50  0000 C CNN
+F 0 "D3" H 10700 2800 50  0000 C CNN
 F 1 "LED" H 10700 2600 50  0000 C CNN
 F 2 "LEDs:LED_0402" H 10700 2700 50  0001 C CNN
@@
 $EndComp
 $Comp
-L R_Small R?
+L R_Small R119
 U 1 1 5B1B2E33
 P 10700 2350
-F 0 "R?" H 10730 2370 50  0000 L CNN
+F 0 "R119" H 10730 2370 50  0000 L CNN
 F 1 "430" H 10730 2310 50  0000 L CNN
 F 2 "Resistors_SMD:R_0402" H 10700 2350 50  0001 C CNN
@@
 	10700 2850 10700 2950
 $Comp
-L GND #PWR?
+L GND #PWR0156
 U 1 1 5B1B2E3B
 P 10700 3700
-F 0 "#PWR?" H 10700 3450 50  0001 C CNN
+F 0 "#PWR0156" H 10700 3450 50  0001 C CNN
 F 1 "GND" H 10700 3550 50  0000 C CNN
 F 2 "" H 10700 3700 50  0001 C CNN
@@
 	10700 3350 10700 3700
 $Comp
-L +3V3 #PWR?
+L +3V3 #PWR0157
 U 1 1 5B1B2E42
 P 10700 2150
-F 0 "#PWR?" H 10700 2000 50  0001 C CNN
+F 0 "#PWR0157" H 10700 2000 50  0001 C CNN
 F 1 "+3V3" H 10700 2290 50  0000 C CNN
 F 2 "" H 10700 2150 50  0001 C CNN
@@
 User LEDs
 $Comp
-L R_Small R?
+L R_Small R115
 U 1 1 5B204015
 P 8800 3350
-F 0 "R?" H 8830 3370 50  0000 L CNN
+F 0 "R115" H 8830 3370 50  0000 L CNN
 F 1 "100k" H 8830 3310 50  0000 L CNN
 F 2 "Resistors_SMD:R_0402" H 8800 3350 50  0001 C CNN
@@
 	10200 3150 10400 3150
 $Comp
-L R_Small R?
+L R_Small R117
 U 1 1 5B20436B
 P 10350 3350
-F 0 "R?" H 10380 3370 50  0000 L CNN
+F 0 "R117" H 10380 3370 50  0000 L CNN
 F 1 "100k" H 10380 3310 50  0000 L CNN
 F 2 "Resistors_SMD:R_0402" H 10350 3350 50  0001 C CNN
@@
 Connection ~ 10700 3550
 $Comp
-L Conn_01x02 J?
+L Conn_01x02 J9
 U 1 1 5B2142B2
 P 10700 4550
-F 0 "J?" H 10700 4650 50  0000 C CNN
+F 0 "J9" H 10700 4650 50  0000 C CNN
 F 1 "Conn_01x02" H 10700 4350 50  0000 C CNN
 F 2 "Pin_Headers:Pin_Header_Angled_1x02_Pitch2.54mm" H 10700 4550 50  0001 C CNN
@@
 	10400 4650 10400 4750
 $Comp
-L GND #PWR?
+L GND #PWR0158
 U 1 1 5B2143F5
 P 10400 4750
-F 0 "#PWR?" H 10400 4500 50  0001 C CNN
+F 0 "#PWR0158" H 10400 4500 50  0001 C CNN
 F 1 "GND" H 10400 4600 50  0000 C CNN
 F 2 "" H 10400 4750 50  0001 C CNN
@@
 $EndComp
 $Comp
-L R_Small R?
+L R_Small R118
 U 1 1 5B214424
 P 10400 4350
-F 0 "R?" H 10430 4370 50  0000 L CNN
+F 0 "R118" H 10430 4370 50  0000 L CNN
 F 1 "DNP" H 10430 4310 50  0000 L CNN
 F 2 "Resistors_SMD:R_0402" H 10400 4350 50  0001 C CNN
@@
 	10300 4550 10500 4550
 $Comp
-L +1V8 #PWR?
+L +1V8 #PWR0159
 U 1 1 5B21453D
 P 10400 4150
-F 0 "#PWR?" H 10400 4000 50  0001 C CNN
+F 0 "#PWR0159" H 10400 4000 50  0001 C CNN
 F 1 "+1V8" H 10400 4290 50  0000 C CNN
 F 2 "" H 10400 4150 50  0001 C CNN

Commit message: Added USB-Uart subschematic. WIP
USB-Uart will be bus powered. Buffer between FTDI and FPGA is missing.
Parts:
- renumbered D1 to D?, D2 to D?, D3 to D?, J8 to J?, J9 to J?, Q3 to Q?, R114 to R?, R116 to R?, R119 to R?, R115 to R?, R117 to R?, R118 to R?
Changed lines of the file:
@@
 LIBS:max14854
 LIBS:switches
+LIBS:ft234xd
 LIBS:zynq_board-cache
 EELAYER 25 0
@@
 $Descr A4 11693 8268
 encoding utf-8
-Sheet 19 20
+Sheet 19 21
 Title ""
 Date ""
@@
 $EndDescr
 $Comp
-L Conn_02x09_Counter_Clockwise J8
+L Conn_02x09_Counter_Clockwise J?
 U 1 1 5B0F5739
 P 5150 3350
-F 0 "J8" H 5200 3850 50  0000 C CNN
+F 0 "J?" H 5200 3850 50  0000 C CNN
 F 1 "Conn_02x09_Counter_Clockwise" H 5200 2850 50  0000 C CNN
 F 2 "" H 5150 3350 50  0001 C CNN
@@
 GPIO_15
 $Comp
-L GND #PWR0150
+L GND #PWR?
 U 1 1 5B0F584E
 P 4950 3750
-F 0 "#PWR0150" H 4950 3500 50  0001 C CNN
+F 0 "#PWR?" H 4950 3500 50  0001 C CNN
 F 1 "GND" V 4950 3550 50  0000 C CNN
 F 2 "" H 4950 3750 50  0001 C CNN
@@
 $EndComp
 $Comp
-L +3V3 #PWR0151
+L +3V3 #PWR?
 U 1 1 5B0F5864
 P 5450 3750
-F 0 "#PWR0151" H 5450 3600 50  0001 C CNN
+F 0 "#PWR?" H 5450 3600 50  0001 C CNN
 F 1 "+3V3" V 5450 4000 50  0000 C CNN
 F 2 "" H 5450 3750 50  0001 C CNN
@@
 $EndComp
 $Comp
-L LED D1
+L LED D?
 U 1 1 5B1B21E2
 P 8000 3150
-F 0 "D1" H 8000 3250 50  0000 C CNN
+F 0 "D?" H 8000 3250 50  0000 C CNN
 F 1 "LED" H 8000 3050 50  0000 C CNN
 F 2 "LEDs:LED_0402" H 8000 3150 50  0001 C CNN
@@
 $EndComp
 $Comp
-L R_Small R114
+L R_Small R?
 U 1 1 5B1B2374
 P 8000 2800
-F 0 "R114" H 8030 2820 50  0000 L CNN
+F 0 "R?" H 8030 2820 50  0000 L CNN
 F 1 "430" H 8030 2760 50  0000 L CNN
 F 2 "Resistors_SMD:R_0402" H 8000 2800 50  0001 C CNN
@@
 GPIOs are 1,8 V only.\n!!!Not 3,3 V or 5 V tolerant!!!
 $Comp
-L +3V3 #PWR0152
+L +3V3 #PWR?
 U 1 1 5B1B2AD0
 P 8000 2550
-F 0 "#PWR0152" H 8000 2400 50  0001 C CNN
+F 0 "#PWR?" H 8000 2400 50  0001 C CNN
 F 1 "+3V3" H 8000 2690 50  0000 C CNN
 F 2 "" H 8000 2550 50  0001 C CNN
@@
 	8000 2550 8000 2700
 $Comp
-L GND #PWR0153
+L GND #PWR?
 U 1 1 5B1B2B0C
 P 8000 3400
-F 0 "#PWR0153" H 8000 3150 50  0001 C CNN
+F 0 "#PWR?" H 8000 3150 50  0001 C CNN
 F 1 "GND" H 8000 3250 50  0000 C CNN
 F 2 "" H 8000 3400 50  0001 C CNN
@@
 	8000 3300 8000 3400
 $Comp
-L BSS138PS Q3
+L BSS138PS Q?
 U 1 1 5B1B2B60
 P 9100 3150
-F 0 "Q3" H 9300 3225 50  0000 L CNN
+F 0 "Q?" H 9300 3225 50  0000 L CNN
 F 1 "BSS138PS" H 9300 3150 50  0000 L CNN
 F 2 "TO_SOT_Packages_SMD:SOT-363_SC-70-6" H 9300 3075 50  0001 L CIN
@@
 $EndComp
 $Comp
-L LED D2
+L LED D?
 U 1 1 5B1B2C38
 P 9200 2700
-F 0 "D2" H 9200 2800 50  0000 C CNN
+F 0 "D?" H 9200 2800 50  0000 C CNN
 F 1 "LED" H 9200 2600 50  0000 C CNN
 F 2 "LEDs:LED_0402" H 9200 2700 50  0001 C CNN
@@
 $EndComp
 $Comp
-L R_Small R116
+L R_Small R?
 U 1 1 5B1B2C8F
 P 9200 2350
-F 0 "R116" H 9230 2370 50  0000 L CNN
+F 0 "R?" H 9230 2370 50  0000 L CNN
 F 1 "430" H 9230 2310 50  0000 L CNN
 F 2 "Resistors_SMD:R_0402" H 9200 2350 50  0001 C CNN
@@
 	9200 2850 9200 2950
 $Comp
-L GND #PWR0154
+L GND #PWR?
 U 1 1 5B1B2D14
 P 9200 3700
-F 0 "#PWR0154" H 9200 3450 50  0001 C CNN
+F 0 "#PWR?" H 9200 3450 50  0001 C CNN
 F 1 "GND" H 9200 3550 50  0000 C CNN
 F 2 "" H 9200 3700 50  0001 C CNN
@@
 	9200 3350 9200 3700
 $Comp
-L +3V3 #PWR0155
+L +3V3 #PWR?
 U 1 1 5B1B2D42
 P 9200 2150
-F 0 "#PWR0155" H 9200 2000 50  0001 C CNN
+F 0 "#PWR?" H 9200 2000 50  0001 C CNN
 F 1 "+3V3" H 9200 2290 50  0000 C CNN
 F 2 "" H 9200 2150 50  0001 C CNN
@@
 LED1
 $Comp
-L BSS138PS Q3
-U 2 1 5B1B2E27
+L BSS138PS Q?
+U 1 1 5B1B2E27
 P 10600 3150
-F 0 "Q3" H 10800 3225 50  0000 L CNN
+F 0 "Q?" H 10800 3225 50  0000 L CNN
 F 1 "BSS138PS" H 10800 3150 50  0000 L CNN
 F 2 "TO_SOT_Packages_SMD:SOT-363_SC-70-6" H 10800 3075 50  0001 L CIN
@@
 F 7 "1" H 10600 3150 60  0001 C CNN "Populated"
 F 8 "SPEC" H 10600 3150 60  0001 C CNN "Source"
-	2    10600 3150
-	1    0    0    -1
-$EndComp
-$Comp
-L LED D3
+	1    10600 3150
+	1    0    0    -1
+$EndComp
+$Comp
+L LED D?
 U 1 1 5B1B2E2D
 P 10700 2700
-F 0 "D3" H 10700 2800 50  0000 C CNN
+F 0 "D?" H 10700 2800 50  0000 C CNN
 F 1 "LED" H 10700 2600 50  0000 C CNN
 F 2 "LEDs:LED_0402" H 10700 2700 50  0001 C CNN
@@
 $EndComp
 $Comp
-L R_Small R119
+L R_Small R?
 U 1 1 5B1B2E33
 P 10700 2350
-F 0 "R119" H 10730 2370 50  0000 L CNN
+F 0 "R?" H 10730 2370 50  0000 L CNN
 F 1 "430" H 10730 2310 50  0000 L CNN
 F 2 "Resistors_SMD:R_0402" H 10700 2350 50  0001 C CNN
@@
 	10700 2850 10700 2950
 $Comp
-L GND #PWR0156
+L GND #PWR?
 U 1 1 5B1B2E3B
 P 10700 3700
-F 0 "#PWR0156" H 10700 3450 50  0001 C CNN
+F 0 "#PWR?" H 10700 3450 50  0001 C CNN
 F 1 "GND" H 10700 3550 50  0000 C CNN
 F 2 "" H 10700 3700 50  0001 C CNN
@@
 	10700 3350 10700 3700
 $Comp
-L +3V3 #PWR0157
+L +3V3 #PWR?
 U 1 1 5B1B2E42
 P 10700 2150
-F 0 "#PWR0157" H 10700 2000 50  0001 C CNN
+F 0 "#PWR?" H 10700 2000 50  0001 C CNN
 F 1 "+3V3" H 10700 2290 50  0000 C CNN
 F 2 "" H 10700 2150 50  0001 C CNN
@@
 User LEDs
 $Comp
-L R_Small R115
+L R_Small R?
 U 1 1 5B204015
 P 8800 3350
-F 0 "R115" H 8830 3370 50  0000 L CNN
+F 0 "R?" H 8830 3370 50  0000 L CNN
 F 1 "100k" H 8830 3310 50  0000 L CNN
 F 2 "Resistors_SMD:R_0402" H 8800 3350 50  0001 C CNN
@@
 	10200 3150 10400 3150
 $Comp
-L R_Small R117
+L R_Small R?
 U 1 1 5B20436B
 P 10350 3350
-F 0 "R117" H 10380 3370 50  0000 L CNN
+F 0 "R?" H 10380 3370 50  0000 L CNN
 F 1 "100k" H 10380 3310 50  0000 L CNN
 F 2 "Resistors_SMD:R_0402" H 10350 3350 50  0001 C CNN
@@
 Connection ~ 10700 3550
 $Comp
-L Conn_01x02 J9
+L Conn_01x02 J?
 U 1 1 5B2142B2
 P 10700 4550
-F 0 "J9" H 10700 4650 50  0000 C CNN
+F 0 "J?" H 10700 4650 50  0000 C CNN
 F 1 "Conn_01x02" H 10700 4350 50  0000 C CNN
 F 2 "Pin_Headers:Pin_Header_Angled_1x02_Pitch2.54mm" H 10700 4550 50  0001 C CNN
@@
 	10400 4650 10400 4750
 $Comp
-L GND #PWR0158
+L GND #PWR?
 U 1 1 5B2143F5
 P 10400 4750
-F 0 "#PWR0158" H 10400 4500 50  0001 C CNN
+F 0 "#PWR?" H 10400 4500 50  0001 C CNN
 F 1 "GND" H 10400 4600 50  0000 C CNN
 F 2 "" H 10400 4750 50  0001 C CNN
@@
 $EndComp
 $Comp
-L R_Small R118
+L R_Small R?
 U 1 1 5B214424
 P 10400 4350
-F 0 "R118" H 10430 4370 50  0000 L CNN
+F 0 "R?" H 10430 4370 50  0000 L CNN
 F 1 "DNP" H 10430 4310 50  0000 L CNN
 F 2 "Resistors_SMD:R_0402" H 10400 4350 50  0001 C CNN
@@
 	10300 4550 10500 4550
 $Comp
-L +1V8 #PWR0159
+L +1V8 #PWR?
 U 1 1 5B21453D
 P 10400 4150
-F 0 "#PWR0159" H 10400 4000 50  0001 C CNN
+F 0 "#PWR?" H 10400 4000 50  0001 C CNN
 F 1 "+1V8" H 10400 4290 50  0000 C CNN
 F 2 "" H 10400 4150 50  0001 C CNN
