File: hardware/gpio.sch (KiCad schematic (older format))
At the start: 13 parts

Commit message: Added a few Todos.
Other:
- note added: "TODO: Select footprint for connector. Maybe something high density. Just in Case for soldering a wire to it or somthing like that."
Changed lines of the file:
@@
 BUTTON1
 Connection ~ 10400 4550
+Text Notes 1600 4250 0    60   ~ 0
+TODO: Select footprint for connector. Maybe something high density. Just in Case for soldering a wire to it or somthing like that.
 $EndSCHEMATC

Commit message: Removed all BSS138PS Transistors due actual unavailability.
Used lsf0102 as Levelshifter for I2C bus, connected LEDs to already existing Levelshifters.
Parts:
- removed D? (x2): LED, LEDs:LED_0402, symbol LED
- removed Q? (x2): BSS138PS, TO_SOT_Packages_SMD:SOT-363_SC-70-6, symbol BSS138PS
- removed R? (x2): 430, Resistors_SMD:R_0402, symbol R_Small
- removed R? (x2): 100k, Resistors_SMD:R_0402, symbol R_Small
Connections:
- net labels removed: +1V8, LED1, LED2
- wire segments 24 -> 8
Other:
- note removed: "User LEDs"

Commit message: Started to route DDR3 Memory.
At first added missing Footprint for Reference- and Terminationvoltage Regulator. Added Powerplanes for GND and VCCO. Added decoupling Network to both DDR3 Memory Chips. There are more small caps, to support Memory from other Manufactors.
Parts:
- gave numbers to parts that had none: 5
Changed lines of the file:
@@
 $EndDescr
 $Comp
-L Conn_02x09_Counter_Clockwise J?
+L Conn_02x09_Counter_Clockwise J8
 U 1 1 5B0F5739
 P 5150 3350
-F 0 "J?" H 5200 3850 50  0000 C CNN
+F 0 "J8" H 5200 3850 50  0000 C CNN
 F 1 "Conn_02x09_Counter_Clockwise" H 5200 2850 50  0000 C CNN
 F 2 "" H 5150 3350 50  0001 C CNN
@@
 GPIO_15
 $Comp
-L GND #PWR?
+L GND #PWR0218
 U 1 1 5B0F584E
 P 4950 3750
-F 0 "#PWR?" H 4950 3500 50  0001 C CNN
+F 0 "#PWR0218" H 4950 3500 50  0001 C CNN
 F 1 "GND" V 4950 3550 50  0000 C CNN
 F 2 "" H 4950 3750 50  0001 C CNN
@@
 $EndComp
 $Comp
-L +3V3 #PWR?
+L +3V3 #PWR0219
 U 1 1 5B0F5864
 P 5450 3750
-F 0 "#PWR?" H 5450 3600 50  0001 C CNN
+F 0 "#PWR0219" H 5450 3600 50  0001 C CNN
 F 1 "+3V3" V 5450 4000 50  0000 C CNN
 F 2 "" H 5450 3750 50  0001 C CNN
@@
 $EndComp
 $Comp
-L LED D?
+L LED D4
 U 1 1 5B1B21E2
 P 10500 3150
-F 0 "D?" H 10500 3250 50  0000 C CNN
+F 0 "D4" H 10500 3250 50  0000 C CNN
 F 1 "LED" H 10500 3050 50  0000 C CNN
 F 2 "LEDs:LED_0402" H 10500 3150 50  0001 C CNN
@@
 $EndComp
 $Comp
-L R_Small R?
+L R_Small R143
 U 1 1 5B1B2374
 P 10500 2800
-F 0 "R?" H 10530 2820 50  0000 L CNN
+F 0 "R143" H 10530 2820 50  0000 L CNN
 F 1 "430" H 10530 2760 50  0000 L CNN
 F 2 "Resistors_SMD:R_0402" H 10500 2800 50  0001 C CNN
@@
 GPIOs are 1,8 V only.\n!!!Not 3,3 V or 5 V tolerant!!!
 $Comp
-L +3V3 #PWR?
+L +3V3 #PWR0220
 U 1 1 5B1B2AD0
 P 10500 2550
-F 0 "#PWR?" H 10500 2400 50  0001 C CNN
+F 0 "#PWR0220" H 10500 2400 50  0001 C CNN
 F 1 "+3V3" H 10500 2690 50  0000 C CNN
 F 2 "" H 10500 2550 50  0001 C CNN
@@
 	10500 2550 10500 2700
 $Comp
-L GND #PWR?
+L GND #PWR0221
 U 1 1 5B1B2B0C
 P 10500 3400
-F 0 "#PWR?" H 10500 3150 50  0001 C CNN
+F 0 "#PWR0221" H 10500 3150 50  0001 C CNN
 F 1 "GND" H 10500 3250 50  0000 C CNN
 F 2 "" H 10500 3400 50  0001 C CNN
@@
 Power Led
 $Comp
-L Conn_01x02 J?
+L Conn_01x02 J9
 U 1 1 5B2142B2
 P 10700 4550
-F 0 "J?" H 10700 4650 50  0000 C CNN
+F 0 "J9" H 10700 4650 50  0000 C CNN
 F 1 "Conn_01x02" H 10700 4350 50  0000 C CNN
 F 2 "Pin_Headers:Pin_Header_Angled_1x02_Pitch2.54mm" H 10700 4550 50  0001 C CNN
@@
 	10400 4650 10400 4750
 $Comp
-L GND #PWR?
+L GND #PWR0222
 U 1 1 5B2143F5
 P 10400 4750
-F 0 "#PWR?" H 10400 4500 50  0001 C CNN
+F 0 "#PWR0222" H 10400 4500 50  0001 C CNN
 F 1 "GND" H 10400 4600 50  0000 C CNN
 F 2 "" H 10400 4750 50  0001 C CNN
@@
 $EndComp
 $Comp
-L R_Small R?
+L R_Small R142
 U 1 1 5B214424
 P 10400 4350
-F 0 "R?" H 10430 4370 50  0000 L CNN
+F 0 "R142" H 10430 4370 50  0000 L CNN
 F 1 "DNP" H 10430 4310 50  0000 L CNN
 F 2 "Resistors_SMD:R_0402" H 10400 4350 50  0001 C CNN

Commit message: Added Power/Protection Circuit
Parts:
- renumbered D4 to D1701, J8 to J1701, J9 to J1702, R142 to R1701, R143 to R1702
Changed lines of the file:
@@
 $EndDescr
 $Comp
-L Conn_02x09_Counter_Clockwise J8
+L Conn_02x09_Counter_Clockwise J1701
 U 1 1 5B0F5739
 P 5150 3350
-F 0 "J8" H 5200 3850 50  0000 C CNN
+F 0 "J1701" H 5200 3850 50  0000 C CNN
 F 1 "Conn_02x09_Counter_Clockwise" H 5200 2850 50  0000 C CNN
 F 2 "" H 5150 3350 50  0001 C CNN
@@
 $EndComp
 $Comp
-L LED D4
+L LED D1701
 U 1 1 5B1B21E2
 P 10500 3150
-F 0 "D4" H 10500 3250 50  0000 C CNN
+F 0 "D1701" H 10500 3250 50  0000 C CNN
 F 1 "LED" H 10500 3050 50  0000 C CNN
 F 2 "LEDs:LED_0402" H 10500 3150 50  0001 C CNN
@@
 $EndComp
 $Comp
-L R_Small R143
+L R_Small R1702
 U 1 1 5B1B2374
 P 10500 2800
-F 0 "R143" H 10530 2820 50  0000 L CNN
+F 0 "R1702" H 10530 2820 50  0000 L CNN
 F 1 "430" H 10530 2760 50  0000 L CNN
 F 2 "Resistors_SMD:R_0402" H 10500 2800 50  0001 C CNN
@@
 Power Led
 $Comp
-L Conn_01x02 J9
+L Conn_01x02 J1702
 U 1 1 5B2142B2
 P 10700 4550
-F 0 "J9" H 10700 4650 50  0000 C CNN
+F 0 "J1702" H 10700 4650 50  0000 C CNN
 F 1 "Conn_01x02" H 10700 4350 50  0000 C CNN
 F 2 "Pin_Headers:Pin_Header_Angled_1x02_Pitch2.54mm" H 10700 4550 50  0001 C CNN
@@
 $EndComp
 $Comp
-L R_Small R142
+L R_Small R1701
 U 1 1 5B214424
 P 10400 4350
-F 0 "R142" H 10430 4370 50  0000 L CNN
+F 0 "R1701" H 10430 4370 50  0000 L CNN
 F 1 "DNP" H 10430 4310 50  0000 L CNN
 F 2 "Resistors_SMD:R_0402" H 10400 4350 50  0001 C CNN
