File: hardware/gpio.sch (KiCad schematic (older format))
At the start: 5 parts, among them J1701 Conn_02x09_Counter_Clockwise, J1702 Conn_01x02

Commit message: Length matched DDR3 Memory again.
Forgot to keep enough space between the traces and between the meander waves.

Also, I switched to Kicad 5.0 RC2.

Swaped a few ddr signals.
Parts:
- D1701: symbol LED -> device:LED
- J1701: symbol Conn_02x09_Counter_Clockwise -> conn:Conn_02x09_Counter_Clockwise
- J1702: symbol Conn_01x02 -> conn:Conn_01x02
- R1701, R1702: symbol R_Small -> device:R_Small
Changed lines of the file:
@@
-EESchema Schematic File Version 2
-LIBS:zynq_board-rescue
-LIBS:power
-LIBS:device
-LIBS:transistors
-LIBS:conn
-LIBS:linear
-LIBS:regul
-LIBS:74xx
-LIBS:cmos4000
-LIBS:adc-dac
-LIBS:memory
-LIBS:xilinx
-LIBS:microcontrollers
-LIBS:dsp
-LIBS:microchip
-LIBS:analog_switches
-LIBS:motorola
-LIBS:texas
-LIBS:intel
-LIBS:audio
-LIBS:interface
-LIBS:digital-audio
-LIBS:philips
-LIBS:display
-LIBS:cypress
-LIBS:siliconi
-LIBS:opto
-LIBS:atmel
-LIBS:contrib
-LIBS:valves
-LIBS:xilinx_zynq_clg485
-LIBS:SFP_plus
-LIBS:ael2005
-LIBS:diff_osc
-LIBS:si53340
-LIBS:usb3320
-LIBS:nx5p3090
-LIBS:smp1255putg
-LIBS:osc
-LIBS:ddr
-LIBS:misc
-LIBS:tlk10031
-LIBS:lshm-150-xxx-x-dv-a-s
-LIBS:sn74axc8t245
-LIBS:sn74lvc2t45
-LIBS:dmf05lcflp
-LIBS:bss138ps
-LIBS:max14854
-LIBS:switches
-LIBS:ft234xd
-LIBS:sn74lv1t126
-LIBS:emif06-msd02n16
-LIBS:cat24c02tdi-gt3
-LIBS:power_symbols
-LIBS:ti_power_modules
-LIBS:mdr20
-LIBS:dm3cs
-LIBS:lsf0102
-LIBS:dmp3056l
+EESchema Schematic File Version 4
 LIBS:zynq_board-cache
-EELAYER 25 0
+EELAYER 26 0
 EELAYER END
 $Descr A4 11693 8268
@@
 $EndDescr
 $Comp
-L Conn_02x09_Counter_Clockwise J1701
+L conn:Conn_02x09_Counter_Clockwise J1701
 U 1 1 5B0F5739
 P 5150 3350
@@
 GPIO_15
 $Comp
-L GND #PWR0220
+L power1:GND #PWR0220
 U 1 1 5B0F584E
 P 4950 3750
@@
 $EndComp
 $Comp
-L +3V3 #PWR0221
+L power1:+3V3 #PWR0221
 U 1 1 5B0F5864
 P 5450 3750
@@
 $EndComp
 $Comp
-L LED D1701
+L device:LED D1701
 U 1 1 5B1B21E2
 P 10500 3150
@@
 $EndComp
 $Comp
-L R_Small R1702
+L device:R_Small R1702
 U 1 1 5B1B2374
 P 10500 2800
@@
 GPIOs are 1,8 V only.\n!!!Not 3,3 V or 5 V tolerant!!!
 $Comp
-L +3V3 #PWR0222
+L power1:+3V3 #PWR0222
 U 1 1 5B1B2AD0
 P 10500 2550
@@
 	10500 2550 10500 2700
 $Comp
-L GND #PWR0223
+L power1:GND #PWR0223
 U 1 1 5B1B2B0C
 P 10500 3400
@@
 Power Led
 $Comp
-L Conn_01x02 J1702
+L conn:Conn_01x02 J1702
 U 1 1 5B2142B2
 P 10700 4550
@@
 	10400 4650 10400 4750
 $Comp
-L GND #PWR0224
+L power1:GND #PWR0224
 U 1 1 5B2143F5
 P 10400 4750
@@
 $EndComp
 $Comp
-L R_Small R1701
+L device:R_Small R1701
 U 1 1 5B214424
 P 10400 4350

Commit message: Layouted USB-UART.
Also moved USB-OTG to the right Side of the Board. To get there
some free Space, i moved the DDR3/Memory and the FPGA a few
Millimeters down.
Parts:
- R1701, R1702: footprint Resistors_SMD:R_0402 -> Resistor_SMD:R_0402_1005Metric
Changed lines of the file:
@@
 F 0 "R1702" H 10530 2820 50  0000 L CNN
 F 1 "430" H 10530 2760 50  0000 L CNN
-F 2 "Resistors_SMD:R_0402" H 10500 2800 50  0001 C CNN
+F 2 "Resistor_SMD:R_0402_1005Metric" H 10500 2800 50  0001 C CNN
 F 3 "" H 10500 2800 50  0001 C CNN
 F 4 "1" H 10500 2800 60  0001 C CNN "Populated"
@@
 F 0 "R1701" H 10430 4370 50  0000 L CNN
 F 1 "DNP" H 10430 4310 50  0000 L CNN
-F 2 "Resistors_SMD:R_0402" H 10400 4350 50  0001 C CNN
+F 2 "Resistor_SMD:R_0402_1005Metric" H 10400 4350 50  0001 C CNN
 F 3 "" H 10400 4350 50  0001 C CNN
 F 4 "0" H 10400 4350 60  0001 C CNN "Populated"

Commit message: Fixed Schematic Symbols
Parts:
- D1701: symbol device:LED -> Device:LED_Small
- J1701: symbol conn:Conn_02x09_Counter_Clockwise -> Connector_Generic:Conn_02x09_Counter_Clockwise
- J1702: symbol conn:Conn_01x02 -> Connector_Generic:Conn_01x02
- R1701, R1702: symbol device:R_Small -> Device:R_Small
Connections:
- wire segments 8 -> 9
Changed lines of the file:
@@
 $Descr A4 11693 8268
 encoding utf-8
-Sheet 17 22
+Sheet 17 21
 Title ""
 Date ""
@@
 $EndDescr
 $Comp
-L conn:Conn_02x09_Counter_Clockwise J1701
+L Connector_Generic:Conn_02x09_Counter_Clockwise J1701
 U 1 1 5B0F5739
 P 5150 3350
@@
 GPIO_15
 $Comp
-L power1:GND #PWR0220
+L power:GND #PWR0220
 U 1 1 5B0F584E
 P 4950 3750
@@
 $EndComp
 $Comp
-L power1:+3V3 #PWR0221
+L power:+3V3 #PWR0221
 U 1 1 5B0F5864
 P 5450 3750
@@
 $EndComp
 $Comp
-L device:LED D1701
+L Device:LED_Small D1701
 U 1 1 5B1B21E2
 P 10500 3150
@@
 $EndComp
 $Comp
-L device:R_Small R1702
+L Device:R_Small R1702
 U 1 1 5B1B2374
 P 10500 2800
@@
 	1    0    0    -1
 $EndComp
-Wire Wire Line
-	10500 2900 10500 3000
 Wire Notes Line
 	4500 2700 4500 3950
@@
 GPIOs are 1,8 V only.\n!!!Not 3,3 V or 5 V tolerant!!!
 $Comp
-L power1:+3V3 #PWR0222
+L power:+3V3 #PWR0222
 U 1 1 5B1B2AD0
 P 10500 2550
@@
 	10500 2550 10500 2700
 $Comp
-L power1:GND #PWR0223
+L power:GND #PWR0223
 U 1 1 5B1B2B0C
 P 10500 3400
@@
 	1    0    0    -1
 $EndComp
-Wire Wire Line
-	10500 3300 10500 3400
 Text Notes 10300 2200 0    60   ~ 0
 Power Led
 $Comp
-L conn:Conn_01x02 J1702
+L Connector_Generic:Conn_01x02 J1702
 U 1 1 5B2142B2
 P 10700 4550
@@
 	10400 4650 10400 4750
 $Comp
-L power1:GND #PWR0224
+L power:GND #PWR0224
 U 1 1 5B2143F5
 P 10400 4750
@@
 $EndComp
 $Comp
-L device:R_Small R1701
+L Device:R_Small R1701
 U 1 1 5B214424
 P 10400 4350
@@
 	10400 4450 10400 4550
 Wire Wire Line
-	10300 4550 10500 4550
+	10300 4550 10400 4550
 Wire Wire Line
 	10400 4150 10400 4250
@@
 Text Notes 1600 4250 0    60   ~ 0
 TODO: Select footprint for connector. Maybe something high density. Just in Case for soldering a wire to it or somthing like that.
+Wire Wire Line
+	10400 4550 10500 4550
+Wire Wire Line
+	10500 3250 10500 3400
+Wire Wire Line
+	10500 2900 10500 3050
 $EndSCHEMATC

Commit message: WIP: TLK Powerdistribution
Parts:
- removed D1701: LED, LEDs:LED_0402, symbol Device:LED_Small
- added D1601: LED_ALT, LED_SMD:LED_0603_1608Metric, symbol Device:LED_ALT
Changed lines of the file:
@@
 EESchema Schematic File Version 4
-LIBS:zynq_board-cache
 EELAYER 26 0
 EELAYER END
 $Descr A4 11693 8268
 encoding utf-8
-Sheet 17 21
+Sheet 16 21
 Title ""
 Date ""
@@
 $EndComp
 $Comp
-L Device:LED_Small D1701
-U 1 1 5B1B21E2
-P 10500 3150
-F 0 "D1701" H 10500 3250 50  0000 C CNN
-F 1 "LED" H 10500 3050 50  0000 C CNN
-F 2 "LEDs:LED_0402" H 10500 3150 50  0001 C CNN
-F 3 "" H 10500 3150 50  0001 C CNN
-F 4 "1" H 10500 3150 60  0001 C CNN "Populated"
-F 5 "SPEC" H 10500 3150 60  0001 C CNN "Source"
-	1    10500 3150
-	0    -1   -1   0
-$EndComp
-$Comp
 L Device:R_Small R1702
 U 1 1 5B1B2374
@@
 Wire Wire Line
 	10400 4550 10500 4550
-Wire Wire Line
-	10500 3250 10500 3400
-Wire Wire Line
-	10500 2900 10500 3050
+$Comp
+L Device:LED_ALT D1601
+U 1 1 5B3144CD
+P 10500 3150
+F 0 "D1601" H 10491 3366 50  0000 C CNN
+F 1 "LED_ALT" H 10491 3275 50  0000 C CNN
+F 2 "LED_SMD:LED_0603_1608Metric" H 10500 3150 50  0001 C CNN
+F 3 "http://www.qt-brightek.com/datasheet/QBLP617_series.pdf" H 10500 3150 50  0001 C CNN
+F 4 "QT Brightek (QTB)" H 10500 3150 50  0001 C CNN "MFG Name"
+F 5 "QBLP617-R" H 10500 3150 50  0001 C CNN "MFG Part Num"
+F 6 "1516-1081-1-ND" H 10500 3150 50  0001 C CNN "Digikey"
+F 7 "1" H 10500 3150 50  0001 C CNN "Populated"
+F 8 "LED RED CLEAR 2SMD R/A" H 10500 3150 50  0001 C CNN "Description"
+F 9 "SPEC" H 10500 3150 50  0001 C CNN "Source"
+F 10 "1" H 10500 3150 50  0001 C CNN "Populate for SBGA485(Z-7030)"
+F 11 "1" H 10500 3150 50  0001 C CNN "Populate for CLG484(Z-7012s/Z-7015)"
+	1    10500 3150
+	0    -1   -1   0
+$EndComp
+Wire Wire Line
+	10500 2900 10500 3000
+Wire Wire Line
+	10500 3400 10500 3300
 $EndSCHEMATC

Commit message: PS Clock, Reset Button, Cam Levelshifters and big 1.0 V Cap placed.
Improved some Footprints and library Symbols.

Also though about Chassis Ground.
Parts:
- J1701: footprint (none) -> footprints:Solder-Pin-Array_18Pins_TestPoint_SMD_0.5mm_0.75mm-pitch; Populate for CLG484(Z-7012s/Z-7015) (none) -> 1; Populate for SBGA485(Z-7030) (none) -> 1; Populated (none) -> 1; Source (none) -> SPEC
Changed lines of the file:
@@
 F 0 "J1701" H 5200 3850 50  0000 C CNN
 F 1 "Conn_02x09_Counter_Clockwise" H 5200 2850 50  0000 C CNN
-F 2 "" H 5150 3350 50  0001 C CNN
+F 2 "footprints:Solder-Pin-Array_18Pins_TestPoint_SMD_0.5mm_0.75mm-pitch" H 5150 3350 50  0001 C CNN
 F 3 "" H 5150 3350 50  0001 C CNN
+F 4 "1" H 5150 3350 50  0001 C CNN "Populated"
+F 5 "SPEC" H 5150 3350 50  0001 C CNN "Source"
+F 6 "1" H 5150 3350 50  0001 C CNN "Populate for SBGA485(Z-7030)"
+F 7 "1" H 5150 3350 50  0001 C CNN "Populate for CLG484(Z-7012s/Z-7015)"
 	1    5150 3350
 	1    0    0    -1

Commit message: WIP: general Routing
Changed lines of the file:
@@
 $Descr A4 11693 8268
 encoding utf-8
-Sheet 15 21
+Sheet 21 21
 Title ""
 Date ""
@@
 	1    0    0    -1
 $EndComp
-Text HLabel 4950 2950 0    60   BiDi ~ 0
-GPIO_0
-Text HLabel 4950 3050 0    60   BiDi ~ 0
-GPIO_1
-Text HLabel 4950 3150 0    60   BiDi ~ 0
-GPIO_2
-Text HLabel 4950 3250 0    60   BiDi ~ 0
-GPIO_3
-Text HLabel 4950 3350 0    60   BiDi ~ 0
-GPIO_4
-Text HLabel 4950 3450 0    60   BiDi ~ 0
-GPIO_5
-Text HLabel 4950 3550 0    60   BiDi ~ 0
-GPIO_6
-Text HLabel 4950 3650 0    60   BiDi ~ 0
-GPIO_7
-Text HLabel 5450 3650 2    60   BiDi ~ 0
-GPIO_8
-Text HLabel 5450 3550 2    60   BiDi ~ 0
-GPIO_9
-Text HLabel 5450 3450 2    60   BiDi ~ 0
-GPIO_10
-Text HLabel 5450 3350 2    60   BiDi ~ 0
-GPIO_11
-Text HLabel 5450 3250 2    60   BiDi ~ 0
-GPIO_12
-Text HLabel 5450 3150 2    60   BiDi ~ 0
-GPIO_13
-Text HLabel 5450 3050 2    60   BiDi ~ 0
-GPIO_14
-Text HLabel 5450 2950 2    60   BiDi ~ 0
-GPIO_15
 $Comp
 L power:GND #PWR0220
@@
 Wire Wire Line
 	10500 3400 10500 3300
+Text GLabel 4950 2950 0    50   BiDi ~ 0
+GPIO_0
+Text GLabel 4950 3050 0    50   BiDi ~ 0
+GPIO_2
+Text GLabel 4950 3150 0    50   BiDi ~ 0
+GPIO_4
+Text GLabel 4950 3250 0    50   BiDi ~ 0
+GPIO_6
+Text GLabel 4950 3350 0    50   BiDi ~ 0
+GPIO_8
+Text GLabel 4950 3450 0    50   BiDi ~ 0
+GPIO_10
+Text GLabel 4950 3550 0    50   BiDi ~ 0
+GPIO_12
+Text GLabel 4950 3650 0    50   BiDi ~ 0
+GPIO_14
+Text GLabel 5450 3650 2    50   BiDi ~ 0
+GPIO_15
+Text GLabel 5450 3550 2    50   BiDi ~ 0
+GPIO_13
+Text GLabel 5450 3450 2    50   BiDi ~ 0
+GPIO_11
+Text GLabel 5450 3350 2    50   BiDi ~ 0
+GPIO_9
+Text GLabel 5450 3250 2    50   BiDi ~ 0
+GPIO_7
+Text GLabel 5450 3150 2    50   BiDi ~ 0
+GPIO_5
+Text GLabel 5450 3050 2    50   BiDi ~ 0
+GPIO_3
+Text GLabel 5450 2950 2    50   BiDi ~ 0
+GPIO_1
 $EndSCHEMATC
