File: hardware/zynq_ps.sch (KiCad schematic (older format))
At the start: 20 parts, among them J2 Micro_SD_Card_Det_Hirose_DM3AT, SW1 SW_Push, U1 xc7z030sbg485

Commit message: Added USB-Uart subschematic. WIP
USB-Uart will be bus powered. Buffer between FTDI and FPGA is missing.
Parts:
- renumbered C14 to C?, J2 to J?, R11 to R?, R9 to R?, R7 to R?, R5 to R?, R3 to R?, R4 to R?, R6 to R?, R8 to R?, R10 to R?, R12 to R?, R121 to R?, R120 to R?, R2 to R?, R1 to R?, R13 to R?, R14 to R?, SW1 to SW?, U1 to U?
Connections:
- net labels added: UART_RX, UART_TX
Changed lines of the file:
@@
 LIBS:max14854
 LIBS:switches
+LIBS:ft234xd
 LIBS:zynq_board-cache
 EELAYER 25 0
@@
 $Descr A4 11693 8268
 encoding utf-8
-Sheet 20 20
+Sheet 20 21
 Title ""
 Date ""
@@
 $EndDescr
 $Comp
-L xc7z030sbg485 U1
+L xc7z030sbg485 U?
 U 6 1 596E7E39
 P 9200 1400
-F 0 "U1" H 9400 1650 60  0000 L CNN
+F 0 "U?" H 9400 1650 60  0000 L CNN
 F 1 "xc7z030sbg485" H 9400 1550 60  0000 L CNN
 F 2 "footprints:SBG485_22x22_19.0x19.0mm_Pitch0.8mm" H 9200 1400 60  0001 C CNN
@@
 $EndComp
 $Comp
-L xc7z030sbg485 U1
+L xc7z030sbg485 U?
 U 7 1 596E7E6B
 P 5500 1450
-F 0 "U1" H 5700 1700 60  0000 L CNN
+F 0 "U?" H 5700 1700 60  0000 L CNN
 F 1 "xc7z030sbg485" H 5700 1600 60  0000 L CNN
 F 2 "footprints:SBG485_22x22_19.0x19.0mm_Pitch0.8mm" H 5500 1450 60  0001 C CNN
@@
 NOTE: The BootROM expects the SD card\nto be connected to MIO pins 40..45 (SDIO0).
 $Comp
-L R R11
+L R R?
 U 1 1 5A98BDBC
 P 7950 1400
-F 0 "R11" V 8030 1400 50  0000 C CNN
+F 0 "R?" V 8030 1400 50  0000 C CNN
 F 1 "DNP" V 7950 1400 50  0000 C CNN
 F 2 "Resistors_SMD:R_0402" V 7880 1400 50  0001 C CNN
@@
 $EndComp
 $Comp
-L R R9
+L R R?
 U 1 1 5A98BDD7
 P 7750 1400
-F 0 "R9" V 7830 1400 50  0000 C CNN
+F 0 "R?" V 7830 1400 50  0000 C CNN
 F 1 "DNP" V 7750 1400 50  0000 C CNN
 F 2 "Resistors_SMD:R_0402" V 7680 1400 50  0001 C CNN
@@
 $EndComp
 $Comp
-L R R7
+L R R?
 U 1 1 5A98BDF4
 P 7550 1400
-F 0 "R7" V 7630 1400 50  0000 C CNN
+F 0 "R?" V 7630 1400 50  0000 C CNN
 F 1 "20k" V 7550 1400 50  0000 C CNN
 F 2 "Resistors_SMD:R_0402" V 7480 1400 50  0001 C CNN
@@
 $EndComp
 $Comp
-L R R5
+L R R?
 U 1 1 5A98BE13
 P 7350 1400
-F 0 "R5" V 7430 1400 50  0000 C CNN
+F 0 "R?" V 7430 1400 50  0000 C CNN
 F 1 "20k" V 7350 1400 50  0000 C CNN
 F 2 "Resistors_SMD:R_0402" V 7280 1400 50  0001 C CNN
@@
 $EndComp
 $Comp
-L R R3
+L R R?
 U 1 1 5A98BE34
 P 7150 1400
-F 0 "R3" V 7230 1400 50  0000 C CNN
+F 0 "R?" V 7230 1400 50  0000 C CNN
 F 1 "DNP" V 7150 1400 50  0000 C CNN
 F 2 "Resistors_SMD:R_0402" V 7080 1400 50  0001 C CNN
@@
 $EndComp
 $Comp
-L R R4
+L R R?
 U 1 1 5A98BE57
 P 7150 2600
-F 0 "R4" V 7230 2600 50  0000 C CNN
+F 0 "R?" V 7230 2600 50  0000 C CNN
 F 1 "20k" V 7150 2600 50  0000 C CNN
 F 2 "Resistors_SMD:R_0402" V 7080 2600 50  0001 C CNN
@@
 $EndComp
 $Comp
-L R R6
+L R R?
 U 1 1 5A98BE7C
 P 7350 2600
-F 0 "R6" V 7430 2600 50  0000 C CNN
+F 0 "R?" V 7430 2600 50  0000 C CNN
 F 1 "DNP" V 7350 2600 50  0000 C CNN
 F 2 "Resistors_SMD:R_0402" V 7280 2600 50  0001 C CNN
@@
 $EndComp
 $Comp
-L R R8
+L R R?
 U 1 1 5A98BEA3
 P 7550 2600
-F 0 "R8" V 7630 2600 50  0000 C CNN
+F 0 "R?" V 7630 2600 50  0000 C CNN
 F 1 "DNP" V 7550 2600 50  0000 C CNN
 F 2 "Resistors_SMD:R_0402" V 7480 2600 50  0001 C CNN
@@
 $EndComp
 $Comp
-L R R10
+L R R?
 U 1 1 5A98BECC
 P 7750 2600
-F 0 "R10" V 7830 2600 50  0000 C CNN
+F 0 "R?" V 7830 2600 50  0000 C CNN
 F 1 "20k" V 7750 2600 50  0000 C CNN
 F 2 "Resistors_SMD:R_0402" V 7680 2600 50  0001 C CNN
@@
 $EndComp
 $Comp
-L R R12
+L R R?
 U 1 1 5A98BEF7
 P 7950 2600
-F 0 "R12" V 8030 2600 50  0000 C CNN
+F 0 "R?" V 8030 2600 50  0000 C CNN
 F 1 "20k" V 7950 2600 50  0000 C CNN
 F 2 "Resistors_SMD:R_0402" V 7880 2600 50  0001 C CNN
@@
 Connection ~ 7750 2850
 $Comp
-L GND #PWR01
+L GND #PWR?
 U 1 1 5A991630
 P 7550 2950
-F 0 "#PWR01" H 7550 2700 50  0001 C CNN
+F 0 "#PWR?" H 7550 2700 50  0001 C CNN
 F 1 "GND" H 7550 2800 50  0000 C CNN
 F 2 "" H 7550 2950 50  0000 C CNN
@@
 TODO: UART, I2C
 $Comp
-L SW_Push SW1
+L SW_Push SW?
 U 1 1 5B1ED103
 P 10400 5550
-F 0 "SW1" H 10450 5650 50  0000 L CNN
+F 0 "SW?" H 10450 5650 50  0000 L CNN
 F 1 "SW_Push" H 10400 5490 50  0000 C CNN
 F 2 "" H 10400 5750 50  0001 C CNN
@@
 	10700 5550 10700 5650
 $Comp
-L GND #PWR02
+L GND #PWR?
 U 1 1 5B1ED412
 P 10700 5650
-F 0 "#PWR02" H 10700 5400 50  0001 C CNN
+F 0 "#PWR?" H 10700 5400 50  0001 C CNN
 F 1 "GND" H 10700 5500 50  0000 C CNN
 F 2 "" H 10700 5650 50  0001 C CNN
@@
 	9400 5550 10200 5550
 $Comp
-L C_Small C14
+L C_Small C?
 U 1 1 5B1EDFD0
 P 10100 5750
-F 0 "C14" H 10110 5820 50  0000 L CNN
+F 0 "C?" H 10110 5820 50  0000 L CNN
 F 1 "100 nF" H 10110 5670 50  0000 L CNN
 F 2 "" H 10100 5750 50  0001 C CNN
@@
 Connection ~ 10100 5550
 $Comp
-L GND #PWR03
+L GND #PWR?
 U 1 1 5B1EE083
 P 10100 5950
-F 0 "#PWR03" H 10100 5700 50  0001 C CNN
+F 0 "#PWR?" H 10100 5700 50  0001 C CNN
 F 1 "GND" H 10100 5800 50  0000 C CNN
 F 2 "" H 10100 5950 50  0001 C CNN
@@
 	8700 3100 9200 3100
 $Comp
-L R_Small R2
+L R_Small R?
 U 1 1 5B1EF27E
 P 10100 5350
-F 0 "R2" H 10130 5370 50  0000 L CNN
+F 0 "R?" H 10130 5370 50  0000 L CNN
 F 1 "10k" H 10130 5310 50  0000 L CNN
 F 2 "" H 10100 5350 50  0001 C CNN
@@
 Reset Button
 $Comp
-L +3V3 #PWR04
+L +3V3 #PWR?
 U 1 1 5B22F1F8
 P 10100 5150
-F 0 "#PWR04" H 10100 5000 50  0001 C CNN
+F 0 "#PWR?" H 10100 5000 50  0001 C CNN
 F 1 "+3V3" H 10100 5290 50  0000 C CNN
 F 2 "" H 10100 5150 50  0001 C CNN
@@
 $EndComp
 $Comp
-L +3V3 #PWR05
+L +3V3 #PWR?
 U 1 1 5B22F273
 P 7550 1050
-F 0 "#PWR05" H 7550 900 50  0001 C CNN
+F 0 "#PWR?" H 7550 900 50  0001 C CNN
 F 1 "+3V3" H 7550 1190 50  0000 C CNN
 F 2 "" H 7550 1050 50  0001 C CNN
@@
 $EndComp
 $Comp
-L +3V3 #PWR06
+L +3V3 #PWR?
 U 1 1 5B22F481
 P 5000 5350
-F 0 "#PWR06" H 5000 5200 50  0001 C CNN
+F 0 "#PWR?" H 5000 5200 50  0001 C CNN
 F 1 "+3V3" H 5000 5490 50  0000 C CNN
 F 2 "" H 5000 5350 50  0001 C CNN
@@
 $EndComp
 $Comp
-L R R1
+L R R?
 U 1 1 5B22F6F0
 P 5250 5350
-F 0 "R1" V 5330 5350 50  0000 C CNN
+F 0 "R?" V 5330 5350 50  0000 C CNN
 F 1 "20k" V 5250 5350 50  0000 C CNN
 F 2 "Resistors_SMD:R_0402" V 5180 5350 50  0001 C CNN
@@
 	5400 5350 5500 5350
 $Comp
-L R R13
+L R R?
 U 1 1 5B22FBB5
 P 8150 2600
-F 0 "R13" V 8230 2600 50  0000 C CNN
+F 0 "R?" V 8230 2600 50  0000 C CNN
 F 1 "20k" V 8150 2600 50  0000 C CNN
 F 2 "Resistors_SMD:R_0402" V 8080 2600 50  0001 C CNN
@@
 $EndComp
 $Comp
-L R R14
+L R R?
 U 1 1 5B22FC2F
 P 8350 2600
-F 0 "R14" V 8430 2600 50  0000 C CNN
+F 0 "R?" V 8430 2600 50  0000 C CNN
 F 1 "20k" V 8350 2600 50  0000 C CNN
 F 2 "Resistors_SMD:R_0402" V 8280 2600 50  0001 C CNN
@@
 Connection ~ 8150 2850
 $Comp
-L Micro_SD_Card_Det_Hirose_DM3AT J2
+L Micro_SD_Card_Det_Hirose_DM3AT J?
 U 1 1 5AD6D576
 P 1800 3850
-F 0 "J2" H 1150 4550 50  0000 C CNN
+F 0 "J?" H 1150 4550 50  0000 C CNN
 F 1 "Micro_SD_Card_Det_Hirose_DM3AT" H 2450 4550 50  0000 R CNN
 F 2 "" H 3850 4550 50  0001 C CNN
@@
 SDIO0_IO3
 $Comp
-L R_Small R121
+L R_Small R?
 U 1 1 5AD6FCC7
 P 2900 3850
-F 0 "R121" H 2930 3870 50  0000 L CNN
+F 0 "R?" H 2930 3870 50  0000 L CNN
 F 1 "43" H 2930 3810 50  0000 L CNN
 F 2 "Resistors_SMD:R_0402" H 2900 3850 50  0001 C CNN
@@
 $EndComp
 $Comp
-L GND #PWR07
+L GND #PWR?
 U 1 1 5AD704C9
 P 2800 3250
-F 0 "#PWR07" H 2800 3000 50  0001 C CNN
+F 0 "#PWR?" H 2800 3000 50  0001 C CNN
 F 1 "GND" H 2800 3100 50  0000 C CNN
 F 2 "" H 2800 3250 50  0000 C CNN
@@
 SDIO0_CD
 $Comp
-L R_Small R120
+L R_Small R?
 U 1 1 5AD70D49
 P 2900 3300
-F 0 "R120" H 2930 3320 50  0000 L CNN
+F 0 "R?" H 2930 3320 50  0000 L CNN
 F 1 "50k" H 2930 3260 50  0000 L CNN
 F 2 "Resistors_SMD:R_0402" H 2900 3300 50  0001 C CNN
@@
 Connection ~ 2900 3450
 $Comp
-L +3V3 #PWR08
+L +3V3 #PWR?
 U 1 1 5AD70E44
 P 2900 3100
-F 0 "#PWR08" H 2900 2950 50  0001 C CNN
+F 0 "#PWR?" H 2900 2950 50  0001 C CNN
 F 1 "+3V3" H 2900 3240 50  0000 C CNN
 F 2 "" H 2900 3100 50  0001 C CNN
@@
 Wire Wire Line
 	900  3350 1000 3350
+Text GLabel 5500 1750 0    60   Output ~ 0
+UART_TX
+Text GLabel 5500 1650 0    60   Input ~ 0
+UART_RX
 $EndSCHEMATC

Commit message: Finished USB Uart.
Also a few more fabrication Informations
Parts:
- added C?: 100 nF, Capacitors_SMD:C_0402, symbol C_Small
Connections:
- net labels added: PS_UART_RX, PS_UART_TX
- net labels removed: UART_RX, UART_TX
- wire segments 57 -> 61
Changed lines of the file:
@@
 LIBS:switches
 LIBS:ft234xd
+LIBS:sn74lv1t126
 LIBS:zynq_board-cache
 EELAYER 25 0
@@
 	900  3350 1000 3350
 Text GLabel 5500 1750 0    60   Output ~ 0
-UART_TX
+PS_UART_TX
 Text GLabel 5500 1650 0    60   Input ~ 0
-UART_RX
+PS_UART_RX
+Wire Wire Line
+	2700 3950 3400 3950
+$Comp
+L GND #PWR?
+U 1 1 5AD94FE0
+P 3400 3950
+F 0 "#PWR?" H 3400 3700 50  0001 C CNN
+F 1 "GND" H 3400 3800 50  0000 C CNN
+F 2 "" H 3400 3950 50  0000 C CNN
+F 3 "" H 3400 3950 50  0000 C CNN
+	1    3400 3950
+	0    -1   -1   0
+$EndComp
+Wire Wire Line
+	2700 3750 3400 3750
+$Comp
+L +3V3 #PWR?
+U 1 1 5AD950A4
+P 3400 3750
+F 0 "#PWR?" H 3400 3600 50  0001 C CNN
+F 1 "+3V3" H 3400 3890 50  0000 C CNN
+F 2 "" H 3400 3750 50  0001 C CNN
+F 3 "" H 3400 3750 50  0001 C CNN
+	1    3400 3750
+	0    1    1    0
+$EndComp
+$Comp
+L C_Small C?
+U 1 1 5AD950DB
+P 1850 2950
+F 0 "C?" H 1860 3020 50  0000 L CNN
+F 1 "100 nF" H 1860 2870 50  0000 L CNN
+F 2 "Capacitors_SMD:C_0402" H 1850 2950 50  0001 C CNN
+F 3 "" H 1850 2950 50  0001 C CNN
+F 4 "1" H 1850 2950 60  0001 C CNN "Populated"
+F 5 "SPEC" H 1850 2950 60  0001 C CNN "Source"
+	1    1850 2950
+	0    -1   -1   0
+$EndComp
+$Comp
+L GND #PWR?
+U 1 1 5AD95198
+P 1650 2950
+F 0 "#PWR?" H 1650 2700 50  0001 C CNN
+F 1 "GND" H 1650 2800 50  0000 C CNN
+F 2 "" H 1650 2950 50  0000 C CNN
+F 3 "" H 1650 2950 50  0000 C CNN
+	1    1650 2950
+	0    1    1    0
+$EndComp
+Wire Wire Line
+	1650 2950 1750 2950
+$Comp
+L +3V3 #PWR?
+U 1 1 5AD9524B
+P 2050 2950
+F 0 "#PWR?" H 2050 2800 50  0001 C CNN
+F 1 "+3V3" H 2050 3090 50  0000 C CNN
+F 2 "" H 2050 2950 50  0001 C CNN
+F 3 "" H 2050 2950 50  0001 C CNN
+	1    2050 2950
+	0    1    1    0
+$EndComp
+Wire Wire Line
+	2050 2950 1950 2950
 $EndSCHEMATC

Commit message: Added ESD Protection for microSD Card Slot.
Also added Fabrication Information to SD-Card Parts and a few Datasheets.
Parts:
- removed R?: 43, Resistors_SMD:R_0402, symbol R_Small
- removed R?: 50k, Resistors_SMD:R_0402, symbol R_Small
- added U?: EMIF06-MSD02N16, footprints:µQFN-16L, symbol EMIF06-MSD02N16
- J?: footprint (none) -> Connectors_Hirose:microSD_Card_Receptacle_Hirose_DM3AT-SF-PEJM5; Digikey (none) -> HR1964CT-ND; MFG Name (none) -> Hirose Electric Co Ltd; MFG Part Num (none) -> DM3AT-SF-PEJM5; Populated (none) -> 1; Source (none) -> SPEC
Connections:
- wire segments 61 -> 71
- no-connect marks 0 -> 1
Other:
- note added: "3,3 V!"
- note added: "ESD/EMI Protection and Filtering IC.\nAlso contains all needed series and\npull-up resistors."

Commit message: Added 2 kbit i2c eeprom connected to ps.
Parts:
- added C?: 100 nF, Capacitors_SMD:C_0402, symbol C_Small
- added R?: DNP, Resistors_SMD:R_0603, symbol R_Small
- added R? (x2): 4k7, Resistors_SMD:R_0603, symbol R_Small
- added U?: CAT24C02TDI-GT3, TO_SOT_Packages_SMD:SOT-23-5, symbol CAT24C02TDI-GT3
Connections:
- net labels added: SCL, SDA
- wire segments 71 -> 86
Changed lines of the file:
@@
 LIBS:sn74lv1t126
 LIBS:emif06-msd02n16
+LIBS:cat24c02tdi-gt3
 LIBS:zynq_board-cache
 EELAYER 25 0
@@
 Text Notes 3150 7750 0    60   ~ 0
 ESD/EMI Protection and Filtering IC.\nAlso contains all needed series and\npull-up resistors.
+$Comp
+L CAT24C02TDI-GT3 U?
+U 1 1 5ADF12BE
+P 2100 2300
+F 0 "U?" H 1850 2000 60  0000 C CNN
+F 1 "CAT24C02TDI-GT3" V 2300 2300 60  0000 C CNN
+F 2 "TO_SOT_Packages_SMD:SOT-23-5" H 2800 1450 60  0001 C CNN
+F 3 "http://www.onsemi.com/pub/Collateral/CAT24C01-D.PDF" H 2800 1450 60  0001 C CNN
+F 4 "ON Semiconductor" H 2100 2300 60  0001 C CNN "MFG Name"
+F 5 "CAT24C02TDI-GT3A" H 2100 2300 60  0001 C CNN "MFG Part Num"
+F 6 "CAT24C02TDI-GT3AOSCT-ND" H 2100 2300 60  0001 C CNN "Digikey"
+F 7 "1" H 2100 2300 60  0001 C CNN "Populated"
+F 8 "SPEC" H 2100 2300 60  0001 C CNN "Source"
+	1    2100 2300
+	1    0    0    -1
+$EndComp
+$Comp
+L C_Small C?
+U 1 1 5ADF17F1
+P 2700 2350
+F 0 "C?" H 2710 2420 50  0000 L CNN
+F 1 "100 nF" H 2710 2270 50  0000 L CNN
+F 2 "Capacitors_SMD:C_0402" H 2700 2350 50  0001 C CNN
+F 3 "" H 2700 2350 50  0001 C CNN
+F 4 "1" H 2700 2350 60  0001 C CNN "Populated"
+F 5 "SPEC" H 2700 2350 60  0001 C CNN "Source"
+	1    2700 2350
+	-1   0    0    1
+$EndComp
+$Comp
+L GND #PWR?
+U 1 1 5ADF17F7
+P 2700 2550
+F 0 "#PWR?" H 2700 2300 50  0001 C CNN
+F 1 "GND" H 2700 2400 50  0000 C CNN
+F 2 "" H 2700 2550 50  0000 C CNN
+F 3 "" H 2700 2550 50  0000 C CNN
+	1    2700 2550
+	1    0    0    -1
+$EndComp
+Wire Wire Line
+	2700 2550 2700 2450
+$Comp
+L +3V3 #PWR?
+U 1 1 5ADF17FE
+P 2700 2150
+F 0 "#PWR?" H 2700 2000 50  0001 C CNN
+F 1 "+3V3" H 2700 2290 50  0000 C CNN
+F 2 "" H 2700 2150 50  0001 C CNN
+F 3 "" H 2700 2150 50  0001 C CNN
+	1    2700 2150
+	1    0    0    -1
+$EndComp
+Wire Wire Line
+	2700 2150 2700 2250
+$Comp
+L R_Small R?
+U 1 1 5ADF2073
+P 1500 2000
+F 0 "R?" H 1530 2020 50  0000 L CNN
+F 1 "DNP" H 1530 1960 50  0000 L CNN
+F 2 "Resistors_SMD:R_0603" H 1500 2000 50  0001 C CNN
+F 3 "" H 1500 2000 50  0001 C CNN
+F 4 "0" H 1500 2000 60  0001 C CNN "Populated"
+F 5 "SPEC" H 1500 2000 60  0001 C CNN "Source"
+	1    1500 2000
+	1    0    0    -1
+$EndComp
+Wire Wire Line
+	1500 2100 1500 2200
+Wire Wire Line
+	1500 2200 1600 2200
+$Comp
+L +3V3 #PWR?
+U 1 1 5ADF21D6
+P 1500 1800
+F 0 "#PWR?" H 1500 1650 50  0001 C CNN
+F 1 "+3V3" H 1500 1940 50  0000 C CNN
+F 2 "" H 1500 1800 50  0001 C CNN
+F 3 "" H 1500 1800 50  0001 C CNN
+	1    1500 1800
+	1    0    0    -1
+$EndComp
+Wire Wire Line
+	1500 1800 1500 1900
+Text Label 1300 2300 0    60   ~ 0
+SCL
+Text Label 1300 2400 0    60   ~ 0
+SDA
+Wire Wire Line
+	1300 2300 1600 2300
+Wire Wire Line
+	1300 2400 1600 2400
+$Comp
+L GND #PWR?
+U 1 1 5ADF2AA7
+P 2100 2850
+F 0 "#PWR?" H 2100 2600 50  0001 C CNN
+F 1 "GND" H 2100 2700 50  0000 C CNN
+F 2 "" H 2100 2850 50  0000 C CNN
+F 3 "" H 2100 2850 50  0000 C CNN
+	1    2100 2850
+	1    0    0    -1
+$EndComp
+Wire Wire Line
+	2100 2850 2100 2750
+$Comp
+L +3V3 #PWR?
+U 1 1 5ADF2B75
+P 2100 1750
+F 0 "#PWR?" H 2100 1600 50  0001 C CNN
+F 1 "+3V3" H 2100 1890 50  0000 C CNN
+F 2 "" H 2100 1750 50  0001 C CNN
+F 3 "" H 2100 1750 50  0001 C CNN
+	1    2100 1750
+	1    0    0    -1
+$EndComp
+Wire Wire Line
+	2100 1750 2100 1850
+Text Label 5200 2050 0    60   ~ 0
+SCL
+Text Label 5200 2150 0    60   ~ 0
+SDA
+Wire Wire Line
+	4050 2050 5500 2050
+Wire Wire Line
+	3850 2150 5500 2150
+$Comp
+L R_Small R?
+U 1 1 5ADF492A
+P 3850 1850
+F 0 "R?" H 3880 1870 50  0000 L CNN
+F 1 "4k7" H 3880 1810 50  0000 L CNN
+F 2 "Resistors_SMD:R_0603" H 3850 1850 50  0001 C CNN
+F 3 "" H 3850 1850 50  0001 C CNN
+F 4 "1" H 3850 1850 60  0001 C CNN "Populated"
+F 5 "SPEC" H 3850 1850 60  0001 C CNN "Source"
+	1    3850 1850
+	1    0    0    -1
+$EndComp
+$Comp
+L +3V3 #PWR?
+U 1 1 5ADF4931
+P 3850 1650
+F 0 "#PWR?" H 3850 1500 50  0001 C CNN
+F 1 "+3V3" H 3850 1790 50  0000 C CNN
+F 2 "" H 3850 1650 50  0001 C CNN
+F 3 "" H 3850 1650 50  0001 C CNN
+	1    3850 1650
+	1    0    0    -1
+$EndComp
+Wire Wire Line
+	3850 1650 3850 1750
+$Comp
+L R_Small R?
+U 1 1 5ADF4A40
+P 4050 1850
+F 0 "R?" H 4080 1870 50  0000 L CNN
+F 1 "4k7" H 4080 1810 50  0000 L CNN
+F 2 "Resistors_SMD:R_0603" H 4050 1850 50  0001 C CNN
+F 3 "" H 4050 1850 50  0001 C CNN
+F 4 "1" H 4050 1850 60  0001 C CNN "Populated"
+F 5 "SPEC" H 4050 1850 60  0001 C CNN "Source"
+	1    4050 1850
+	1    0    0    -1
+$EndComp
+$Comp
+L +3V3 #PWR?
+U 1 1 5ADF4A46
+P 4050 1650
+F 0 "#PWR?" H 4050 1500 50  0001 C CNN
+F 1 "+3V3" H 4050 1790 50  0000 C CNN
+F 2 "" H 4050 1650 50  0001 C CNN
+F 3 "" H 4050 1650 50  0001 C CNN
+	1    4050 1650
+	1    0    0    -1
+$EndComp
+Wire Wire Line
+	4050 1650 4050 1750
+Wire Wire Line
+	4050 2050 4050 1950
+Wire Wire Line
+	3850 2150 3850 1950
 $EndSCHEMATC

Commit message: Connect MGT Supplies, POR_B, change reset button, add missing dcm files
Parts:
- removed R?: 20k, Resistors_SMD:R_0402, symbol R
Connections:
- net labels added: PS_POR_B
- wire segments 86 -> 107
Other:
- note added: "TODO: UART, I2C, Clock"
- note removed: "3,3 V!"
- note removed: "TODO: UART, I2C"
- note removed: "TODO: decide on MIO voltage"

Commit message: Added a first Version of footprints.
Some of them are made using the 'kicad footprint generator'-scripting libary. Source code of them is currently not in this repository.
Connections:
- wire segments 107 -> 89
Changed lines of the file:
@@
 LIBS:cat24c02tdi-gt3
 LIBS:power_symbols
-LIBS:zynq_board-cache
+LIBS:ti_power_modules
 EELAYER 25 0
 EELAYER END
@@
 	7950 1700 9200 1700
 Wire Wire Line
-	7950 1550 7950 1700
-Wire Wire Line
-	7950 1700 7950 2450
-Wire Wire Line
-	7750 1550 7750 1800
-Wire Wire Line
-	7750 1800 7750 2450
-Wire Wire Line
-	7550 1550 7550 1900
-Wire Wire Line
-	7550 1900 7550 2450
-Wire Wire Line
-	7350 1550 7350 2000
-Wire Wire Line
-	7350 2000 7350 2450
-Wire Wire Line
-	7150 1550 7150 2100
-Wire Wire Line
-	7150 2100 7150 2450
+	7950 1550 7950 2450
+Wire Wire Line
+	7750 1550 7750 2450
+Wire Wire Line
+	7550 1550 7550 2450
+Wire Wire Line
+	7350 1550 7350 2450
+Wire Wire Line
+	7150 1550 7150 2450
 Connection ~ 7950 1700
 Connection ~ 7750 1800
@@
 	7150 1250 7150 1150
 Wire Wire Line
-	7150 1150 7350 1150
-Wire Wire Line
-	7350 1150 7550 1150
-Wire Wire Line
-	7550 1150 7750 1150
-Wire Wire Line
-	7750 1150 7950 1150
+	7150 1150 7950 1150
 Wire Wire Line
 	7950 1150 7950 1250
@@
 Connection ~ 7350 1150
 Wire Wire Line
-	7550 1050 7550 1150
-Wire Wire Line
-	7550 1150 7550 1250
+	7550 1050 7550 1250
 Connection ~ 7550 1150
 Wire Wire Line
@@
 Connection ~ 7350 2850
 Wire Wire Line
-	7550 2750 7550 2850
-Wire Wire Line
-	7550 2850 7550 2950
+	7550 2750 7550 2950
 Connection ~ 7550 2850
 Wire Wire Line
@@
 	7150 2750 7150 2850
 Wire Wire Line
-	7150 2850 7350 2850
-Wire Wire Line
-	7350 2850 7550 2850
-Wire Wire Line
-	7550 2850 7750 2850
-Wire Wire Line
-	7750 2850 7950 2850
-Wire Wire Line
-	7950 2850 8150 2850
-Wire Wire Line
-	8150 2850 8350 2850
+	7150 2850 8350 2850
 Wire Wire Line
 	950  6250 1050 6250
@@
 	3050 7250 2950 7250
 Wire Wire Line
-	2950 7250 2950 7300
-Wire Wire Line
-	2950 7300 2950 7350
+	2950 7250 2950 7350
 Wire Wire Line
 	2950 7350 3050 7350
@@
 Connection ~ 10100 5550
 Wire Wire Line
-	10100 5450 10100 5550
-Wire Wire Line
-	10100 5550 10100 5650
+	10100 5450 10100 5650
 $Comp
 L C_Small C?
@@
 $EndComp
 Wire Wire Line
-	9400 5550 10100 5550
-Wire Wire Line
-	10100 5550 10200 5550
+	9400 5550 10200 5550
 Text Label 9400 5550 0    60   ~ 0
 PS_RESET
