File: hardware/zynq_ps.sch (KiCad schematic (older format))
At the start: 27 parts, among them J10 DM3CS, SW1 SW_Push, U1 xc7z030sbg485, U36 CAT24C02TDI-GT3, U37 EMIF06-MSD02N16, U38 33.333MHZ

Commit message: Added Power/Protection Circuit
Parts:
- renumbered C239 to C1801, C240 to C1802, C241 to C1803, C242 to C1804, J10 to J1801, R144 to R1801, R145 to R1802, R146 to R1803, R147 to R1804, R148 to R1805, R149 to R1806, R150 to R1807, R151 to R1808, R152 to R1809, R153 to R1810, R154 to R1811, R155 to R1812, R156 to R1813, R157 to R1814, R158 to R1815, R159 to R1816, R160 to R1817, SW1 to SW1801, U36 to U1801, U37 to U1802, U38 to U1803, U1 to U201
Changed lines of the file:
@@
 $EndDescr
 $Comp
-L xc7z030sbg485 U1
+L xc7z030sbg485 U201
 U 6 1 596E7E39
 P 9200 1400
-F 0 "U1" H 9400 1650 60  0000 L CNN
+F 0 "U201" H 9400 1650 60  0000 L CNN
 F 1 "xc7z030sbg485" H 9400 1550 60  0000 L CNN
 F 2 "footprints:SBG485_22x22_19.0x19.0mm_Pitch0.8mm" H 9200 1400 60  0001 C CNN
@@
 $EndComp
 $Comp
-L xc7z030sbg485 U1
+L xc7z030sbg485 U201
 U 7 1 596E7E6B
 P 5500 1450
-F 0 "U1" H 5700 1700 60  0000 L CNN
+F 0 "U201" H 5700 1700 60  0000 L CNN
 F 1 "xc7z030sbg485" H 5700 1600 60  0000 L CNN
 F 2 "footprints:SBG485_22x22_19.0x19.0mm_Pitch0.8mm" H 5500 1450 60  0001 C CNN
@@
 NOTE: The BootROM expects the SD card\nto be connected to MIO pins 40..45 (SDIO0).
 $Comp
-L R R155
+L R R1812
 U 1 1 5A98BDBC
 P 7950 1400
-F 0 "R155" V 8030 1400 50  0000 C CNN
+F 0 "R1812" V 8030 1400 50  0000 C CNN
 F 1 "DNP" V 7950 1400 50  0000 C CNN
 F 2 "Resistors_SMD:R_0402" V 7880 1400 50  0001 C CNN
@@
 $EndComp
 $Comp
-L R R153
+L R R1810
 U 1 1 5A98BDD7
 P 7750 1400
-F 0 "R153" V 7830 1400 50  0000 C CNN
+F 0 "R1810" V 7830 1400 50  0000 C CNN
 F 1 "DNP" V 7750 1400 50  0000 C CNN
 F 2 "Resistors_SMD:R_0402" V 7680 1400 50  0001 C CNN
@@
 $EndComp
 $Comp
-L R R151
+L R R1808
 U 1 1 5A98BDF4
 P 7550 1400
-F 0 "R151" V 7630 1400 50  0000 C CNN
+F 0 "R1808" V 7630 1400 50  0000 C CNN
 F 1 "20k" V 7550 1400 50  0000 C CNN
 F 2 "Resistors_SMD:R_0402" V 7480 1400 50  0001 C CNN
@@
 $EndComp
 $Comp
-L R R149
+L R R1806
 U 1 1 5A98BE13
 P 7350 1400
-F 0 "R149" V 7430 1400 50  0000 C CNN
+F 0 "R1806" V 7430 1400 50  0000 C CNN
 F 1 "20k" V 7350 1400 50  0000 C CNN
 F 2 "Resistors_SMD:R_0402" V 7280 1400 50  0001 C CNN
@@
 $EndComp
 $Comp
-L R R147
+L R R1804
 U 1 1 5A98BE34
 P 7150 1400
-F 0 "R147" V 7230 1400 50  0000 C CNN
+F 0 "R1804" V 7230 1400 50  0000 C CNN
 F 1 "DNP" V 7150 1400 50  0000 C CNN
 F 2 "Resistors_SMD:R_0402" V 7080 1400 50  0001 C CNN
@@
 $EndComp
 $Comp
-L R R148
+L R R1805
 U 1 1 5A98BE57
 P 7150 2600
-F 0 "R148" V 7230 2600 50  0000 C CNN
+F 0 "R1805" V 7230 2600 50  0000 C CNN
 F 1 "20k" V 7150 2600 50  0000 C CNN
 F 2 "Resistors_SMD:R_0402" V 7080 2600 50  0001 C CNN
@@
 $EndComp
 $Comp
-L R R150
+L R R1807
 U 1 1 5A98BE7C
 P 7350 2600
-F 0 "R150" V 7430 2600 50  0000 C CNN
+F 0 "R1807" V 7430 2600 50  0000 C CNN
 F 1 "DNP" V 7350 2600 50  0000 C CNN
 F 2 "Resistors_SMD:R_0402" V 7280 2600 50  0001 C CNN
@@
 $EndComp
 $Comp
-L R R152
+L R R1809
 U 1 1 5A98BEA3
 P 7550 2600
-F 0 "R152" V 7630 2600 50  0000 C CNN
+F 0 "R1809" V 7630 2600 50  0000 C CNN
 F 1 "DNP" V 7550 2600 50  0000 C CNN
 F 2 "Resistors_SMD:R_0402" V 7480 2600 50  0001 C CNN
@@
 $EndComp
 $Comp
-L R R154
+L R R1811
 U 1 1 5A98BECC
 P 7750 2600
-F 0 "R154" V 7830 2600 50  0000 C CNN
+F 0 "R1811" V 7830 2600 50  0000 C CNN
 F 1 "20k" V 7750 2600 50  0000 C CNN
 F 2 "Resistors_SMD:R_0402" V 7680 2600 50  0001 C CNN
@@
 $EndComp
 $Comp
-L R R156
+L R R1813
 U 1 1 5A98BEF7
 P 7950 2600
-F 0 "R156" V 8030 2600 50  0000 C CNN
+F 0 "R1813" V 8030 2600 50  0000 C CNN
 F 1 "20k" V 7950 2600 50  0000 C CNN
 F 2 "Resistors_SMD:R_0402" V 7880 2600 50  0001 C CNN
@@
 $EndComp
 $Comp
-L R R157
+L R R1814
 U 1 1 5B22FBB5
 P 8150 2600
-F 0 "R157" V 8230 2600 50  0000 C CNN
+F 0 "R1814" V 8230 2600 50  0000 C CNN
 F 1 "20k" V 8150 2600 50  0000 C CNN
 F 2 "Resistors_SMD:R_0402" V 8080 2600 50  0001 C CNN
@@
 $EndComp
 $Comp
-L R R158
+L R R1815
 U 1 1 5B22FC2F
 P 8350 2600
-F 0 "R158" V 8430 2600 50  0000 C CNN
+F 0 "R1815" V 8430 2600 50  0000 C CNN
 F 1 "20k" V 8350 2600 50  0000 C CNN
 F 2 "Resistors_SMD:R_0402" V 8280 2600 50  0001 C CNN
@@
 $EndComp
 $Comp
-L DM3CS J10
+L DM3CS J1801
 U 1 1 5AD6D576
 P 1850 6750
-F 0 "J10" H 1200 7450 50  0000 C CNN
+F 0 "J1801" H 1200 7450 50  0000 C CNN
 F 1 "DM3CS" H 2500 7450 50  0000 R CNN
 F 2 "footprints:DM3CS" H 3900 7450 50  0001 C CNN
@@
 PS_UART_RX
 $Comp
-L C_Small C239
+L C_Small C1801
 U 1 1 5AD950DB
 P 1900 5850
-F 0 "C239" H 1910 5920 50  0000 L CNN
+F 0 "C1801" H 1910 5920 50  0000 L CNN
 F 1 "100 nF" H 1910 5770 50  0000 L CNN
 F 2 "Capacitors_SMD:C_0402" H 1900 5850 50  0001 C CNN
@@
 $EndComp
 $Comp
-L EMIF06-MSD02N16 U37
+L EMIF06-MSD02N16 U1802
 U 1 1 5ADAA7F4
 P 3750 6750
-F 0 "U37" H 3700 6050 60  0000 C CNN
+F 0 "U1802" H 3700 6050 60  0000 C CNN
 F 1 "EMIF06-MSD02N16" V 3750 6800 60  0000 C CNN
 F 2 "footprints:µQFN-16L" H 3400 5800 60  0001 C CNN
@@
 ESD/EMI Protection and Filtering IC.\nAlso contains all needed series and\npull-up resistors.
 $Comp
-L CAT24C02TDI-GT3 U36
+L CAT24C02TDI-GT3 U1801
 U 1 1 5ADF12BE
 P 2100 2300
-F 0 "U36" H 1850 2000 60  0000 C CNN
+F 0 "U1801" H 1850 2000 60  0000 C CNN
 F 1 "CAT24C02TDI-GT3" V 2300 2300 60  0000 C CNN
 F 2 "TO_SOT_Packages_SMD:SOT-23-5" H 2800 1450 60  0001 C CNN
@@
 $EndComp
 $Comp
-L C_Small C240
+L C_Small C1802
 U 1 1 5ADF17F1
 P 2700 2350
-F 0 "C240" H 2710 2420 50  0000 L CNN
+F 0 "C1802" H 2710 2420 50  0000 L CNN
 F 1 "100 nF" H 2710 2270 50  0000 L CNN
 F 2 "Capacitors_SMD:C_0402" H 2700 2350 50  0001 C CNN
@@
 $EndComp
 $Comp
-L R_Small R144
+L R_Small R1801
 U 1 1 5ADF2073
 P 1500 2000
-F 0 "R144" H 1530 2020 50  0000 L CNN
+F 0 "R1801" H 1530 2020 50  0000 L CNN
 F 1 "DNP" H 1530 1960 50  0000 L CNN
 F 2 "Resistors_SMD:R_0603" H 1500 2000 50  0001 C CNN
@@
 SDA
 $Comp
-L R_Small R145
+L R_Small R1802
 U 1 1 5ADF492A
 P 3850 1850
-F 0 "R145" H 3880 1870 50  0000 L CNN
+F 0 "R1802" H 3880 1870 50  0000 L CNN
 F 1 "4k7" H 3880 1810 50  0000 L CNN
 F 2 "Resistors_SMD:R_0603" H 3850 1850 50  0001 C CNN
@@
 $EndComp
 $Comp
-L R_Small R146
+L R_Small R1803
 U 1 1 5ADF4A40
 P 4050 1850
-F 0 "R146" H 4080 1870 50  0000 L CNN
+F 0 "R1803" H 4080 1870 50  0000 L CNN
 F 1 "4k7" H 4080 1810 50  0000 L CNN
 F 2 "Resistors_SMD:R_0603" H 4050 1850 50  0001 C CNN
@@
 	10100 5150 10100 5250
 $Comp
-L R_Small R160
+L R_Small R1817
 U 1 1 5B1EF27E
 P 10100 5350
-F 0 "R160" H 10130 5370 50  0000 L CNN
+F 0 "R1817" H 10130 5370 50  0000 L CNN
 F 1 "10k" H 10130 5310 50  0000 L CNN
 F 2 "" H 10100 5350 50  0001 C CNN
@@
 	10100 5450 10100 5650
 $Comp
-L C_Small C242
+L C_Small C1804
 U 1 1 5B1EDFD0
 P 10100 5750
-F 0 "C242" H 10110 5820 50  0000 L CNN
+F 0 "C1804" H 10110 5820 50  0000 L CNN
 F 1 "100 nF" H 10110 5670 50  0000 L CNN
 F 2 "" H 10100 5750 50  0001 C CNN
@@
 	10600 5550 10700 5550
 $Comp
-L SW_Push SW1
+L SW_Push SW1801
 U 1 1 5B1ED103
 P 10400 5550
-F 0 "SW1" H 10450 5650 50  0000 L CNN
+F 0 "SW1801" H 10450 5650 50  0000 L CNN
 F 1 "SW_Push" H 10400 5490 50  0000 C CNN
 F 2 "" H 10400 5750 50  0001 C CNN
@@
 	8900 3200 9200 3200
 $Comp
-L OSC U38
+L OSC U1803
 U 1 1 5B025E58
 P 7950 5450
-F 0 "U38" H 7950 5400 60  0000 C CNN
+F 0 "U1803" H 7950 5400 60  0000 C CNN
 F 1 "33.333MHZ" H 7950 5500 60  0000 C CNN
 F 2 "footprints:ASDMB_2.5x2.0mm_1.65mm_pitch" H 7950 5450 60  0001 C CNN
@@
 Connection ~ 8550 5350
 $Comp
-L C_Small C241
+L C_Small C1803
 U 1 1 5B026A7D
 P 7150 5450
-F 0 "C241" H 7160 5520 50  0000 L CNN
+F 0 "C1803" H 7160 5520 50  0000 L CNN
 F 1 "100 nF" H 7160 5370 50  0000 L CNN
 F 2 "Capacitors_SMD:C_0402" H 7150 5450 50  0001 C CNN
@@
 	8700 1400 9200 1400
 $Comp
-L R_Small R159
+L R_Small R1816
 U 1 1 5B047F57
 P 8650 5550
-F 0 "R159" H 8680 5570 50  0000 L CNN
+F 0 "R1816" H 8680 5570 50  0000 L CNN
 F 1 "40,2" V 8650 5550 31  0000 C CNN
 F 2 "Resistors_SMD:R_0402" H 8650 5550 50  0001 C CNN

Commit message: Length matched DDR3 Memory again.
Forgot to keep enough space between the traces and between the meander waves.

Also, I switched to Kicad 5.0 RC2.

Swaped a few ddr signals.
Parts:
- C1801, C1802, C1803, C1804: symbol C_Small -> device:C_Small
- J1801: symbol DM3CS -> dm3cs:DM3CS
- R1801, R1802, R1803, R1816, R1817: symbol R_Small -> device:R_Small
- R1804, R1805, R1806, R1807, R1808, R1809, R1810, R1811, R1812, R1813, R1814, R1815: symbol R -> device:R
- SW1801: symbol SW_Push -> switches:SW_Push
- U1801: symbol CAT24C02TDI-GT3 -> cat24c02tdi-gt3:CAT24C02TDI-GT3
- U1802: symbol EMIF06-MSD02N16 -> emif06-msd02n16:EMIF06-MSD02N16
- U1803: symbol OSC -> osc:OSC
- U201: symbol xc7z030sbg485 -> xilinx_zynq_clg485:xc7z030sbg485
Changed lines of the file:
@@
-EESchema Schematic File Version 2
-LIBS:zynq_board-rescue
-LIBS:power
-LIBS:device
-LIBS:transistors
-LIBS:conn
-LIBS:linear
-LIBS:regul
-LIBS:74xx
-LIBS:cmos4000
-LIBS:adc-dac
-LIBS:memory
-LIBS:xilinx
-LIBS:microcontrollers
-LIBS:dsp
-LIBS:microchip
-LIBS:analog_switches
-LIBS:motorola
-LIBS:texas
-LIBS:intel
-LIBS:audio
-LIBS:interface
-LIBS:digital-audio
-LIBS:philips
-LIBS:display
-LIBS:cypress
-LIBS:siliconi
-LIBS:opto
-LIBS:atmel
-LIBS:contrib
-LIBS:valves
-LIBS:xilinx_zynq_clg485
-LIBS:SFP_plus
-LIBS:ael2005
-LIBS:diff_osc
-LIBS:si53340
-LIBS:usb3320
-LIBS:nx5p3090
-LIBS:smp1255putg
-LIBS:osc
-LIBS:ddr
-LIBS:misc
-LIBS:tlk10031
-LIBS:lshm-150-xxx-x-dv-a-s
-LIBS:sn74axc8t245
-LIBS:sn74lvc2t45
-LIBS:dmf05lcflp
-LIBS:bss138ps
-LIBS:max14854
-LIBS:switches
-LIBS:ft234xd
-LIBS:sn74lv1t126
-LIBS:emif06-msd02n16
-LIBS:cat24c02tdi-gt3
-LIBS:power_symbols
-LIBS:ti_power_modules
-LIBS:mdr20
-LIBS:dm3cs
-LIBS:lsf0102
-LIBS:dmp3056l
+EESchema Schematic File Version 4
 LIBS:zynq_board-cache
-EELAYER 25 0
+EELAYER 26 0
 EELAYER END
 $Descr A4 11693 8268
@@
 $EndDescr
 $Comp
-L xc7z030sbg485 U201
+L xilinx_zynq_clg485:xc7z030sbg485 U201
 U 6 1 596E7E39
 P 9200 1400
@@
 $EndComp
 $Comp
-L xc7z030sbg485 U201
+L xilinx_zynq_clg485:xc7z030sbg485 U201
 U 7 1 596E7E6B
 P 5500 1450
@@
 NOTE: The BootROM expects the SD card\nto be connected to MIO pins 40..45 (SDIO0).
 $Comp
-L R R1812
+L device:R R1812
 U 1 1 5A98BDBC
 P 7950 1400
@@
 $EndComp
 $Comp
-L R R1810
+L device:R R1810
 U 1 1 5A98BDD7
 P 7750 1400
@@
 $EndComp
 $Comp
-L R R1808
+L device:R R1808
 U 1 1 5A98BDF4
 P 7550 1400
@@
 $EndComp
 $Comp
-L R R1806
+L device:R R1806
 U 1 1 5A98BE13
 P 7350 1400
@@
 $EndComp
 $Comp
-L R R1804
+L device:R R1804
 U 1 1 5A98BE34
 P 7150 1400
@@
 $EndComp
 $Comp
-L R R1805
+L device:R R1805
 U 1 1 5A98BE57
 P 7150 2600
@@
 $EndComp
 $Comp
-L R R1807
+L device:R R1807
 U 1 1 5A98BE7C
 P 7350 2600
@@
 $EndComp
 $Comp
-L R R1809
+L device:R R1809
 U 1 1 5A98BEA3
 P 7550 2600
@@
 $EndComp
 $Comp
-L R R1811
+L device:R R1811
 U 1 1 5A98BECC
 P 7750 2600
@@
 $EndComp
 $Comp
-L R R1813
+L device:R R1813
 U 1 1 5A98BEF7
 P 7950 2600
@@
 $EndComp
 $Comp
-L GND #PWR0225
+L power1:GND #PWR0225
 U 1 1 5A991630
 P 7550 2950
@@
 NOTE: pulls must be 20k.
 $Comp
-L +3V3 #PWR0226
+L power1:+3V3 #PWR0226
 U 1 1 5B22F273
 P 7550 1050
@@
 $EndComp
 $Comp
-L R R1814
+L device:R R1814
 U 1 1 5B22FBB5
 P 8150 2600
@@
 $EndComp
 $Comp
-L R R1815
+L device:R R1815
 U 1 1 5B22FC2F
 P 8350 2600
@@
 $EndComp
 $Comp
-L DM3CS J1801
+L dm3cs:DM3CS J1801
 U 1 1 5AD6D576
 P 1850 6750
@@
 SDIO0_CD
 $Comp
-L +3V3 #PWR0227
+L power1:+3V3 #PWR0227
 U 1 1 5AD70E44
 P 2900 6850
@@
 $EndComp
 $Comp
-L GND #PWR0228
+L power1:GND #PWR0228
 U 1 1 5AD853F0
 P 950 6250
@@
 PS_UART_RX
 $Comp
-L C_Small C1801
+L device:C_Small C1801
 U 1 1 5AD950DB
 P 1900 5850
@@
 $EndComp
 $Comp
-L GND #PWR0229
+L power1:GND #PWR0229
 U 1 1 5AD95198
 P 1700 5850
@@
 $EndComp
 $Comp
-L +3V3 #PWR0230
+L power1:+3V3 #PWR0230
 U 1 1 5AD9524B
 P 2100 5850
@@
 $EndComp
 $Comp
-L EMIF06-MSD02N16 U1802
+L emif06-msd02n16:EMIF06-MSD02N16 U1802
 U 1 1 5ADAA7F4
 P 3750 6750
@@
 $EndComp
 $Comp
-L +3V3 #PWR0231
+L power1:+3V3 #PWR0231
 U 1 1 5ADAB627
 P 2850 7300
@@
 $EndComp
 $Comp
-L GND #PWR0232
+L power1:GND #PWR0232
 U 1 1 5ADAB6E8
 P 4600 6150
@@
 NoConn ~ 4500 7250
 $Comp
-L GND #PWR0233
+L power1:GND #PWR0233
 U 1 1 5ADABBC7
 P 2900 6650
@@
 ESD/EMI Protection and Filtering IC.\nAlso contains all needed series and\npull-up resistors.
 $Comp
-L CAT24C02TDI-GT3 U1801
+L cat24c02tdi-gt3:CAT24C02TDI-GT3 U1801
 U 1 1 5ADF12BE
 P 2100 2300
@@
 $EndComp
 $Comp
-L C_Small C1802
+L device:C_Small C1802
 U 1 1 5ADF17F1
 P 2700 2350
@@
 $EndComp
 $Comp
-L GND #PWR0234
+L power1:GND #PWR0234
 U 1 1 5ADF17F7
 P 2700 2550
@@
 $EndComp
 $Comp
-L +3V3 #PWR0235
+L power1:+3V3 #PWR0235
 U 1 1 5ADF17FE
 P 2700 2150
@@
 $EndComp
 $Comp
-L R_Small R1801
+L device:R_Small R1801
 U 1 1 5ADF2073
 P 1500 2000
@@
 $EndComp
 $Comp
-L +3V3 #PWR0236
+L power1:+3V3 #PWR0236
 U 1 1 5ADF21D6
 P 1500 1750
@@
 SDA
 $Comp
-L GND #PWR0237
+L power1:GND #PWR0237
 U 1 1 5ADF2AA7
 P 2100 2850
@@
 $EndComp
 $Comp
-L +3V3 #PWR0238
+L power1:+3V3 #PWR0238
 U 1 1 5ADF2B75
 P 2100 1750
@@
 SDA
 $Comp
-L R_Small R1802
+L device:R_Small R1802
 U 1 1 5ADF492A
 P 3850 1850
@@
 $EndComp
 $Comp
-L +3V3 #PWR0239
+L power1:+3V3 #PWR0239
 U 1 1 5ADF4931
 P 3850 1650
@@
 $EndComp
 $Comp
-L R_Small R1803
+L device:R_Small R1803
 U 1 1 5ADF4A40
 P 4050 1850
@@
 $EndComp
 $Comp
-L +3V3 #PWR0240
+L power1:+3V3 #PWR0240
 U 1 1 5ADF4A46
 P 4050 1650
@@
 	3850 2150 3850 1950
 $Comp
-L +3V3 #PWR0241
+L power1:+3V3 #PWR0241
 U 1 1 5B22F1F8
 P 10100 5150
@@
 	10100 5150 10100 5250
 $Comp
-L R_Small R1817
+L device:R_Small R1817
 U 1 1 5B1EF27E
 P 10100 5350
@@
 	10100 5950 10100 5850
 $Comp
-L GND #PWR0242
+L power1:GND #PWR0242
 U 1 1 5B1EE083
 P 10100 5950
@@
 	10100 5450 10100 5650
 $Comp
-L C_Small C1804
+L device:C_Small C1804
 U 1 1 5B1EDFD0
 P 10100 5750
@@
 PS_RESET
 $Comp
-L GND #PWR0243
+L power1:GND #PWR0243
 U 1 1 5B1ED412
 P 10700 5650
@@
 	10600 5550 10700 5550
 $Comp
-L SW_Push SW1801
+L switches:SW_Push SW1801
 U 1 1 5B1ED103
 P 10400 5550
@@
 	8900 3200 9200 3200
 $Comp
-L OSC U1803
+L osc:OSC U1803
 U 1 1 5B025E58
 P 7950 5450
@@
 $EndComp
 $Comp
-L GND #PWR0244
+L power1:GND #PWR0244
 U 1 1 5B02614D
 P 7350 5650
@@
 	7150 5550 7450 5550
 $Comp
-L +3V3 #PWR0245
+L power1:+3V3 #PWR0245
 U 1 1 5B02628C
 P 8650 5250
@@
 Connection ~ 8550 5350
 $Comp
-L C_Small C1803
+L device:C_Small C1803
 U 1 1 5B026A7D
 P 7150 5450
@@
 	8700 1400 9200 1400
 $Comp
-L R_Small R1816
+L device:R_Small R1816
 U 1 1 5B047F57
 P 8650 5550

Commit message: Layouted most of the Power Circuit and Triggerbus Levelshifters.
Added Footprint for Tantal Caps. Modified Footprint for MDR20 Connector, SD-Card.

Fixed Symbol and Circuit for Power Supervisor/Delay IC.

Also fixed some smaller things in the schematics.
Parts:
- removed R1817: 10k, symbol device:R_Small
- added C1805: 100 nF, Capacitors_SMD:C_0201, symbol device:C_Small
- added R1817: 3M, Resistor_SMD:R_0402_1005Metric, symbol device:R
- added R1818: 560k, Resistor_SMD:R_0402_1005Metric, symbol device:R
- added R1819: 100k, Resistor_SMD:R_0402_1005Metric, symbol device:R
- added U1804: TPS3808G01, Package_DFN_QFN:Texas_S-PWSON-N6, symbol ti_power_modules:TPS3808
- C1804: value 100 nF -> 1nF; footprint (none) -> Capacitor_SMD:C_0402_1005Metric; Description (none) -> CAP CER 1000PF 6.3V X5R 0402; Digikey (none) -> 490-6285-1-ND; MFG Name (none) -> Murata Electronics North America; MFG Part Num (none) -> GRM155R60J102KA01D; Populate for CLG484(Z-7012s/Z-7015) (none) -> 1; Populate for SBGA485(Z-7030) (none) -> 1; Populated (none) -> 1; Source (none) -> SPEC; Voltage (none) -> 6,3 V
- SW1801: footprint (none) -> Button_Switch_SMD:SW_SPST_PTS645; Description (none) -> SWITCH TACTILE SPST-NO 0.05A 12V; Digikey (none) -> CKN9087CT-ND; MFG Name (none) -> C&K; MFG Part Num (none) -> PTS645SK50SMTR92 LFS; Populate for CLG484(Z-7012s/Z-7015) (none) -> 1; Populate for SBGA485(Z-7030) (none) -> 1; Populated (none) -> 1; Source (none) -> SPEC
Connections:
- net labels added: 3,3V
- wire segments 98 -> 143
Other:
- note added: "500ms ~RESET~ Delay"
- note added: "R1+R2 ~~ 4MΩ\n"
- note added: "Sense Threshold 2,7 V\n(Monitor POR)"
- note added: "V_ref = 0.4V"
- note removed: "Reset Button"
- moved on the sheet: U1803

Commit message: Layouted USB-UART.
Also moved USB-OTG to the right Side of the Board. To get there
some free Space, i moved the DDR3/Memory and the FPGA a few
Millimeters down.
Parts:
- R1804, R1805, R1806, R1807, R1808, R1809, R1810, R1811, R1812, R1813, R1814, R1815, R1816: footprint Resistors_SMD:R_0402 -> Resistor_SMD:R_0402_1005Metric
Changed lines of the file:
@@
 F 0 "R1812" V 8030 1400 50  0000 C CNN
 F 1 "DNP" V 7950 1400 50  0000 C CNN
-F 2 "Resistors_SMD:R_0402" V 7880 1400 50  0001 C CNN
+F 2 "Resistor_SMD:R_0402_1005Metric" V 7880 1400 50  0001 C CNN
 F 3 "" H 7950 1400 50  0000 C CNN
 	1    7950 1400
@@
 F 0 "R1810" V 7830 1400 50  0000 C CNN
 F 1 "DNP" V 7750 1400 50  0000 C CNN
-F 2 "Resistors_SMD:R_0402" V 7680 1400 50  0001 C CNN
+F 2 "Resistor_SMD:R_0402_1005Metric" V 7680 1400 50  0001 C CNN
 F 3 "" H 7750 1400 50  0000 C CNN
 	1    7750 1400
@@
 F 0 "R1808" V 7630 1400 50  0000 C CNN
 F 1 "20k" V 7550 1400 50  0000 C CNN
-F 2 "Resistors_SMD:R_0402" V 7480 1400 50  0001 C CNN
+F 2 "Resistor_SMD:R_0402_1005Metric" V 7480 1400 50  0001 C CNN
 F 3 "" H 7550 1400 50  0000 C CNN
 	1    7550 1400
@@
 F 0 "R1806" V 7430 1400 50  0000 C CNN
 F 1 "20k" V 7350 1400 50  0000 C CNN
-F 2 "Resistors_SMD:R_0402" V 7280 1400 50  0001 C CNN
+F 2 "Resistor_SMD:R_0402_1005Metric" V 7280 1400 50  0001 C CNN
 F 3 "" H 7350 1400 50  0000 C CNN
 	1    7350 1400
@@
 F 0 "R1804" V 7230 1400 50  0000 C CNN
 F 1 "DNP" V 7150 1400 50  0000 C CNN
-F 2 "Resistors_SMD:R_0402" V 7080 1400 50  0001 C CNN
+F 2 "Resistor_SMD:R_0402_1005Metric" V 7080 1400 50  0001 C CNN
 F 3 "" H 7150 1400 50  0000 C CNN
 	1    7150 1400
@@
 F 0 "R1805" V 7230 2600 50  0000 C CNN
 F 1 "20k" V 7150 2600 50  0000 C CNN
-F 2 "Resistors_SMD:R_0402" V 7080 2600 50  0001 C CNN
+F 2 "Resistor_SMD:R_0402_1005Metric" V 7080 2600 50  0001 C CNN
 F 3 "" H 7150 2600 50  0000 C CNN
 	1    7150 2600
@@
 F 0 "R1807" V 7430 2600 50  0000 C CNN
 F 1 "DNP" V 7350 2600 50  0000 C CNN
-F 2 "Resistors_SMD:R_0402" V 7280 2600 50  0001 C CNN
+F 2 "Resistor_SMD:R_0402_1005Metric" V 7280 2600 50  0001 C CNN
 F 3 "" H 7350 2600 50  0000 C CNN
 	1    7350 2600
@@
 F 0 "R1809" V 7630 2600 50  0000 C CNN
 F 1 "DNP" V 7550 2600 50  0000 C CNN
-F 2 "Resistors_SMD:R_0402" V 7480 2600 50  0001 C CNN
+F 2 "Resistor_SMD:R_0402_1005Metric" V 7480 2600 50  0001 C CNN
 F 3 "" H 7550 2600 50  0000 C CNN
 	1    7550 2600
@@
 F 0 "R1811" V 7830 2600 50  0000 C CNN
 F 1 "20k" V 7750 2600 50  0000 C CNN
-F 2 "Resistors_SMD:R_0402" V 7680 2600 50  0001 C CNN
+F 2 "Resistor_SMD:R_0402_1005Metric" V 7680 2600 50  0001 C CNN
 F 3 "" H 7750 2600 50  0000 C CNN
 	1    7750 2600
@@
 F 0 "R1813" V 8030 2600 50  0000 C CNN
 F 1 "20k" V 7950 2600 50  0000 C CNN
-F 2 "Resistors_SMD:R_0402" V 7880 2600 50  0001 C CNN
+F 2 "Resistor_SMD:R_0402_1005Metric" V 7880 2600 50  0001 C CNN
 F 3 "" H 7950 2600 50  0000 C CNN
 	1    7950 2600
@@
 F 0 "R1814" V 8230 2600 50  0000 C CNN
 F 1 "20k" V 8150 2600 50  0000 C CNN
-F 2 "Resistors_SMD:R_0402" V 8080 2600 50  0001 C CNN
+F 2 "Resistor_SMD:R_0402_1005Metric" V 8080 2600 50  0001 C CNN
 F 3 "" H 8150 2600 50  0000 C CNN
 	1    8150 2600
@@
 F 0 "R1815" V 8430 2600 50  0000 C CNN
 F 1 "20k" V 8350 2600 50  0000 C CNN
-F 2 "Resistors_SMD:R_0402" V 8280 2600 50  0001 C CNN
+F 2 "Resistor_SMD:R_0402_1005Metric" V 8280 2600 50  0001 C CNN
 F 3 "" H 8350 2600 50  0000 C CNN
 	1    8350 2600
@@
 F 0 "R1816" H 2880 4970 50  0000 L CNN
 F 1 "40,2" V 2850 4950 31  0000 C CNN
-F 2 "Resistors_SMD:R_0402" H 2850 4950 50  0001 C CNN
+F 2 "Resistor_SMD:R_0402_1005Metric" H 2850 4950 50  0001 C CNN
 F 3 "" H 2850 4950 50  0001 C CNN
 F 4 "1" H 2850 4950 60  0001 C CNN "Populated"
