File: hardware/zynq_ps.sch (KiCad schematic (older format))
At the start: 31 parts, among them J1801 DM3CS, SW1801 SW_Push, U1801 CAT24C02TDI-GT3, U1802 EMIF06-MSD02N16, U1803 33.333MHZ, U1804 TPS3808G01, U201 xc7z030sbg485

Commit message: Improved Powerdistribution Network of the FPGA.
Also started to layout USB.
Parts:
- removed C1804: 1nF, Capacitor_SMD:C_0402_1005Metric, symbol device:C_Small
- removed C1805: 100 nF, Capacitors_SMD:C_0201, symbol device:C_Small
- removed R1817: 3M, Resistor_SMD:R_0402_1005Metric, symbol device:R
- removed R1818: 560k, Resistor_SMD:R_0402_1005Metric, symbol device:R
- removed U1804: TPS3808G01, Package_DFN_QFN:Texas_S-PWSON-N6, symbol ti_power_modules:TPS3808
- C1801, C1802, C1803: footprint Capacitors_SMD:C_0402 -> Capacitor_SMD:C_0402_1005Metric
- R1819: value 100k -> 10k
Connections:
- net labels removed: 3,3V
- wire segments 143 -> 116
Other:
- note removed: "500ms ~RESET~ Delay"
- note removed: "R1+R2 ~~ 4MΩ\n"
- note removed: "Sense Threshold 2,7 V\n(Monitor POR)"
- note removed: "V_ref = 0.4V"
Changed lines of the file:
@@
 F 0 "C1801" H 1910 5920 50  0000 L CNN
 F 1 "100 nF" H 1910 5770 50  0000 L CNN
-F 2 "Capacitors_SMD:C_0402" H 1900 5850 50  0001 C CNN
+F 2 "Capacitor_SMD:C_0402_1005Metric" H 1900 5850 50  0001 C CNN
 F 3 "" H 1900 5850 50  0001 C CNN
 F 4 "1" H 1900 5850 60  0001 C CNN "Populated"
@@
 F 0 "C1802" H 2710 2420 50  0000 L CNN
 F 1 "100 nF" H 2710 2270 50  0000 L CNN
-F 2 "Capacitors_SMD:C_0402" H 2700 2350 50  0001 C CNN
+F 2 "Capacitor_SMD:C_0402_1005Metric" H 2700 2350 50  0001 C CNN
 F 3 "" H 2700 2350 50  0001 C CNN
 F 4 "1" H 2700 2350 60  0001 C CNN "Populated"
@@
 F 0 "C1803" H 1360 4920 50  0000 L CNN
 F 1 "100 nF" H 1360 4770 50  0000 L CNN
-F 2 "Capacitors_SMD:C_0402" H 1350 4850 50  0001 C CNN
+F 2 "Capacitor_SMD:C_0402_1005Metric" H 1350 4850 50  0001 C CNN
 F 3 "" H 1350 4850 50  0001 C CNN
 F 4 "1" H 1350 4850 60  0001 C CNN "Populated"
@@
 Wire Wire Line
 	1550 4950 1650 4950
-$Comp
-L device:R R1817
-U 1 1 5B36AFCF
-P 7850 5150
-F 0 "R1817" V 7930 5150 50  0000 C CNN
-F 1 "3M" V 7850 5150 50  0000 C CNN
-F 2 "Resistor_SMD:R_0402_1005Metric" V 7780 5150 50  0001 C CNN
-F 3 "" H 7850 5150 50  0001 C CNN
-F 4 "1" H 7850 5150 60  0001 C CNN "Populated"
-F 5 "SPEC" H 7850 5150 60  0001 C CNN "Source"
-F 6 "1" H 7850 5150 50  0001 C CNN "Populate for SBGA485(Z-7030)"
-F 7 "1" H 7850 5150 50  0001 C CNN "Populate for CLG484(Z-7012s/Z-7015)"
-	1    7850 5150
-	1    0    0    -1
-$EndComp
-$Comp
-L device:R R1818
-U 1 1 5B36AFDA
-P 7850 5650
-F 0 "R1818" V 7930 5650 50  0000 C CNN
-F 1 "560k" V 7850 5650 50  0000 C CNN
-F 2 "Resistor_SMD:R_0402_1005Metric" V 7780 5650 50  0001 C CNN
-F 3 "" H 7850 5650 50  0001 C CNN
-F 4 "1" H 7850 5650 60  0001 C CNN "Populated"
-F 5 "SPEC" H 7850 5650 60  0001 C CNN "Source"
-F 6 "1" H 7850 5650 50  0001 C CNN "Populate for SBGA485(Z-7030)"
-F 7 "1" H 7850 5650 50  0001 C CNN "Populate for CLG484(Z-7012s/Z-7015)"
-	1    7850 5650
-	1    0    0    -1
-$EndComp
-$Comp
-L device:C_Small C1804
-U 1 1 5B36AFEA
-P 7650 5650
-F 0 "C1804" H 7660 5720 50  0000 L CNN
-F 1 "1nF" H 7660 5570 50  0000 L CNN
-F 2 "Capacitor_SMD:C_0402_1005Metric" H 7650 5650 50  0001 C CNN
-F 3 "http://search.murata.co.jp/Ceramy/image/img/A01X/G101/ENG/GRM155R60J102KA01-01.pdf" H 7650 5650 50  0001 C CNN
-F 4 "Murata Electronics North America" H 7650 5650 50  0001 C CNN "MFG Name"
-F 5 "GRM155R60J102KA01D" H 7650 5650 50  0001 C CNN "MFG Part Num"
-F 6 "490-6285-1-ND" H 7650 5650 50  0001 C CNN "Digikey"
-F 7 "1" H 7650 5650 50  0001 C CNN "Populated"
-F 8 "CAP CER 1000PF 6.3V X5R 0402 " H 7650 5650 50  0001 C CNN "Description"
-F 9 "SPEC" H 7650 5650 50  0001 C CNN "Source"
-F 10 "1" H 7650 5650 50  0001 C CNN "Populate for SBGA485(Z-7030)"
-F 11 "1" H 7650 5650 50  0001 C CNN "Populate for CLG484(Z-7012s/Z-7015)"
-F 12 "6,3 V" H 7750 5500 50  0000 C CNN "Voltage"
-	1    7650 5650
-	-1   0    0    -1
-$EndComp
-Text Notes 7100 5250 0    60   ~ 0
-R1+R2 ~~ 4MΩ\n
-Text Notes 7100 5350 0    60   ~ 0
-V_ref = 0.4V
-Text Notes 7100 5000 0    60   ~ 0
-Sense Threshold 2,7 V\n(Monitor POR)
-Text Label 7050 4900 0    60   ~ 0
-3,3V
-$Comp
-L ti_power_modules:TPS3808 U1804
-U 1 1 5B36AFFD
-P 8850 5400
-F 0 "U1804" H 8550 5700 60  0000 C CNN
-F 1 "TPS3808G01" H 8850 5200 60  0000 C CNN
-F 2 "Package_DFN_QFN:Texas_S-PWSON-N6" H 8550 5450 60  0001 C CNN
-F 3 "http://www.ti.com/lit/ds/symlink/tps3808.pdf" H 8550 5450 60  0001 C CNN
-F 4 "Texas Instruments" H 8850 5400 60  0001 C CNN "MFG Name"
-F 5 "TPS3808G01" H 8850 5400 60  0001 C CNN "MFG Part Num"
-F 6 "296-23656-1-ND" H 8850 5400 60  0001 C CNN "Digikey"
-F 7 "1" H 8850 5400 60  0001 C CNN "Populated"
-F 8 "IC VOLT SUPERVISOR ADJ 6SON" H 8850 5400 60  0001 C CNN "Description"
-F 9 "SPEC" H 8850 5400 60  0001 C CNN "Source"
-F 10 "1" H 8850 5400 50  0001 C CNN "Populate for SBGA485(Z-7030)"
-F 11 "1" H 8850 5400 50  0001 C CNN "Populate for CLG484(Z-7012s/Z-7015)"
-	1    8850 5400
-	1    0    0    -1
-$EndComp
-Text Notes 8400 5000 0    60   ~ 0
-500ms ~RESET~ Delay
-$Comp
-L power1:GND #PWR01801
-U 1 1 5B36B008
-P 8750 6300
-F 0 "#PWR01801" H 8750 6050 50  0001 C CNN
-F 1 "GND" H 8750 6150 50  0000 C CNN
-F 2 "" H 8750 6300 50  0001 C CNN
-F 3 "" H 8750 6300 50  0001 C CNN
-	1    8750 6300
-	1    0    0    -1
-$EndComp
-Wire Wire Line
-	9450 5300 9600 5300
-Wire Wire Line
-	9450 5500 9550 5500
-Wire Wire Line
-	9550 5500 9550 6150
-Wire Wire Line
-	7650 5400 7850 5400
-Wire Wire Line
-	7850 5300 7850 5400
-Connection ~ 7850 5400
-Wire Wire Line
-	7850 5000 7850 4900
-Wire Wire Line
-	7050 4900 7850 4900
-Wire Wire Line
-	8150 5300 8250 5300
-Wire Wire Line
-	7850 5800 7850 6150
-Wire Wire Line
-	7650 5550 7650 5400
-Wire Wire Line
-	7650 5750 7650 6150
-Connection ~ 7850 6150
-Wire Wire Line
-	7650 6150 7850 6150
-Wire Wire Line
-	8250 5500 8150 5500
-Wire Wire Line
-	8150 5500 8150 5650
 Wire Wire Line
 	8150 6150 8150 6050
-Connection ~ 8150 6150
-Wire Wire Line
-	8750 6300 8750 6150
-Connection ~ 8750 6150
-Wire Wire Line
-	7850 5400 8250 5400
-Wire Wire Line
-	7850 5400 7850 5500
-Wire Wire Line
-	7850 6150 8150 6150
-Wire Wire Line
-	8150 6150 8750 6150
-Wire Wire Line
-	8750 6150 9550 6150
-Text Label 10100 5300 2    60   ~ 0
+Text Label 8650 5250 2    60   ~ 0
 PS_RESET
 Text GLabel 8150 4600 1    60   Input ~ 0
 VCCO_MIO1
-Text HLabel 7050 4750 1    60   Input ~ 0
-PS_POR_B
 $Comp
 L device:R R1819
 U 1 1 5B3A2046
-P 9600 5050
-F 0 "R1819" V 9680 5050 50  0000 C CNN
-F 1 "100k" V 9600 5050 50  0000 C CNN
-F 2 "Resistor_SMD:R_0402_1005Metric" V 9530 5050 50  0001 C CNN
-F 3 "" H 9600 5050 50  0001 C CNN
-F 4 "1" H 9600 5050 60  0001 C CNN "Populated"
-F 5 "SPEC" H 9600 5050 60  0001 C CNN "Source"
-F 6 "1" H 9600 5050 50  0001 C CNN "Populate for SBGA485(Z-7030)"
-F 7 "1" H 9600 5050 50  0001 C CNN "Populate for CLG484(Z-7012s/Z-7015)"
-	1    9600 5050
-	1    0    0    -1
-$EndComp
-Wire Wire Line
-	9600 5200 9600 5300
-Connection ~ 9600 5300
-Wire Wire Line
-	9600 5300 10100 5300
-Wire Wire Line
-	9600 4900 9600 4800
-Wire Wire Line
-	9600 4800 8150 4800
-Connection ~ 8150 4800
-Wire Wire Line
-	8150 4800 8150 5300
-Wire Wire Line
-	7050 4900 7050 4750
-Wire Wire Line
-	8150 4600 8150 4800
-$Comp
-L device:C_Small C1805
-U 1 1 5B3E6117
-P 9800 5700
-F 0 "C1805" H 9650 5650 50  0000 L CNN
-F 1 "100 nF" H 9500 5800 50  0000 L CNN
-F 2 "Capacitors_SMD:C_0201" H 9800 5700 50  0001 C CNN
-F 3 "http://search.murata.co.jp/Ceramy/image/img/A01X/G101/ENG/GRM033R60J104KE19-01.pdf" H 9800 5700 50  0001 C CNN
-F 4 "Murata Electronics North America" H 9800 5700 60  0001 C CNN "MFG Name"
-F 5 "GRM033R60J104KE19D" H 9800 5700 60  0001 C CNN "MFG Part Num"
-F 6 "490-3167-1-ND" H 9800 5700 60  0001 C CNN "Digikey"
-F 7 "1" V 9800 5700 60  0001 C CNN "Populated"
-F 8 "SPEC" H 9800 5700 60  0001 C CNN "Source"
-F 9 "1" H 9800 5700 50  0001 C CNN "Populate for SBGA485(Z-7030)"
-F 10 "1" H 9800 5700 50  0001 C CNN "Populate for CLG484(Z-7012s/Z-7015)"
-	1    9800 5700
-	-1   0    0    1
-$EndComp
-Wire Wire Line
-	9800 5400 9800 5600
-Wire Wire Line
-	9450 5400 9800 5400
-Wire Wire Line
-	9800 5800 9800 6150
-Wire Wire Line
-	9800 6150 9550 6150
-Connection ~ 9550 6150
+P 8150 5000
+F 0 "R1819" V 8230 5000 50  0000 C CNN
+F 1 "10k" V 8150 5000 50  0000 C CNN
+F 2 "Resistor_SMD:R_0402_1005Metric" V 8080 5000 50  0001 C CNN
+F 3 "" H 8150 5000 50  0001 C CNN
+F 4 "1" H 8150 5000 60  0001 C CNN "Populated"
+F 5 "SPEC" H 8150 5000 60  0001 C CNN "Source"
+F 6 "1" H 8150 5000 50  0001 C CNN "Populate for SBGA485(Z-7030)"
+F 7 "1" H 8150 5000 50  0001 C CNN "Populate for CLG484(Z-7012s/Z-7015)"
+	1    8150 5000
+	1    0    0    -1
+$EndComp
+Wire Wire Line
+	8150 5150 8150 5250
+Wire Wire Line
+	8150 5250 8650 5250
+Wire Wire Line
+	8150 4600 8150 4850
+Wire Wire Line
+	8150 5250 8150 5650
+Connection ~ 8150 5250
+$Comp
+L power1:GND #PWR01801
+U 1 1 5B36B008
+P 8150 6150
+F 0 "#PWR01801" H 8150 5900 50  0001 C CNN
+F 1 "GND" H 8150 6000 50  0000 C CNN
+F 2 "" H 8150 6150 50  0001 C CNN
+F 3 "" H 8150 6150 50  0001 C CNN
+	1    8150 6150
+	1    0    0    -1
+$EndComp
 $EndSCHEMATC

Commit message: Fixed Schematic Symbols
Parts:
- C1801, C1802, C1803: symbol device:C_Small -> Device:C_Small
- R1801, R1802, R1803, R1816: symbol device:R_Small -> Device:R_Small
- R1804, R1805, R1806, R1807, R1808, R1809, R1810, R1811, R1812, R1813, R1814, R1815, R1819: symbol device:R -> Device:R
- SW1801: symbol switches:SW_Push -> Switch:SW_Push
Changed lines of the file:
@@
 $Descr A4 11693 8268
 encoding utf-8
-Sheet 18 22
+Sheet 17 21
 Title ""
 Date ""
@@
 NOTE: The BootROM expects the SD card\nto be connected to MIO pins 40..45 (SDIO0).
 $Comp
-L device:R R1812
+L Device:R R1812
 U 1 1 5A98BDBC
 P 7950 1400
@@
 $EndComp
 $Comp
-L device:R R1810
+L Device:R R1810
 U 1 1 5A98BDD7
 P 7750 1400
@@
 $EndComp
 $Comp
-L device:R R1808
+L Device:R R1808
 U 1 1 5A98BDF4
 P 7550 1400
@@
 $EndComp
 $Comp
-L device:R R1806
+L Device:R R1806
 U 1 1 5A98BE13
 P 7350 1400
@@
 $EndComp
 $Comp
-L device:R R1804
+L Device:R R1804
 U 1 1 5A98BE34
 P 7150 1400
@@
 $EndComp
 $Comp
-L device:R R1805
+L Device:R R1805
 U 1 1 5A98BE57
 P 7150 2600
@@
 $EndComp
 $Comp
-L device:R R1807
+L Device:R R1807
 U 1 1 5A98BE7C
 P 7350 2600
@@
 $EndComp
 $Comp
-L device:R R1809
+L Device:R R1809
 U 1 1 5A98BEA3
 P 7550 2600
@@
 $EndComp
 $Comp
-L device:R R1811
+L Device:R R1811
 U 1 1 5A98BECC
 P 7750 2600
@@
 $EndComp
 $Comp
-L device:R R1813
+L Device:R R1813
 U 1 1 5A98BEF7
 P 7950 2600
@@
 $EndComp
 $Comp
-L power1:GND #PWR0225
+L power:GND #PWR0225
 U 1 1 5A991630
 P 7550 2950
@@
 NOTE: pulls must be 20k.
 $Comp
-L power1:+3V3 #PWR0226
+L power:+3V3 #PWR0226
 U 1 1 5B22F273
 P 7550 1050
@@
 $EndComp
 $Comp
-L device:R R1814
+L Device:R R1814
 U 1 1 5B22FBB5
 P 8150 2600
@@
 $EndComp
 $Comp
-L device:R R1815
+L Device:R R1815
 U 1 1 5B22FC2F
 P 8350 2600
@@
 SDIO0_CD
 $Comp
-L power1:+3V3 #PWR0227
+L power:+3V3 #PWR0227
 U 1 1 5AD70E44
 P 2900 6850
@@
 $EndComp
 $Comp
-L power1:GND #PWR0228
+L power:GND #PWR0228
 U 1 1 5AD853F0
 P 950 6250
@@
 PS_UART_RX
 $Comp
-L device:C_Small C1801
+L Device:C_Small C1801
 U 1 1 5AD950DB
 P 1900 5850
@@
 $EndComp
 $Comp
-L power1:GND #PWR0229
+L power:GND #PWR0229
 U 1 1 5AD95198
 P 1700 5850
@@
 $EndComp
 $Comp
-L power1:+3V3 #PWR0230
+L power:+3V3 #PWR0230
 U 1 1 5AD9524B
 P 2100 5850
@@
 $EndComp
 $Comp
-L power1:+3V3 #PWR0231
+L power:+3V3 #PWR0231
 U 1 1 5ADAB627
 P 2850 7300
@@
 $EndComp
 $Comp
-L power1:GND #PWR0232
+L power:GND #PWR0232
 U 1 1 5ADAB6E8
 P 4600 6150
@@
 NoConn ~ 4500 7250
 $Comp
-L power1:GND #PWR0233
+L power:GND #PWR0233
 U 1 1 5ADABBC7
 P 2900 6650
@@
 $EndComp
 $Comp
-L device:C_Small C1802
+L Device:C_Small C1802
 U 1 1 5ADF17F1
 P 2700 2350
@@
 $EndComp
 $Comp
-L power1:GND #PWR0234
+L power:GND #PWR0234
 U 1 1 5ADF17F7
 P 2700 2550
@@
 $EndComp
 $Comp
-L power1:+3V3 #PWR0235
+L power:+3V3 #PWR0235
 U 1 1 5ADF17FE
 P 2700 2150
@@
 $EndComp
 $Comp
-L device:R_Small R1801
+L Device:R_Small R1801
 U 1 1 5ADF2073
 P 1500 2000
@@
 $EndComp
 $Comp
-L power1:+3V3 #PWR0236
+L power:+3V3 #PWR0236
 U 1 1 5ADF21D6
 P 1500 1750
@@
 SDA
 $Comp
-L power1:GND #PWR0237
+L power:GND #PWR0237
 U 1 1 5ADF2AA7
 P 2100 2850
@@
 $EndComp
 $Comp
-L power1:+3V3 #PWR0238
+L power:+3V3 #PWR0238
 U 1 1 5ADF2B75
 P 2100 1750
@@
 SDA
 $Comp
-L device:R_Small R1802
+L Device:R_Small R1802
 U 1 1 5ADF492A
 P 3850 1850
@@
 $EndComp
 $Comp
-L power1:+3V3 #PWR0239
+L power:+3V3 #PWR0239
 U 1 1 5ADF4931
 P 3850 1650
@@
 $EndComp
 $Comp
-L device:R_Small R1803
+L Device:R_Small R1803
 U 1 1 5ADF4A40
 P 4050 1850
@@
 $EndComp
 $Comp
-L power1:+3V3 #PWR0240
+L power:+3V3 #PWR0240
 U 1 1 5ADF4A46
 P 4050 1650
@@
 	3850 2150 3850 1950
 $Comp
-L switches:SW_Push SW1801
+L Switch:SW_Push SW1801
 U 1 1 5B1ED103
 P 8150 5850
@@
 $EndComp
 $Comp
-L power1:GND #PWR0244
+L power:GND #PWR0244
 U 1 1 5B02614D
 P 1550 5050
@@
 	1350 4950 1550 4950
 $Comp
-L power1:+3V3 #PWR0245
+L power:+3V3 #PWR0245
 U 1 1 5B02628C
 P 2850 4650
@@
 Connection ~ 2750 4750
 $Comp
-L device:C_Small C1803
+L Device:C_Small C1803
 U 1 1 5B026A7D
 P 1350 4850
@@
 	8700 1400 9200 1400
 $Comp
-L device:R_Small R1816
+L Device:R_Small R1816
 U 1 1 5B047F57
 P 2850 4950
@@
 VCCO_MIO1
 $Comp
-L device:R R1819
+L Device:R R1819
 U 1 1 5B3A2046
 P 8150 5000
@@
 Connection ~ 8150 5250
 $Comp
-L power1:GND #PWR01801
+L power:GND #PWR01801
 U 1 1 5B36B008
 P 8150 6150

Commit message: WIP: route GPIOs/Levelshifters
Parts:
- R1802, R1803: footprint Resistors_SMD:R_0603 -> Resistor_SMD:R_0402_1005Metric; Populate for CLG484(Z-7012s/Z-7015) (none) -> 1; Populate for SBGA485(Z-7030) (none) -> 1
Changed lines of the file:
@@
 F 0 "R1802" H 3880 1870 50  0000 L CNN
 F 1 "4k7" H 3880 1810 50  0000 L CNN
-F 2 "Resistors_SMD:R_0603" H 3850 1850 50  0001 C CNN
+F 2 "Resistor_SMD:R_0402_1005Metric" H 3850 1850 50  0001 C CNN
 F 3 "" H 3850 1850 50  0001 C CNN
 F 4 "1" H 3850 1850 60  0001 C CNN "Populated"
 F 5 "SPEC" H 3850 1850 60  0001 C CNN "Source"
+F 6 "1" H 3850 1850 50  0001 C CNN "Populate for SBGA485(Z-7030)"
+F 7 "1" H 3850 1850 50  0001 C CNN "Populate for CLG484(Z-7012s/Z-7015)"
 	1    3850 1850
 	1    0    0    -1
@@
 F 0 "R1803" H 4080 1870 50  0000 L CNN
 F 1 "4k7" H 4080 1810 50  0000 L CNN
-F 2 "Resistors_SMD:R_0603" H 4050 1850 50  0001 C CNN
+F 2 "Resistor_SMD:R_0402_1005Metric" H 4050 1850 50  0001 C CNN
 F 3 "" H 4050 1850 50  0001 C CNN
 F 4 "1" H 4050 1850 60  0001 C CNN "Populated"
 F 5 "SPEC" H 4050 1850 60  0001 C CNN "Source"
+F 6 "1" H 4050 1850 50  0001 C CNN "Populate for SBGA485(Z-7030)"
+F 7 "1" H 4050 1850 50  0001 C CNN "Populate for CLG484(Z-7012s/Z-7015)"
 	1    4050 1850
 	1    0    0    -1
