File: hardware/ddr.sch (KiCad schematic (older format))
At the start: 45 parts

Commit message: Added decoupling Capacitors for the Zynq. Also added the 2,5 V Power supply.
The 2,5 V supply was implemented as LDO and is sourced by the 3,3 V Line.
Parts:
- added C? (x2): 0.01µF, Capacitors_SMD:C_0402, symbol C_Small
- added R? (x2): 80.6Ω, R402, symbol R_Small
Connections:
- net labels added: +V_DDR, VCCO_DDR, VREF
- net labels removed: +1V5
- wire segments 377 -> 391
Changed lines of the file:
@@
 Text Label 14050 5250 0    60   ~ 0
 A0
-$Comp
-L +1V5 #PWR?
-U 1 1 5985C8D0
-P 10650 2900
-F 0 "#PWR?" H 10650 2750 50  0001 C CNN
-F 1 "+1V5" H 10650 3040 50  0000 C CNN
-F 2 "" H 10650 2900 50  0001 C CNN
-F 3 "" H 10650 2900 50  0001 C CNN
-	1    10650 2900
-	1    0    0    -1
-$EndComp
-$Comp
-L +1V5 #PWR?
-U 1 1 5985CE11
-P 2800 8850
-F 0 "#PWR?" H 2800 8700 50  0001 C CNN
-F 1 "+1V5" H 2800 8990 50  0000 C CNN
-F 2 "" H 2800 8850 50  0001 C CNN
-F 3 "" H 2800 8850 50  0001 C CNN
-	1    2800 8850
-	1    0    0    -1
-$EndComp
-$Comp
-L +1V5 #PWR?
-U 1 1 5985EA7B
-P 5550 2900
-F 0 "#PWR?" H 5550 2750 50  0001 C CNN
-F 1 "+1V5" H 5550 3040 50  0000 C CNN
-F 2 "" H 5550 2900 50  0001 C CNN
-F 3 "" H 5550 2900 50  0001 C CNN
-	1    5550 2900
-	1    0    0    -1
-$EndComp
 Text Label 14800 3550 3    60   ~ 0
 VTT
@@
 Wire Wire Line
 	19050 9300 20050 9300
+Text GLabel 19600 9400 0    60   Input ~ 0
+VCCO_DDR
+Wire Wire Line
+	19600 9400 20050 9400
+$Comp
+L R_Small R?
+U 1 1 5AF40F8D
+P 19800 9100
+F 0 "R?" V 19750 9100 50  0000 C BNN
+F 1 "80.6Ω" V 19800 9100 31  0000 C CNN
+F 2 "R402" H 19800 9100 50  0001 C CNN
+F 3 "" H 19800 9100 50  0001 C CNN
+F 4 "1" H 19800 9100 60  0001 C CNN "Populated"
+F 5 "R0402 40.2Ω 1%" V 19800 9100 60  0001 C CNN "Description"
+	1    19800 9100
+	0    1    1    0
+$EndComp
+$Comp
+L R_Small R?
+U 1 1 5AF412AF
+P 19800 9200
+F 0 "R?" V 19750 9200 50  0000 C BNN
+F 1 "80.6Ω" V 19800 9200 31  0000 C CNN
+F 2 "R402" H 19800 9200 50  0001 C CNN
+F 3 "" H 19800 9200 50  0001 C CNN
+F 4 "1" H 19800 9200 60  0001 C CNN "Populated"
+F 5 "R0402 40.2Ω 1%" V 19800 9200 60  0001 C CNN "Description"
+	1    19800 9200
+	0    -1   -1   0
+$EndComp
+$Comp
+L GND #PWR?
+U 1 1 5AF4192D
+P 19100 9200
+F 0 "#PWR?" H 19100 8950 50  0001 C CNN
+F 1 "GND" H 19100 9050 50  0000 C CNN
+F 2 "" H 19100 9200 50  0001 C CNN
+F 3 "" H 19100 9200 50  0001 C CNN
+	1    19100 9200
+	0    1    1    0
+$EndComp
+Wire Wire Line
+	19100 9200 19700 9200
+Wire Wire Line
+	19900 9200 20050 9200
+Wire Wire Line
+	20050 9100 19900 9100
+Text GLabel 19600 9100 0    60   Input ~ 0
+VCCO_DDR
+Wire Wire Line
+	19600 9100 19700 9100
+$Comp
+L +V_DDR #PWR?
+U 1 1 5AF4B702
+P 2800 8850
+F 0 "#PWR?" H 2800 8700 50  0001 C CNN
+F 1 "+V_DDR" H 2800 8990 50  0000 C CNN
+F 2 "" H 2800 8850 50  0001 C CNN
+F 3 "" H 2800 8850 50  0001 C CNN
+	1    2800 8850
+	1    0    0    -1
+$EndComp
+$Comp
+L +V_DDR #PWR?
+U 1 1 5AF4B7A1
+P 5550 2900
+F 0 "#PWR?" H 5550 2750 50  0001 C CNN
+F 1 "+V_DDR" H 5550 3040 50  0000 C CNN
+F 2 "" H 5550 2900 50  0001 C CNN
+F 3 "" H 5550 2900 50  0001 C CNN
+	1    5550 2900
+	1    0    0    -1
+$EndComp
+$Comp
+L +V_DDR #PWR?
+U 1 1 5AF4B9E0
+P 10650 2900
+F 0 "#PWR?" H 10650 2750 50  0001 C CNN
+F 1 "+V_DDR" H 10650 3040 50  0000 C CNN
+F 2 "" H 10650 2900 50  0001 C CNN
+F 3 "" H 10650 2900 50  0001 C CNN
+	1    10650 2900
+	1    0    0    -1
+$EndComp
+Wire Wire Line
+	17850 8900 20050 8900
+Wire Wire Line
+	20050 9000 19950 9000
+Wire Wire Line
+	19950 9000 19950 8900
+Connection ~ 19950 8900
+Text Label 19050 8900 0    60   ~ 0
+VREF
+$Comp
+L C_Small C?
+U 1 1 5AF79FC3
+P 18200 9100
+F 0 "C?" H 18210 9170 50  0000 L CNN
+F 1 "0.01µF" H 18210 9020 50  0000 L CNN
+F 2 "Capacitors_SMD:C_0402" H 18200 9100 50  0001 C CNN
+F 3 "" H 18200 9100 50  0001 C CNN
+F 4 "1" H 18200 9100 60  0001 C CNN "Populated"
+	1    18200 9100
+	1    0    0    -1
+$EndComp
+$Comp
+L C_Small C?
+U 1 1 5AF7A0D7
+P 17850 9100
+F 0 "C?" H 17860 9170 50  0000 L CNN
+F 1 "0.01µF" H 17860 9020 50  0000 L CNN
+F 2 "Capacitors_SMD:C_0402" H 17850 9100 50  0001 C CNN
+F 3 "" H 17850 9100 50  0001 C CNN
+F 4 "1" H 17850 9100 60  0001 C CNN "Populated"
+	1    17850 9100
+	1    0    0    -1
+$EndComp
+Wire Wire Line
+	17850 9200 17850 9300
+Wire Wire Line
+	17850 9300 18200 9300
+Wire Wire Line
+	18200 9300 18200 9200
+Wire Wire Line
+	17850 9000 17850 8900
+Wire Wire Line
+	18200 9000 18200 8900
+Connection ~ 18200 8900
+$Comp
+L GND #PWR?
+U 1 1 5AF7A86C
+P 18050 9400
+F 0 "#PWR?" H 18050 9150 50  0001 C CNN
+F 1 "GND" H 18050 9250 50  0000 C CNN
+F 2 "" H 18050 9400 50  0001 C CNN
+F 3 "" H 18050 9400 50  0001 C CNN
+	1    18050 9400
+	1    0    0    -1
+$EndComp
+Wire Wire Line
+	18050 9400 18050 9300
+Connection ~ 18050 9300
+Text Label 17850 8900 0    60   ~ 0
+VTT_REF
 $EndSCHEMATC

Commit message: Removed all BSS138PS Transistors due actual unavailability.
Used lsf0102 as Levelshifter for I2C bus, connected LEDs to already existing Levelshifters.
Other:
- note removed: "TODO: VREFx, VRx, VCCO_DDR"
Changed lines of the file:
@@
 LIBS:mdr20
 LIBS:dm3cs
+LIBS:lsf0102
 LIBS:zynq_board-cache
 EELAYER 25 0
@@
 Text Label 18350 4600 0    60   ~ 0
 DQ0
-Text Notes 19900 9900 0    60   ~ 0
-TODO: VREFx, VRx, VCCO_DDR
 Wire Wire Line
 	6800 5250 7000 5250

Commit message: Enhanced Power Connector and Filtering.
Also added a few more production informations.
Parts:
- added C? (x2): 10 µF, Capacitors_SMD:C_0603, symbol C_Small
- added C? (x16): 100 nF, Capacitors_SMD:C_0201, symbol C_Small
- U?: Digikey (none) -> 296-28767-1-ND; Populate for CLG484(Z-7012s/Z-7015) (none) -> 1; Populate for SBGA485(Z-7030) (none) -> 1
Connections:
- wire segments 391 -> 439
Other:
- note added: "Additional Decoupling Capacitors. May not be populated."

Commit message: Started to route DDR3 Memory.
At first added missing Footprint for Reference- and Terminationvoltage Regulator. Added Powerplanes for GND and VCCO. Added decoupling Network to both DDR3 Memory Chips. There are more small caps, to support Memory from other Manufactors.
Parts:
- removed C?: 10 µF, Capacitors_SMD:C_0603, symbol C_Small
- removed C? (x8): 100 nF, Capacitors_SMD:C_0201, symbol C_Small
- added C101, C102, C104, C106, C107, C109, C110, C111, C112, C113, C115, C116, C117, C118, C119, C120, C121, C122, C123, C124, C125, C126, C127, C128, C129, C130, C132, C134: 100 nF, Capacitors_SMD:C_0201, symbol C_Small
- added C114: 10 µF, Capacitors_SMD:C_0603, symbol C_Small
- C133, C136: renamed from C?; footprint C0603 -> Capacitors_SMD:C_0603; Populate for CLG484(Z-7012s/Z-7015) (none) -> 1; Populate for SBGA485(Z-7030) (none) -> 1
- C137: renamed from C?; footprint C0402 -> Capacitors_SMD:C_0402; Populate for CLG484(Z-7012s/Z-7015) (none) -> 1; Populate for SBGA485(Z-7030) (none) -> 1
- R40, R41: renamed from R?; footprint R402 -> Resistors_SMD:R_0402; Populate for CLG484(Z-7012s/Z-7015) (none) -> 1; Populate for SBGA485(Z-7030) (none) -> 1
- U13: renamed from U?; footprint S-PWSON-N10 -> footprints:TI_PWSON-N10_2.0x2.0mm
- gave numbers to parts that had none: 52
Connections:
- wire segments 439 -> 479

Commit message: Corrected two mistakes in the DDR Sheet. Changed bit sequence a bit to ease routing. Added more decoupling Caps Termination Voltage.
Mistakes: the Bank Address was not terminated. The Reset Line was connected like it's an terminated Signal. Reset should be connected through an PD Resistor to GND.
Parts:
- added C252, C253: 100 µF, Capacitors_SMD:C_1210, symbol C_Small
- added C254, C255: 4,7 µF, Capacitors_SMD:C_0402, symbol C_Small
- added C256, C257, C258, C259: 10 nF, Capacitors_SMD:C_0201, symbol C_Small
- added R166, R167, R168: 40.2Ω, Resistors_SMD:R_0402, symbol R_Small
- R43, R44, R45, R46, R47, R48, R49, R50, R51, R53, R54, R55, R56, R57, R58, R59, R60, R61, R62, R63, R64, R65, R66, R67: footprint R402 -> Resistors_SMD:R_0402
- R52: value 40.2Ω -> 4.7 kΩ; footprint R402 -> Resistors_SMD:R_0402; Description R0402 40.2Ω 1% -> R0402 4.7 kΩ; Populate for CLG484(Z-7012s/Z-7015) (none) -> 1; Populate for SBGA485(Z-7030) (none) -> 1; Source (none) -> SPEC
- U1: footprint (none) -> footprints:SBG485_22x22_19.0x19.0mm_Pitch0.8mm
Connections:
- wire segments 479 -> 505
Other:
- note added: "VTT Decoupling"
