File: hardware/ddr.sch (KiCad schematic (older format))
At the start: 98 parts, among them U201 xc7z030sbg485, U701 MT41K128M8, U702 TPS51206, U703 MT41K128M8

Commit message: Layouted USB-UART.
Also moved USB-OTG to the right Side of the Board. To get there
some free Space, i moved the DDR3/Memory and the FPGA a few
Millimeters down.
Parts:
- R701, R702, R703, R704, R705, R706, R707, R708, R709, R710, R711, R712, R713, R714, R715, R716, R717, R718, R719, R720, R721, R722, R723, R724, R725, R726, R727, R728, R729, R730, R731, R732: footprint Resistors_SMD:R_0402 -> Resistor_SMD:R_0402_1005Metric
Changed lines of the file:
@@
 F 0 "R701" H 7080 6920 50  0000 L CNN
 F 1 "240Ω" H 7080 6860 50  0000 L CNN
-F 2 "Resistors_SMD:R_0402" H 7050 6900 50  0001 C CNN
+F 2 "Resistor_SMD:R_0402_1005Metric" H 7050 6900 50  0001 C CNN
 F 3 "" H 7050 6900 50  0001 C CNN
 	1    7050 6900
@@
 F 0 "R704" H 12230 6920 50  0000 L CNN
 F 1 "240Ω" H 12230 6860 50  0000 L CNN
-F 2 "Resistors_SMD:R_0402" H 12200 6900 50  0001 C CNN
+F 2 "Resistor_SMD:R_0402_1005Metric" H 12200 6900 50  0001 C CNN
 F 3 "" H 12200 6900 50  0001 C CNN
 	1    12200 6900
@@
 F 0 "R717" V 14550 3850 50  0000 C BNN
 F 1 "40.2Ω" V 14600 3850 31  0000 C CNN
-F 2 "Resistors_SMD:R_0402" H 14600 3850 50  0001 C CNN
+F 2 "Resistor_SMD:R_0402_1005Metric" H 14600 3850 50  0001 C CNN
 F 3 "" H 14600 3850 50  0001 C CNN
 F 4 "1" H 14600 3850 60  0001 C CNN "Populated"
@@
 F 0 "R718" V 14550 4050 50  0000 C BNN
 F 1 "40.2Ω" V 14600 4050 31  0000 C CNN
-F 2 "Resistors_SMD:R_0402" H 14600 4050 50  0001 C CNN
+F 2 "Resistor_SMD:R_0402_1005Metric" H 14600 4050 50  0001 C CNN
 F 3 "" H 14600 4050 50  0001 C CNN
 F 4 "1" H 14600 4050 60  0001 C CNN "Populated"
@@
 F 0 "R719" V 14550 4250 50  0000 C BNN
 F 1 "40.2Ω" V 14600 4250 31  0000 C CNN
-F 2 "Resistors_SMD:R_0402" H 14600 4250 50  0001 C CNN
+F 2 "Resistor_SMD:R_0402_1005Metric" H 14600 4250 50  0001 C CNN
 F 3 "" H 14600 4250 50  0001 C CNN
 F 4 "1" H 14600 4250 60  0001 C CNN "Populated"
@@
 F 0 "R720" V 14550 4450 50  0000 C BNN
 F 1 "40.2Ω" V 14600 4450 31  0000 C CNN
-F 2 "Resistors_SMD:R_0402" H 14600 4450 50  0001 C CNN
+F 2 "Resistor_SMD:R_0402_1005Metric" H 14600 4450 50  0001 C CNN
 F 3 "" H 14600 4450 50  0001 C CNN
 F 4 "1" H 14600 4450 60  0001 C CNN "Populated"
@@
 F 0 "R721" V 14550 4650 50  0000 C BNN
 F 1 "40.2Ω" V 14600 4650 31  0000 C CNN
-F 2 "Resistors_SMD:R_0402" H 14600 4650 50  0001 C CNN
+F 2 "Resistor_SMD:R_0402_1005Metric" H 14600 4650 50  0001 C CNN
 F 3 "" H 14600 4650 50  0001 C CNN
 F 4 "1" H 14600 4650 60  0001 C CNN "Populated"
@@
 F 0 "R722" V 14550 4850 50  0000 C BNN
 F 1 "40.2Ω" V 14600 4850 31  0000 C CNN
-F 2 "Resistors_SMD:R_0402" H 14600 4850 50  0001 C CNN
+F 2 "Resistor_SMD:R_0402_1005Metric" H 14600 4850 50  0001 C CNN
 F 3 "" H 14600 4850 50  0001 C CNN
 F 4 "1" H 14600 4850 60  0001 C CNN "Populated"
@@
 F 0 "R723" V 14550 5050 50  0000 C BNN
 F 1 "40.2Ω" V 14600 5050 31  0000 C CNN
-F 2 "Resistors_SMD:R_0402" H 14600 5050 50  0001 C CNN
+F 2 "Resistor_SMD:R_0402_1005Metric" H 14600 5050 50  0001 C CNN
 F 3 "" H 14600 5050 50  0001 C CNN
 F 4 "1" H 14600 5050 60  0001 C CNN "Populated"
@@
 F 0 "R724" V 14550 5250 50  0000 C BNN
 F 1 "40.2Ω" V 14600 5250 31  0000 C CNN
-F 2 "Resistors_SMD:R_0402" H 14600 5250 50  0001 C CNN
+F 2 "Resistor_SMD:R_0402_1005Metric" H 14600 5250 50  0001 C CNN
 F 3 "" H 14600 5250 50  0001 C CNN
 F 4 "1" H 14600 5250 60  0001 C CNN "Populated"
@@
 F 0 "R711" V 14300 5150 50  0000 C BNN
 F 1 "40.2Ω" V 14350 5150 31  0000 C CNN
-F 2 "Resistors_SMD:R_0402" H 14350 5150 50  0001 C CNN
+F 2 "Resistor_SMD:R_0402_1005Metric" H 14350 5150 50  0001 C CNN
 F 3 "" H 14350 5150 50  0001 C CNN
 F 4 "1" H 14350 5150 60  0001 C CNN "Populated"
@@
 F 0 "R710" V 14300 4950 50  0000 C BNN
 F 1 "40.2Ω" V 14350 4950 31  0000 C CNN
-F 2 "Resistors_SMD:R_0402" H 14350 4950 50  0001 C CNN
+F 2 "Resistor_SMD:R_0402_1005Metric" H 14350 4950 50  0001 C CNN
 F 3 "" H 14350 4950 50  0001 C CNN
 F 4 "1" H 14350 4950 60  0001 C CNN "Populated"
@@
 F 0 "R709" V 14300 4750 50  0000 C BNN
 F 1 "40.2Ω" V 14350 4750 31  0000 C CNN
-F 2 "Resistors_SMD:R_0402" H 14350 4750 50  0001 C CNN
+F 2 "Resistor_SMD:R_0402_1005Metric" H 14350 4750 50  0001 C CNN
 F 3 "" H 14350 4750 50  0001 C CNN
 F 4 "1" H 14350 4750 60  0001 C CNN "Populated"
@@
 F 0 "R708" V 14300 4550 50  0000 C BNN
 F 1 "40.2Ω" V 14350 4550 31  0000 C CNN
-F 2 "Resistors_SMD:R_0402" H 14350 4550 50  0001 C CNN
+F 2 "Resistor_SMD:R_0402_1005Metric" H 14350 4550 50  0001 C CNN
 F 3 "" H 14350 4550 50  0001 C CNN
 F 4 "1" H 14350 4550 60  0001 C CNN "Populated"
@@
 F 0 "R707" V 14300 4350 50  0000 C BNN
 F 1 "40.2Ω" V 14350 4350 31  0000 C CNN
-F 2 "Resistors_SMD:R_0402" H 14350 4350 50  0001 C CNN
+F 2 "Resistor_SMD:R_0402_1005Metric" H 14350 4350 50  0001 C CNN
 F 3 "" H 14350 4350 50  0001 C CNN
 F 4 "1" H 14350 4350 60  0001 C CNN "Populated"
@@
 F 0 "R706" V 14300 4150 50  0000 C BNN
 F 1 "40.2Ω" V 14350 4150 31  0000 C CNN
-F 2 "Resistors_SMD:R_0402" H 14350 4150 50  0001 C CNN
+F 2 "Resistor_SMD:R_0402_1005Metric" H 14350 4150 50  0001 C CNN
 F 3 "" H 14350 4150 50  0001 C CNN
 F 4 "1" H 14350 4150 60  0001 C CNN "Populated"
@@
 F 0 "R705" V 14300 3950 50  0000 C BNN
 F 1 "40.2Ω" V 14350 3950 31  0000 C CNN
-F 2 "Resistors_SMD:R_0402" H 14350 3950 50  0001 C CNN
+F 2 "Resistor_SMD:R_0402_1005Metric" H 14350 3950 50  0001 C CNN
 F 3 "" H 14350 3950 50  0001 C CNN
 F 4 "1" H 14350 3950 60  0001 C CNN "Populated"
@@
 F 0 "R725" V 14550 5500 50  0000 C BNN
 F 1 "40.2Ω" V 14600 5500 31  0000 C CNN
-F 2 "Resistors_SMD:R_0402" H 14600 5500 50  0001 C CNN
+F 2 "Resistor_SMD:R_0402_1005Metric" H 14600 5500 50  0001 C CNN
 F 3 "" H 14600 5500 50  0001 C CNN
 F 4 "1" H 14600 5500 60  0001 C CNN "Populated"
@@
 F 0 "R726" V 14550 5700 50  0000 C BNN
 F 1 "40.2Ω" V 14600 5700 31  0000 C CNN
-F 2 "Resistors_SMD:R_0402" H 14600 5700 50  0001 C CNN
+F 2 "Resistor_SMD:R_0402_1005Metric" H 14600 5700 50  0001 C CNN
 F 3 "" H 14600 5700 50  0001 C CNN
 F 4 "1" H 14600 5700 60  0001 C CNN "Populated"
@@
 F 0 "R727" V 14550 5900 50  0000 C BNN
 F 1 "40.2Ω" V 14600 5900 31  0000 C CNN
-F 2 "Resistors_SMD:R_0402" H 14600 5900 50  0001 C CNN
+F 2 "Resistor_SMD:R_0402_1005Metric" H 14600 5900 50  0001 C CNN
 F 3 "" H 14600 5900 50  0001 C CNN
 F 4 "1" H 14600 5900 60  0001 C CNN "Populated"
@@
 F 0 "R728" V 14550 6100 50  0000 C BNN
 F 1 "40.2Ω" V 14600 6100 31  0000 C CNN
-F 2 "Resistors_SMD:R_0402" H 14600 6100 50  0001 C CNN
+F 2 "Resistor_SMD:R_0402_1005Metric" H 14600 6100 50  0001 C CNN
 F 3 "" H 14600 6100 50  0001 C CNN
 F 4 "1" H 14600 6100 60  0001 C CNN "Populated"
@@
 F 0 "R716" V 14350 7400 50  0000 C BNN
 F 1 "4.7 kΩ" V 14400 7400 31  0000 C CNN
-F 2 "Resistors_SMD:R_0402" H 14400 7400 50  0001 C CNN
+F 2 "Resistor_SMD:R_0402_1005Metric" H 14400 7400 50  0001 C CNN
 F 3 "" H 14400 7400 50  0001 C CNN
 F 4 "1" H 14400 7400 60  0001 C CNN "Populated"
@@
 F 0 "R713" V 14300 5600 50  0000 C BNN
 F 1 "40.2Ω" V 14350 5600 31  0000 C CNN
-F 2 "Resistors_SMD:R_0402" H 14350 5600 50  0001 C CNN
+F 2 "Resistor_SMD:R_0402_1005Metric" H 14350 5600 50  0001 C CNN
 F 3 "" H 14350 5600 50  0001 C CNN
 F 4 "1" H 14350 5600 60  0001 C CNN "Populated"
@@
 F 0 "R712" V 14300 5400 50  0000 C BNN
 F 1 "40.2Ω" V 14350 5400 31  0000 C CNN
-F 2 "Resistors_SMD:R_0402" H 14350 5400 50  0001 C CNN
+F 2 "Resistor_SMD:R_0402_1005Metric" H 14350 5400 50  0001 C CNN
 F 3 "" H 14350 5400 50  0001 C CNN
 F 4 "1" H 14350 5400 60  0001 C CNN "Populated"
@@
 F 0 "R715" V 14300 6700 50  0000 C BNN
 F 1 "80.6Ω" V 14350 6700 31  0000 C CNN
-F 2 "Resistors_SMD:R_0402" H 14350 6700 50  0001 C CNN
+F 2 "Resistor_SMD:R_0402_1005Metric" H 14350 6700 50  0001 C CNN
 F 3 "" H 14350 6700 50  0001 C CNN
 F 4 "1" H 14350 6700 60  0001 C CNN "Populated"
@@
 F 0 "R702" V 8200 9350 50  0000 C BNN
 F 1 "10kΩ" V 8250 9350 31  0000 C CNN
-F 2 "Resistors_SMD:R_0402" H 8250 9350 50  0001 C CNN
+F 2 "Resistor_SMD:R_0402_1005Metric" H 8250 9350 50  0001 C CNN
 F 3 "" H 8250 9350 50  0001 C CNN
 F 4 "1" H 8250 9350 60  0001 C CNN "Populated"
@@
 F 0 "R703" V 8200 9450 50  0000 C BNN
 F 1 "10kΩ" V 8250 9450 31  0000 C CNN
-F 2 "Resistors_SMD:R_0402" H 8250 9450 50  0001 C CNN
+F 2 "Resistor_SMD:R_0402_1005Metric" H 8250 9450 50  0001 C CNN
 F 3 "" H 8250 9450 50  0001 C CNN
 F 4 "1" H 8250 9450 60  0001 C CNN "Populated"
@@
 F 0 "R731" V 19750 9100 50  0000 C BNN
 F 1 "80.6Ω" V 19800 9100 31  0000 C CNN
-F 2 "Resistors_SMD:R_0402" H 19800 9100 50  0001 C CNN
+F 2 "Resistor_SMD:R_0402_1005Metric" H 19800 9100 50  0001 C CNN
 F 3 "" H 19800 9100 50  0001 C CNN
 F 4 "1" H 19800 9100 60  0001 C CNN "Populated"
@@
 F 0 "R732" V 19750 9200 50  0000 C BNN
 F 1 "80.6Ω" V 19800 9200 31  0000 C CNN
-F 2 "Resistors_SMD:R_0402" H 19800 9200 50  0001 C CNN
+F 2 "Resistor_SMD:R_0402_1005Metric" H 19800 9200 50  0001 C CNN
 F 3 "" H 19800 9200 50  0001 C CNN
 F 4 "1" H 19800 9200 60  0001 C CNN "Populated"
@@
 F 0 "R729" V 14550 6300 50  0000 C BNN
 F 1 "40.2Ω" V 14600 6300 31  0000 C CNN
-F 2 "Resistors_SMD:R_0402" H 14600 6300 50  0001 C CNN
+F 2 "Resistor_SMD:R_0402_1005Metric" H 14600 6300 50  0001 C CNN
 F 3 "" H 14600 6300 50  0001 C CNN
 F 4 "1" H 14600 6300 60  0001 C CNN "Populated"
@@
 F 0 "R714" V 14300 6400 50  0000 C BNN
 F 1 "40.2Ω" V 14350 6400 31  0000 C CNN
-F 2 "Resistors_SMD:R_0402" H 14350 6400 50  0001 C CNN
+F 2 "Resistor_SMD:R_0402_1005Metric" H 14350 6400 50  0001 C CNN
 F 3 "" H 14350 6400 50  0001 C CNN
 F 4 "1" H 14350 6400 60  0001 C CNN "Populated"
@@
 F 0 "R730" V 14550 6500 50  0000 C BNN
 F 1 "40.2Ω" V 14600 6500 31  0000 C CNN
-F 2 "Resistors_SMD:R_0402" H 14600 6500 50  0001 C CNN
+F 2 "Resistor_SMD:R_0402_1005Metric" H 14600 6500 50  0001 C CNN
 F 3 "" H 14600 6500 50  0001 C CNN
 F 4 "1" H 14600 6500 60  0001 C CNN "Populated"

Commit message: Improved Powerdistribution Network of the FPGA.
Also started to layout USB.
Parts:
- removed C752, C753: 100 µF, Capacitors_SMD:C_1210, symbol device:C_Small
- C701, C728, C747, C750: footprint Capacitors_SMD:C_0603 -> Capacitor_SMD:C_0603_1608Metric
- C702, C704, C707, C710, C714, C717, C719, C722, C751, C754, C755: footprint Capacitors_SMD:C_0402 -> Capacitor_SMD:C_0402_1005Metric
- C703, C705, C706, C708, C709, C711, C712, C713, C715, C716, C718, C720, C721, C723, C724, C725, C726, C727, C729, C730, C731, C732, C733, C734, C735, C736, C737, C738, C739, C740, C741, C742, C743, C744, C745, C746, C748, C749, C756, C757, C758, C759, C760, C761, C762: footprint Capacitors_SMD:C_0201 -> Capacitor_SMD:C_0201_0603Metric
Connections:
- wire segments 719 -> 711

Commit message: Fixed Schematic Symbols
Parts:
- C701, C702, C703, C704, C705, C706, C707, C708, C709, C710, C711, C712, C713, C714, C715, C716, C717, C718, C719, C720, C721, C722, C723, C724, C725, C726, C727, C728, C729, C730, C731, C732, C733, C734, C735, C736, C737, C738, C739, C740, C741, C742, C743, C744, C745, C746, C747, C748, C749, C750, C751, C754, C755, C756, C757, C758, C759, C760, C761, C762: symbol device:C_Small -> Device:C_Small
- R701, R702, R703, R704, R705, R706, R707, R708, R709, R710, R711, R712, R713, R714, R715, R716, R717, R718, R719, R720, R721, R722, R723, R724, R725, R726, R727, R728, R729, R730, R731, R732: symbol device:R_Small -> Device:R_Small

Commit message: SFP+ Power Filter, Levelshifter and MGT/TLK Clock Distribution.
Parts:
- added C623, C624: 100uF, Capacitor_SMD:C_1210_3225Metric, symbol Device:C_Small
- added TP601: Test_Point, footprints:TestPoint_SMD_0.5mm, symbol Connector:Test_Point
Connections:
- wire segments 711 -> 720
Other:
- note added: "Two 100 µF Bulk Caps and two additional 4 to 7 µF deoupling Caps\nas recommended at Micron TN-46-14 Page 6"
Changed lines of the file:
@@
 	8400 9000 8500 9000
 Wire Wire Line
-	9850 9000 10000 9000
+	9850 9000 9950 9000
 Wire Wire Line
 	6950 6350 7500 6350
@@
 Wire Wire Line
 	6350 3200 6450 3200
+$Comp
+L Device:C_Small C623
+U 1 1 5B5B50E2
+P 11300 9250
+F 0 "C623" H 11100 9350 50  0000 L CNN
+F 1 "100uF" H 11050 9200 50  0000 L CNN
+F 2 "Capacitor_SMD:C_1210_3225Metric" H 11300 9250 50  0001 C CNN
+F 3 "http://search.murata.co.jp/Ceramy/image/img/A01X/G101/ENG/GRM32ER60J107ME20-01.pdf" H 11300 9250 50  0001 C CNN
+F 4 "Murata" H 11300 9250 60  0001 C CNN "MFG Name"
+F 5 "GRM32ER60J107M" H 11300 9250 60  0001 C CNN "MFG Part Num"
+F 6 "490-3390-1-ND" H 11300 9250 50  0001 C CNN "Digikey"
+F 7 "1" H 11300 9250 60  0001 C CNN "Populated"
+F 8 "CAP CER 100UF 6.3V X5R 1210" H 11300 9250 50  0001 C CNN "Description"
+F 9 "SPEC" H 11300 9250 60  0001 C CNN "Source"
+F 10 "1" H 11300 9250 50  0001 C CNN "Populate for SBGA485(Z-7030)"
+F 11 "1" H 11300 9250 50  0001 C CNN "Populate for CLG484(Z-7012s/Z-7015)"
+F 12 "6.3V" H 11150 9100 50  0000 C CNN "Voltage"
+	1    11300 9250
+	1    0    0    -1
+$EndComp
+Wire Wire Line
+	11300 9150 11300 9050
+Wire Wire Line
+	11300 9050 11650 9050
+Connection ~ 12050 9050
+Wire Wire Line
+	12050 9450 11650 9450
+Wire Wire Line
+	11300 9450 11300 9350
+Connection ~ 12050 9450
+$Comp
+L Device:C_Small C624
+U 1 1 5B8F1E5B
+P 11650 9250
+F 0 "C624" H 11450 9350 50  0000 L CNN
+F 1 "100uF" H 11400 9200 50  0000 L CNN
+F 2 "Capacitor_SMD:C_1210_3225Metric" H 11650 9250 50  0001 C CNN
+F 3 "http://search.murata.co.jp/Ceramy/image/img/A01X/G101/ENG/GRM32ER60J107ME20-01.pdf" H 11650 9250 50  0001 C CNN
+F 4 "Murata" H 11650 9250 60  0001 C CNN "MFG Name"
+F 5 "GRM32ER60J107M" H 11650 9250 60  0001 C CNN "MFG Part Num"
+F 6 "490-3390-1-ND" H 11650 9250 50  0001 C CNN "Digikey"
+F 7 "1" H 11650 9250 60  0001 C CNN "Populated"
+F 8 "CAP CER 100UF 6.3V X5R 1210" H 11650 9250 50  0001 C CNN "Description"
+F 9 "SPEC" H 11650 9250 60  0001 C CNN "Source"
+F 10 "1" H 11650 9250 50  0001 C CNN "Populate for SBGA485(Z-7030)"
+F 11 "1" H 11650 9250 50  0001 C CNN "Populate for CLG484(Z-7012s/Z-7015)"
+F 12 "6.3V" H 11500 9100 50  0000 C CNN "Voltage"
+	1    11650 9250
+	1    0    0    -1
+$EndComp
+Wire Wire Line
+	11650 9150 11650 9050
+Connection ~ 11650 9050
+Wire Wire Line
+	11650 9050 12050 9050
+Wire Wire Line
+	11650 9350 11650 9450
+Connection ~ 11650 9450
+Wire Wire Line
+	11650 9450 11300 9450
+Text Notes 11050 10150 0    50   ~ 0
+Two 100 µF Bulk Caps and two additional 4 to 7 µF deoupling Caps\nas recommended at Micron TN-46-14 Page 6
+$Comp
+L Connector:Test_Point TP601
+U 1 1 5BA77F6A
+P 9950 9000
+F 0 "TP601" H 10008 9120 50  0000 L CNN
+F 1 "Test_Point" H 10008 9029 50  0000 L CNN
+F 2 "footprints:TestPoint_SMD_0.5mm" H 10150 9000 50  0001 C CNN
+F 3 "~" H 10150 9000 50  0001 C CNN
+F 4 "1" H 9950 9000 50  0001 C CNN "Populated"
+F 5 "SPEC" H 9950 9000 50  0001 C CNN "Source"
+F 6 "1" H 9950 9000 50  0001 C CNN "Populate for SBGA485(Z-7030)"
+F 7 "1" H 9950 9000 50  0001 C CNN "Populate for CLG484(Z-7012s/Z-7015)"
+	1    9950 9000
+	1    0    0    -1
+$EndComp
 Wire Bus Line
 	7100 2000 18200 2000
@@
 Wire Bus Line
 	18200 2000 18200 7600
+Connection ~ 9950 9000
+Wire Wire Line
+	9950 9000 10000 9000
 $EndSCHEMATC

Commit message: Routed extra GPIO Solder Pads, reannotated the whole schematic to make it consistent.
Power Distribution routing WIP
Parts:
- U1: renamed from U201; Populate for CLG484(Z-7012s/Z-7015) (none) -> 1; Populate for SBGA485(Z-7030) (none) -> 1; Populated (none) -> 1; Source (none) -> SPEC
- renumbered C701 to C601, C702 to C602, C703 to C603, C704 to C604, C705 to C605, C706 to C606, C707 to C607, C708 to C608, C709 to C609, C710 to C610, C711 to C611, C712 to C612, C713 to C613, C714 to C614, C715 to C615, C716 to C616, C717 to C617, C718 to C618, C719 to C619, C720 to C620, C721 to C621, C722 to C622, C723 to C623, C724 to C624, C725 to C625, C726 to C626, C727 to C627, C728 to C628, C729 to C629, C730 to C630, C731 to C631, C732 to C632, C733 to C633, C734 to C634, C735 to C635, C736 to C636, C737 to C637, C738 to C638, C739 to C639, C740 to C640, C741 to C641, C742 to C642, C743 to C643, C744 to C644, C745 to C645, C746 to C646, C747 to C647, C748 to C648, C749 to C649, C750 to C650, C751 to C651, C623 to C652, C624 to C653, C754 to C654, C755 to C655, C756 to C656, C757 to C657, C758 to C658, C759 to C659, C760 to C660, C761 to C661, C762 to C662, R701 to R601, R702 to R602, R703 to R603, R704 to R604, R705 to R605, R706 to R606, R707 to R607, R708 to R608, R709 to R609, R710 to R610, R711 to R611, R712 to R612, R713 to R613, R714 to R614, R715 to R615, R716 to R616, R717 to R617, R718 to R618, R719 to R619, R720 to R620, R721 to R621, R722 to R622, R723 to R623, R724 to R624, R725 to R625, R726 to R626, R727 to R627, R728 to R628, R729 to R629, R730 to R630, R731 to R631, R732 to R632, U701 to U601, U702 to U602, U703 to U603

Commit message: First Version without any Net not routed.
Parts:
- U601, U603: footprint Housings_BGA:BGA-96_2x3x16_9.0x13.0mm_Pitch0.8mm -> Package_BGA:BGA-96_9.0x13.0mm_Layout2x3x16_P0.8mm
Changed lines of the file:
@@
 F 0 "U601" H 5550 5000 60  0000 C CNN
 F 1 "MT41K128M8" H 5550 5400 60  0000 C CNN
-F 2 "Housings_BGA:BGA-96_2x3x16_9.0x13.0mm_Pitch0.8mm" H 5550 5200 60  0001 C CNN
+F 2 "Package_BGA:BGA-96_9.0x13.0mm_Layout2x3x16_P0.8mm" H 5550 5200 60  0001 C CNN
 F 3 "https://www.micron.com/~/media/documents/products/data-sheet/dram/ddr3/1gb_1_35v_ddr3l.pdf" H 5550 5200 60  0001 C CNN
 F 4 "Micron" H 5550 5200 60  0001 C CNN "MFG Name"
@@
 F 0 "U603" H 10700 5000 60  0000 C CNN
 F 1 "MT41K128M8" H 10700 5400 60  0000 C CNN
-F 2 "Housings_BGA:BGA-96_2x3x16_9.0x13.0mm_Pitch0.8mm" H 10700 5200 60  0001 C CNN
+F 2 "Package_BGA:BGA-96_9.0x13.0mm_Layout2x3x16_P0.8mm" H 10700 5200 60  0001 C CNN
 F 3 "https://www.micron.com/~/media/documents/products/data-sheet/dram/ddr3/1gb_1_35v_ddr3l.pdf" H 10700 5200 60  0001 C CNN
 F 4 "Micron" H 10700 5200 60  0001 C CNN "MFG Name"
