File: hardware/pmic.sch (KiCad schematic (older format))
At the start: 55 parts

Commit message: Added a few Todos.
Other:
- note added: "Missing:\n* Input Protection\n* Input Connector\n* evtl. 2,5 V supply. May be needed for Bank 13."
- note removed: "Missing:\n* Input Protection\n* Input Connector"
Changed lines of the file:
@@
 5V
 Text Notes 1100 1000 0    60   ~ 0
-Missing:\n* Input Protection\n* Input Connector
+Missing:\n* Input Protection\n* Input Connector\n* evtl. 2,5 V supply. May be needed for Bank 13.
 Text Label 7150 2350 2    60   ~ 0
 PG_5V

Commit message: Added decoupling Capacitors for the Zynq. Also added the 2,5 V Power supply.
The 2,5 V supply was implemented as LDO and is sourced by the 3,3 V Line.
Parts:
- added C? (x2): 1 µF 6.3 V, Capacitors_SMD:C_0402, symbol C_Small
- added U?: MCP1700-2502E_SOT23, TO_SOT_Packages_SMD:SOT-23, symbol MCP1700-2502E_SOT23
Connections:
- net labels added: +2V5
- wire segments 353 -> 363
Other:
- note added: "2,5 V Source for Bank 13.\nLDO here, because there should\nno heavy current."
- note added: "2.5V"
Changed lines of the file:
@@
 Wire Wire Line
 	4250 5000 4250 5100
+$Comp
+L MCP1700-2502E_SOT23 U?
+U 1 1 5AFABD17
+P 14500 6300
+F 0 "U?" H 14650 6050 50  0000 C CNN
+F 1 "MCP1700-2502E_SOT23" H 14050 6450 50  0000 L CNN
+F 2 "TO_SOT_Packages_SMD:SOT-23" H 14500 6525 50  0001 C CNN
+F 3 "http://www.microchip.com/mymicrochip/filehandler.aspx?ddocname=en011779" H 14500 6300 50  0001 C CNN
+F 4 "Microchip Technology" H 14500 6300 60  0001 C CNN "MFG Name"
+F 5 "MCP1700T-2502E/TT" H 14500 6300 60  0001 C CNN "MFG Part Num"
+F 6 "MCP1700T-2502E/TTCT-ND" H 14500 6300 60  0001 C CNN "Digikey"
+F 7 "1" H 14500 6300 60  0001 C CNN "Populated"
+F 8 " IC REG LINEAR 2.5V 250MA SOT23-3" H 14500 6300 60  0001 C CNN "Description"
+F 9 "SPEC" H 14500 6300 60  0001 C CNN "Source"
+	1    14500 6300
+	1    0    0    -1
+$EndComp
+$Comp
+L GND #PWR?
+U 1 1 5AFAC292
+P 14500 6800
+F 0 "#PWR?" H 14500 6550 50  0001 C CNN
+F 1 "GND" H 14500 6650 50  0000 C CNN
+F 2 "" H 14500 6800 50  0001 C CNN
+F 3 "" H 14500 6800 50  0001 C CNN
+	1    14500 6800
+	1    0    0    -1
+$EndComp
+$Comp
+L C_Small C?
+U 1 1 5AFAD2F1
+P 14100 6500
+F 0 "C?" H 14110 6570 50  0000 L CNN
+F 1 "1 µF 6.3 V" H 14110 6420 50  0000 L CNN
+F 2 "Capacitors_SMD:C_0402" H 14100 6500 50  0001 C CNN
+F 3 "http://search.murata.co.jp/Ceramy/image/img/A01X/G101/ENG/GRM152R60J105ME15-01.pdf" H 14100 6500 50  0001 C CNN
+F 4 "Murata Electronics North America" H 14100 6500 60  0001 C CNN "MFG Name"
+F 5 "GRM152R60J105ME15D" H 14100 6500 60  0001 C CNN "MFG Part Num"
+F 6 "490-10006-1-ND" H 14100 6500 60  0001 C CNN "Digikey"
+F 7 "1" H 14100 6500 60  0001 C CNN "Populated"
+F 8 "CAP CER 1UF 6.3V X5R 0402" H 14100 6500 60  0001 C CNN "Description"
+F 9 "SPEC" H 14100 6500 60  0001 C CNN "Source"
+	1    14100 6500
+	1    0    0    -1
+$EndComp
+Wire Wire Line
+	14100 6400 14100 6300
+Wire Wire Line
+	14000 6300 14200 6300
+Wire Wire Line
+	14800 6300 15000 6300
+Wire Wire Line
+	14900 6300 14900 6400
+Wire Wire Line
+	14500 6600 14500 6800
+Wire Wire Line
+	14100 6600 14100 6700
+Wire Wire Line
+	14100 6700 14900 6700
+Connection ~ 14500 6700
+Wire Wire Line
+	14900 6700 14900 6600
+Wire Wire Line
+	15000 6300 15000 6200
+Connection ~ 14900 6300
+$Comp
+L +2V5 #PWR?
+U 1 1 5AFAEE44
+P 15000 6200
+F 0 "#PWR?" H 15000 6050 50  0001 C CNN
+F 1 "+2V5" H 15000 6340 50  0000 C CNN
+F 2 "" H 15000 6200 50  0001 C CNN
+F 3 "" H 15000 6200 50  0001 C CNN
+	1    15000 6200
+	1    0    0    -1
+$EndComp
+Wire Wire Line
+	14000 6300 14000 6200
+Connection ~ 14100 6300
+$Comp
+L +3V3 #PWR?
+U 1 1 5AFAF34B
+P 14000 6200
+F 0 "#PWR?" H 14000 6050 50  0001 C CNN
+F 1 "+3V3" H 14000 6340 50  0000 C CNN
+F 2 "" H 14000 6200 50  0001 C CNN
+F 3 "" H 14000 6200 50  0001 C CNN
+	1    14000 6200
+	1    0    0    -1
+$EndComp
+$Comp
+L C_Small C?
+U 1 1 5AFC1BC9
+P 14900 6500
+F 0 "C?" H 14910 6570 50  0000 L CNN
+F 1 "1 µF 6.3 V" H 14910 6420 50  0000 L CNN
+F 2 "Capacitors_SMD:C_0402" H 14900 6500 50  0001 C CNN
+F 3 "http://search.murata.co.jp/Ceramy/image/img/A01X/G101/ENG/GRM152R60J105ME15-01.pdf" H 14900 6500 50  0001 C CNN
+F 4 "Murata Electronics North America" H 14900 6500 60  0001 C CNN "MFG Name"
+F 5 "GRM152R60J105ME15D" H 14900 6500 60  0001 C CNN "MFG Part Num"
+F 6 "490-10006-1-ND" H 14900 6500 60  0001 C CNN "Digikey"
+F 7 "1" H 14900 6500 60  0001 C CNN "Populated"
+F 8 "CAP CER 1UF 6.3V X5R 0402" H 14900 6500 60  0001 C CNN "Description"
+F 9 "SPEC" H 14900 6500 60  0001 C CNN "Source"
+	1    14900 6500
+	1    0    0    -1
+$EndComp
+Text Notes 13850 7300 0    60   ~ 0
+2,5 V Source for Bank 13.\nLDO here, because there should\nno heavy current.
+Text Notes 14200 5250 0    157  ~ 31
+2.5V
 $EndSCHEMATC

Commit message: Removed all BSS138PS Transistors due actual unavailability.
Used lsf0102 as Levelshifter for I2C bus, connected LEDs to already existing Levelshifters.
Connections:
- no-connect marks 3 -> 4
Changed lines of the file:
@@
 LIBS:mdr20
 LIBS:dm3cs
+LIBS:lsf0102
 LIBS:zynq_board-cache
 EELAYER 25 0
@@
 Text Notes 14200 5250 0    157  ~ 31
 2.5V
+NoConn ~ 11950 3000
 $EndSCHEMATC

Commit message: First version of Power Input.
Connections:
- net labels added: V_IN
- wire segments 363 -> 269

Commit message: Started to route DDR3 Memory.
At first added missing Footprint for Reference- and Terminationvoltage Regulator. Added Powerplanes for GND and VCCO. Added decoupling Network to both DDR3 Memory Chips. There are more small caps, to support Memory from other Manufactors.
Parts:
- gave numbers to parts that had none: 58

Commit message: Added Power/Protection Circuit
Parts:
- renumbered C65 to C601, C66 to C602, C67 to C603, C68 to C604, C69 to C605, C70 to C606, C71 to C607, C72 to C608, C73 to C609, C74 to C610, C75 to C611, C76 to C612, C77 to C613, C78 to C614, C79 to C615, C80 to C616, C81 to C617, C82 to C618, C83 to C619, C84 to C620, C85 to C621, C86 to C622, R12 to R601, R13 to R602, R14 to R603, R15 to R604, R16 to R605, R17 to R606, R18 to R607, R19 to R608, R20 to R609, R21 to R610, R22 to R611, R23 to R612, R24 to R613, R25 to R614, R26 to R615, R27 to R616, R28 to R617, R29 to R618, R30 to R619, R31 to R620, R32 to R621, R33 to R622, R34 to R623, R35 to R624, R36 to R625, R37 to R626, R38 to R627, U3 to U601, U4 to U602, U5 to U603, U6 to U604, U7 to U605, U8 to U606, U9 to U607, U10 to U608, U11 to U609
