File: hardware/pmic.sch (KiCad schematic (older format))
At the start: 58 parts, among them U601 TPS8208x, U602 TPS8208x, U603 TPSM84424, U604 TPSM84424, U605 TPS8208x, U606 TPS8208x, U607 TPS8208x, U608 TPS3808G01, U609 MCP1700-2502E_SOT23

Commit message: Length matched DDR3 Memory again.
Forgot to keep enough space between the traces and between the meander waves.

Also, I switched to Kicad 5.0 RC2.

Swaped a few ddr signals.
Parts:
- C601, C602, C603, C604, C605, C606, C607, C608, C609, C610, C611, C614, C615, C616, C617, C618, C619, C620, C621, C622: symbol C_Small -> device:C_Small
- C612, C613: symbol CP_Small -> device:CP_Small
- R601, R602, R603, R604, R605, R606, R607, R608, R609, R610, R611, R612, R613, R614, R615, R616, R617, R618, R619, R620, R621, R622, R623, R624, R625, R626, R627: symbol R -> device:R
- U601, U602, U605, U606, U607: symbol TPS8208x -> ti_power_modules:TPS8208x
- U603, U604: symbol TPSM84824 -> ti_power_modules:TPSM84824
- U608: symbol TPS3890-Q1 -> ti_power_modules:TPS3890-Q1
- U609: symbol MCP1700-2502E_SOT23 -> regul:MCP1700-2502E_SOT23

Commit message: Layouted most of the Power Circuit and Triggerbus Levelshifters.
Added Footprint for Tantal Caps. Modified Footprint for MDR20 Connector, SD-Card.

Fixed Symbol and Circuit for Power Supervisor/Delay IC.

Also fixed some smaller things in the schematics.
Parts:
- added R628: 43k, Resistor_SMD:R_0402_1005Metric, symbol device:R
- C601, C602, C603, C604: footprint (none) -> Capacitor_SMD:C_1210_3225Metric; Description (none) -> CAP CER 10UF 25V X7R 1210; Digikey (none) -> 490-1867-1-ND; Populate for CLG484(Z-7012s/Z-7015) (none) -> 1; Populate for SBGA485(Z-7030) (none) -> 1
- C605, C606, C615, C616, C617: value 10uF 25V -> 10uF; footprint (none) -> Capacitor_SMD:C_0805_2012Metric; Description (none) -> CAP CER 10UF 10V X7R 0805; Digikey (none) -> 490-10516-1-ND; MFG Part Num GRM32DR71E106KA12L -> GRM21BR71A106KA73L; Populate for CLG484(Z-7012s/Z-7015) (none) -> 1; Populate for SBGA485(Z-7030) (none) -> 1; Voltage (none) -> 10 V
- C607, C608, C609, C618, C619, C620: footprint (none) -> Capacitor_SMD:C_1210_3225Metric; Description (none) -> CAP CER 47UF 6.3V X7R 1210; Digikey (none) -> 490-4844-1-ND; Populate for CLG484(Z-7012s/Z-7015) (none) -> 1; Populate for SBGA485(Z-7030) (none) -> 1
- C610, C611: footprint (none) -> Capacitor_SMD:C_1210_3225Metric; Description (none) -> CAP CER 100UF 6.3V X5R 1210; Digikey (none) -> 490-3390-1-ND; Populate for CLG484(Z-7012s/Z-7015) (none) -> 1; Populate for SBGA485(Z-7030) (none) -> 1
- C612, C613: footprint (none) -> footprints:C7343-31_KEMET-D_10.22x5.6mm; Digikey (none) -> 399-10341-1-ND; Populate for CLG484(Z-7012s/Z-7015) (none) -> 1; Populate for SBGA485(Z-7030) (none) -> 1
- C614: footprint (none) -> Capacitor_SMD:C_0402_1005Metric; Description (none) -> CAP CER 1000PF 6.3V X5R 0402; Digikey (none) -> 490-6285-1-ND; MFG Name (none) -> Murata Electronics North America; MFG Part Num (none) -> GRM155R60J102KA01D; Populate for CLG484(Z-7012s/Z-7015) (none) -> 1; Populate for SBGA485(Z-7030) (none) -> 1; Populated (none) -> 1; Source (none) -> SPEC; Voltage (none) -> 6,3 V
- R601, R602, R607, R609, R611, R612, R613, R614, R615, R616, R617, R618, R619, R620, R621, R622, R623, R624, R625, R626, R627: footprint (none) -> Resistor_SMD:R_0402_1005Metric; Populate for CLG484(Z-7012s/Z-7015) (none) -> 1; Populate for SBGA485(Z-7030) (none) -> 1
- R603, R604, R605, R606, R608, R610: footprint (none) -> Resistor_SMD:R_0402_1005Metric; Populate for CLG484(Z-7012s/Z-7015) (none) -> 1; Populate for SBGA485(Z-7030) (none) -> 1; Populated (none) -> 1; Source (none) -> SPEC
- U608: footprint Housings_DFN_QFN:DFN-6-1EP_2x2mm_Pitch0.65mm -> Package_DFN_QFN:Texas_S-PWSON-N6; symbol ti_power_modules:TPS3890-Q1 -> ti_power_modules:TPS3808; Populate for CLG484(Z-7012s/Z-7015) (none) -> 1; Populate for SBGA485(Z-7030) (none) -> 1
Connections:
- wire segments 269 -> 396
Other:
- note added: "For 300 ms Delay a 40 kΩ to 200 kΩ\nResistor must be used!"
- note added: "NO, POR can be triggered\nby disconnecting Power ..."

Commit message: Improved Powerdistribution Network of the FPGA.
Also started to layout USB.
Parts:
- C621, C622: footprint Capacitors_SMD:C_0402 -> Capacitor_SMD:C_0402_1005Metric
Changed lines of the file:
@@
 F 0 "C621" H 14110 6570 50  0000 L CNN
 F 1 "1 µF 6.3 V" H 14110 6420 50  0000 L CNN
-F 2 "Capacitors_SMD:C_0402" H 14100 6500 50  0001 C CNN
+F 2 "Capacitor_SMD:C_0402_1005Metric" H 14100 6500 50  0001 C CNN
 F 3 "http://search.murata.co.jp/Ceramy/image/img/A01X/G101/ENG/GRM152R60J105ME15-01.pdf" H 14100 6500 50  0001 C CNN
 F 4 "Murata Electronics North America" H 14100 6500 60  0001 C CNN "MFG Name"
@@
 F 0 "C622" H 14910 6570 50  0000 L CNN
 F 1 "1 µF 6.3 V" H 14910 6420 50  0000 L CNN
-F 2 "Capacitors_SMD:C_0402" H 14900 6500 50  0001 C CNN
+F 2 "Capacitor_SMD:C_0402_1005Metric" H 14900 6500 50  0001 C CNN
 F 3 "http://search.murata.co.jp/Ceramy/image/img/A01X/G101/ENG/GRM152R60J105ME15-01.pdf" H 14900 6500 50  0001 C CNN
 F 4 "Murata Electronics North America" H 14900 6500 60  0001 C CNN "MFG Name"

Commit message: Fixed Schematic Symbols
Parts:
- C601, C602, C603, C604, C605, C606, C607, C608, C609, C610, C611, C614, C615, C616, C617, C618, C619, C620, C621, C622: symbol device:C_Small -> Device:C_Small
- C612, C613: symbol device:CP_Small -> Device:CP_Small
- R601, R602, R603, R604, R605, R606, R607, R608, R609, R610, R611, R612, R613, R614, R615, R616, R617, R618, R619, R620, R621, R622, R623, R624, R625, R626, R627, R628: symbol device:R -> Device:R
- U609: symbol regul:MCP1700-2502E_SOT23 -> Regulator_Linear:MCP1700-2502E_SOT23

Commit message: SFP+ Power Filter, Levelshifter and MGT/TLK Clock Distribution.
Parts:
- added TP501, TP502, TP503, TP504, TP505, TP506, TP507, TP508, TP509, TP510, TP511, TP512, TP513: Test_Point, footprints:TestPoint_SMD_0.5mm, symbol Connector:Test_Point
Connections:
- wire segments 396 -> 408

Commit message: WIP: routing the HF Part of the Camera Connector. I have to move the clock away from the left border.
TODO: Fix DDR3 RAM.
Connections:
- net labels added: +V_IN, VCCO_MIO0
- net labels removed: V_IN
- wire segments 408 -> 399
- no-connect marks 4 -> 3
Changed lines of the file:
@@
 	1    0    0    -1
 $EndComp
-NoConn ~ 9400 2300
-NoConn ~ 9400 2150
 $Bitmap
 Pos 14450 2000
@@
 PS_POR_B
 $Comp
-L power:+3V3 #PWR046
-U 1 1 5AE3F062
-P 12100 1150
-F 0 "#PWR046" H 12100 1000 50  0001 C CNN
-F 1 "+3V3" H 12100 1290 50  0000 C CNN
-F 2 "" H 12100 1150 50  0001 C CNN
-F 3 "" H 12100 1150 50  0001 C CNN
-	1    12100 1150
-	1    0    0    -1
-$EndComp
-$Comp
 L power:+5V #PWR047
 U 1 1 5AE3F924
@@
 NoConn ~ 11950 3000
 Wire Wire Line
-	5400 1500 5500 1500
-Wire Wire Line
-	5500 1500 5500 1400
-Wire Wire Line
-	5400 1400 5500 1400
-Connection ~ 5500 1400
-Wire Wire Line
 	5750 1400 5750 1450
 Connection ~ 5750 1400
@@
 Connection ~ 11300 3800
 Wire Wire Line
-	5400 3900 5500 3900
-Wire Wire Line
-	5500 3900 5500 3800
-Wire Wire Line
-	5400 3800 5500 3800
-Connection ~ 5500 3800
-Wire Wire Line
 	5750 3800 5750 3850
 Connection ~ 5750 3800
@@
 Wire Wire Line
 	8900 2400 9100 2400
-Wire Wire Line
-	9500 2000 9400 2000
-Wire Wire Line
-	9400 2000 9400 2150
-Wire Wire Line
-	9400 2400 9400 2300
-Connection ~ 9400 2400
 Connection ~ 9100 1400
 Wire Wire Line
@@
 Wire Wire Line
 	3600 1400 3500 1400
-Text HLabel 2450 1400 0    60   Input ~ 0
-V_IN
 $Comp
 L Device:C_Small C603
@@
 $EndComp
 Wire Wire Line
-	5500 1400 5750 1400
-Wire Wire Line
 	5750 1400 5950 1400
 Wire Wire Line
@@
 	11300 3800 11300 4150
 Wire Wire Line
-	5500 3800 5750 3800
-Wire Wire Line
 	5750 3800 6050 3800
 Wire Wire Line
@@
 Wire Wire Line
 	9100 1900 9100 2000
-Wire Wire Line
-	9100 2400 9400 2400
-Wire Wire Line
-	9400 2400 10000 2400
 Wire Wire Line
 	9100 1400 9400 1400
@@
 Wire Wire Line
 	6350 7650 7600 7650
+Wire Wire Line
+	5400 3800 5750 3800
+Wire Wire Line
+	5400 1400 5750 1400
+$Comp
+L power_symbols:+V_IN #PWR0188
+U 1 1 5BE97F97
+P 2450 1250
+F 0 "#PWR0188" H 2450 1100 50  0001 C CNN
+F 1 "+V_IN" H 2465 1423 50  0000 C CNN
+F 2 "" H 2450 1250 50  0001 C CNN
+F 3 "" H 2450 1250 50  0001 C CNN
+	1    2450 1250
+	1    0    0    -1
+$EndComp
+Wire Wire Line
+	2450 1250 2450 1400
+Text GLabel 12100 1150 1    60   Input ~ 0
+VCCO_MIO0
+Wire Wire Line
+	9100 2400 10000 2400
+NoConn ~ 9500 2000
 $EndSCHEMATC
