File: hardware/SFP_plus.sch (KiCad schematic (older format))
At the start: 20 parts

Commit message: Started to route DDR3 Memory.
At first added missing Footprint for Reference- and Terminationvoltage Regulator. Added Powerplanes for GND and VCCO. Added decoupling Network to both DDR3 Memory Chips. There are more small caps, to support Memory from other Manufactors.
Parts:
- gave numbers to parts that had none: 20
Changed lines of the file:
@@
 $EndDescr
 $Comp
-L SFPP_CONN U?
+L SFPP_CONN U2
 U 1 1 5973C22F
 P 5400 3900
-F 0 "U?" H 5400 3850 60  0000 C CNN
+F 0 "U2" H 5400 3850 60  0000 C CNN
 F 1 "SFPP_CONN" H 5400 3950 60  0000 C CNN
 F 2 "footprints:SFP+_Connector_with_Cage" H 5400 3900 60  0001 C CNN
@@
 $EndComp
 $Comp
-L C C?
+L C C63
 U 1 1 5973C515
 P 3300 3450
-F 0 "C?" H 3325 3550 50  0000 L CNN
+F 0 "C63" H 3325 3550 50  0000 L CNN
 F 1 "0.1uF" H 3325 3350 50  0000 L CNN
 F 2 "Capacitors_SMD:C_0402" H 3338 3300 50  0001 C CNN
@@
 $EndComp
 $Comp
-L C C?
+L C C61
 U 1 1 5973C862
 P 3000 3450
-F 0 "C?" H 3025 3550 50  0000 L CNN
+F 0 "C61" H 3025 3550 50  0000 L CNN
 F 1 "22uF" H 3025 3350 50  0000 L CNN
 F 2 "Capacitors_SMD:C_0402" H 3038 3300 50  0001 C CNN
@@
 $EndComp
 $Comp
-L C C?
+L C C59
 U 1 1 5973C883
 P 2300 3450
-F 0 "C?" H 2325 3550 50  0000 L CNN
+F 0 "C59" H 2325 3550 50  0000 L CNN
 F 1 "0.1uF" H 2325 3350 50  0000 L CNN
 F 2 "Capacitors_SMD:C_0402" H 2338 3300 50  0001 C CNN
@@
 $EndComp
 $Comp
-L C C?
+L C C64
 U 1 1 5973C8C6
 P 3300 4350
-F 0 "C?" H 3325 4450 50  0000 L CNN
+F 0 "C64" H 3325 4450 50  0000 L CNN
 F 1 "0.1uF" H 3325 4250 50  0000 L CNN
 F 2 "Capacitors_SMD:C_0402" H 3338 4200 50  0001 C CNN
@@
 $EndComp
 $Comp
-L C C?
+L C C62
 U 1 1 5973C8FD
 P 3000 4350
-F 0 "C?" H 3025 4450 50  0000 L CNN
+F 0 "C62" H 3025 4450 50  0000 L CNN
 F 1 "22uF" H 3025 4250 50  0000 L CNN
 F 2 "Capacitors_SMD:C_0402" H 3038 4200 50  0001 C CNN
@@
 $EndComp
 $Comp
-L C C?
+L C C60
 U 1 1 5973C92A
 P 2300 4350
-F 0 "C?" H 2325 4450 50  0000 L CNN
+F 0 "C60" H 2325 4450 50  0000 L CNN
 F 1 "0.1uF" H 2325 4250 50  0000 L CNN
 F 2 "Capacitors_SMD:C_0402" H 2338 4200 50  0001 C CNN
@@
 $EndComp
 $Comp
-L L_Small L?
+L L_Small L3
 U 1 1 5973CA0B
 P 2650 3200
-F 0 "L?" V 2750 3200 50  0000 C CNN
+F 0 "L3" V 2750 3200 50  0000 C CNN
 F 1 "4.7uH" V 2550 3200 50  0000 C CNN
 F 2 "" H 2650 3200 50  0001 C CNN
@@
 $EndComp
 $Comp
-L L_Small L?
+L L_Small L4
 U 1 1 5973CA4A
 P 2650 4100
-F 0 "L?" V 2750 4100 50  0000 C CNN
+F 0 "L4" V 2750 4100 50  0000 C CNN
 F 1 "4.7uH" V 2550 4100 50  0000 C CNN
 F 2 "" H 2650 4100 50  0001 C CNN
@@
 Connection ~ 3000 4100
 $Comp
-L +3V3 #PWR?
+L +3V3 #PWR026
 U 1 1 5973CBAF
 P 2300 3150
-F 0 "#PWR?" H 2300 3000 50  0001 C CNN
+F 0 "#PWR026" H 2300 3000 50  0001 C CNN
 F 1 "+3V3" H 2300 3290 50  0000 C CNN
 F 2 "" H 2300 3150 50  0000 C CNN
@@
 $EndComp
 $Comp
-L +3V3 #PWR?
+L +3V3 #PWR027
 U 1 1 5973CBD5
 P 2300 4050
-F 0 "#PWR?" H 2300 3900 50  0001 C CNN
+F 0 "#PWR027" H 2300 3900 50  0001 C CNN
 F 1 "+3V3" H 2300 4190 50  0000 C CNN
 F 2 "" H 2300 4050 50  0000 C CNN
@@
 Connection ~ 2300 4100
 $Comp
-L GND #PWR?
+L GND #PWR028
 U 1 1 5973CC3E
 P 3300 3600
-F 0 "#PWR?" H 3300 3350 50  0001 C CNN
+F 0 "#PWR028" H 3300 3350 50  0001 C CNN
 F 1 "GND" H 3300 3450 50  0000 C CNN
 F 2 "" H 3300 3600 50  0000 C CNN
@@
 $EndComp
 $Comp
-L GND #PWR?
+L GND #PWR029
 U 1 1 5973CC64
 P 3000 3600
-F 0 "#PWR?" H 3000 3350 50  0001 C CNN
+F 0 "#PWR029" H 3000 3350 50  0001 C CNN
 F 1 "GND" H 3000 3450 50  0000 C CNN
 F 2 "" H 3000 3600 50  0000 C CNN
@@
 $EndComp
 $Comp
-L GND #PWR?
+L GND #PWR030
 U 1 1 5973CD98
 P 2300 3600
-F 0 "#PWR?" H 2300 3350 50  0001 C CNN
+F 0 "#PWR030" H 2300 3350 50  0001 C CNN
 F 1 "GND" H 2300 3450 50  0000 C CNN
 F 2 "" H 2300 3600 50  0000 C CNN
@@
 $EndComp
 $Comp
-L GND #PWR?
+L GND #PWR031
 U 1 1 5973CDD0
 P 3300 4500
-F 0 "#PWR?" H 3300 4250 50  0001 C CNN
+F 0 "#PWR031" H 3300 4250 50  0001 C CNN
 F 1 "GND" H 3300 4350 50  0000 C CNN
 F 2 "" H 3300 4500 50  0000 C CNN
@@
 $EndComp
 $Comp
-L GND #PWR?
+L GND #PWR032
 U 1 1 5973CDF6
 P 3000 4500
-F 0 "#PWR?" H 3000 4250 50  0001 C CNN
+F 0 "#PWR032" H 3000 4250 50  0001 C CNN
 F 1 "GND" H 3000 4350 50  0000 C CNN
 F 2 "" H 3000 4500 50  0000 C CNN
@@
 $EndComp
 $Comp
-L GND #PWR?
+L GND #PWR033
 U 1 1 5973CE1C
 P 2300 4500
-F 0 "#PWR?" H 2300 4250 50  0001 C CNN
+F 0 "#PWR033" H 2300 4250 50  0001 C CNN
 F 1 "GND" H 2300 4350 50  0000 C CNN
 F 2 "" H 2300 4500 50  0000 C CNN
@@
 Connection ~ 3300 4100
 $Comp
-L GND #PWR?
+L GND #PWR034
 U 1 1 5973DD7C
 P 4500 4500
-F 0 "#PWR?" H 4500 4250 50  0001 C CNN
+F 0 "#PWR034" H 4500 4250 50  0001 C CNN
 F 1 "GND" H 4500 4350 50  0000 C CNN
 F 2 "" H 4500 4500 50  0000 C CNN
@@
 Connection ~ 6450 4300
 $Comp
-L GND #PWR?
+L GND #PWR035
 U 1 1 5973DEDC
 P 6450 4500
-F 0 "#PWR?" H 6450 4250 50  0001 C CNN
+F 0 "#PWR035" H 6450 4250 50  0001 C CNN
 F 1 "GND" H 6450 4350 50  0000 C CNN
 F 2 "" H 6450 4500 50  0000 C CNN
@@
 $EndComp
 $Comp
-L R R?
+L R R1
 U 1 1 5973DF65
 P 6800 3050
-F 0 "R?" V 6880 3050 50  0000 C CNN
+F 0 "R1" V 6880 3050 50  0000 C CNN
 F 1 "10k" V 6800 3050 50  0000 C CNN
 F 2 "Resistors_SMD:R_0402" V 6730 3050 50  0001 C CNN
@@
 $EndComp
 $Comp
-L R R?
+L R R3
 U 1 1 5973DF9C
 P 7000 3050
-F 0 "R?" V 7080 3050 50  0000 C CNN
+F 0 "R3" V 7080 3050 50  0000 C CNN
 F 1 "10k" V 7000 3050 50  0000 C CNN
 F 2 "Resistors_SMD:R_0402" V 6930 3050 50  0001 C CNN
@@
 $EndComp
 $Comp
-L R R?
+L R R4
 U 1 1 5973DFC7
 P 7200 3050
-F 0 "R?" V 7280 3050 50  0000 C CNN
+F 0 "R4" V 7280 3050 50  0000 C CNN
 F 1 "10k" V 7200 3050 50  0000 C CNN
 F 2 "Resistors_SMD:R_0402" V 7130 3050 50  0001 C CNN
@@
 $EndComp
 $Comp
-L R R?
+L R R6
 U 1 1 5973DFF4
 P 7400 3050
-F 0 "R?" V 7480 3050 50  0000 C CNN
+F 0 "R6" V 7480 3050 50  0000 C CNN
 F 1 "10k" V 7400 3050 50  0000 C CNN
 F 2 "Resistors_SMD:R_0402" V 7330 3050 50  0001 C CNN
@@
 $EndComp
 $Comp
-L R R?
+L R R7
 U 1 1 5973E023
 P 7600 3050
-F 0 "R?" V 7680 3050 50  0000 C CNN
+F 0 "R7" V 7680 3050 50  0000 C CNN
 F 1 "10k" V 7600 3050 50  0000 C CNN
 F 2 "Resistors_SMD:R_0402" V 7530 3050 50  0001 C CNN
@@
 $EndComp
 $Comp
-L R R?
+L R R8
 U 1 1 5973E070
 P 7800 3050
-F 0 "R?" V 7880 3050 50  0000 C CNN
+F 0 "R8" V 7880 3050 50  0000 C CNN
 F 1 "10k" V 7800 3050 50  0000 C CNN
 F 2 "Resistors_SMD:R_0402" V 7730 3050 50  0001 C CNN
@@
 $EndComp
 $Comp
-L R R?
+L R R9
 U 1 1 5973E0A7
 P 8000 3050
-F 0 "R?" V 8080 3050 50  0000 C CNN
+F 0 "R9" V 8080 3050 50  0000 C CNN
 F 1 "10k" V 8000 3050 50  0000 C CNN
 F 2 "Resistors_SMD:R_0402" V 7930 3050 50  0001 C CNN
@@
 Connection ~ 7800 2800
 $Comp
-L +3V3 #PWR?
+L +3V3 #PWR036
 U 1 1 5973E37C
 P 7400 2700
-F 0 "#PWR?" H 7400 2550 50  0001 C CNN
+F 0 "#PWR036" H 7400 2550 50  0001 C CNN
 F 1 "+3V3" H 7400 2840 50  0000 C CNN
 F 2 "" H 7400 2700 50  0000 C CNN
@@
 	8000 4200 8000 3200
 $Comp
-L R R?
+L R R10
 U 1 1 5973E623
 P 8300 3450
-F 0 "R?" V 8380 3450 50  0000 C CNN
+F 0 "R10" V 8380 3450 50  0000 C CNN
 F 1 "1k" V 8300 3450 50  0000 C CNN
 F 2 "Resistors_SMD:R_0402" V 8230 3450 50  0001 C CNN
@@
 $EndComp
 $Comp
-L R R?
+L R R11
 U 1 1 5973E65E
 P 8300 3650
-F 0 "R?" V 8380 3650 50  0000 C CNN
+F 0 "R11" V 8380 3650 50  0000 C CNN
 F 1 "1k" V 8300 3650 50  0000 C CNN
 F 2 "Resistors_SMD:R_0402" V 8230 3650 50  0001 C CNN
@@
 SFP_GPIO
 $Comp
-L R R?
+L R R2
 U 1 1 5973F1E4
 P 6800 4450
-F 0 "R?" V 6880 4450 50  0000 C CNN
+F 0 "R2" V 6880 4450 50  0000 C CNN
 F 1 "DNP" V 6800 4450 50  0000 C CNN
 F 2 "Resistors_SMD:R_0402" V 6730 4450 50  0001 C CNN
@@
 $EndComp
 $Comp
-L R R?
+L R R5
 U 1 1 5973F225
 P 7200 4450
-F 0 "R?" V 7280 4450 50  0000 C CNN
+F 0 "R5" V 7280 4450 50  0000 C CNN
 F 1 "DNP" V 7200 4450 50  0000 C CNN
 F 2 "Resistors_SMD:R_0402" V 7130 4450 50  0001 C CNN
@@
 $EndComp
 $Comp
-L GND #PWR?
+L GND #PWR037
 U 1 1 5973F2EE
 P 7000 4700
-F 0 "#PWR?" H 7000 4450 50  0001 C CNN
+F 0 "#PWR037" H 7000 4450 50  0001 C CNN
 F 1 "GND" H 7000 4550 50  0000 C CNN
 F 2 "" H 7000 4700 50  0000 C CNN

Commit message: Added Power/Protection Circuit
Parts:
- renumbered C59 to C501, C60 to C502, C61 to C503, C62 to C504, C63 to C505, C64 to C506, L3 to L501, L4 to L502, R1 to R501, R2 to R502, R3 to R503, R4 to R504, R5 to R505, R6 to R506, R7 to R507, R8 to R508, R9 to R509, R10 to R510, R11 to R511, U2 to U501
Changed lines of the file:
@@
 $EndDescr
 $Comp
-L SFPP_CONN U2
+L SFPP_CONN U501
 U 1 1 5973C22F
 P 5400 3900
-F 0 "U2" H 5400 3850 60  0000 C CNN
+F 0 "U501" H 5400 3850 60  0000 C CNN
 F 1 "SFPP_CONN" H 5400 3950 60  0000 C CNN
 F 2 "footprints:SFP+_Connector_with_Cage" H 5400 3900 60  0001 C CNN
@@
 $EndComp
 $Comp
-L C C63
+L C C505
 U 1 1 5973C515
 P 3300 3450
-F 0 "C63" H 3325 3550 50  0000 L CNN
+F 0 "C505" H 3325 3550 50  0000 L CNN
 F 1 "0.1uF" H 3325 3350 50  0000 L CNN
 F 2 "Capacitors_SMD:C_0402" H 3338 3300 50  0001 C CNN
@@
 $EndComp
 $Comp
-L C C61
+L C C503
 U 1 1 5973C862
 P 3000 3450
-F 0 "C61" H 3025 3550 50  0000 L CNN
+F 0 "C503" H 3025 3550 50  0000 L CNN
 F 1 "22uF" H 3025 3350 50  0000 L CNN
 F 2 "Capacitors_SMD:C_0402" H 3038 3300 50  0001 C CNN
@@
 $EndComp
 $Comp
-L C C59
+L C C501
 U 1 1 5973C883
 P 2300 3450
-F 0 "C59" H 2325 3550 50  0000 L CNN
+F 0 "C501" H 2325 3550 50  0000 L CNN
 F 1 "0.1uF" H 2325 3350 50  0000 L CNN
 F 2 "Capacitors_SMD:C_0402" H 2338 3300 50  0001 C CNN
@@
 $EndComp
 $Comp
-L C C64
+L C C506
 U 1 1 5973C8C6
 P 3300 4350
-F 0 "C64" H 3325 4450 50  0000 L CNN
+F 0 "C506" H 3325 4450 50  0000 L CNN
 F 1 "0.1uF" H 3325 4250 50  0000 L CNN
 F 2 "Capacitors_SMD:C_0402" H 3338 4200 50  0001 C CNN
@@
 $EndComp
 $Comp
-L C C62
+L C C504
 U 1 1 5973C8FD
 P 3000 4350
-F 0 "C62" H 3025 4450 50  0000 L CNN
+F 0 "C504" H 3025 4450 50  0000 L CNN
 F 1 "22uF" H 3025 4250 50  0000 L CNN
 F 2 "Capacitors_SMD:C_0402" H 3038 4200 50  0001 C CNN
@@
 $EndComp
 $Comp
-L C C60
+L C C502
 U 1 1 5973C92A
 P 2300 4350
-F 0 "C60" H 2325 4450 50  0000 L CNN
+F 0 "C502" H 2325 4450 50  0000 L CNN
 F 1 "0.1uF" H 2325 4250 50  0000 L CNN
 F 2 "Capacitors_SMD:C_0402" H 2338 4200 50  0001 C CNN
@@
 $EndComp
 $Comp
-L L_Small L3
+L L_Small L501
 U 1 1 5973CA0B
 P 2650 3200
-F 0 "L3" V 2750 3200 50  0000 C CNN
+F 0 "L501" V 2750 3200 50  0000 C CNN
 F 1 "4.7uH" V 2550 3200 50  0000 C CNN
 F 2 "" H 2650 3200 50  0001 C CNN
@@
 $EndComp
 $Comp
-L L_Small L4
+L L_Small L502
 U 1 1 5973CA4A
 P 2650 4100
-F 0 "L4" V 2750 4100 50  0000 C CNN
+F 0 "L502" V 2750 4100 50  0000 C CNN
 F 1 "4.7uH" V 2550 4100 50  0000 C CNN
 F 2 "" H 2650 4100 50  0001 C CNN
@@
 $EndComp
 $Comp
-L R R1
+L R R501
 U 1 1 5973DF65
 P 6800 3050
-F 0 "R1" V 6880 3050 50  0000 C CNN
+F 0 "R501" V 6880 3050 50  0000 C CNN
 F 1 "10k" V 6800 3050 50  0000 C CNN
 F 2 "Resistors_SMD:R_0402" V 6730 3050 50  0001 C CNN
@@
 $EndComp
 $Comp
-L R R3
+L R R503
 U 1 1 5973DF9C
 P 7000 3050
-F 0 "R3" V 7080 3050 50  0000 C CNN
+F 0 "R503" V 7080 3050 50  0000 C CNN
 F 1 "10k" V 7000 3050 50  0000 C CNN
 F 2 "Resistors_SMD:R_0402" V 6930 3050 50  0001 C CNN
@@
 $EndComp
 $Comp
-L R R4
+L R R504
 U 1 1 5973DFC7
 P 7200 3050
-F 0 "R4" V 7280 3050 50  0000 C CNN
+F 0 "R504" V 7280 3050 50  0000 C CNN
 F 1 "10k" V 7200 3050 50  0000 C CNN
 F 2 "Resistors_SMD:R_0402" V 7130 3050 50  0001 C CNN
@@
 $EndComp
 $Comp
-L R R6
+L R R506
 U 1 1 5973DFF4
 P 7400 3050
-F 0 "R6" V 7480 3050 50  0000 C CNN
+F 0 "R506" V 7480 3050 50  0000 C CNN
 F 1 "10k" V 7400 3050 50  0000 C CNN
 F 2 "Resistors_SMD:R_0402" V 7330 3050 50  0001 C CNN
@@
 $EndComp
 $Comp
-L R R7
+L R R507
 U 1 1 5973E023
 P 7600 3050
-F 0 "R7" V 7680 3050 50  0000 C CNN
+F 0 "R507" V 7680 3050 50  0000 C CNN
 F 1 "10k" V 7600 3050 50  0000 C CNN
 F 2 "Resistors_SMD:R_0402" V 7530 3050 50  0001 C CNN
@@
 $EndComp
 $Comp
-L R R8
+L R R508
 U 1 1 5973E070
 P 7800 3050
-F 0 "R8" V 7880 3050 50  0000 C CNN
+F 0 "R508" V 7880 3050 50  0000 C CNN
 F 1 "10k" V 7800 3050 50  0000 C CNN
 F 2 "Resistors_SMD:R_0402" V 7730 3050 50  0001 C CNN
@@
 $EndComp
 $Comp
-L R R9
+L R R509
 U 1 1 5973E0A7
 P 8000 3050
-F 0 "R9" V 8080 3050 50  0000 C CNN
+F 0 "R509" V 8080 3050 50  0000 C CNN
 F 1 "10k" V 8000 3050 50  0000 C CNN
 F 2 "Resistors_SMD:R_0402" V 7930 3050 50  0001 C CNN
@@
 	8000 4200 8000 3200
 $Comp
-L R R10
+L R R510
 U 1 1 5973E623
 P 8300 3450
-F 0 "R10" V 8380 3450 50  0000 C CNN
+F 0 "R510" V 8380 3450 50  0000 C CNN
 F 1 "1k" V 8300 3450 50  0000 C CNN
 F 2 "Resistors_SMD:R_0402" V 8230 3450 50  0001 C CNN
@@
 $EndComp
 $Comp
-L R R11
+L R R511
 U 1 1 5973E65E
 P 8300 3650
-F 0 "R11" V 8380 3650 50  0000 C CNN
+F 0 "R511" V 8380 3650 50  0000 C CNN
 F 1 "1k" V 8300 3650 50  0000 C CNN
 F 2 "Resistors_SMD:R_0402" V 8230 3650 50  0001 C CNN
@@
 SFP_GPIO
 $Comp
-L R R2
+L R R502
 U 1 1 5973F1E4
 P 6800 4450
-F 0 "R2" V 6880 4450 50  0000 C CNN
+F 0 "R502" V 6880 4450 50  0000 C CNN
 F 1 "DNP" V 6800 4450 50  0000 C CNN
 F 2 "Resistors_SMD:R_0402" V 6730 4450 50  0001 C CNN
@@
 $EndComp
 $Comp
-L R R5
+L R R505
 U 1 1 5973F225
 P 7200 4450
-F 0 "R5" V 7280 4450 50  0000 C CNN
+F 0 "R505" V 7280 4450 50  0000 C CNN
 F 1 "DNP" V 7200 4450 50  0000 C CNN
 F 2 "Resistors_SMD:R_0402" V 7130 4450 50  0001 C CNN

Commit message: Length matched DDR3 Memory again.
Forgot to keep enough space between the traces and between the meander waves.

Also, I switched to Kicad 5.0 RC2.

Swaped a few ddr signals.
Parts:
- C501, C502, C503, C504, C505, C506: symbol C -> device:C
- L501, L502: symbol L_Small -> device:L_Small
- R501, R502, R503, R504, R505, R506, R507, R508, R509, R510, R511: symbol R -> device:R
- U501: symbol SFPP_CONN -> SFP_plus:SFPP_CONN
Changed lines of the file:
@@
-EESchema Schematic File Version 2
-LIBS:zynq_board-rescue
-LIBS:power
-LIBS:device
-LIBS:transistors
-LIBS:conn
-LIBS:linear
-LIBS:regul
-LIBS:74xx
-LIBS:cmos4000
-LIBS:adc-dac
-LIBS:memory
-LIBS:xilinx
-LIBS:microcontrollers
-LIBS:dsp
-LIBS:microchip
-LIBS:analog_switches
-LIBS:motorola
-LIBS:texas
-LIBS:intel
-LIBS:audio
-LIBS:interface
-LIBS:digital-audio
-LIBS:philips
-LIBS:display
-LIBS:cypress
-LIBS:siliconi
-LIBS:opto
-LIBS:atmel
-LIBS:contrib
-LIBS:valves
-LIBS:xilinx_zynq_clg485
-LIBS:SFP_plus
-LIBS:ael2005
-LIBS:diff_osc
-LIBS:si53340
-LIBS:usb3320
-LIBS:nx5p3090
-LIBS:smp1255putg
-LIBS:osc
-LIBS:ddr
-LIBS:misc
-LIBS:tlk10031
-LIBS:lshm-150-xxx-x-dv-a-s
-LIBS:sn74axc8t245
-LIBS:sn74lvc2t45
-LIBS:dmf05lcflp
-LIBS:bss138ps
-LIBS:max14854
-LIBS:switches
-LIBS:ft234xd
-LIBS:sn74lv1t126
-LIBS:emif06-msd02n16
-LIBS:cat24c02tdi-gt3
-LIBS:power_symbols
-LIBS:ti_power_modules
-LIBS:mdr20
-LIBS:dm3cs
-LIBS:lsf0102
-LIBS:dmp3056l
+EESchema Schematic File Version 4
 LIBS:zynq_board-cache
-EELAYER 25 0
+EELAYER 26 0
 EELAYER END
 $Descr A4 11693 8268
@@
 $EndDescr
 $Comp
-L SFPP_CONN U501
+L SFP_plus:SFPP_CONN U501
 U 1 1 5973C22F
 P 5400 3900
@@
 $EndComp
 $Comp
-L C C505
+L device:C C505
 U 1 1 5973C515
 P 3300 3450
@@
 $EndComp
 $Comp
-L C C503
+L device:C C503
 U 1 1 5973C862
 P 3000 3450
@@
 $EndComp
 $Comp
-L C C501
+L device:C C501
 U 1 1 5973C883
 P 2300 3450
@@
 $EndComp
 $Comp
-L C C506
+L device:C C506
 U 1 1 5973C8C6
 P 3300 4350
@@
 $EndComp
 $Comp
-L C C504
+L device:C C504
 U 1 1 5973C8FD
 P 3000 4350
@@
 $EndComp
 $Comp
-L C C502
+L device:C C502
 U 1 1 5973C92A
 P 2300 4350
@@
 $EndComp
 $Comp
-L L_Small L501
+L device:L_Small L501
 U 1 1 5973CA0B
 P 2650 3200
@@
 $EndComp
 $Comp
-L L_Small L502
+L device:L_Small L502
 U 1 1 5973CA4A
 P 2650 4100
@@
 Connection ~ 3000 4100
 $Comp
-L +3V3 #PWR026
+L power1:+3V3 #PWR026
 U 1 1 5973CBAF
 P 2300 3150
@@
 $EndComp
 $Comp
-L +3V3 #PWR027
+L power1:+3V3 #PWR027
 U 1 1 5973CBD5
 P 2300 4050
@@
 Connection ~ 2300 4100
 $Comp
-L GND #PWR028
+L power1:GND #PWR028
 U 1 1 5973CC3E
 P 3300 3600
@@
 $EndComp
 $Comp
-L GND #PWR029
+L power1:GND #PWR029
 U 1 1 5973CC64
 P 3000 3600
@@
 $EndComp
 $Comp
-L GND #PWR030
+L power1:GND #PWR030
 U 1 1 5973CD98
 P 2300 3600
@@
 $EndComp
 $Comp
-L GND #PWR031
+L power1:GND #PWR031
 U 1 1 5973CDD0
 P 3300 4500
@@
 $EndComp
 $Comp
-L GND #PWR032
+L power1:GND #PWR032
 U 1 1 5973CDF6
 P 3000 4500
@@
 $EndComp
 $Comp
-L GND #PWR033
+L power1:GND #PWR033
 U 1 1 5973CE1C
 P 2300 4500
@@
 Connection ~ 3300 4100
 $Comp
-L GND #PWR034
+L power1:GND #PWR034
 U 1 1 5973DD7C
 P 4500 4500
@@
 Connection ~ 6450 4300
 $Comp
-L GND #PWR035
+L power1:GND #PWR035
 U 1 1 5973DEDC
 P 6450 4500
@@
 $EndComp
 $Comp
-L R R501
+L device:R R501
 U 1 1 5973DF65
 P 6800 3050
@@
 $EndComp
 $Comp
-L R R503
+L device:R R503
 U 1 1 5973DF9C
 P 7000 3050
@@
 $EndComp
 $Comp
-L R R504
+L device:R R504
 U 1 1 5973DFC7
 P 7200 3050
@@
 $EndComp
 $Comp
-L R R506
+L device:R R506
 U 1 1 5973DFF4
 P 7400 3050
@@
 $EndComp
 $Comp
-L R R507
+L device:R R507
 U 1 1 5973E023
 P 7600 3050
@@
 $EndComp
 $Comp
-L R R508
+L device:R R508
 U 1 1 5973E070
 P 7800 3050
@@
 $EndComp
 $Comp
-L R R509
+L device:R R509
 U 1 1 5973E0A7
 P 8000 3050
@@
 Connection ~ 7800 2800
 $Comp
-L +3V3 #PWR036
+L power1:+3V3 #PWR036
 U 1 1 5973E37C
 P 7400 2700
@@
 	8000 4200 8000 3200
 $Comp
-L R R510
+L device:R R510
 U 1 1 5973E623
 P 8300 3450
@@
 $EndComp
 $Comp
-L R R511
+L device:R R511
 U 1 1 5973E65E
 P 8300 3650
@@
 SFP_GPIO
 $Comp
-L R R502
+L device:R R502
 U 1 1 5973F1E4
 P 6800 4450
@@
 $EndComp
 $Comp
-L R R505
+L device:R R505
 U 1 1 5973F225
 P 7200 4450
@@
 $EndComp
 $Comp
-L GND #PWR037
+L power1:GND #PWR037
 U 1 1 5973F2EE
 P 7000 4700

Commit message: Layouted most of the Power Circuit and Triggerbus Levelshifters.
Added Footprint for Tantal Caps. Modified Footprint for MDR20 Connector, SD-Card.

Fixed Symbol and Circuit for Power Supervisor/Delay IC.

Also fixed some smaller things in the schematics.
Connections:
- wire segments 58 -> 85
Changed lines of the file:
@@
 	3300 3300 3300 3200
 Wire Wire Line
-	2750 3200 3600 3200
+	2750 3200 3000 3200
 Wire Wire Line
 	3000 3300 3000 3200
@@
 	2300 3200 2550 3200
 Wire Wire Line
-	2300 3150 2300 3300
-Wire Wire Line
-	2300 4050 2300 4200
+	2300 3150 2300 3200
+Wire Wire Line
+	2300 4050 2300 4100
 Wire Wire Line
 	2300 4100 2550 4100
@@
 	3000 4200 3000 4100
 Wire Wire Line
-	2750 4100 3600 4100
+	2750 4100 3000 4100
 Wire Wire Line
 	3300 4200 3300 4100
@@
 $EndComp
 Wire Wire Line
-	4500 3450 4500 4500
+	4500 3450 4500 3750
 Wire Wire Line
 	6300 3400 6450 3400
 Wire Wire Line
-	6450 3400 6450 4500
+	6450 3400 6450 4300
 Wire Wire Line
 	6300 4300 6450 4300
@@
 	6800 2900 6800 2800
 Wire Wire Line
-	6800 2800 8000 2800
+	6800 2800 7000 2800
 Wire Wire Line
 	8000 2800 8000 2900
@@
 Connection ~ 7200 2800
 Wire Wire Line
-	7400 2700 7400 2900
+	7400 2700 7400 2800
 Connection ~ 7400 2800
 Wire Wire Line
@@
 $EndComp
 Wire Wire Line
-	6300 3500 8150 3500
-Wire Wire Line
-	6800 3200 6800 4300
-Wire Wire Line
-	6300 3600 8650 3600
+	6300 3500 6800 3500
+Wire Wire Line
+	6800 3200 6800 3500
+Wire Wire Line
+	6300 3600 7000 3600
 Wire Wire Line
 	7000 3600 7000 3200
 Wire Wire Line
-	6300 3700 8150 3700
-Wire Wire Line
-	7200 3200 7200 4300
-Wire Wire Line
-	6300 3800 8650 3800
+	6300 3700 7200 3700
+Wire Wire Line
+	7200 3200 7200 3700
+Wire Wire Line
+	6300 3800 7400 3800
 Wire Wire Line
 	7400 3800 7400 3200
 Wire Wire Line
-	6300 3900 8650 3900
+	6300 3900 7600 3900
 Wire Wire Line
 	7600 3900 7600 3200
 Wire Wire Line
-	6300 4000 8650 4000
+	6300 4000 7800 4000
 Wire Wire Line
 	7800 4000 7800 3200
 Wire Wire Line
-	6300 4200 8650 4200
+	6300 4200 8000 4200
 Wire Wire Line
 	8000 4200 8000 3200
@@
 Connection ~ 6800 3500
 Wire Wire Line
-	8450 3450 8650 3450
+	8450 3450 8550 3450
 Connection ~ 8550 3450
 Connection ~ 7400 3800
@@
 	6800 4600 6800 4650
 Wire Wire Line
-	6800 4650 7200 4650
+	6800 4650 7000 4650
 Wire Wire Line
 	7000 4650 7000 4700
@@
 Text Notes 2300 2150 0    60   ~ 0
 Peak module current (3V3): 1200 mA\n(see SFF-8431 for details)
+Wire Wire Line
+	3000 3200 3300 3200
+Wire Wire Line
+	3000 4100 3300 4100
+Wire Wire Line
+	2300 3200 2300 3300
+Wire Wire Line
+	2300 4100 2300 4200
+Wire Wire Line
+	4500 4350 4500 4500
+Wire Wire Line
+	4500 4050 4500 4350
+Wire Wire Line
+	4500 3750 4500 4050
+Wire Wire Line
+	3300 4100 3600 4100
+Wire Wire Line
+	6450 4300 6450 4500
+Wire Wire Line
+	7000 2800 7200 2800
+Wire Wire Line
+	7200 2800 7400 2800
+Wire Wire Line
+	7400 2800 7400 2900
+Wire Wire Line
+	7400 2800 7600 2800
+Wire Wire Line
+	7600 2800 7800 2800
+Wire Wire Line
+	7800 2800 8000 2800
+Wire Wire Line
+	7000 3600 8650 3600
+Wire Wire Line
+	7200 3700 8150 3700
+Wire Wire Line
+	7200 3700 7200 4300
+Wire Wire Line
+	6800 3500 8150 3500
+Wire Wire Line
+	6800 3500 6800 4300
+Wire Wire Line
+	8550 3450 8650 3450
+Wire Wire Line
+	7400 3800 8650 3800
+Wire Wire Line
+	7600 3900 8650 3900
+Wire Wire Line
+	7800 4000 8650 4000
+Wire Wire Line
+	8000 4200 8650 4200
+Wire Wire Line
+	7000 4650 7200 4650
+Wire Wire Line
+	3300 3200 3600 3200
 $EndSCHEMATC
