File: hardware/SFP_plus.sch (KiCad schematic (older format))
At the start: 26 parts, among them U501 SFPP_CONN

Commit message: Routed a first Version of the High Speed Part of the Camera Connector. The optional LVDS Clocks are left unconnected. I couldn't keep the Connectors Pin Assignment because it was just impossible to route.
WIP: general Routing

Fixed: DDR3 Trace Length Matching
Parts:
- removed PO401, PO402: POWER_OUTPUT, footprints:EMPTY, symbol fixme:POWER_OUTPUT
Changed lines of the file:
@@
 	0    1    -1   0
 $EndComp
-Wire Wire Line
-	2750 3200 2800 3200
 Connection ~ 3000 3200
 Wire Wire Line
@@
 Wire Wire Line
 	2300 4450 2550 4450
-Wire Wire Line
-	2750 4450 2800 4450
 Connection ~ 3000 4450
 $Comp
@@
 Peak module current (3V3): 1200 mA\n(see SFF-8431 for details)
 Wire Wire Line
-	3000 3200 3300 3200
-Wire Wire Line
-	3000 4450 3300 4450
+	3000 3200 3150 3200
+Wire Wire Line
+	3000 4450 3200 4450
 Wire Wire Line
 	4500 4350 4500 4500
@@
 	1    0    0    -1
 $EndComp
-$Comp
-L fixme:POWER_OUTPUT PO401
-U 1 1 5BEC3DBF
-P 2800 3100
-F 0 "PO401" H 2800 3100 50  0001 C CNN
-F 1 "POWER_OUTPUT" H 2800 3250 50  0001 C CNN
-F 2 "footprints:EMPTY" H 2800 3100 50  0001 C CNN
-F 3 "" H 2800 3100 50  0001 C CNN
-	1    2800 3100
-	1    0    0    -1
-$EndComp
-Connection ~ 2800 3200
-Wire Wire Line
-	2800 3200 3000 3200
-$Comp
-L fixme:POWER_OUTPUT PO402
-U 1 1 5BEC3F5D
-P 2800 4350
-F 0 "PO402" H 2800 4350 50  0001 C CNN
-F 1 "POWER_OUTPUT" H 2800 4500 50  0001 C CNN
-F 2 "footprints:EMPTY" H 2800 4350 50  0001 C CNN
-F 3 "" H 2800 4350 50  0001 C CNN
-	1    2800 4350
-	1    0    0    -1
-$EndComp
-Connection ~ 2800 4450
-Wire Wire Line
-	2800 4450 3000 4450
+Wire Wire Line
+	2750 3200 3000 3200
+Wire Wire Line
+	2750 4450 3000 4450
+$Comp
+L power:PWR_FLAG #FLG0103
+U 1 1 5C1F039D
+P 3150 3200
+F 0 "#FLG0103" H 3150 3275 50  0001 C CNN
+F 1 "PWR_FLAG" H 3150 3374 50  0000 C CNN
+F 2 "" H 3150 3200 50  0001 C CNN
+F 3 "~" H 3150 3200 50  0001 C CNN
+	1    3150 3200
+	1    0    0    -1
+$EndComp
+Connection ~ 3150 3200
+Wire Wire Line
+	3150 3200 3300 3200
+$Comp
+L power:PWR_FLAG #FLG0104
+U 1 1 5C1F0411
+P 3200 4450
+F 0 "#FLG0104" H 3200 4525 50  0001 C CNN
+F 1 "PWR_FLAG" H 3200 4624 50  0000 C CNN
+F 2 "" H 3200 4450 50  0001 C CNN
+F 3 "~" H 3200 4450 50  0001 C CNN
+	1    3200 4450
+	1    0    0    -1
+$EndComp
+Connection ~ 3200 4450
+Wire Wire Line
+	3200 4450 3300 4450
 $EndSCHEMATC
