File: hardware/pwr_con_fuse_filter.sch (KiCad schematic (older format))
At the start: 6 parts

Commit message: Enhanced Power Connector and Filtering.
Also added a few more production informations.
Parts:
- removed C?: 100 nF/16 V, Capacitors_SMD:C_0402, symbol C_Small
- added D?: TN1515-600B-TR, TO_SOT_Packages_SMD:TO-252-2, symbol Q_Thyristor_KAG
- added D?: 15 V, Diodes_SMD:D_SOD-123, symbol D_Zener
- F?: Description (none) -> FUSE BOARD MOUNT 2.5A 32VDC 0402; Digikey (none) -> P15129CT-ND; MFG Name (none) -> Panasonic Electronic Components; MFG Part Num (none) -> ERB-RD2R50X
- T?: Digikey 490-11112-2-ND -> 490-11112-1-ND

Commit message: Started to route DDR3 Memory.
At first added missing Footprint for Reference- and Terminationvoltage Regulator. Added Powerplanes for GND and VCCO. Added decoupling Network to both DDR3 Memory Chips. There are more small caps, to support Memory from other Manufactors.
Parts:
- gave numbers to parts that had none: 7
Changed lines of the file:
@@
 $EndDescr
 $Comp
-L Conn_01x02 J?
+L Conn_01x02 J12
 U 1 1 5AFB123F
 P 1550 2800
-F 0 "J?" H 1550 2900 50  0000 C CNN
+F 0 "J12" H 1550 2900 50  0000 C CNN
 F 1 "Conn_01x02" H 1550 2600 50  0000 C CNN
 F 2 "footprints:WAGO-890-802" H 1550 2800 50  0001 C CNN
@@
 $EndComp
 $Comp
-L Transformer_1P_1S T?
+L Transformer_1P_1S T1
 U 1 1 5AFB12DF
 P 2550 2850
-F 0 "T?" H 2550 3100 50  0000 C CNN
+F 0 "T1" H 2550 3100 50  0000 C CNN
 F 1 "500 Ohm@100 MHz" H 2550 2550 50  0000 C CNN
 F 2 "" H 2550 2850 50  0001 C CNN
@@
 V_IN
 $Comp
-L DMP3056L Q?
+L DMP3056L Q1
 U 1 1 5AFC9627
 P 3900 2550
-F 0 "Q?" H 4100 2625 50  0000 L CNN
+F 0 "Q1" H 4100 2625 50  0000 L CNN
 F 1 "DMP3056L" H 4100 2550 50  0000 L CNN
 F 2 "TO_SOT_Packages_SMD:SOT-23" H 4100 2475 50  0001 L CIN
@@
 $EndComp
 $Comp
-L Fuse F?
+L Fuse F1
 U 1 1 5AFC9CDC
 P 3000 2450
-F 0 "F?" V 3080 2450 50  0000 C CNN
+F 0 "F1" V 3080 2450 50  0000 C CNN
 F 1 "Fuse" V 2925 2450 50  0000 C CNN
 F 2 "Resistors_SMD:R_0402" V 2930 2450 50  0001 C CNN
@@
 	3450 3250 3450 3450
 $Comp
-L D_TVS D?
+L D_TVS D5
 U 1 1 5AFCA27A
 P 2050 2850
-F 0 "D?" H 2050 2950 50  0000 C CNN
+F 0 "D5" H 2050 2950 50  0000 C CNN
 F 1 "P0220SCMCLRP" H 2050 2750 50  0000 C CNN
 F 2 "" H 2050 2850 50  0001 C CNN
@@
 Connection ~ 3450 3250
 $Comp
-L GND #PWR?
+L GND #PWR0261
 U 1 1 5AFCA36D
 P 3450 3450
-F 0 "#PWR?" H 3450 3200 50  0001 C CNN
+F 0 "#PWR0261" H 3450 3200 50  0001 C CNN
 F 1 "GND" H 3450 3300 50  0000 C CNN
 F 2 "" H 3450 3450 50  0001 C CNN
@@
 Connection ~ 2050 3250
 $Comp
-L Q_Thyristor_KAG D?
+L Q_Thyristor_KAG D7
 U 1 1 5B01386E
 P 3550 3000
-F 0 "D?" H 3625 3025 50  0000 L CNN
+F 0 "D7" H 3625 3025 50  0000 L CNN
 F 1 "TN1515-600B-TR" H 3625 2950 50  0000 L CNN
 F 2 "TO_SOT_Packages_SMD:TO-252-2" V 3550 3000 50  0001 C CNN
@@
 	3550 3250 3550 3150
 $Comp
-L D_Zener D?
+L D_Zener D6
 U 1 1 5B01397F
 P 3300 2750
-F 0 "D?" H 3300 2850 50  0000 C CNN
+F 0 "D6" H 3300 2850 50  0000 C CNN
 F 1 "15 V" H 3300 2650 50  0000 C CNN
 F 2 "Diodes_SMD:D_SOD-123" H 3300 2750 50  0001 C CNN

Commit message: Added Power/Protection Circuit
Parts:
- added D2204: BAT54GWJ, Diodes_SMD:D_SOD-123, symbol D_Schottky
- D2201: renamed from D5; footprint (none) -> footprints:DO-214AA
- F2201: renamed from F1; footprint Resistors_SMD:R_0402 -> Fuse_Holders_and_Fuses:Fuse_SMD1206_Reflow; Description FUSE BOARD MOUNT 2.5A 32VDC 0402 -> FUSE BOARD MOUNT 2.5A 32VDC 1206; Digikey P15129CT-ND -> P16740CT-ND; MFG Part Num ERB-RD2R50X -> ERB-RG2R50V
- T2201: renamed from T1; footprint (none) -> footprints:DLW5BTM_5.00x5.00mm
- renumbered D6 to D2202, D7 to D2203, J12 to J2201, Q1 to Q2201
Connections:
- wire segments 19 -> 18

Commit message: Length matched DDR3 Memory again.
Forgot to keep enough space between the traces and between the meander waves.

Also, I switched to Kicad 5.0 RC2.

Swaped a few ddr signals.
Parts:
- D2201: symbol D_TVS -> device:D_TVS
- D2202: symbol D_Zener -> device:D_Zener
- D2203: symbol Q_Thyristor_KAG -> device:Q_Thyristor_KAG
- D2204: symbol D_Schottky -> device:D_Schottky
- F2201: symbol Fuse -> device:Fuse
- J2201: symbol Conn_01x02 -> conn:Conn_01x02
- Q2201: symbol DMP3056L -> dmp3056l:DMP3056L
- T2201: symbol Transformer_1P_1S -> device:Transformer_1P_1S
Connections:
- wire segments 18 -> 24
Changed lines of the file:
@@
-EESchema Schematic File Version 2
-LIBS:zynq_board-rescue
-LIBS:power
-LIBS:device
-LIBS:transistors
-LIBS:conn
-LIBS:linear
-LIBS:regul
-LIBS:74xx
-LIBS:cmos4000
-LIBS:adc-dac
-LIBS:memory
-LIBS:xilinx
-LIBS:microcontrollers
-LIBS:dsp
-LIBS:microchip
-LIBS:analog_switches
-LIBS:motorola
-LIBS:texas
-LIBS:intel
-LIBS:audio
-LIBS:interface
-LIBS:digital-audio
-LIBS:philips
-LIBS:display
-LIBS:cypress
-LIBS:siliconi
-LIBS:opto
-LIBS:atmel
-LIBS:contrib
-LIBS:valves
-LIBS:xilinx_zynq_clg485
-LIBS:SFP_plus
-LIBS:ael2005
-LIBS:diff_osc
-LIBS:si53340
-LIBS:usb3320
-LIBS:nx5p3090
-LIBS:smp1255putg
-LIBS:osc
-LIBS:ddr
-LIBS:misc
-LIBS:tlk10031
-LIBS:lshm-150-xxx-x-dv-a-s
-LIBS:sn74axc8t245
-LIBS:sn74lvc2t45
-LIBS:dmf05lcflp
-LIBS:bss138ps
-LIBS:max14854
-LIBS:switches
-LIBS:ft234xd
-LIBS:sn74lv1t126
-LIBS:emif06-msd02n16
-LIBS:cat24c02tdi-gt3
-LIBS:power_symbols
-LIBS:ti_power_modules
-LIBS:mdr20
-LIBS:dm3cs
-LIBS:lsf0102
-LIBS:dmp3056l
+EESchema Schematic File Version 4
 LIBS:zynq_board-cache
-EELAYER 25 0
+EELAYER 26 0
 EELAYER END
 $Descr A4 11693 8268
@@
 $EndDescr
 $Comp
-L Conn_01x02 J2201
+L conn:Conn_01x02 J2201
 U 1 1 5AFB123F
 P 1550 2800
@@
 $EndComp
 $Comp
-L Transformer_1P_1S T2201
+L device:Transformer_1P_1S T2201
 U 1 1 5AFB12DF
 P 3000 2850
@@
 V_IN
 $Comp
-L DMP3056L Q2201
+L dmp3056l:DMP3056L Q2201
 U 1 1 5AFC9627
 P 4050 2550
@@
 $EndComp
 $Comp
-L Fuse F2201
+L device:Fuse F2201
 U 1 1 5AFC9CDC
 P 2150 2450
@@
 $EndComp
 Wire Wire Line
-	2300 2450 2800 2450
+	2300 2450 2500 2450
 Wire Wire Line
 	1850 2450 1850 2800
@@
 	1850 2900 1850 3250
 Wire Wire Line
-	1850 3250 2800 3250
-Wire Wire Line
-	3200 2450 3850 2450
-Wire Wire Line
-	3200 3250 4050 3250
+	1850 3250 2500 3250
+Wire Wire Line
+	3200 2450 3450 2450
+Wire Wire Line
+	3200 3250 3600 3250
 Wire Wire Line
 	4050 3250 4050 2750
@@
 	3600 3250 3600 3450
 $Comp
-L D_TVS D2201
+L device:D_TVS D2201
 U 1 1 5AFCA27A
 P 2500 2850
@@
 Connection ~ 3600 3250
 $Comp
-L GND #PWR0263
+L power1:GND #PWR0263
 U 1 1 5AFCA36D
 P 3600 3450
@@
 Connection ~ 2500 3250
 $Comp
-L Q_Thyristor_KAG D2203
+L device:Q_Thyristor_KAG D2203
 U 1 1 5B01386E
 P 3700 3000
@@
 	3700 3250 3700 3150
 $Comp
-L D_Zener D2202
+L device:D_Zener D2202
 U 1 1 5B01397F
 P 3450 2650
@@
 	2000 2450 1850 2450
 $Comp
-L D_Schottky D2204
+L device:D_Schottky D2204
 U 1 1 5B074FD5
 P 3450 2950
@@
 	0    -1   -1   0
 $EndComp
+Wire Wire Line
+	3600 3250 3700 3250
+Wire Wire Line
+	2500 2450 2800 2450
+Wire Wire Line
+	2500 3250 2800 3250
+Wire Wire Line
+	3450 2450 3700 2450
+Wire Wire Line
+	3700 2450 3850 2450
+Wire Wire Line
+	3700 3250 4050 3250
 $EndSCHEMATC

Commit message: Layouted most of the Power Circuit and Triggerbus Levelshifters.
Added Footprint for Tantal Caps. Modified Footprint for MDR20 Connector, SD-Card.

Fixed Symbol and Circuit for Power Supervisor/Delay IC.

Also fixed some smaller things in the schematics.
Parts:
- D2204: value BAT54GWJ -> PMEG3020EGWX; Description DIODE SCHOTTKY 30V 200MA SOD123 -> DIODE SCHOTTKY 30V 2A SOD123; Digikey 1727-7328-1-ND -> 1727-7331-1-ND; MFG Part Num BAT54GWJ -> PMEG3020EGWX
Changed lines of the file:
@@
 Wire Wire Line
 	2000 2450 1850 2450
-$Comp
-L device:D_Schottky D2204
-U 1 1 5B074FD5
-P 3450 2950
-F 0 "D2204" H 3450 2850 50  0000 C CNN
-F 1 "BAT54GWJ" H 3400 3050 50  0000 C CNN
-F 2 "Diodes_SMD:D_SOD-123" H 3450 2950 50  0001 C CNN
-F 3 "https://assets.nexperia.com/documents/data-sheet/BAT54GW.pdf" H 3450 2950 50  0001 C CNN
-F 4 "Nexperia USA Inc." H 3450 2950 60  0001 C CNN "MFG Name"
-F 5 "BAT54GWJ" H 3450 2950 60  0001 C CNN "MFG Part Num"
-F 6 "1727-7328-1-ND" H 3450 2950 60  0001 C CNN "Digikey"
-F 7 "1" H 3450 2950 60  0001 C CNN "Populated"
-F 8 "DIODE SCHOTTKY 30V 200MA SOD123" H 3450 2950 60  0001 C CNN "Description"
-F 9 "SPEC" H 3450 2950 60  0001 C CNN "Source"
-F 10 "1" H 3450 2950 60  0001 C CNN "Populate for SBGA485(Z-7030)"
-F 11 "1" H 3450 2950 60  0001 C CNN "Populate for CLG484(Z-7012s/Z-7015)"
-	1    3450 2950
-	0    -1   -1   0
-$EndComp
 Wire Wire Line
 	3600 3250 3700 3250
@@
 Wire Wire Line
 	3700 3250 4050 3250
+$Comp
+L device:D_Schottky D2204
+U 1 1 5B1B8794
+P 3450 2950
+F 0 "D2204" H 3450 3050 50  0000 C CNN
+F 1 "PMEG3020EGWX" H 3250 2850 50  0000 C CNN
+F 2 "Diodes_SMD:D_SOD-123" H 3450 2950 50  0001 C CNN
+F 3 "https://assets.nexperia.com/documents/data-sheet/PMEG3020EGW.pdf" H 3450 2950 50  0001 C CNN
+F 4 "Nexperia USA Inc." H 3450 2950 50  0001 C CNN "MFG Name"
+F 5 "PMEG3020EGWX" H 3450 2950 50  0001 C CNN "MFG Part Num"
+F 6 "1727-7331-1-ND" H 3450 2950 50  0001 C CNN "Digikey"
+F 7 "1" H 3450 2950 50  0001 C CNN "Populated"
+F 8 "DIODE SCHOTTKY 30V 2A SOD123" H 3450 2950 50  0001 C CNN "Description"
+F 9 "SPEC" H 3450 2950 50  0001 C CNN "Source"
+F 10 "1" H 3450 2950 50  0001 C CNN "Populate for SBGA485(Z-7030)"
+F 11 "1" H 3450 2950 50  0001 C CNN "Populate for CLG484(Z-7012s/Z-7015)"
+	1    3450 2950
+	0    -1   -1   0
+$EndComp
 $EndSCHEMATC

Commit message: Layouted USB-UART.
Also moved USB-OTG to the right Side of the Board. To get there
some free Space, i moved the DDR3/Memory and the FPGA a few
Millimeters down.
Parts:
- F2201: footprint Fuse_Holders_and_Fuses:Fuse_SMD1206_Reflow -> Fuse:Fuse_1206_3216Metric
Changed lines of the file:
@@
 F 0 "F2201" V 2230 2450 50  0000 C CNN
 F 1 "Fuse" V 2075 2450 50  0000 C CNN
-F 2 "Fuse_Holders_and_Fuses:Fuse_SMD1206_Reflow" V 2080 2450 50  0001 C CNN
+F 2 "Fuse:Fuse_1206_3216Metric" V 2080 2450 50  0001 C CNN
 F 3 "https://industrial.panasonic.com/cdbs/www-data/pdf/AFA0000/AFA0000C7.pdf" H 2150 2450 50  0001 C CNN
 F 4 "Panasonic Electronic Components" H 2150 2450 60  0001 C CNN "MFG Name"

Commit message: Fixed Schematic Symbols
Parts:
- D2201: symbol device:D_TVS -> Device:D_TVS
- D2202: symbol device:D_Zener -> Device:D_Zener
- D2203: symbol device:Q_Thyristor_KAG -> Device:Q_SCR_KAG
- D2204: symbol device:D_Schottky -> Device:D_Schottky
- F2201: symbol device:Fuse -> Device:Fuse
- J2201: symbol conn:Conn_01x02 -> Connector_Generic:Conn_01x02
- T2201: symbol device:Transformer_1P_1S -> Device:Transformer_1P_1S
Changed lines of the file:
@@
 $Descr A4 11693 8268
 encoding utf-8
-Sheet 22 22
+Sheet 21 21
 Title ""
 Date ""
@@
 $EndDescr
 $Comp
-L conn:Conn_01x02 J2201
+L Connector_Generic:Conn_01x02 J2201
 U 1 1 5AFB123F
 P 1550 2800
@@
 $EndComp
 $Comp
-L device:Transformer_1P_1S T2201
+L Device:Transformer_1P_1S T2201
 U 1 1 5AFB12DF
 P 3000 2850
@@
 $EndComp
 $Comp
-L device:Fuse F2201
+L Device:Fuse F2201
 U 1 1 5AFC9CDC
 P 2150 2450
@@
 	3600 3250 3600 3450
 $Comp
-L device:D_TVS D2201
+L Device:D_TVS D2201
 U 1 1 5AFCA27A
 P 2500 2850
@@
 Connection ~ 3600 3250
 $Comp
-L power1:GND #PWR0263
+L power:GND #PWR0263
 U 1 1 5AFCA36D
 P 3600 3450
@@
 Connection ~ 2500 3250
 $Comp
-L device:Q_Thyristor_KAG D2203
+L Device:Q_SCR_KAG D2203
 U 1 1 5B01386E
 P 3700 3000
@@
 	3700 3250 3700 3150
 $Comp
-L device:D_Zener D2202
+L Device:D_Zener D2202
 U 1 1 5B01397F
 P 3450 2650
@@
 	3700 3250 4050 3250
 $Comp
-L device:D_Schottky D2204
+L Device:D_Schottky D2204
 U 1 1 5B1B8794
 P 3450 2950
