File: hardware/TLK10031.sch (KiCad schematic (older format))
At the start: 44 parts, among them J1301 TEST_1P, J1302 TEST_1P, J1303 Conn_01x06, U1201 TLK10031

Commit message: Length matched DDR3 Memory again.
Forgot to keep enough space between the traces and between the meander waves.

Also, I switched to Kicad 5.0 RC2.

Swaped a few ddr signals.
Parts:
- C1301, C1302, C1303, C1304, C1305, C1306, C1307, C1308, C1309, C1310, C1311, C1312, C1313, C1314, C1315, C1316, C1317, C1318, C1319, C1320: symbol C_Small -> device:C_Small
- J1301, J1302: symbol TEST_1P -> conn:TEST_1P
- J1303: symbol Conn_01x06 -> conn:Conn_01x06
- R1301, R1302, R1303, R1304, R1305, R1306, R1307, R1308, R1309, R1310, R1311, R1312, R1313, R1314, R1315, R1316, R1317, R1318, R1319, R1320: symbol R -> device:R
- U1201: symbol TLK10031 -> tlk10031:TLK10031
Changed lines of the file:
@@
-EESchema Schematic File Version 2
-LIBS:zynq_board-rescue
-LIBS:power
-LIBS:device
-LIBS:transistors
-LIBS:conn
-LIBS:linear
-LIBS:regul
-LIBS:74xx
-LIBS:cmos4000
-LIBS:adc-dac
-LIBS:memory
-LIBS:xilinx
-LIBS:microcontrollers
-LIBS:dsp
-LIBS:microchip
-LIBS:analog_switches
-LIBS:motorola
-LIBS:texas
-LIBS:intel
-LIBS:audio
-LIBS:interface
-LIBS:digital-audio
-LIBS:philips
-LIBS:display
-LIBS:cypress
-LIBS:siliconi
-LIBS:opto
-LIBS:atmel
-LIBS:contrib
-LIBS:valves
-LIBS:xilinx_zynq_clg485
-LIBS:SFP_plus
-LIBS:ael2005
-LIBS:diff_osc
-LIBS:si53340
-LIBS:usb3320
-LIBS:nx5p3090
-LIBS:smp1255putg
-LIBS:osc
-LIBS:ddr
-LIBS:misc
-LIBS:tlk10031
-LIBS:lshm-150-xxx-x-dv-a-s
-LIBS:sn74axc8t245
-LIBS:sn74lvc2t45
-LIBS:dmf05lcflp
-LIBS:bss138ps
-LIBS:max14854
-LIBS:switches
-LIBS:ft234xd
-LIBS:sn74lv1t126
-LIBS:emif06-msd02n16
-LIBS:cat24c02tdi-gt3
-LIBS:power_symbols
-LIBS:ti_power_modules
-LIBS:mdr20
-LIBS:dm3cs
-LIBS:lsf0102
-LIBS:dmp3056l
+EESchema Schematic File Version 4
 LIBS:zynq_board-cache
-EELAYER 25 0
+EELAYER 26 0
 EELAYER END
 $Descr A4 11693 8268
@@
 $EndDescr
 $Comp
-L TLK10031 U1201
+L tlk10031:TLK10031 U1201
 U 1 1 5ACA3102
 P 5150 3450
@@
 INA[0]_N
 $Comp
-L C_Small C1301
+L device:C_Small C1301
 U 1 1 5ACAE246
 P 2400 1050
@@
 OUTA[0]_N
 $Comp
-L R R1314
+L device:R R1314
 U 1 1 5ACB0AA4
 P 3600 3050
@@
 $EndComp
 $Comp
-L GND #PWR0144
+L power1:GND #PWR0144
 U 1 1 5ACB0BCF
 P 3350 3050
@@
 HSRXA_N
 $Comp
-L GND #PWR0145
+L power1:GND #PWR0145
 U 1 1 5ACC67F6
 P 3950 5300
@@
 $EndComp
 $Comp
-L R R1303
+L device:R R1303
 U 1 1 5ACCADAC
 P 1100 4500
@@
 $EndComp
 $Comp
-L R R1305
+L device:R R1305
 U 1 1 5ACCAF62
 P 1250 4500
@@
 $EndComp
 $Comp
-L R R1307
+L device:R R1307
 U 1 1 5ACCB198
 P 1400 4500
@@
 $EndComp
 $Comp
-L R R1309
+L device:R R1309
 U 1 1 5ACCB19E
 P 1550 4500
@@
 $EndComp
 $Comp
-L R R1304
+L device:R R1304
 U 1 1 5ACCB916
 P 1100 5400
@@
 $EndComp
 $Comp
-L R R1306
+L device:R R1306
 U 1 1 5ACCB9E9
 P 1250 5400
@@
 $EndComp
 $Comp
-L R R1308
+L device:R R1308
 U 1 1 5ACCBA49
 P 1400 5400
@@
 $EndComp
 $Comp
-L R R1310
+L device:R R1310
 U 1 1 5ACCBAB0
 P 1550 5400
@@
 $EndComp
 $Comp
-L GND #PWR0146
+L power1:GND #PWR0146
 U 1 1 5ACCBE2D
 P 1250 5750
@@
 $EndComp
 $Comp
-L C_Small C1319
+L device:C_Small C1319
 U 1 1 5ACCC8EE
 P 3700 3250
@@
 $EndComp
 $Comp
-L C_Small C1320
+L device:C_Small C1320
 U 1 1 5ACCC9AB
 P 3700 3650
@@
 $EndComp
 $Comp
-L R R1313
+L device:R R1313
 U 1 1 5ACCCAE1
 P 3450 3450
@@
 MDC
 $Comp
-L Conn_01x06 J1303
+L conn:Conn_01x06 J1303
 U 1 1 5AC7786C
 P 8050 3050
@@
 $EndComp
 $Comp
-L GND #PWR0147
+L power1:GND #PWR0147
 U 1 1 5AC77C0F
 P 7750 3450
@@
 $EndComp
 $Comp
-L R R1320
+L device:R R1320
 U 1 1 5AC79DD9
 P 7550 3350
@@
 $EndComp
 $Comp
-L R R1315
+L device:R R1315
 U 1 1 5AC7A06C
 P 6700 3550
@@
 $EndComp
 $Comp
-L R R1318
+L device:R R1318
 U 1 1 5AC7A140
 P 6950 3650
@@
 $EndComp
 $Comp
-L R R1316
+L device:R R1316
 U 1 1 5AC7A1F2
 P 6700 3750
@@
 $EndComp
 $Comp
-L R R1319
+L device:R R1319
 U 1 1 5AC7A28E
 P 6950 3850
@@
 $EndComp
 $Comp
-L R R1317
+L device:R R1317
 U 1 1 5AC7A32D
 P 6950 3450
@@
 Same as VDDO
 $Comp
-L GND #PWR0148
+L power1:GND #PWR0148
 U 1 1 5AC7C5FF
 P 7300 3650
@@
 What to do with\nunsed output clocks?
 $Comp
-L TEST_1P J1301
+L conn:TEST_1P J1301
 U 1 1 5AC7FBF4
 P 2450 3950
@@
 $EndComp
 $Comp
-L R R1311
+L device:R R1311
 U 1 1 5AC82864
 P 2850 4250
@@
 Same as VDDO
 $Comp
-L TEST_1P J1302
+L conn:TEST_1P J1302
 U 1 1 5AC8C54E
 P 2450 4550
@@
 	2450 4550 3950 4550
 $Comp
-L R R1302
+L device:R R1302
 U 1 1 5AC8C9C3
 P 950 5400
@@
 $EndComp
 $Comp
-L R R1301
+L device:R R1301
 U 1 1 5AC8CA81
 P 950 4500
@@
 	2450 5650 3950 5650
 $Comp
-L R R1312
+L device:R R1312
 U 1 1 5AC9120F
 P 3150 5750
@@
 	2300 2750 2150 2750
 $Comp
-L +1V8 #PWR0149
+L power1:+1V8 #PWR0149
 U 1 1 5AC92C58
 P 2450 4250
@@
 $EndComp
 $Comp
-L +1V8 #PWR0150
+L power1:+1V8 #PWR0150
 U 1 1 5AC92CEE
 P 1250 4100
@@
 $EndComp
 $Comp
-L +1V8 #PWR0151
+L power1:+1V8 #PWR0151
 U 1 1 5AC92E59
 P 2900 5750
@@
 $EndComp
 $Comp
-L +1V8 #PWR0152
+L power1:+1V8 #PWR0152
 U 1 1 5AC92F40
 P 7100 3450
@@
 HSRXA_N
 $Comp
-L C_Small C1306
+L device:C_Small C1306
 U 1 1 5AE3C4AB
 P 2650 1150
@@
 $EndComp
 $Comp
-L C_Small C1311
+L device:C_Small C1311
 U 1 1 5AE3C523
 P 2900 1250
@@
 $EndComp
 $Comp
-L C_Small C1315
+L device:C_Small C1315
 U 1 1 5AE3C59E
 P 3150 1350
@@
 $EndComp
 $Comp
-L C_Small C1302
+L device:C_Small C1302
 U 1 1 5AE3C61E
 P 2400 1450
@@
 $EndComp
 $Comp
-L C_Small C1307
+L device:C_Small C1307
 U 1 1 5AE3C728
 P 2650 1550
@@
 $EndComp
 $Comp
-L C_Small C1312
+L device:C_Small C1312
 U 1 1 5AE3C7AA
 P 2900 1650
@@
 $EndComp
 $Comp
-L C_Small C1316
+L device:C_Small C1316
 U 1 1 5AE3C833
 P 3150 1750
@@
 $EndComp
 $Comp
-L C_Small C1303
+L device:C_Small C1303
 U 1 1 5AE3C8C1
 P 2400 1900
@@
 $EndComp
 $Comp
-L C_Small C1308
+L device:C_Small C1308
 U 1 1 5AE3C960
 P 2650 2000
@@
 $EndComp
 $Comp
-L C_Small C1313
+L device:C_Small C1313
 U 1 1 5AE3CA70
 P 2900 2100
@@
 $EndComp
 $Comp
-L C_Small C1317
+L device:C_Small C1317
 U 1 1 5AE3CB13
 P 3150 2200
@@
 $EndComp
 $Comp
-L C_Small C1304
+L device:C_Small C1304
 U 1 1 5AE3CBAD
 P 2400 2300
@@
 $EndComp
 $Comp
-L C_Small C1309
+L device:C_Small C1309
 U 1 1 5AE3CC68
 P 2650 2400
@@
 $EndComp
 $Comp
-L C_Small C1314
+L device:C_Small C1314
 U 1 1 5AE3CD12
 P 2900 2500
@@
 $EndComp
 $Comp
-L C_Small C1318
+L device:C_Small C1318
 U 1 1 5AE3CDAF
 P 3150 2600
@@
 $EndComp
 $Comp
-L C_Small C1305
+L device:C_Small C1305
 U 1 1 5AE3CE51
 P 2400 2750
@@
 $EndComp
 $Comp
-L C_Small C1310
+L device:C_Small C1310
 U 1 1 5AE3CF12
 P 2650 2850

Commit message: Layouted most of the Power Circuit and Triggerbus Levelshifters.
Added Footprint for Tantal Caps. Modified Footprint for MDR20 Connector, SD-Card.

Fixed Symbol and Circuit for Power Supervisor/Delay IC.

Also fixed some smaller things in the schematics.
Parts:
- C1301: Populate for CLG484(Z-7012s/Z-7015) (none) -> 1; Populate for SBGA485(Z-7030) (none) -> 1
Connections:
- wire segments 109 -> 130
Changed lines of the file:
@@
 F 7 "1" V 2400 1050 60  0001 C CNN "Populated"
 F 8 "SPEC" H 2400 1050 60  0001 C CNN "Source"
+F 9 "1" H 2400 1050 50  0001 C CNN "Populate for SBGA485(Z-7030)"
+F 10 "1" H 2400 1050 50  0001 C CNN "Populate for CLG484(Z-7012s/Z-7015)"
 	1    2400 1050
 	0    1    1    0
@@
 	3950 3000 3900 3000
 Wire Wire Line
-	3900 3000 3900 3100
+	3900 3000 3900 3050
 Wire Wire Line
 	3900 3100 3950 3100
@@
 	3950 4900 1550 4900
 Wire Wire Line
-	1550 4650 1550 5250
+	1550 4650 1550 4900
 Wire Wire Line
 	3950 5000 1400 5000
 Wire Wire Line
-	1400 4650 1400 5250
+	1400 4650 1400 5000
 Wire Wire Line
 	3950 5100 1250 5100
 Wire Wire Line
-	1250 4650 1250 5250
-Wire Wire Line
-	1100 4650 1100 5250
+	1250 4650 1250 5100
+Wire Wire Line
+	1100 4650 1100 5200
 Wire Wire Line
 	1100 5200 3950 5200
@@
 	6350 3050 7850 3050
 Wire Wire Line
-	7850 3150 6350 3150
+	7850 3150 7350 3150
 Wire Wire Line
 	6350 3250 7850 3250
@@
 Connection ~ 7350 3150
 Wire Wire Line
-	7700 3350 7850 3350
+	7700 3350 7750 3350
 Wire Wire Line
 	7400 3350 7350 3350
 Wire Wire Line
-	6550 3550 6350 3550
+	6550 3550 6450 3550
 Wire Wire Line
 	6800 3450 6450 3450
@@
 	6850 3550 7200 3550
 Wire Wire Line
-	7200 3550 7200 3850
+	7200 3550 7200 3650
 Wire Wire Line
 	7200 3850 7100 3850
@@
 Connection ~ 7200 3750
 Wire Wire Line
-	7100 3650 7300 3650
+	7100 3650 7200 3650
 Connection ~ 7200 3650
 Wire Wire Line
 	1100 4350 1100 4250
 Wire Wire Line
-	950  4250 1550 4250
+	950  4250 1100 4250
 Wire Wire Line
 	1550 4250 1550 4350
@@
 Connection ~ 1400 4250
 Wire Wire Line
-	1250 4100 1250 4350
+	1250 4100 1250 4250
 Connection ~ 1250 4250
 Wire Wire Line
 	1100 5550 1100 5650
 Wire Wire Line
-	950  5650 1550 5650
+	950  5650 1100 5650
 Wire Wire Line
 	1550 5650 1550 5550
@@
 Connection ~ 1400 5650
 Wire Wire Line
-	1250 5550 1250 5750
+	1250 5550 1250 5650
 Connection ~ 1250 5650
 Wire Wire Line
@@
 Connection ~ 1100 5650
 Wire Wire Line
-	950  4650 950  5250
+	950  4650 950  4750
 Wire Wire Line
 	3950 4750 950  4750
@@
 MDIO
 Wire Wire Line
-	2450 5650 3950 5650
+	2450 5650 3400 5650
 $Comp
 L device:R R1312
@@
 Text Notes 1350 7600 0    60   ~ 0
 TODO: Select Footprint for JTAG Connector.\nFor Just in Case. We don't have enough information to do even an\nboundary scan. So it may not be useful ....
+Wire Wire Line
+	3900 3050 3900 3100
+Wire Wire Line
+	1100 5200 1100 5250
+Wire Wire Line
+	1250 5100 1250 5250
+Wire Wire Line
+	1400 5000 1400 5250
+Wire Wire Line
+	1550 4900 1550 5250
+Wire Wire Line
+	7750 3350 7850 3350
+Wire Wire Line
+	7350 3150 6350 3150
+Wire Wire Line
+	6450 3550 6350 3550
+Wire Wire Line
+	7200 3750 7200 3850
+Wire Wire Line
+	7200 3650 7200 3750
+Wire Wire Line
+	7200 3650 7300 3650
+Wire Wire Line
+	1400 4250 1550 4250
+Wire Wire Line
+	1250 4250 1400 4250
+Wire Wire Line
+	1250 4250 1250 4350
+Wire Wire Line
+	1400 5650 1550 5650
+Wire Wire Line
+	1250 5650 1400 5650
+Wire Wire Line
+	1250 5650 1250 5750
+Wire Wire Line
+	1100 4250 1250 4250
+Wire Wire Line
+	1100 5650 1250 5650
+Wire Wire Line
+	950  4750 950  5250
+Wire Wire Line
+	3400 5650 3950 5650
 $EndSCHEMATC

Commit message: Layouted USB-UART.
Also moved USB-OTG to the right Side of the Board. To get there
some free Space, i moved the DDR3/Memory and the FPGA a few
Millimeters down.
Parts:
- R1301, R1302, R1303, R1304, R1305, R1306, R1307, R1308, R1309, R1310, R1311, R1312, R1313, R1314, R1315, R1316, R1317, R1318, R1319, R1320: footprint Resistors_SMD:R_0402 -> Resistor_SMD:R_0402_1005Metric
Changed lines of the file:
@@
 F 0 "R1314" V 3680 3050 50  0000 C CNN
 F 1 "100" V 3600 3050 50  0000 C CNN
-F 2 "Resistors_SMD:R_0402" V 3530 3050 50  0001 C CNN
+F 2 "Resistor_SMD:R_0402_1005Metric" V 3530 3050 50  0001 C CNN
 F 3 "" H 3600 3050 50  0001 C CNN
 F 4 "1" V 3600 3050 60  0001 C CNN "Populated"
@@
 F 0 "R1303" V 1180 4500 50  0000 C CNN
 F 1 "DNP" V 1100 4500 50  0000 C CNN
-F 2 "Resistors_SMD:R_0402" V 1030 4500 50  0001 C CNN
+F 2 "Resistor_SMD:R_0402_1005Metric" V 1030 4500 50  0001 C CNN
 F 3 "" H 1100 4500 50  0001 C CNN
 F 4 "0" V 1100 4500 60  0001 C CNN "Populated"
@@
 F 0 "R1305" V 1330 4500 50  0000 C CNN
 F 1 "DNP" V 1250 4500 50  0000 C CNN
-F 2 "Resistors_SMD:R_0402" V 1180 4500 50  0001 C CNN
+F 2 "Resistor_SMD:R_0402_1005Metric" V 1180 4500 50  0001 C CNN
 F 3 "" H 1250 4500 50  0001 C CNN
 F 4 "0" V 1250 4500 60  0001 C CNN "Populated"
@@
 F 0 "R1307" V 1480 4500 50  0000 C CNN
 F 1 "DNP" V 1400 4500 50  0000 C CNN
-F 2 "Resistors_SMD:R_0402" V 1330 4500 50  0001 C CNN
+F 2 "Resistor_SMD:R_0402_1005Metric" V 1330 4500 50  0001 C CNN
 F 3 "" H 1400 4500 50  0001 C CNN
 F 4 "0" V 1400 4500 60  0001 C CNN "Populated"
@@
 F 0 "R1309" V 1630 4500 50  0000 C CNN
 F 1 "DNP" V 1550 4500 50  0000 C CNN
-F 2 "Resistors_SMD:R_0402" V 1480 4500 50  0001 C CNN
+F 2 "Resistor_SMD:R_0402_1005Metric" V 1480 4500 50  0001 C CNN
 F 3 "" H 1550 4500 50  0001 C CNN
 F 4 "0" V 1550 4500 60  0001 C CNN "Populated"
@@
 F 0 "R1304" V 1180 5400 50  0000 C CNN
 F 1 "0" V 1100 5400 50  0000 C CNN
-F 2 "Resistors_SMD:R_0402" V 1030 5400 50  0001 C CNN
+F 2 "Resistor_SMD:R_0402_1005Metric" V 1030 5400 50  0001 C CNN
 F 3 "" H 1100 5400 50  0001 C CNN
 F 4 "1" V 1100 5400 60  0001 C CNN "Populated"
@@
 F 0 "R1306" V 1330 5400 50  0000 C CNN
 F 1 "0" V 1250 5400 50  0000 C CNN
-F 2 "Resistors_SMD:R_0402" V 1180 5400 50  0001 C CNN
+F 2 "Resistor_SMD:R_0402_1005Metric" V 1180 5400 50  0001 C CNN
 F 3 "" H 1250 5400 50  0001 C CNN
 F 4 "1" V 1250 5400 60  0001 C CNN "Populated"
@@
 F 0 "R1308" V 1480 5400 50  0000 C CNN
 F 1 "0" V 1400 5400 50  0000 C CNN
-F 2 "Resistors_SMD:R_0402" V 1330 5400 50  0001 C CNN
+F 2 "Resistor_SMD:R_0402_1005Metric" V 1330 5400 50  0001 C CNN
 F 3 "" H 1400 5400 50  0001 C CNN
 F 4 "1" V 1400 5400 60  0001 C CNN "Populated"
@@
 F 0 "R1310" V 1630 5400 50  0000 C CNN
 F 1 "0" V 1550 5400 50  0000 C CNN
-F 2 "Resistors_SMD:R_0402" V 1480 5400 50  0001 C CNN
+F 2 "Resistor_SMD:R_0402_1005Metric" V 1480 5400 50  0001 C CNN
 F 3 "" H 1550 5400 50  0001 C CNN
 F 4 "1" V 1550 5400 60  0001 C CNN "Populated"
@@
 F 0 "R1313" V 3530 3450 50  0000 C CNN
 F 1 "DNP" V 3450 3450 50  0000 C CNN
-F 2 "Resistors_SMD:R_0402" V 3380 3450 50  0001 C CNN
+F 2 "Resistor_SMD:R_0402_1005Metric" V 3380 3450 50  0001 C CNN
 F 3 "" H 3450 3450 50  0001 C CNN
 F 4 "0" V 3450 3450 60  0001 C CNN "Populated"
@@
 F 0 "R1320" V 7630 3350 50  0000 C CNN
 F 1 "R" V 7550 3350 50  0000 C CNN
-F 2 "Resistors_SMD:R_0402" V 7480 3350 50  0001 C CNN
+F 2 "Resistor_SMD:R_0402_1005Metric" V 7480 3350 50  0001 C CNN
 F 3 "" H 7550 3350 50  0001 C CNN
 F 4 "1" V 7550 3350 60  0001 C CNN "Populated"
@@
 F 0 "R1315" V 6780 3550 50  0000 C CNN
 F 1 "R" V 6700 3550 50  0000 C CNN
-F 2 "Resistors_SMD:R_0402" V 6630 3550 50  0001 C CNN
+F 2 "Resistor_SMD:R_0402_1005Metric" V 6630 3550 50  0001 C CNN
 F 3 "" H 6700 3550 50  0001 C CNN
 F 4 "1" V 6700 3550 60  0001 C CNN "Populated"
@@
 F 0 "R1318" V 7030 3650 50  0000 C CNN
 F 1 "R" V 6950 3650 50  0000 C CNN
-F 2 "Resistors_SMD:R_0402" V 6880 3650 50  0001 C CNN
+F 2 "Resistor_SMD:R_0402_1005Metric" V 6880 3650 50  0001 C CNN
 F 3 "" H 6950 3650 50  0001 C CNN
 F 4 "1" V 6950 3650 60  0001 C CNN "Populated"
@@
 F 0 "R1316" V 6780 3750 50  0000 C CNN
 F 1 "R" V 6700 3750 50  0000 C CNN
-F 2 "Resistors_SMD:R_0402" V 6630 3750 50  0001 C CNN
+F 2 "Resistor_SMD:R_0402_1005Metric" V 6630 3750 50  0001 C CNN
 F 3 "" H 6700 3750 50  0001 C CNN
 F 4 "1" V 6700 3750 60  0001 C CNN "Populated"
@@
 F 0 "R1319" V 7030 3850 50  0000 C CNN
 F 1 "R" V 6950 3850 50  0000 C CNN
-F 2 "Resistors_SMD:R_0402" V 6880 3850 50  0001 C CNN
+F 2 "Resistor_SMD:R_0402_1005Metric" V 6880 3850 50  0001 C CNN
 F 3 "" H 6950 3850 50  0001 C CNN
 F 4 "1" V 6950 3850 60  0001 C CNN "Populated"
@@
 F 0 "R1317" V 7030 3450 50  0000 C CNN
 F 1 "DNP" V 6950 3450 50  0000 C CNN
-F 2 "Resistors_SMD:R_0402" V 6880 3450 50  0001 C CNN
+F 2 "Resistor_SMD:R_0402_1005Metric" V 6880 3450 50  0001 C CNN
 F 3 "" H 6950 3450 50  0001 C CNN
 F 4 "0" V 6950 3450 60  0001 C CNN "Populated"
@@
 F 0 "R1311" V 2930 4250 50  0000 C CNN
 F 1 "R" V 2850 4250 50  0000 C CNN
-F 2 "Resistors_SMD:R_0402" V 2780 4250 50  0001 C CNN
+F 2 "Resistor_SMD:R_0402_1005Metric" V 2780 4250 50  0001 C CNN
 F 3 "" H 2850 4250 50  0001 C CNN
 F 4 "1" V 2850 4250 60  0001 C CNN "Populated"
@@
 F 0 "R1302" V 1030 5400 50  0000 C CNN
 F 1 "0" V 950 5400 50  0000 C CNN
-F 2 "Resistors_SMD:R_0402" V 880 5400 50  0001 C CNN
+F 2 "Resistor_SMD:R_0402_1005Metric" V 880 5400 50  0001 C CNN
 F 3 "" H 950 5400 50  0001 C CNN
 F 4 "1" V 950 5400 60  0001 C CNN "Populated"
@@
 F 0 "R1301" V 1030 4500 50  0000 C CNN
 F 1 "DNP" V 950 4500 50  0000 C CNN
-F 2 "Resistors_SMD:R_0402" V 880 4500 50  0001 C CNN
+F 2 "Resistor_SMD:R_0402_1005Metric" V 880 4500 50  0001 C CNN
 F 3 "" H 950 4500 50  0001 C CNN
 F 4 "0" V 950 4500 60  0001 C CNN "Populated"
@@
 F 0 "R1312" V 3230 5750 50  0000 C CNN
 F 1 "2k" V 3150 5750 50  0000 C CNN
-F 2 "Resistors_SMD:R_0402" V 3080 5750 50  0001 C CNN
+F 2 "Resistor_SMD:R_0402_1005Metric" V 3080 5750 50  0001 C CNN
 F 3 "" H 3150 5750 50  0001 C CNN
 F 4 "1" V 3150 5750 60  0001 C CNN "Populated"
