File: hardware/TLK10031.sch (KiCad schematic (older format))
At the start: 44 parts, among them J1301 TEST_1P, J1302 TEST_1P, J1303 Conn_01x06, U1201 TLK10031

Commit message: Improved Powerdistribution Network of the FPGA.
Also started to layout USB.
Parts:
- C1301, C1302, C1303, C1304, C1305, C1306, C1307, C1308, C1309, C1310, C1311, C1312, C1313, C1314, C1315, C1316, C1317, C1318: footprint Capacitors_SMD:C_0201 -> Capacitor_SMD:C_0201_0603Metric
- C1319, C1320: footprint Capacitors_SMD:C_0402 -> Capacitor_SMD:C_0402_1005Metric
Changed lines of the file:
@@
 F 0 "C1301" V 2450 1100 50  0000 L CNN
 F 1 "100 nF" V 2350 1100 50  0000 L CNN
-F 2 "Capacitors_SMD:C_0201" H 2400 1050 50  0001 C CNN
+F 2 "Capacitor_SMD:C_0201_0603Metric" H 2400 1050 50  0001 C CNN
 F 3 "http://search.murata.co.jp/Ceramy/image/img/A01X/G101/ENG/GRM033R60J104KE19-01.pdf" H 2400 1050 50  0001 C CNN
 F 4 "Murata Electronics North America" H 2400 1050 60  0001 C CNN "MFG Name"
@@
 F 0 "C1319" H 3710 3320 50  0000 L CNN
 F 1 "DNP" H 3710 3170 50  0000 L CNN
-F 2 "Capacitors_SMD:C_0402" H 3700 3250 50  0001 C CNN
+F 2 "Capacitor_SMD:C_0402_1005Metric" H 3700 3250 50  0001 C CNN
 F 3 "" H 3700 3250 50  0001 C CNN
 F 4 "0" H 3700 3250 60  0001 C CNN "Populated"
@@
 F 0 "C1320" H 3710 3720 50  0000 L CNN
 F 1 "DNP" H 3710 3570 50  0000 L CNN
-F 2 "Capacitors_SMD:C_0402" H 3700 3650 50  0001 C CNN
+F 2 "Capacitor_SMD:C_0402_1005Metric" H 3700 3650 50  0001 C CNN
 F 3 "" H 3700 3650 50  0001 C CNN
 	1    3700 3650
@@
 F 0 "C1306" V 2700 1200 50  0000 L CNN
 F 1 "100 nF" V 2600 1200 50  0000 L CNN
-F 2 "Capacitors_SMD:C_0201" H 2650 1150 50  0001 C CNN
+F 2 "Capacitor_SMD:C_0201_0603Metric" H 2650 1150 50  0001 C CNN
 F 3 "http://search.murata.co.jp/Ceramy/image/img/A01X/G101/ENG/GRM033R60J104KE19-01.pdf" H 2650 1150 50  0001 C CNN
 F 4 "Murata Electronics North America" H 2650 1150 60  0001 C CNN "MFG Name"
@@
 F 0 "C1311" V 2950 1300 50  0000 L CNN
 F 1 "100 nF" V 2850 1300 50  0000 L CNN
-F 2 "Capacitors_SMD:C_0201" H 2900 1250 50  0001 C CNN
+F 2 "Capacitor_SMD:C_0201_0603Metric" H 2900 1250 50  0001 C CNN
 F 3 "http://search.murata.co.jp/Ceramy/image/img/A01X/G101/ENG/GRM033R60J104KE19-01.pdf" H 2900 1250 50  0001 C CNN
 F 4 "Murata Electronics North America" H 2900 1250 60  0001 C CNN "MFG Name"
@@
 F 0 "C1315" V 3200 1400 50  0000 L CNN
 F 1 "100 nF" V 3100 1400 50  0000 L CNN
-F 2 "Capacitors_SMD:C_0201" H 3150 1350 50  0001 C CNN
+F 2 "Capacitor_SMD:C_0201_0603Metric" H 3150 1350 50  0001 C CNN
 F 3 "http://search.murata.co.jp/Ceramy/image/img/A01X/G101/ENG/GRM033R60J104KE19-01.pdf" H 3150 1350 50  0001 C CNN
 F 4 "Murata Electronics North America" H 3150 1350 60  0001 C CNN "MFG Name"
@@
 F 0 "C1302" V 2450 1500 50  0000 L CNN
 F 1 "100 nF" V 2350 1500 50  0000 L CNN
-F 2 "Capacitors_SMD:C_0201" H 2400 1450 50  0001 C CNN
+F 2 "Capacitor_SMD:C_0201_0603Metric" H 2400 1450 50  0001 C CNN
 F 3 "http://search.murata.co.jp/Ceramy/image/img/A01X/G101/ENG/GRM033R60J104KE19-01.pdf" H 2400 1450 50  0001 C CNN
 F 4 "Murata Electronics North America" H 2400 1450 60  0001 C CNN "MFG Name"
@@
 F 0 "C1307" V 2700 1600 50  0000 L CNN
 F 1 "100 nF" V 2600 1600 50  0000 L CNN
-F 2 "Capacitors_SMD:C_0201" H 2650 1550 50  0001 C CNN
+F 2 "Capacitor_SMD:C_0201_0603Metric" H 2650 1550 50  0001 C CNN
 F 3 "http://search.murata.co.jp/Ceramy/image/img/A01X/G101/ENG/GRM033R60J104KE19-01.pdf" H 2650 1550 50  0001 C CNN
 F 4 "Murata Electronics North America" H 2650 1550 60  0001 C CNN "MFG Name"
@@
 F 0 "C1312" V 2950 1700 50  0000 L CNN
 F 1 "100 nF" V 2850 1700 50  0000 L CNN
-F 2 "Capacitors_SMD:C_0201" H 2900 1650 50  0001 C CNN
+F 2 "Capacitor_SMD:C_0201_0603Metric" H 2900 1650 50  0001 C CNN
 F 3 "http://search.murata.co.jp/Ceramy/image/img/A01X/G101/ENG/GRM033R60J104KE19-01.pdf" H 2900 1650 50  0001 C CNN
 F 4 "Murata Electronics North America" H 2900 1650 60  0001 C CNN "MFG Name"
@@
 F 0 "C1316" V 3200 1800 50  0000 L CNN
 F 1 "100 nF" V 3100 1800 50  0000 L CNN
-F 2 "Capacitors_SMD:C_0201" H 3150 1750 50  0001 C CNN
+F 2 "Capacitor_SMD:C_0201_0603Metric" H 3150 1750 50  0001 C CNN
 F 3 "http://search.murata.co.jp/Ceramy/image/img/A01X/G101/ENG/GRM033R60J104KE19-01.pdf" H 3150 1750 50  0001 C CNN
 F 4 "Murata Electronics North America" H 3150 1750 60  0001 C CNN "MFG Name"
@@
 F 0 "C1303" V 2450 1950 50  0000 L CNN
 F 1 "100 nF" V 2350 1950 50  0000 L CNN
-F 2 "Capacitors_SMD:C_0201" H 2400 1900 50  0001 C CNN
+F 2 "Capacitor_SMD:C_0201_0603Metric" H 2400 1900 50  0001 C CNN
 F 3 "http://search.murata.co.jp/Ceramy/image/img/A01X/G101/ENG/GRM033R60J104KE19-01.pdf" H 2400 1900 50  0001 C CNN
 F 4 "Murata Electronics North America" H 2400 1900 60  0001 C CNN "MFG Name"
@@
 F 0 "C1308" V 2700 2050 50  0000 L CNN
 F 1 "100 nF" V 2600 2050 50  0000 L CNN
-F 2 "Capacitors_SMD:C_0201" H 2650 2000 50  0001 C CNN
+F 2 "Capacitor_SMD:C_0201_0603Metric" H 2650 2000 50  0001 C CNN
 F 3 "http://search.murata.co.jp/Ceramy/image/img/A01X/G101/ENG/GRM033R60J104KE19-01.pdf" H 2650 2000 50  0001 C CNN
 F 4 "Murata Electronics North America" H 2650 2000 60  0001 C CNN "MFG Name"
@@
 F 0 "C1313" V 2950 2150 50  0000 L CNN
 F 1 "100 nF" V 2850 2150 50  0000 L CNN
-F 2 "Capacitors_SMD:C_0201" H 2900 2100 50  0001 C CNN
+F 2 "Capacitor_SMD:C_0201_0603Metric" H 2900 2100 50  0001 C CNN
 F 3 "http://search.murata.co.jp/Ceramy/image/img/A01X/G101/ENG/GRM033R60J104KE19-01.pdf" H 2900 2100 50  0001 C CNN
 F 4 "Murata Electronics North America" H 2900 2100 60  0001 C CNN "MFG Name"
@@
 F 0 "C1317" V 3200 2250 50  0000 L CNN
 F 1 "100 nF" V 3100 2250 50  0000 L CNN
-F 2 "Capacitors_SMD:C_0201" H 3150 2200 50  0001 C CNN
+F 2 "Capacitor_SMD:C_0201_0603Metric" H 3150 2200 50  0001 C CNN
 F 3 "http://search.murata.co.jp/Ceramy/image/img/A01X/G101/ENG/GRM033R60J104KE19-01.pdf" H 3150 2200 50  0001 C CNN
 F 4 "Murata Electronics North America" H 3150 2200 60  0001 C CNN "MFG Name"
@@
 F 0 "C1304" V 2450 2350 50  0000 L CNN
 F 1 "100 nF" V 2350 2350 50  0000 L CNN
-F 2 "Capacitors_SMD:C_0201" H 2400 2300 50  0001 C CNN
+F 2 "Capacitor_SMD:C_0201_0603Metric" H 2400 2300 50  0001 C CNN
 F 3 "http://search.murata.co.jp/Ceramy/image/img/A01X/G101/ENG/GRM033R60J104KE19-01.pdf" H 2400 2300 50  0001 C CNN
 F 4 "Murata Electronics North America" H 2400 2300 60  0001 C CNN "MFG Name"
@@
 F 0 "C1309" V 2700 2450 50  0000 L CNN
 F 1 "100 nF" V 2600 2450 50  0000 L CNN
-F 2 "Capacitors_SMD:C_0201" H 2650 2400 50  0001 C CNN
+F 2 "Capacitor_SMD:C_0201_0603Metric" H 2650 2400 50  0001 C CNN
 F 3 "http://search.murata.co.jp/Ceramy/image/img/A01X/G101/ENG/GRM033R60J104KE19-01.pdf" H 2650 2400 50  0001 C CNN
 F 4 "Murata Electronics North America" H 2650 2400 60  0001 C CNN "MFG Name"
@@
 F 0 "C1314" V 2950 2550 50  0000 L CNN
 F 1 "100 nF" V 2850 2550 50  0000 L CNN
-F 2 "Capacitors_SMD:C_0201" H 2900 2500 50  0001 C CNN
+F 2 "Capacitor_SMD:C_0201_0603Metric" H 2900 2500 50  0001 C CNN
 F 3 "http://search.murata.co.jp/Ceramy/image/img/A01X/G101/ENG/GRM033R60J104KE19-01.pdf" H 2900 2500 50  0001 C CNN
 F 4 "Murata Electronics North America" H 2900 2500 60  0001 C CNN "MFG Name"
@@
 F 0 "C1318" V 3200 2650 50  0000 L CNN
 F 1 "100 nF" V 3100 2650 50  0000 L CNN
-F 2 "Capacitors_SMD:C_0201" H 3150 2600 50  0001 C CNN
+F 2 "Capacitor_SMD:C_0201_0603Metric" H 3150 2600 50  0001 C CNN
 F 3 "http://search.murata.co.jp/Ceramy/image/img/A01X/G101/ENG/GRM033R60J104KE19-01.pdf" H 3150 2600 50  0001 C CNN
 F 4 "Murata Electronics North America" H 3150 2600 60  0001 C CNN "MFG Name"
@@
 F 0 "C1305" V 2450 2800 50  0000 L CNN
 F 1 "100 nF" V 2350 2800 50  0000 L CNN
-F 2 "Capacitors_SMD:C_0201" H 2400 2750 50  0001 C CNN
+F 2 "Capacitor_SMD:C_0201_0603Metric" H 2400 2750 50  0001 C CNN
 F 3 "http://search.murata.co.jp/Ceramy/image/img/A01X/G101/ENG/GRM033R60J104KE19-01.pdf" H 2400 2750 50  0001 C CNN
 F 4 "Murata Electronics North America" H 2400 2750 60  0001 C CNN "MFG Name"
@@
 F 0 "C1310" V 2700 2900 50  0000 L CNN
 F 1 "100 nF" V 2600 2900 50  0000 L CNN
-F 2 "Capacitors_SMD:C_0201" H 2650 2850 50  0001 C CNN
+F 2 "Capacitor_SMD:C_0201_0603Metric" H 2650 2850 50  0001 C CNN
 F 3 "http://search.murata.co.jp/Ceramy/image/img/A01X/G101/ENG/GRM033R60J104KE19-01.pdf" H 2650 2850 50  0001 C CNN
 F 4 "Murata Electronics North America" H 2650 2850 60  0001 C CNN "MFG Name"

Commit message: Fixed Schematic Symbols
Parts:
- C1301, C1302, C1303, C1304, C1305, C1306, C1307, C1308, C1309, C1310, C1311, C1312, C1313, C1314, C1315, C1316, C1317, C1318, C1319, C1320: symbol device:C_Small -> Device:C_Small
- J1301, J1302: symbol conn:TEST_1P -> Connector:Test_Point
- J1303: symbol conn:Conn_01x06 -> Connector_Generic:Conn_01x06
- R1301, R1302, R1303, R1304, R1305, R1306, R1307, R1308, R1309, R1310, R1311, R1312, R1313, R1314, R1315, R1316, R1317, R1318, R1319, R1320: symbol device:R -> Device:R
Changed lines of the file:
@@
 $Descr A4 11693 8268
 encoding utf-8
-Sheet 13 22
+Sheet 13 21
 Title ""
 Date ""
@@
 INA[0]_N
 $Comp
-L device:C_Small C1301
+L Device:C_Small C1301
 U 1 1 5ACAE246
 P 2400 1050
@@
 OUTA[0]_N
 $Comp
-L device:R R1314
+L Device:R R1314
 U 1 1 5ACB0AA4
 P 3600 3050
@@
 $EndComp
 $Comp
-L power1:GND #PWR0144
+L power:GND #PWR0144
 U 1 1 5ACB0BCF
 P 3350 3050
@@
 HSRXA_N
 $Comp
-L power1:GND #PWR0145
+L power:GND #PWR0145
 U 1 1 5ACC67F6
 P 3950 5300
@@
 $EndComp
 $Comp
-L device:R R1303
+L Device:R R1303
 U 1 1 5ACCADAC
 P 1100 4500
@@
 $EndComp
 $Comp
-L device:R R1305
+L Device:R R1305
 U 1 1 5ACCAF62
 P 1250 4500
@@
 $EndComp
 $Comp
-L device:R R1307
+L Device:R R1307
 U 1 1 5ACCB198
 P 1400 4500
@@
 $EndComp
 $Comp
-L device:R R1309
+L Device:R R1309
 U 1 1 5ACCB19E
 P 1550 4500
@@
 $EndComp
 $Comp
-L device:R R1304
+L Device:R R1304
 U 1 1 5ACCB916
 P 1100 5400
@@
 $EndComp
 $Comp
-L device:R R1306
+L Device:R R1306
 U 1 1 5ACCB9E9
 P 1250 5400
@@
 $EndComp
 $Comp
-L device:R R1308
+L Device:R R1308
 U 1 1 5ACCBA49
 P 1400 5400
@@
 $EndComp
 $Comp
-L device:R R1310
+L Device:R R1310
 U 1 1 5ACCBAB0
 P 1550 5400
@@
 $EndComp
 $Comp
-L power1:GND #PWR0146
+L power:GND #PWR0146
 U 1 1 5ACCBE2D
 P 1250 5750
@@
 $EndComp
 $Comp
-L device:C_Small C1319
+L Device:C_Small C1319
 U 1 1 5ACCC8EE
 P 3700 3250
@@
 $EndComp
 $Comp
-L device:C_Small C1320
+L Device:C_Small C1320
 U 1 1 5ACCC9AB
 P 3700 3650
@@
 $EndComp
 $Comp
-L device:R R1313
+L Device:R R1313
 U 1 1 5ACCCAE1
 P 3450 3450
@@
 MDC
 $Comp
-L conn:Conn_01x06 J1303
+L Connector_Generic:Conn_01x06 J1303
 U 1 1 5AC7786C
 P 8050 3050
@@
 $EndComp
 $Comp
-L power1:GND #PWR0147
+L power:GND #PWR0147
 U 1 1 5AC77C0F
 P 7750 3450
@@
 $EndComp
 $Comp
-L device:R R1320
+L Device:R R1320
 U 1 1 5AC79DD9
 P 7550 3350
@@
 $EndComp
 $Comp
-L device:R R1315
+L Device:R R1315
 U 1 1 5AC7A06C
 P 6700 3550
@@
 $EndComp
 $Comp
-L device:R R1318
+L Device:R R1318
 U 1 1 5AC7A140
 P 6950 3650
@@
 $EndComp
 $Comp
-L device:R R1316
+L Device:R R1316
 U 1 1 5AC7A1F2
 P 6700 3750
@@
 $EndComp
 $Comp
-L device:R R1319
+L Device:R R1319
 U 1 1 5AC7A28E
 P 6950 3850
@@
 $EndComp
 $Comp
-L device:R R1317
+L Device:R R1317
 U 1 1 5AC7A32D
 P 6950 3450
@@
 Same as VDDO
 $Comp
-L power1:GND #PWR0148
+L power:GND #PWR0148
 U 1 1 5AC7C5FF
 P 7300 3650
@@
 What to do with\nunsed output clocks?
 $Comp
-L conn:TEST_1P J1301
+L Connector:Test_Point J1301
 U 1 1 5AC7FBF4
 P 2450 3950
@@
 $EndComp
 $Comp
-L device:R R1311
+L Device:R R1311
 U 1 1 5AC82864
 P 2850 4250
@@
 Same as VDDO
 $Comp
-L conn:TEST_1P J1302
+L Connector:Test_Point J1302
 U 1 1 5AC8C54E
 P 2450 4550
@@
 	2450 4550 3950 4550
 $Comp
-L device:R R1302
+L Device:R R1302
 U 1 1 5AC8C9C3
 P 950 5400
@@
 $EndComp
 $Comp
-L device:R R1301
+L Device:R R1301
 U 1 1 5AC8CA81
 P 950 4500
@@
 	2450 5650 3400 5650
 $Comp
-L device:R R1312
+L Device:R R1312
 U 1 1 5AC9120F
 P 3150 5750
@@
 	2300 2750 2150 2750
 $Comp
-L power1:+1V8 #PWR0149
+L power:+1V8 #PWR0149
 U 1 1 5AC92C58
 P 2450 4250
@@
 $EndComp
 $Comp
-L power1:+1V8 #PWR0150
+L power:+1V8 #PWR0150
 U 1 1 5AC92CEE
 P 1250 4100
@@
 $EndComp
 $Comp
-L power1:+1V8 #PWR0151
+L power:+1V8 #PWR0151
 U 1 1 5AC92E59
 P 2900 5750
@@
 $EndComp
 $Comp
-L power1:+1V8 #PWR0152
+L power:+1V8 #PWR0152
 U 1 1 5AC92F40
 P 7100 3450
@@
 HSRXA_N
 $Comp
-L device:C_Small C1306
+L Device:C_Small C1306
 U 1 1 5AE3C4AB
 P 2650 1150
@@
 $EndComp
 $Comp
-L device:C_Small C1311
+L Device:C_Small C1311
 U 1 1 5AE3C523
 P 2900 1250
@@
 $EndComp
 $Comp
-L device:C_Small C1315
+L Device:C_Small C1315
 U 1 1 5AE3C59E
 P 3150 1350
@@
 $EndComp
 $Comp
-L device:C_Small C1302
+L Device:C_Small C1302
 U 1 1 5AE3C61E
 P 2400 1450
@@
 $EndComp
 $Comp
-L device:C_Small C1307
+L Device:C_Small C1307
 U 1 1 5AE3C728
 P 2650 1550
@@
 $EndComp
 $Comp
-L device:C_Small C1312
+L Device:C_Small C1312
 U 1 1 5AE3C7AA
 P 2900 1650
@@
 $EndComp
 $Comp
-L device:C_Small C1316
+L Device:C_Small C1316
 U 1 1 5AE3C833
 P 3150 1750
@@
 $EndComp
 $Comp
-L device:C_Small C1303
+L Device:C_Small C1303
 U 1 1 5AE3C8C1
 P 2400 1900
@@
 $EndComp
 $Comp
-L device:C_Small C1308
+L Device:C_Small C1308
 U 1 1 5AE3C960
 P 2650 2000
@@
 $EndComp
 $Comp
-L device:C_Small C1313
+L Device:C_Small C1313
 U 1 1 5AE3CA70
 P 2900 2100
@@
 $EndComp
 $Comp
-L device:C_Small C1317
+L Device:C_Small C1317
 U 1 1 5AE3CB13
 P 3150 2200
@@
 $EndComp
 $Comp
-L device:C_Small C1304
+L Device:C_Small C1304
 U 1 1 5AE3CBAD
 P 2400 2300
@@
 $EndComp
 $Comp
-L device:C_Small C1309
+L Device:C_Small C1309
 U 1 1 5AE3CC68
 P 2650 2400
@@
 $EndComp
 $Comp
-L device:C_Small C1314
+L Device:C_Small C1314
 U 1 1 5AE3CD12
 P 2900 2500
@@
 $EndComp
 $Comp
-L device:C_Small C1318
+L Device:C_Small C1318
 U 1 1 5AE3CDAF
 P 3150 2600
@@
 $EndComp
 $Comp
-L device:C_Small C1305
+L Device:C_Small C1305
 U 1 1 5AE3CE51
 P 2400 2750
@@
 $EndComp
 $Comp
-L device:C_Small C1310
+L Device:C_Small C1310
 U 1 1 5AE3CF12
 P 2650 2850

Commit message: Xaui lanes
Parts:
- removed J1303: Conn_01x06, symbol Connector_Generic:Conn_01x06
- added J1201, J1202, J1203, J1204, J1205: TEST_1P, footprints:TestPoint_SMD_0.5mm, symbol Connector:Test_Point
- J1301, J1302: footprint (none) -> footprints:TestPoint_SMD_0.5mm; Populate for CLG484(Z-7012s/Z-7015) (none) -> 1; Populate for SBGA485(Z-7030) (none) -> 1; Populated (none) -> 1; Source (none) -> SPEC
Connections:
- net labels added: OC_N, OC_P
- no-connect marks 0 -> 1
Changed lines of the file:
@@
 MDC
-$Comp
-L Connector_Generic:Conn_01x06 J1303
-U 1 1 5AC7786C
-P 8050 3050
-F 0 "J1303" H 8050 3350 50  0000 C CNN
-F 1 "Conn_01x06" H 8050 2650 50  0000 C CNN
-F 2 "" H 8050 3050 50  0001 C CNN
-F 3 "" H 8050 3050 50  0001 C CNN
-	1    8050 3050
-	1    0    0    -1
-$EndComp
 $Comp
 L power:GND #PWR0147
@@
 P 2450 3950
 F 0 "J1301" H 2450 4220 50  0000 C CNN
-F 1 "TEST_1P" H 2450 4150 50  0000 C CNN
-F 2 "" H 2650 3950 50  0001 C CNN
+F 1 "TEST_1P" H 2450 4150 50  0001 C CNN
+F 2 "footprints:TestPoint_SMD_0.5mm" H 2650 3950 50  0001 C CNN
 F 3 "" H 2650 3950 50  0001 C CNN
+F 4 "1" H 2450 3950 50  0001 C CNN "Populated"
+F 5 "SPEC" H 2450 3950 50  0001 C CNN "Source"
+F 6 "1" H 2450 3950 50  0001 C CNN "Populate for SBGA485(Z-7030)"
+F 7 "1" H 2450 3950 50  0001 C CNN "Populate for CLG484(Z-7012s/Z-7015)"
 	1    2450 3950
 	0    -1   -1   0
@@
 P 2450 4550
 F 0 "J1302" H 2450 4820 50  0000 C CNN
-F 1 "TEST_1P" H 2450 4750 50  0000 C CNN
-F 2 "" H 2650 4550 50  0001 C CNN
+F 1 "TEST_1P" H 2450 4750 50  0001 C CNN
+F 2 "footprints:TestPoint_SMD_0.5mm" H 2650 4550 50  0001 C CNN
 F 3 "" H 2650 4550 50  0001 C CNN
+F 4 "1" H 2450 4550 50  0001 C CNN "Populated"
+F 5 "SPEC" H 2450 4550 50  0001 C CNN "Source"
+F 6 "1" H 2450 4550 50  0001 C CNN "Populate for SBGA485(Z-7030)"
+F 7 "1" H 2450 4550 50  0001 C CNN "Populate for CLG484(Z-7012s/Z-7015)"
 	1    2450 4550
 	0    -1   -1   0
@@
 Wire Wire Line
 	3400 5650 3950 5650
+$Comp
+L Connector:Test_Point J1201
+U 1 1 5B369D0D
+P 7850 2850
+F 0 "J1201" V 7850 3150 50  0000 C CNN
+F 1 "TEST_1P" H 7850 3050 50  0001 C CNN
+F 2 "footprints:TestPoint_SMD_0.5mm" H 8050 2850 50  0001 C CNN
+F 3 "" H 8050 2850 50  0001 C CNN
+F 4 "1" H 7850 2850 50  0001 C CNN "Populated"
+F 5 "SPEC" H 7850 2850 50  0001 C CNN "Source"
+F 6 "1" H 7850 2850 50  0001 C CNN "Populate for SBGA485(Z-7030)"
+F 7 "1" H 7850 2850 50  0001 C CNN "Populate for CLG484(Z-7012s/Z-7015)"
+	1    7850 2850
+	0    1    1    0
+$EndComp
+NoConn ~ 7850 3350
+$Comp
+L Connector:Test_Point J1202
+U 1 1 5B376607
+P 7850 2950
+F 0 "J1202" V 7850 3250 50  0000 C CNN
+F 1 "TEST_1P" H 7850 3150 50  0001 C CNN
+F 2 "footprints:TestPoint_SMD_0.5mm" H 8050 2950 50  0001 C CNN
+F 3 "" H 8050 2950 50  0001 C CNN
+F 4 "1" H 7850 2950 50  0001 C CNN "Populated"
+F 5 "SPEC" H 7850 2950 50  0001 C CNN "Source"
+F 6 "1" H 7850 2950 50  0001 C CNN "Populate for SBGA485(Z-7030)"
+F 7 "1" H 7850 2950 50  0001 C CNN "Populate for CLG484(Z-7012s/Z-7015)"
+	1    7850 2950
+	0    1    1    0
+$EndComp
+$Comp
+L Connector:Test_Point J1203
+U 1 1 5B376681
+P 7850 3050
+F 0 "J1203" V 7850 3350 50  0000 C CNN
+F 1 "TEST_1P" H 7850 3250 50  0001 C CNN
+F 2 "footprints:TestPoint_SMD_0.5mm" H 8050 3050 50  0001 C CNN
+F 3 "" H 8050 3050 50  0001 C CNN
+F 4 "1" H 7850 3050 50  0001 C CNN "Populated"
+F 5 "SPEC" H 7850 3050 50  0001 C CNN "Source"
+F 6 "1" H 7850 3050 50  0001 C CNN "Populate for SBGA485(Z-7030)"
+F 7 "1" H 7850 3050 50  0001 C CNN "Populate for CLG484(Z-7012s/Z-7015)"
+	1    7850 3050
+	0    1    1    0
+$EndComp
+$Comp
+L Connector:Test_Point J1204
+U 1 1 5B3766FB
+P 7850 3150
+F 0 "J1204" V 7850 3450 50  0000 C CNN
+F 1 "TEST_1P" H 7850 3350 50  0001 C CNN
+F 2 "footprints:TestPoint_SMD_0.5mm" H 8050 3150 50  0001 C CNN
+F 3 "" H 8050 3150 50  0001 C CNN
+F 4 "1" H 7850 3150 50  0001 C CNN "Populated"
+F 5 "SPEC" H 7850 3150 50  0001 C CNN "Source"
+F 6 "1" H 7850 3150 50  0001 C CNN "Populate for SBGA485(Z-7030)"
+F 7 "1" H 7850 3150 50  0001 C CNN "Populate for CLG484(Z-7012s/Z-7015)"
+	1    7850 3150
+	0    1    1    0
+$EndComp
+$Comp
+L Connector:Test_Point J1205
+U 1 1 5B376775
+P 7850 3250
+F 0 "J1205" V 7850 3550 50  0000 C CNN
+F 1 "TEST_1P" H 7850 3450 50  0001 C CNN
+F 2 "footprints:TestPoint_SMD_0.5mm" H 8050 3250 50  0001 C CNN
+F 3 "" H 8050 3250 50  0001 C CNN
+F 4 "1" H 7850 3250 50  0001 C CNN "Populated"
+F 5 "SPEC" H 7850 3250 50  0001 C CNN "Source"
+F 6 "1" H 7850 3250 50  0001 C CNN "Populate for SBGA485(Z-7030)"
+F 7 "1" H 7850 3250 50  0001 C CNN "Populate for CLG484(Z-7012s/Z-7015)"
+	1    7850 3250
+	0    1    1    0
+$EndComp
+Text Label 3850 3250 0    50   ~ 0
+OC_P
+Text Label 3900 3600 1    50   ~ 0
+OC_N
 $EndSCHEMATC

Commit message: SFP+ Power Filter, Levelshifter and MGT/TLK Clock Distribution.
Connections:
- net labels added: REFCLK_N, REFCLK_P
Changed lines of the file:
@@
 Text Label 3900 3600 1    50   ~ 0
 OC_N
+Text Label 3600 2750 0    50   ~ 0
+REFCLK_P
+Text Label 3600 2850 0    50   ~ 0
+REFCLK_N
 $EndSCHEMATC
