File: hardware/TLK10031.sch (KiCad schematic (older format))
At the start: 48 parts, among them J1201 TEST_1P, J1202 TEST_1P, J1203 TEST_1P, J1204 TEST_1P, J1205 TEST_1P, J1301 TEST_1P, J1302 TEST_1P, U1201 TLK10031

Commit message: WIP: routing the HF Part of the Camera Connector. I have to move the clock away from the left border.
TODO: Fix DDR3 RAM.
Parts:
- U1201: Populate for CLG484(Z-7012s/Z-7015) (none) -> 1; Populate for SBGA485(Z-7030) (none) -> 1
Connections:
- net labels added: REFCLK_TLK_N, REFCLK_TLK_P, ~TLK_RESET_18~
- net labels removed: REFCLK0_N, REFCLK0_P, ~TLK_RESET~
- wire segments 130 -> 129
Changed lines of the file:
@@
 $Descr A4 11693 8268
 encoding utf-8
-Sheet 12 21
+Sheet 11 21
 Title ""
 Date ""
@@
 F 8 "1" H 5150 3450 60  0001 C CNN "Populated"
 F 9 "SPEC" H 5150 3450 60  0001 C CNN "Source"
+F 10 "1" H 5150 3450 50  0001 C CNN "Populate for SBGA485(Z-7030)"
+F 11 "1" H 5150 3450 50  0001 C CNN "Populate for CLG484(Z-7012s/Z-7015)"
 	1    5150 3450
 	1    0    0    -1
@@
 Text Notes 1250 3150 0    60   ~ 0
 Not used Ref Clocks should be grounded\nthrough an shared 100 Ω Resistor
-Text HLabel 2150 2750 0    60   Input ~ 0
-REFCLK0_P
-Text HLabel 2150 2850 0    60   Input ~ 0
-REFCLK0_N
 Text HLabel 7100 1050 2    60   Output ~ 0
 HSTXA_P
@@
 Text Notes 3700 5400 2    60   ~ 0
 TLK10031 only supports\n4 Bit MDIO Addresses
-Text HLabel 2450 5450 0    60   Input ~ 0
-~TLK_RESET~
 Text HLabel 2450 5550 0    60   Input ~ 0
 MDC
@@
 Text Notes 7650 1350 0    60   ~ 0
 AC-coupling Capacitors\nare inside the SFP+ Module
-Wire Wire Line
-	2450 5450 3950 5450
 Wire Wire Line
 	3950 5550 2450 5550
@@
 Text Label 3600 2850 0    50   ~ 0
 REFCLK_N
+Text GLabel 3950 5450 0    50   Input ~ 0
+~TLK_RESET_18~
+Text GLabel 2150 2850 0    50   Input ~ 0
+REFCLK_TLK_N
+Text GLabel 2150 2750 0    50   Input ~ 0
+REFCLK_TLK_P
 $EndSCHEMATC

Commit message: Added Courtyard to selfmade Footprints. Also general Routing WIP.
Other:
- note added: "TODO: Needs MDC an Pull-UP? AFAIK it does"
- note removed: "TODO: Select Footprint for JTAG Connector.\nFor Just in Case. We don't have enough information to do even an\nboundary scan. So it may not be useful ...."
- note removed: "What to do with\nunsed output clocks?"
Changed lines of the file:
@@
 EESchema Schematic File Version 4
+LIBS:zynq_board-cache
 EELAYER 26 0
 EELAYER END
@@
 	0    -1   -1   0
 $EndComp
-Text Notes 3750 3550 0    60   ~ 0
-What to do with\nunsed output clocks?
 $Comp
 L Connector:Test_Point J1301
@@
 	0    1    1    0
 $EndComp
-Text Notes 1350 7600 0    60   ~ 0
-TODO: Select Footprint for JTAG Connector.\nFor Just in Case. We don't have enough information to do even an\nboundary scan. So it may not be useful ....
 Wire Wire Line
 	3900 3050 3900 3100
@@
 Text GLabel 2150 2750 0    50   Input ~ 0
 REFCLK_TLK_P
+Text Notes 1900 6350 0    50   ~ 0
+TODO: Needs MDC an Pull-UP? AFAIK it does
 $EndSCHEMATC

Commit message: WIP: general Routing
Other:
- note added: "TODO: Needs MDC an Pull-UP? AFAIK it does not,\nbecause MDC is driven Push-Pull by the FPGA GPIO"
- note removed: "TODO: Needs MDC an Pull-UP? AFAIK it does"
Changed lines of the file:
@@
 REFCLK_TLK_P
 Text Notes 1900 6350 0    50   ~ 0
-TODO: Needs MDC an Pull-UP? AFAIK it does
+TODO: Needs MDC an Pull-UP? AFAIK it does not,\nbecause MDC is driven Push-Pull by the FPGA GPIO
 $EndSCHEMATC

Commit message: Routed extra GPIO Solder Pads, reannotated the whole schematic to make it consistent.
Power Distribution routing WIP
Parts:
- renumbered C1301 to C1101, C1302 to C1102, C1303 to C1103, C1304 to C1104, C1305 to C1105, C1306 to C1106, C1307 to C1107, C1308 to C1108, C1309 to C1109, C1310 to C1110, C1311 to C1111, C1312 to C1112, C1313 to C1113, C1314 to C1114, C1315 to C1115, C1316 to C1116, C1317 to C1117, C1318 to C1118, C1319 to C1119, C1320 to C1120, J1301 to J1101, J1302 to J1102, J1201 to J1103, J1202 to J1104, J1203 to J1105, J1204 to J1106, J1205 to J1107, R1301 to R1101, R1302 to R1102, R1303 to R1103, R1304 to R1104, R1305 to R1105, R1306 to R1106, R1307 to R1107, R1308 to R1108, R1309 to R1109, R1310 to R1110, R1311 to R1111, R1312 to R1112, R1313 to R1113, R1314 to R1114, R1315 to R1115, R1316 to R1116, R1317 to R1117, R1318 to R1118, R1319 to R1119, R1320 to R1120, U1201 to U1001

Commit message: general routing mainly power distribution, fixed some footprints
Connections:
- wire segments 129 -> 128
- no-connect marks 1 -> 0
Changed lines of the file:
@@
 Wire Wire Line
 	7750 3350 7750 3450
-Connection ~ 7750 3350
 Wire Wire Line
 	7350 3350 7350 3150
@@
 	1550 4900 1550 5250
 Wire Wire Line
-	7750 3350 7850 3350
-Wire Wire Line
 	7350 3150 6350 3150
 Wire Wire Line
@@
 	0    1    1    0
 $EndComp
-NoConn ~ 7850 3350
 $Comp
 L Connector:Test_Point J1104

Commit message: Add sym-lib-table and fp-lib-table, fixes for KiCad 5
Parts:
- J1101, J1102, J1103, J1104, J1105, J1106, J1107: symbol Connector:Test_Point -> Connector:TestPoint
Changed lines of the file:
@@
 $EndComp
 $Comp
-L Connector:Test_Point J1101
+L Connector:TestPoint J1101
 U 1 1 5AC7FBF4
 P 2450 3950
@@
 Same as VDDO
 $Comp
-L Connector:Test_Point J1102
+L Connector:TestPoint J1102
 U 1 1 5AC8C54E
 P 2450 4550
@@
 	3400 5650 3950 5650
 $Comp
-L Connector:Test_Point J1103
+L Connector:TestPoint J1103
 U 1 1 5B369D0D
 P 7850 2850
@@
 $EndComp
 $Comp
-L Connector:Test_Point J1104
+L Connector:TestPoint J1104
 U 1 1 5B376607
 P 7850 2950
@@
 $EndComp
 $Comp
-L Connector:Test_Point J1105
+L Connector:TestPoint J1105
 U 1 1 5B376681
 P 7850 3050
@@
 $EndComp
 $Comp
-L Connector:Test_Point J1106
+L Connector:TestPoint J1106
 U 1 1 5B3766FB
 P 7850 3150
@@
 $EndComp
 $Comp
-L Connector:Test_Point J1107
+L Connector:TestPoint J1107
 U 1 1 5B376775
 P 7850 3250

Commit message: Added Step Models, fixed some footprints(e.g. added solderpaste), cleaned up a bit
Parts:
- U1001: footprint footprints:TI-CTR_FCBGA_N144_12x12_13x13mm_Pitch1.0mm -> footprints:Texas_CTR_FCBGA_N144_12x12_13x13mm_Pitch1.0mm
Changed lines of the file:
@@
 EESchema Schematic File Version 4
 LIBS:zynq_board-cache
-EELAYER 26 0
+EELAYER 29 0
 EELAYER END
 $Descr A4 11693 8268
@@
 F 0 "U1001" H 5150 3400 60  0000 C CNN
 F 1 "TLK10031" H 5150 3500 60  0000 C CNN
-F 2 "footprints:TI-CTR_FCBGA_N144_12x12_13x13mm_Pitch1.0mm" H 4850 2950 60  0001 C CNN
+F 2 "footprints:Texas_CTR_FCBGA_N144_12x12_13x13mm_Pitch1.0mm" H 4850 2950 60  0001 C CNN
 F 3 "http://www.ti.com/lit/ds/symlink/tlk10031.pdf" H 4850 2950 60  0001 C CNN
 F 4 "Texas Instruments" H 5150 3450 60  0001 C CNN "MFG Name"
