File: hardware/usb_uart.sch (KiCad schematic (older format))
At the start: 20 parts, among them J1901 USB_OTG, U1901 SMP1255PUTG, U1902 FT234XD, U1903 SN74LV1T126, U1904 SN74LV1T126

Commit message: Layouted most of the Power Circuit and Triggerbus Levelshifters.
Added Footprint for Tantal Caps. Modified Footprint for MDR20 Connector, SD-Card.

Fixed Symbol and Circuit for Power Supervisor/Delay IC.

Also fixed some smaller things in the schematics.
Connections:
- net labels added: USB_UART_N, USB_UART_P
Changed lines of the file:
@@
 Wire Wire Line
 	4050 4550 3800 4550
+Text Label 2450 2900 0    50   ~ 0
+USB_UART_P
+Text Label 2450 3000 0    50   ~ 0
+USB_UART_N
 $EndSCHEMATC

Commit message: Layouted USB-UART.
Also moved USB-OTG to the right Side of the Board. To get there
some free Space, i moved the DDR3/Memory and the FPGA a few
Millimeters down.
Parts:
- added D1901: LED_ALT, LED_SMD:LED_0603_1608Metric, symbol Device:LED_ALT
- added R1906: 270, Resistor_SMD:R_0402_1005Metric, symbol device:R_Small
- C1901, C1906: footprint Capacitors_SMD:C_0402 -> Capacitor_SMD:C_0201_0603Metric; Description (none) -> CAP CER 10000PF 6.3V X5R 0201; Digikey (none) -> 490-17060-1-ND; MFG Name (none) -> Murata Electronics North America; MFG Part Num (none) -> GRM033R60J103KA01E; Populate for CLG484(Z-7012s/Z-7015) (none) -> 1; Populate for SBGA485(Z-7030) (none) -> 1; Voltage (none) -> 6,3 V
- C1902: value 4,7 µF -> 4.7µF; Description (none) -> CAP CER 4.7UF 10V X7R 0805; Digikey (none) -> 490-6479-1-ND; MFG Name (none) -> Murata; MFG Part Num (none) -> GRM21BR71A475KA73
- C1903, C1905: footprint Capacitors_SMD:C_0402 -> Capacitor_SMD:C_0201_0603Metric; Description (none) -> CAP CER 47PF 50V C0G/NP0 0201; MFG Name (none) -> Murata Electronics North America; MFG Part Num (none) -> GRM0335C1H470JA01D; Populate for CLG484(Z-7012s/Z-7015) (none) -> 1; Populate for SBGA485(Z-7030) (none) -> 1; Populated 0 -> DNP; Voltage (none) -> 50 V
- C1904, C1907, C1908, C1909: footprint Capacitors_SMD:C_0402 -> Capacitor_SMD:C_0201_0603Metric; Description (none) -> CAP CER 0.1UF 6.3V X5R 0201; Digikey (none) -> 490-3167-1-ND; MFG Name (none) -> Murata Electronics North America; MFG Part Num (none) -> GRM033R60J104KE19D; Populate for CLG484(Z-7012s/Z-7015) (none) -> 1; Populate for SBGA485(Z-7030) (none) -> 1
- R1901, R1902, R1903, R1904, R1905: footprint Resistors_SMD:R_0402 -> Resistor_SMD:R_0402_1005Metric
Connections:
- wire segments 73 -> 96
- no-connect marks 3 -> 2

Commit message: Improved Powerdistribution Network of the FPGA.
Also started to layout USB.
Parts:
- C1902: footprint Capacitors_SMD:C_0805 -> Capacitor_SMD:C_0805_2012Metric
Changed lines of the file:
@@
 F 0 "C1902" H 3460 2020 50  0000 L CNN
 F 1 "4.7µF" H 3460 1870 50  0000 L CNN
-F 2 "Capacitors_SMD:C_0805" H 3450 1950 50  0001 C CNN
+F 2 "Capacitor_SMD:C_0805_2012Metric" H 3450 1950 50  0001 C CNN
 F 3 "http://search.murata.co.jp/Ceramy/image/img/A01X/G101/ENG/GRM21BR71A475KA73-01.pdf" H 3450 1950 50  0001 C CNN
 F 4 "Murata" H 3450 1950 60  0001 C CNN "MFG Name"

Commit message: Fixed Schematic Symbols
Parts:
- C1901, C1902, C1903, C1904, C1905, C1906, C1907, C1908, C1909: symbol device:C_Small -> Device:C_Small
- J1901: symbol conn:USB_OTG -> Connector:USB_OTG
- L1901: symbol device:L_Small -> Device:L_Small
- R1901, R1902, R1903, R1904, R1905, R1906: symbol device:R_Small -> Device:R_Small
Changed lines of the file:
@@
 $Descr A4 11693 8268
 encoding utf-8
-Sheet 19 22
+Sheet 18 21
 Title ""
 Date ""
@@
 PS_UART_TX
 $Comp
-L conn:USB_OTG J1901
+L Connector:USB_OTG J1901
 U 1 1 5AD9C9C2
 P 1350 2900
@@
 $EndComp
 $Comp
-L device:R_Small R1902
+L Device:R_Small R1902
 U 1 1 5AD9CAF7
 P 4650 2900
@@
 $EndComp
 $Comp
-L device:R_Small R1903
+L Device:R_Small R1903
 U 1 1 5AD9CB9D
 P 4650 3000
@@
 $EndComp
 $Comp
-L power1:GND #PWR0246
+L power:GND #PWR0246
 U 1 1 5AD9D27D
 P 1300 3550
@@
 $EndComp
 $Comp
-L power1:GND #PWR0247
+L power:GND #PWR0247
 U 1 1 5AD9D2C5
 P 5600 3800
@@
 $EndComp
 $Comp
-L power1:GND #PWR0248
+L power:GND #PWR0248
 U 1 1 5AD9D3A1
 P 4400 2350
@@
 $EndComp
 $Comp
-L device:C_Small C1903
+L Device:C_Small C1903
 U 1 1 5AD9E9AF
 P 3550 3350
@@
 $EndComp
 $Comp
-L power1:GND #PWR0249
+L power:GND #PWR0249
 U 1 1 5AD9EB01
 P 3850 3650
@@
 $EndComp
 $Comp
-L power1:GND #PWR0250
+L power:GND #PWR0250
 U 1 1 5AD9EB21
 P 3550 3650
@@
 $EndComp
 $Comp
-L device:C_Small C1901
+L Device:C_Small C1901
 U 1 1 5AD9EC24
 P 3250 3350
@@
 $EndComp
 $Comp
-L power1:GND #PWR0251
+L power:GND #PWR0251
 U 1 1 5AD9EC9D
 P 3250 3650
@@
 $EndComp
 $Comp
-L device:L_Small L1901
+L Device:L_Small L1901
 U 1 1 5AD9ECD6
 P 3250 2500
@@
 VBUS
 $Comp
-L power1:GND #PWR0252
+L power:GND #PWR0252
 U 1 1 5ADA11B7
 P 3600 2250
@@
 $EndComp
 $Comp
-L power1:GND #PWR0253
+L power:GND #PWR0253
 U 1 1 5ADA1328
 P 4150 3650
@@
 $EndComp
 $Comp
-L device:R_Small R1901
+L Device:R_Small R1901
 U 1 1 5ADA14ED
 P 4150 1950
@@
 	8150 3150 8850 3150
 $Comp
-L power1:+3V3 #PWR0254
+L power:+3V3 #PWR0254
 U 1 1 5AD8CC08
 P 9750 2350
@@
 	9750 2450 9650 2450
 $Comp
-L power1:GND #PWR0255
+L power:GND #PWR0255
 U 1 1 5AD8CC90
 P 9700 3450
@@
 	9700 3350 9700 3450
 $Comp
-L power1:GND #PWR0256
+L power:GND #PWR0256
 U 1 1 5AD8CD22
 P 8750 2750
@@
 	8600 2650 8750 2650
 $Comp
-L device:R_Small R1905
+L Device:R_Small R1905
 U 1 1 5AD8CDB8
 P 9950 3150
@@
 $EndComp
 $Comp
-L power1:+3V3 #PWR0257
+L power:+3V3 #PWR0257
 U 1 1 5AD8CF57
 P 9750 3050
@@
 	9750 3150 9750 3050
 $Comp
-L device:R_Small R1904
+L Device:R_Small R1904
 U 1 1 5AD8CF83
 P 8500 2650
@@
 VCCIO
 $Comp
-L power1:+3V3 #PWR0258
+L power:+3V3 #PWR0258
 U 1 1 5AD8D3A3
 P 10650 2350
@@
 	10650 2350 10650 2450
 $Comp
-L power1:GND #PWR0259
+L power:GND #PWR0259
 U 1 1 5AD8D43B
 P 10650 2750
@@
 	10650 3050 10650 3150
 $Comp
-L power1:GND #PWR0260
+L power:GND #PWR0260
 U 1 1 5AD8D581
 P 10650 3450
@@
 Connection ~ 9750 3150
 $Comp
-L power1:GND #PWR0261
+L power:GND #PWR0261
 U 1 1 5AD8FB0C
 P 10150 3150
@@
 	3950 4750 3800 4750
 $Comp
-L power1:GND #PWR0262
+L power:GND #PWR0262
 U 1 1 5ADA9D3F
 P 4100 4700
@@
 	3950 4700 3950 4750
 $Comp
-L device:C_Small C1904
+L Device:C_Small C1904
 U 1 1 5B50328E
 P 3750 1950
@@
 $EndComp
 $Comp
-L device:C_Small C1907
+L Device:C_Small C1907
 U 1 1 5B50569A
 P 4600 2350
@@
 $EndComp
 $Comp
-L device:C_Small C1908
+L Device:C_Small C1908
 U 1 1 5B5057FF
 P 10650 2550
@@
 $EndComp
 $Comp
-L device:C_Small C1909
+L Device:C_Small C1909
 U 1 1 5B5059A3
 P 10650 3250
@@
 $EndComp
 $Comp
-L device:C_Small C1902
+L Device:C_Small C1902
 U 1 1 5B506935
 P 3450 1950
@@
 $EndComp
 $Comp
-L device:R_Small R1906
+L Device:R_Small R1906
 U 1 1 5B518666
 P 6450 3150
@@
 	6350 3150 6250 3150
 $Comp
-L device:C_Small C1906
+L Device:C_Small C1906
 U 1 1 5B522417
 P 4150 3350
@@
 $EndComp
 $Comp
-L device:C_Small C1905
+L Device:C_Small C1905
 U 1 1 5B5231A0
 P 3850 3350

Commit message: WIP: routing the HF Part of the Camera Connector. I have to move the clock away from the left border.
TODO: Fix DDR3 RAM.
Parts:
- added PO1801: POWER_OUTPUT, footprints:EMPTY, symbol fixme:POWER_OUTPUT
Connections:
- wire segments 96 -> 93
Changed lines of the file:
@@
 L power:GND #PWR0247
 U 1 1 5AD9D2C5
-P 5600 3800
-F 0 "#PWR0247" H 5600 3550 50  0001 C CNN
-F 1 "GND" H 5600 3650 50  0000 C CNN
-F 2 "" H 5600 3800 50  0001 C CNN
-F 3 "" H 5600 3800 50  0001 C CNN
-	1    5600 3800
+P 5650 3700
+F 0 "#PWR0247" H 5650 3450 50  0001 C CNN
+F 1 "GND" H 5650 3550 50  0000 C CNN
+F 2 "" H 5650 3700 50  0001 C CNN
+F 3 "" H 5650 3700 50  0001 C CNN
+	1    5650 3700
 	1    0    0    -1
 $EndComp
@@
 Connection ~ 1300 3400
 Wire Wire Line
-	5550 3600 5550 3700
-Wire Wire Line
-	5550 3700 5600 3700
-Wire Wire Line
 	5650 3700 5650 3600
-Wire Wire Line
-	5600 3800 5600 3700
-Connection ~ 5600 3700
 Wire Wire Line
 	4950 2750 4800 2750
@@
 Connection ~ 3250 2700
 Wire Wire Line
-	3250 2400 3250 1750
+	3250 2400 3250 2350
 Wire Wire Line
 	3250 1750 3450 1750
@@
 	1300 3400 1350 3400
 Wire Wire Line
-	5600 3700 5650 3700
-Wire Wire Line
 	4800 2350 4800 2000
 Wire Wire Line
@@
 Wire Wire Line
 	2000 4550 2200 4550
+$Comp
+L fixme:POWER_OUTPUT PO1801
+U 1 1 5BEDB612
+P 3150 2350
+F 0 "PO1801" H 3150 2350 50  0001 C CNN
+F 1 "POWER_OUTPUT" H 3150 2500 50  0001 C CNN
+F 2 "footprints:EMPTY" H 3150 2350 50  0001 C CNN
+F 3 "" H 3150 2350 50  0001 C CNN
+F 4 "1" H 3150 2350 50  0001 C CNN "Populated"
+F 5 "SPEC" H 3150 2350 50  0001 C CNN "Source"
+F 6 "1" H 3150 2350 50  0001 C CNN "Populate for SBGA485(Z-7030)"
+F 7 "1" H 3150 2350 50  0001 C CNN "Populate for CLG484(Z-7012s/Z-7015)"
+	1    3150 2350
+	0    -1   -1   0
+$EndComp
+Connection ~ 3250 2350
+Wire Wire Line
+	3250 2350 3250 1750
 $EndSCHEMATC

Commit message: Routed a first Version of the High Speed Part of the Camera Connector. The optional LVDS Clocks are left unconnected. I couldn't keep the Connectors Pin Assignment because it was just impossible to route.
WIP: general Routing

Fixed: DDR3 Trace Length Matching
Parts:
- removed PO1801: POWER_OUTPUT, footprints:EMPTY, symbol fixme:POWER_OUTPUT
Changed lines of the file:
@@
 $Descr A4 11693 8268
 encoding utf-8
-Sheet 18 21
+Sheet 17 21
 Title ""
 Date ""
@@
 Connection ~ 3250 2700
 Wire Wire Line
-	3250 2400 3250 2350
-Wire Wire Line
 	3250 1750 3450 1750
 Wire Wire Line
@@
 	3250 2700 3250 3250
 Wire Wire Line
-	3450 1750 3750 1750
+	3450 1750 3600 1750
 Wire Wire Line
 	3750 1750 4150 1750
@@
 Wire Wire Line
 	2000 4550 2200 4550
-$Comp
-L fixme:POWER_OUTPUT PO1801
-U 1 1 5BEDB612
-P 3150 2350
-F 0 "PO1801" H 3150 2350 50  0001 C CNN
-F 1 "POWER_OUTPUT" H 3150 2500 50  0001 C CNN
-F 2 "footprints:EMPTY" H 3150 2350 50  0001 C CNN
-F 3 "" H 3150 2350 50  0001 C CNN
-F 4 "1" H 3150 2350 50  0001 C CNN "Populated"
-F 5 "SPEC" H 3150 2350 50  0001 C CNN "Source"
-F 6 "1" H 3150 2350 50  0001 C CNN "Populate for SBGA485(Z-7030)"
-F 7 "1" H 3150 2350 50  0001 C CNN "Populate for CLG484(Z-7012s/Z-7015)"
-	1    3150 2350
-	0    -1   -1   0
-$EndComp
-Connection ~ 3250 2350
-Wire Wire Line
-	3250 2350 3250 1750
+Wire Wire Line
+	3250 1750 3250 2400
+$Comp
+L power:PWR_FLAG #FLG0111
+U 1 1 5C1EF5C0
+P 3600 1750
+F 0 "#FLG0111" H 3600 1825 50  0001 C CNN
+F 1 "PWR_FLAG" H 3600 1924 50  0000 C CNN
+F 2 "" H 3600 1750 50  0001 C CNN
+F 3 "~" H 3600 1750 50  0001 C CNN
+	1    3600 1750
+	1    0    0    -1
+$EndComp
+Connection ~ 3600 1750
+Wire Wire Line
+	3600 1750 3750 1750
 $EndSCHEMATC
