File: hardware/usb_uart.sch (KiCad schematic (older format))
At the start: 20 parts

Commit message: Removed all BSS138PS Transistors due actual unavailability.
Used lsf0102 as Levelshifter for I2C bus, connected LEDs to already existing Levelshifters.
Parts:
- U? (x2): Mouser (none) -> 595-SN74LV1T126DBVR; Populate for CLG484(Z-7012s/Z-7015) (none) -> 1; Populate for SBGA485(Z-7030) (none) -> 1
- U?: footprint (none) -> Housings_DFN_QFN:DFN-12-1EP_3x3mm_Pitch0.45mm; Populate for CLG484(Z-7012s/Z-7015) (none) -> 1; Populate for SBGA485(Z-7030) (none) -> 1
- U?: footprint (none) -> footprints:SMC_MicroDFN_1.8x2.0mm_0.4mm_Pitch; Populate for CLG484(Z-7012s/Z-7015) (none) -> 1; Populate for SBGA485(Z-7030) (none) -> 1
Changed lines of the file:
@@
 LIBS:mdr20
 LIBS:dm3cs
+LIBS:lsf0102
 LIBS:zynq_board-cache
 EELAYER 25 0
@@
 F 0 "U?" H 6350 2600 60  0000 C CNN
 F 1 "FT234XD" V 5600 3000 60  0000 C CNN
-F 2 "" H 5650 3250 60  0001 C CNN
+F 2 "Housings_DFN_QFN:DFN-12-1EP_3x3mm_Pitch0.45mm" H 5650 3250 60  0001 C CNN
 F 3 "http://www.ftdichip.com/Support/Documents/DataSheets/ICs/DS_FT234XD.pdf" H 5650 3250 60  0001 C CNN
 F 4 "FTDI, Future Technology Devices International Ltd" H 5600 2950 60  0001 C CNN "MFG Name"
@@
 F 7 "1" H 5600 2950 60  0001 C CNN "Populated"
 F 8 "SPEC" H 5600 2950 60  0001 C CNN "Source"
+F 9 "1" H 5600 2950 60  0001 C CNN "Populate for SBGA485(Z-7030)"
+F 10 "1" H 5600 2950 60  0001 C CNN "Populate for CLG484(Z-7012s/Z-7015)"
 	1    5600 2950
 	1    0    0    -1
@@
 F 5 "SN74LV1T126DBVR" H 9250 2550 60  0001 C CNN "MFG Part Num"
 F 6 "296-37174-6-ND" H 9250 2550 60  0001 C CNN "Digikey"
-F 7 "1" H 9250 2550 60  0001 C CNN "Populated"
-F 8 "SPEC" H 9250 2550 60  0001 C CNN "Source"
+F 7 "595-SN74LV1T126DBVR" H 9250 2550 60  0001 C CNN "Mouser"
+F 8 "1" H 9250 2550 60  0001 C CNN "Populated"
+F 9 "SPEC" H 9250 2550 60  0001 C CNN "Source"
+F 10 "1" H 9250 2550 60  0001 C CNN "Populate for SBGA485(Z-7030)"
+F 11 "1" H 9250 2550 60  0001 C CNN "Populate for CLG484(Z-7012s/Z-7015)"
 	1    9250 2550
 	1    0    0    -1
@@
 F 5 "SN74LV1T126DBVR" H 9250 3250 60  0001 C CNN "MFG Part Num"
 F 6 "296-37174-6-ND" H 9250 3250 60  0001 C CNN "Digikey"
-F 7 "1" H 9250 3250 60  0001 C CNN "Populated"
-F 8 "SPEC" H 9250 3250 60  0001 C CNN "Source"
+F 7 "595-SN74LV1T126DBVR" H 9250 3250 60  0001 C CNN "Mouser"
+F 8 "1" H 9250 3250 60  0001 C CNN "Populated"
+F 9 "SPEC" H 9250 3250 60  0001 C CNN "Source"
+F 10 "1" H 9250 3250 60  0001 C CNN "Populate for SBGA485(Z-7030)"
+F 11 "1" H 9250 3250 60  0001 C CNN "Populate for CLG484(Z-7012s/Z-7015)"
 	1    9250 3250
 	-1   0    0    -1
@@
 F 0 "U?" H 3000 4600 60  0000 C CNN
 F 1 "SMP1255PUTG" H 3000 4700 60  0000 C CNN
-F 2 "" H 3000 4650 60  0001 C CNN
+F 2 "footprints:SMC_MicroDFN_1.8x2.0mm_0.4mm_Pitch" H 3000 4650 60  0001 C CNN
 F 3 "http://www.smc-diodes.com/propdf/SMP1255PUTG%20N1749%20REV.A.pdf" H 3000 4650 60  0001 C CNN
 F 4 "SMC Diode Solutions" H 3000 4650 60  0001 C CNN "MFG Name"
@@
 F 7 "1" H 3000 4650 60  0001 C CNN "Populated"
 F 8 "SPEC" H 3000 4650 60  0001 C CNN "Source"
+F 9 "1" H 3000 4650 60  0001 C CNN "Populate for SBGA485(Z-7030)"
+F 10 "1" H 3000 4650 60  0001 C CNN "Populate for CLG484(Z-7012s/Z-7015)"
 	1    3000 4650
 	1    0    0    -1

Commit message: Started to route DDR3 Memory.
At first added missing Footprint for Reference- and Terminationvoltage Regulator. Added Powerplanes for GND and VCCO. Added decoupling Network to both DDR3 Memory Chips. There are more small caps, to support Memory from other Manufactors.
Parts:
- gave numbers to parts that had none: 20
Changed lines of the file:
@@
 $EndDescr
 $Comp
-L FT234XD U?
+L FT234XD U40
 U 1 1 5AD9638F
 P 5600 2950
-F 0 "U?" H 6350 2600 60  0000 C CNN
+F 0 "U40" H 6350 2600 60  0000 C CNN
 F 1 "FT234XD" V 5600 3000 60  0000 C CNN
 F 2 "Housings_DFN_QFN:DFN-12-1EP_3x3mm_Pitch0.45mm" H 5650 3250 60  0001 C CNN
@@
 PS_UART_TX
 $Comp
-L USB_OTG J?
+L USB_OTG J11
 U 1 1 5AD9C9C2
 P 1350 2900
-F 0 "J?" H 1150 3350 50  0000 L CNN
+F 0 "J11" H 1150 3350 50  0000 L CNN
 F 1 "USB_OTG" H 1150 3250 50  0000 L CNN
 F 2 "Connectors:USB_Micro-B" H 1500 2850 50  0001 C CNN
@@
 $EndComp
 $Comp
-L R_Small R?
+L R_Small R162
 U 1 1 5AD9CAF7
 P 4650 2900
-F 0 "R?" V 4700 2950 50  0000 L CNN
+F 0 "R162" V 4700 2950 50  0000 L CNN
 F 1 "27" V 4700 2750 50  0000 L CNN
 F 2 "Resistors_SMD:R_0402" H 4650 2900 50  0001 C CNN
@@
 $EndComp
 $Comp
-L R_Small R?
+L R_Small R163
 U 1 1 5AD9CB9D
 P 4650 3000
-F 0 "R?" V 4700 2850 50  0000 L CNN
+F 0 "R163" V 4700 2850 50  0000 L CNN
 F 1 "27" V 4700 3100 50  0000 L CNN
 F 2 "Resistors_SMD:R_0402" H 4650 3000 50  0001 C CNN
@@
 $EndComp
 $Comp
-L GND #PWR?
+L GND #PWR0244
 U 1 1 5AD9D27D
 P 1300 3550
-F 0 "#PWR?" H 1300 3300 50  0001 C CNN
+F 0 "#PWR0244" H 1300 3300 50  0001 C CNN
 F 1 "GND" H 1300 3400 50  0000 C CNN
 F 2 "" H 1300 3550 50  0001 C CNN
@@
 $EndComp
 $Comp
-L GND #PWR?
+L GND #PWR0245
 U 1 1 5AD9D2C5
 P 5600 3800
-F 0 "#PWR?" H 5600 3550 50  0001 C CNN
+F 0 "#PWR0245" H 5600 3550 50  0001 C CNN
 F 1 "GND" H 5600 3650 50  0000 C CNN
 F 2 "" H 5600 3800 50  0001 C CNN
@@
 $EndComp
 $Comp
-L C_Small C?
+L C_Small C249
 U 1 1 5AD9D30F
 P 4600 2350
-F 0 "C?" V 4700 2300 50  0000 L CNN
+F 0 "C249" V 4700 2300 50  0000 L CNN
 F 1 "100 nF" V 4500 2200 50  0000 L CNN
 F 2 "Capacitors_SMD:C_0402" H 4600 2350 50  0001 C CNN
@@
 $EndComp
 $Comp
-L GND #PWR?
+L GND #PWR0246
 U 1 1 5AD9D3A1
 P 4400 2350
-F 0 "#PWR?" H 4400 2100 50  0001 C CNN
+F 0 "#PWR0246" H 4400 2100 50  0001 C CNN
 F 1 "GND" H 4400 2200 50  0000 C CNN
 F 2 "" H 4400 2350 50  0001 C CNN
@@
 $EndComp
 $Comp
-L C_Small C?
+L C_Small C245
 U 1 1 5AD9E9AF
 P 3550 3350
-F 0 "C?" H 3560 3420 50  0000 L CNN
+F 0 "C245" H 3560 3420 50  0000 L CNN
 F 1 "47 pF" H 3560 3270 50  0000 L CNN
 F 2 "Capacitors_SMD:C_0402" H 3550 3350 50  0001 C CNN
@@
 $EndComp
 $Comp
-L C_Small C?
+L C_Small C247
 U 1 1 5AD9EA7E
 P 3850 3350
-F 0 "C?" H 3860 3420 50  0000 L CNN
+F 0 "C247" H 3860 3420 50  0000 L CNN
 F 1 "47 pF" H 3860 3270 50  0000 L CNN
 F 2 "Capacitors_SMD:C_0402" H 3850 3350 50  0001 C CNN
@@
 $EndComp
 $Comp
-L GND #PWR?
+L GND #PWR0247
 U 1 1 5AD9EB01
 P 3850 3650
-F 0 "#PWR?" H 3850 3400 50  0001 C CNN
+F 0 "#PWR0247" H 3850 3400 50  0001 C CNN
 F 1 "GND" H 3850 3500 50  0000 C CNN
 F 2 "" H 3850 3650 50  0001 C CNN
@@
 $EndComp
 $Comp
-L GND #PWR?
+L GND #PWR0248
 U 1 1 5AD9EB21
 P 3550 3650
-F 0 "#PWR?" H 3550 3400 50  0001 C CNN
+F 0 "#PWR0248" H 3550 3400 50  0001 C CNN
 F 1 "GND" H 3550 3500 50  0000 C CNN
 F 2 "" H 3550 3650 50  0001 C CNN
@@
 $EndComp
 $Comp
-L C_Small C?
+L C_Small C243
 U 1 1 5AD9EC24
 P 3250 3350
-F 0 "C?" H 3260 3420 50  0000 L CNN
+F 0 "C243" H 3260 3420 50  0000 L CNN
 F 1 "10 nF" H 3260 3270 50  0000 L CNN
 F 2 "Capacitors_SMD:C_0402" H 3250 3350 50  0001 C CNN
@@
 $EndComp
 $Comp
-L GND #PWR?
+L GND #PWR0249
 U 1 1 5AD9EC9D
 P 3250 3650
-F 0 "#PWR?" H 3250 3400 50  0001 C CNN
+F 0 "#PWR0249" H 3250 3400 50  0001 C CNN
 F 1 "GND" H 3250 3500 50  0000 C CNN
 F 2 "" H 3250 3650 50  0001 C CNN
@@
 $EndComp
 $Comp
-L L_Small L?
+L L_Small L5
 U 1 1 5AD9ECD6
 P 3250 2500
-F 0 "L?" H 3280 2540 50  0000 L CNN
+F 0 "L5" H 3280 2540 50  0000 L CNN
 F 1 "600R@100MHz" H 3280 2460 50  0000 L CNN
 F 2 "Inductors_SMD:L_0603" H 3250 2500 50  0001 C CNN
@@
 VBUS
 $Comp
-L C_Small C?
+L C_Small C244
 U 1 1 5ADA0DF8
 P 3450 1950
-F 0 "C?" H 3460 2020 50  0000 L CNN
+F 0 "C244" H 3460 2020 50  0000 L CNN
 F 1 "4,7 µF" H 3460 1870 50  0000 L CNN
 F 2 "Capacitors_SMD:C_0805" H 3450 1950 50  0001 C CNN
@@
 $EndComp
 $Comp
-L C_Small C?
+L C_Small C246
 U 1 1 5ADA1011
 P 3750 1950
-F 0 "C?" H 3760 2020 50  0000 L CNN
+F 0 "C246" H 3760 2020 50  0000 L CNN
 F 1 "100 nF" H 3760 1870 50  0000 L CNN
 F 2 "Capacitors_SMD:C_0402" H 3750 1950 50  0001 C CNN
@@
 $EndComp
 $Comp
-L GND #PWR?
+L GND #PWR0250
 U 1 1 5ADA11B7
 P 3600 2250
-F 0 "#PWR?" H 3600 2000 50  0001 C CNN
+F 0 "#PWR0250" H 3600 2000 50  0001 C CNN
 F 1 "GND" H 3600 2100 50  0000 C CNN
 F 2 "" H 3600 2250 50  0001 C CNN
@@
 $EndComp
 $Comp
-L C_Small C?
+L C_Small C248
 U 1 1 5ADA1247
 P 4150 3350
-F 0 "C?" H 4160 3420 50  0000 L CNN
+F 0 "C248" H 4160 3420 50  0000 L CNN
 F 1 "10 nF" H 4160 3270 50  0000 L CNN
 F 2 "Capacitors_SMD:C_0402" H 4150 3350 50  0001 C CNN
@@
 $EndComp
 $Comp
-L GND #PWR?
+L GND #PWR0251
 U 1 1 5ADA1328
 P 4150 3650
-F 0 "#PWR?" H 4150 3400 50  0001 C CNN
+F 0 "#PWR0251" H 4150 3400 50  0001 C CNN
 F 1 "GND" H 4150 3500 50  0000 C CNN
 F 2 "" H 4150 3650 50  0001 C CNN
@@
 $EndComp
 $Comp
-L R_Small R?
+L R_Small R161
 U 1 1 5ADA14ED
 P 4150 1950
-F 0 "R?" H 4180 1970 50  0000 L CNN
+F 0 "R161" H 4180 1970 50  0000 L CNN
 F 1 "10k" H 4180 1910 50  0000 L CNN
 F 2 "Resistors_SMD:R_0402" H 4150 1950 50  0001 C CNN
@@
 	6250 2700 6900 2700
 $Comp
-L SN74LV1T126 U?
+L SN74LV1T126 U41
 U 1 1 5AD8BC5F
 P 9250 2550
-F 0 "U?" H 9250 2350 60  0000 C CNN
+F 0 "U41" H 9250 2350 60  0000 C CNN
 F 1 "SN74LV1T126" H 9250 2750 60  0000 C CNN
 F 2 "TO_SOT_Packages_SMD:SOT-23-5" H 9250 2550 60  0001 C CNN
@@
 	8150 3150 8850 3150
 $Comp
-L +3V3 #PWR?
+L +3V3 #PWR0252
 U 1 1 5AD8CC08
 P 9750 2350
-F 0 "#PWR?" H 9750 2200 50  0001 C CNN
+F 0 "#PWR0252" H 9750 2200 50  0001 C CNN
 F 1 "+3V3" H 9750 2490 50  0000 C CNN
 F 2 "" H 9750 2350 50  0001 C CNN
@@
 	9750 2450 9650 2450
 $Comp
-L GND #PWR?
+L GND #PWR0253
 U 1 1 5AD8CC90
 P 9700 3450
-F 0 "#PWR?" H 9700 3200 50  0001 C CNN
+F 0 "#PWR0253" H 9700 3200 50  0001 C CNN
 F 1 "GND" H 9700 3300 50  0000 C CNN
 F 2 "" H 9700 3450 50  0001 C CNN
@@
 	9700 3350 9700 3450
 $Comp
-L GND #PWR?
+L GND #PWR0254
 U 1 1 5AD8CD22
 P 8750 2750
-F 0 "#PWR?" H 8750 2500 50  0001 C CNN
+F 0 "#PWR0254" H 8750 2500 50  0001 C CNN
 F 1 "GND" H 8750 2600 50  0000 C CNN
 F 2 "" H 8750 2750 50  0001 C CNN
@@
 	8600 2650 8850 2650
 $Comp
-L R_Small R?
+L R_Small R165
 U 1 1 5AD8CDB8
 P 9950 3150
-F 0 "R?" H 9980 3170 50  0000 L CNN
+F 0 "R165" H 9980 3170 50  0000 L CNN
 F 1 "100k" H 9980 3110 50  0000 L CNN
 F 2 "Resistors_SMD:R_0402" H 9950 3150 50  0001 C CNN
@@
 $EndComp
 $Comp
-L +3V3 #PWR?
+L +3V3 #PWR0255
 U 1 1 5AD8CF57
 P 9750 3050
-F 0 "#PWR?" H 9750 2900 50  0001 C CNN
+F 0 "#PWR0255" H 9750 2900 50  0001 C CNN
 F 1 "+3V3" H 9750 3190 50  0000 C CNN
 F 2 "" H 9750 3050 50  0001 C CNN
@@
 	9750 3150 9750 3050
 $Comp
-L R_Small R?
+L R_Small R164
 U 1 1 5AD8CF83
 P 8500 2650
-F 0 "R?" H 8530 2670 50  0000 L CNN
+F 0 "R164" H 8530 2670 50  0000 L CNN
 F 1 "100k" H 8530 2610 50  0000 L CNN
 F 2 "Resistors_SMD:R_0402" H 8500 2650 50  0001 C CNN
@@
 VCCIO
 $Comp
-L C_Small C?
+L C_Small C250
 U 1 1 5AD8D14F
 P 10650 2550
-F 0 "C?" H 10660 2620 50  0000 L CNN
+F 0 "C250" H 10660 2620 50  0000 L CNN
 F 1 "100 nF" H 10660 2470 50  0000 L CNN
 F 2 "Capacitors_SMD:C_0402" H 10650 2550 50  0001 C CNN
@@
 $EndComp
 $Comp
-L +3V3 #PWR?
+L +3V3 #PWR0256
 U 1 1 5AD8D3A3
 P 10650 2350
-F 0 "#PWR?" H 10650 2200 50  0001 C CNN
+F 0 "#PWR0256" H 10650 2200 50  0001 C CNN
 F 1 "+3V3" H 10650 2490 50  0000 C CNN
 F 2 "" H 10650 2350 50  0001 C CNN
@@
 	10650 2350 10650 2450
 $Comp
-L GND #PWR?
+L GND #PWR0257
 U 1 1 5AD8D43B
 P 10650 2750
-F 0 "#PWR?" H 10650 2500 50  0001 C CNN
+F 0 "#PWR0257" H 10650 2500 50  0001 C CNN
 F 1 "GND" H 10650 2600 50  0000 C CNN
 F 2 "" H 10650 2750 50  0001 C CNN
@@
 	10650 2750 10650 2650
 $Comp
-L C_Small C?
+L C_Small C251
 U 1 1 5AD8D574
 P 10650 3250
-F 0 "C?" H 10660 3320 50  0000 L CNN
+F 0 "C251" H 10660 3320 50  0000 L CNN
 F 1 "100 nF" H 10660 3170 50  0000 L CNN
 F 2 "Capacitors_SMD:C_0402" H 10650 3250 50  0001 C CNN
@@
 	10650 3050 10650 3150
 $Comp
-L GND #PWR?
+L GND #PWR0258
 U 1 1 5AD8D581
 P 10650 3450
-F 0 "#PWR?" H 10650 3200 50  0001 C CNN
+F 0 "#PWR0258" H 10650 3200 50  0001 C CNN
 F 1 "GND" H 10650 3300 50  0000 C CNN
 F 2 "" H 10650 3450 50  0001 C CNN
@@
 	11000 1950 7800 1950
 $Comp
-L SN74LV1T126 U?
+L SN74LV1T126 U42
 U 1 1 5AD8DFD6
 P 9250 3250
-F 0 "U?" H 9250 3050 60  0000 C CNN
+F 0 "U42" H 9250 3050 60  0000 C CNN
 F 1 "SN74LV1T126" H 9250 3450 60  0000 C CNN
 F 2 "TO_SOT_Packages_SMD:SOT-23-5" H 9250 3250 60  0001 C CNN
@@
 Connection ~ 9750 3150
 $Comp
-L GND #PWR?
+L GND #PWR0259
 U 1 1 5AD8FB0C
 P 10150 3150
-F 0 "#PWR?" H 10150 2900 50  0001 C CNN
+F 0 "#PWR0259" H 10150 2900 50  0001 C CNN
 F 1 "GND" H 10150 3000 50  0000 C CNN
 F 2 "" H 10150 3150 50  0001 C CNN
@@
 NoConn ~ 6250 3150
 $Comp
-L SMP1255PUTG U?
+L SMP1255PUTG U39
 U 1 1 5ADA96D5
 P 3000 4650
-F 0 "U?" H 3000 4600 60  0000 C CNN
+F 0 "U39" H 3000 4600 60  0000 C CNN
 F 1 "SMP1255PUTG" H 3000 4700 60  0000 C CNN
 F 2 "footprints:SMC_MicroDFN_1.8x2.0mm_0.4mm_Pitch" H 3000 4650 60  0001 C CNN
@@
 	3950 4750 3800 4750
 $Comp
-L GND #PWR?
+L GND #PWR0260
 U 1 1 5ADA9D3F
 P 4100 4700
-F 0 "#PWR?" H 4100 4450 50  0001 C CNN
+F 0 "#PWR0260" H 4100 4450 50  0001 C CNN
 F 1 "GND" H 4100 4550 50  0000 C CNN
 F 2 "" H 4100 4700 50  0001 C CNN

Commit message: Added Power/Protection Circuit
Parts:
- renumbered C243 to C1901, C244 to C1902, C245 to C1903, C246 to C1904, C247 to C1905, C248 to C1906, C249 to C1907, C250 to C1908, C251 to C1909, J11 to J1901, L5 to L1901, R161 to R1901, R162 to R1902, R163 to R1903, R164 to R1904, R165 to R1905, U39 to U1901, U40 to U1902, U41 to U1903, U42 to U1904
Changed lines of the file:
@@
 $EndDescr
 $Comp
-L FT234XD U40
+L FT234XD U1902
 U 1 1 5AD9638F
 P 5600 2950
-F 0 "U40" H 6350 2600 60  0000 C CNN
+F 0 "U1902" H 6350 2600 60  0000 C CNN
 F 1 "FT234XD" V 5600 3000 60  0000 C CNN
 F 2 "Housings_DFN_QFN:DFN-12-1EP_3x3mm_Pitch0.45mm" H 5650 3250 60  0001 C CNN
@@
 PS_UART_TX
 $Comp
-L USB_OTG J11
+L USB_OTG J1901
 U 1 1 5AD9C9C2
 P 1350 2900
-F 0 "J11" H 1150 3350 50  0000 L CNN
+F 0 "J1901" H 1150 3350 50  0000 L CNN
 F 1 "USB_OTG" H 1150 3250 50  0000 L CNN
 F 2 "Connectors:USB_Micro-B" H 1500 2850 50  0001 C CNN
@@
 $EndComp
 $Comp
-L R_Small R162
+L R_Small R1902
 U 1 1 5AD9CAF7
 P 4650 2900
-F 0 "R162" V 4700 2950 50  0000 L CNN
+F 0 "R1902" V 4700 2950 50  0000 L CNN
 F 1 "27" V 4700 2750 50  0000 L CNN
 F 2 "Resistors_SMD:R_0402" H 4650 2900 50  0001 C CNN
@@
 $EndComp
 $Comp
-L R_Small R163
+L R_Small R1903
 U 1 1 5AD9CB9D
 P 4650 3000
-F 0 "R163" V 4700 2850 50  0000 L CNN
+F 0 "R1903" V 4700 2850 50  0000 L CNN
 F 1 "27" V 4700 3100 50  0000 L CNN
 F 2 "Resistors_SMD:R_0402" H 4650 3000 50  0001 C CNN
@@
 $EndComp
 $Comp
-L C_Small C249
+L C_Small C1907
 U 1 1 5AD9D30F
 P 4600 2350
-F 0 "C249" V 4700 2300 50  0000 L CNN
+F 0 "C1907" V 4700 2300 50  0000 L CNN
 F 1 "100 nF" V 4500 2200 50  0000 L CNN
 F 2 "Capacitors_SMD:C_0402" H 4600 2350 50  0001 C CNN
@@
 $EndComp
 $Comp
-L C_Small C245
+L C_Small C1903
 U 1 1 5AD9E9AF
 P 3550 3350
-F 0 "C245" H 3560 3420 50  0000 L CNN
+F 0 "C1903" H 3560 3420 50  0000 L CNN
 F 1 "47 pF" H 3560 3270 50  0000 L CNN
 F 2 "Capacitors_SMD:C_0402" H 3550 3350 50  0001 C CNN
@@
 $EndComp
 $Comp
-L C_Small C247
+L C_Small C1905
 U 1 1 5AD9EA7E
 P 3850 3350
-F 0 "C247" H 3860 3420 50  0000 L CNN
+F 0 "C1905" H 3860 3420 50  0000 L CNN
 F 1 "47 pF" H 3860 3270 50  0000 L CNN
 F 2 "Capacitors_SMD:C_0402" H 3850 3350 50  0001 C CNN
@@
 $EndComp
 $Comp
-L C_Small C243
+L C_Small C1901
 U 1 1 5AD9EC24
 P 3250 3350
-F 0 "C243" H 3260 3420 50  0000 L CNN
+F 0 "C1901" H 3260 3420 50  0000 L CNN
 F 1 "10 nF" H 3260 3270 50  0000 L CNN
 F 2 "Capacitors_SMD:C_0402" H 3250 3350 50  0001 C CNN
@@
 $EndComp
 $Comp
-L L_Small L5
+L L_Small L1901
 U 1 1 5AD9ECD6
 P 3250 2500
-F 0 "L5" H 3280 2540 50  0000 L CNN
+F 0 "L1901" H 3280 2540 50  0000 L CNN
 F 1 "600R@100MHz" H 3280 2460 50  0000 L CNN
 F 2 "Inductors_SMD:L_0603" H 3250 2500 50  0001 C CNN
@@
 VBUS
 $Comp
-L C_Small C244
+L C_Small C1902
 U 1 1 5ADA0DF8
 P 3450 1950
-F 0 "C244" H 3460 2020 50  0000 L CNN
+F 0 "C1902" H 3460 2020 50  0000 L CNN
 F 1 "4,7 µF" H 3460 1870 50  0000 L CNN
 F 2 "Capacitors_SMD:C_0805" H 3450 1950 50  0001 C CNN
@@
 $EndComp
 $Comp
-L C_Small C246
+L C_Small C1904
 U 1 1 5ADA1011
 P 3750 1950
-F 0 "C246" H 3760 2020 50  0000 L CNN
+F 0 "C1904" H 3760 2020 50  0000 L CNN
 F 1 "100 nF" H 3760 1870 50  0000 L CNN
 F 2 "Capacitors_SMD:C_0402" H 3750 1950 50  0001 C CNN
@@
 $EndComp
 $Comp
-L C_Small C248
+L C_Small C1906
 U 1 1 5ADA1247
 P 4150 3350
-F 0 "C248" H 4160 3420 50  0000 L CNN
+F 0 "C1906" H 4160 3420 50  0000 L CNN
 F 1 "10 nF" H 4160 3270 50  0000 L CNN
 F 2 "Capacitors_SMD:C_0402" H 4150 3350 50  0001 C CNN
@@
 $EndComp
 $Comp
-L R_Small R161
+L R_Small R1901
 U 1 1 5ADA14ED
 P 4150 1950
-F 0 "R161" H 4180 1970 50  0000 L CNN
+F 0 "R1901" H 4180 1970 50  0000 L CNN
 F 1 "10k" H 4180 1910 50  0000 L CNN
 F 2 "Resistors_SMD:R_0402" H 4150 1950 50  0001 C CNN
@@
 	6250 2700 6900 2700
 $Comp
-L SN74LV1T126 U41
+L SN74LV1T126 U1903
 U 1 1 5AD8BC5F
 P 9250 2550
-F 0 "U41" H 9250 2350 60  0000 C CNN
+F 0 "U1903" H 9250 2350 60  0000 C CNN
 F 1 "SN74LV1T126" H 9250 2750 60  0000 C CNN
 F 2 "TO_SOT_Packages_SMD:SOT-23-5" H 9250 2550 60  0001 C CNN
@@
 	8600 2650 8850 2650
 $Comp
-L R_Small R165
+L R_Small R1905
 U 1 1 5AD8CDB8
 P 9950 3150
-F 0 "R165" H 9980 3170 50  0000 L CNN
+F 0 "R1905" H 9980 3170 50  0000 L CNN
 F 1 "100k" H 9980 3110 50  0000 L CNN
 F 2 "Resistors_SMD:R_0402" H 9950 3150 50  0001 C CNN
@@
 	9750 3150 9750 3050
 $Comp
-L R_Small R164
+L R_Small R1904
 U 1 1 5AD8CF83
 P 8500 2650
-F 0 "R164" H 8530 2670 50  0000 L CNN
+F 0 "R1904" H 8530 2670 50  0000 L CNN
 F 1 "100k" H 8530 2610 50  0000 L CNN
 F 2 "Resistors_SMD:R_0402" H 8500 2650 50  0001 C CNN
@@
 VCCIO
 $Comp
-L C_Small C250
+L C_Small C1908
 U 1 1 5AD8D14F
 P 10650 2550
-F 0 "C250" H 10660 2620 50  0000 L CNN
+F 0 "C1908" H 10660 2620 50  0000 L CNN
 F 1 "100 nF" H 10660 2470 50  0000 L CNN
 F 2 "Capacitors_SMD:C_0402" H 10650 2550 50  0001 C CNN
@@
 	10650 2750 10650 2650
 $Comp
-L C_Small C251
+L C_Small C1909
 U 1 1 5AD8D574
 P 10650 3250
-F 0 "C251" H 10660 3320 50  0000 L CNN
+F 0 "C1909" H 10660 3320 50  0000 L CNN
 F 1 "100 nF" H 10660 3170 50  0000 L CNN
 F 2 "Capacitors_SMD:C_0402" H 10650 3250 50  0001 C CNN
@@
 	11000 1950 7800 1950
 $Comp
-L SN74LV1T126 U42
+L SN74LV1T126 U1904
 U 1 1 5AD8DFD6
 P 9250 3250
-F 0 "U42" H 9250 3050 60  0000 C CNN
+F 0 "U1904" H 9250 3050 60  0000 C CNN
 F 1 "SN74LV1T126" H 9250 3450 60  0000 C CNN
 F 2 "TO_SOT_Packages_SMD:SOT-23-5" H 9250 3250 60  0001 C CNN
@@
 NoConn ~ 6250 3150
 $Comp
-L SMP1255PUTG U39
+L SMP1255PUTG U1901
 U 1 1 5ADA96D5
 P 3000 4650
-F 0 "U39" H 3000 4600 60  0000 C CNN
+F 0 "U1901" H 3000 4600 60  0000 C CNN
 F 1 "SMP1255PUTG" H 3000 4700 60  0000 C CNN
 F 2 "footprints:SMC_MicroDFN_1.8x2.0mm_0.4mm_Pitch" H 3000 4650 60  0001 C CNN
