File: hardware/usb_uart.sch (KiCad schematic (older format))
At the start: 20 parts, among them J1901 USB_OTG, U1901 SMP1255PUTG, U1902 FT234XD, U1903 SN74LV1T126, U1904 SN74LV1T126

Commit message: Length matched DDR3 Memory again.
Forgot to keep enough space between the traces and between the meander waves.

Also, I switched to Kicad 5.0 RC2.

Swaped a few ddr signals.
Parts:
- C1901, C1902, C1903, C1904, C1905, C1906, C1907, C1908, C1909: symbol C_Small -> device:C_Small
- J1901: symbol USB_OTG -> conn:USB_OTG
- L1901: symbol L_Small -> device:L_Small
- R1901, R1902, R1903, R1904, R1905: symbol R_Small -> device:R_Small
- U1901: symbol SMP1255PUTG -> smp1255putg:SMP1255PUTG
- U1902: symbol FT234XD -> ft234xd:FT234XD
- U1903, U1904: symbol SN74LV1T126 -> sn74lv1t126:SN74LV1T126
Changed lines of the file:
@@
-EESchema Schematic File Version 2
-LIBS:zynq_board-rescue
-LIBS:power
-LIBS:device
-LIBS:transistors
-LIBS:conn
-LIBS:linear
-LIBS:regul
-LIBS:74xx
-LIBS:cmos4000
-LIBS:adc-dac
-LIBS:memory
-LIBS:xilinx
-LIBS:microcontrollers
-LIBS:dsp
-LIBS:microchip
-LIBS:analog_switches
-LIBS:motorola
-LIBS:texas
-LIBS:intel
-LIBS:audio
-LIBS:interface
-LIBS:digital-audio
-LIBS:philips
-LIBS:display
-LIBS:cypress
-LIBS:siliconi
-LIBS:opto
-LIBS:atmel
-LIBS:contrib
-LIBS:valves
-LIBS:xilinx_zynq_clg485
-LIBS:SFP_plus
-LIBS:ael2005
-LIBS:diff_osc
-LIBS:si53340
-LIBS:usb3320
-LIBS:nx5p3090
-LIBS:smp1255putg
-LIBS:osc
-LIBS:ddr
-LIBS:misc
-LIBS:tlk10031
-LIBS:lshm-150-xxx-x-dv-a-s
-LIBS:sn74axc8t245
-LIBS:sn74lvc2t45
-LIBS:dmf05lcflp
-LIBS:bss138ps
-LIBS:max14854
-LIBS:switches
-LIBS:ft234xd
-LIBS:sn74lv1t126
-LIBS:emif06-msd02n16
-LIBS:cat24c02tdi-gt3
-LIBS:power_symbols
-LIBS:ti_power_modules
-LIBS:mdr20
-LIBS:dm3cs
-LIBS:lsf0102
-LIBS:dmp3056l
+EESchema Schematic File Version 4
 LIBS:zynq_board-cache
-EELAYER 25 0
+EELAYER 26 0
 EELAYER END
 $Descr A4 11693 8268
@@
 $EndDescr
 $Comp
-L FT234XD U1902
+L ft234xd:FT234XD U1902
 U 1 1 5AD9638F
 P 5600 2950
@@
 PS_UART_TX
 $Comp
-L USB_OTG J1901
+L conn:USB_OTG J1901
 U 1 1 5AD9C9C2
 P 1350 2900
@@
 $EndComp
 $Comp
-L R_Small R1902
+L device:R_Small R1902
 U 1 1 5AD9CAF7
 P 4650 2900
@@
 $EndComp
 $Comp
-L R_Small R1903
+L device:R_Small R1903
 U 1 1 5AD9CB9D
 P 4650 3000
@@
 $EndComp
 $Comp
-L GND #PWR0246
+L power1:GND #PWR0246
 U 1 1 5AD9D27D
 P 1300 3550
@@
 $EndComp
 $Comp
-L GND #PWR0247
+L power1:GND #PWR0247
 U 1 1 5AD9D2C5
 P 5600 3800
@@
 $EndComp
 $Comp
-L C_Small C1907
+L device:C_Small C1907
 U 1 1 5AD9D30F
 P 4600 2350
@@
 $EndComp
 $Comp
-L GND #PWR0248
+L power1:GND #PWR0248
 U 1 1 5AD9D3A1
 P 4400 2350
@@
 $EndComp
 $Comp
-L C_Small C1903
+L device:C_Small C1903
 U 1 1 5AD9E9AF
 P 3550 3350
@@
 $EndComp
 $Comp
-L C_Small C1905
+L device:C_Small C1905
 U 1 1 5AD9EA7E
 P 3850 3350
@@
 $EndComp
 $Comp
-L GND #PWR0249
+L power1:GND #PWR0249
 U 1 1 5AD9EB01
 P 3850 3650
@@
 $EndComp
 $Comp
-L GND #PWR0250
+L power1:GND #PWR0250
 U 1 1 5AD9EB21
 P 3550 3650
@@
 $EndComp
 $Comp
-L C_Small C1901
+L device:C_Small C1901
 U 1 1 5AD9EC24
 P 3250 3350
@@
 $EndComp
 $Comp
-L GND #PWR0251
+L power1:GND #PWR0251
 U 1 1 5AD9EC9D
 P 3250 3650
@@
 $EndComp
 $Comp
-L L_Small L1901
+L device:L_Small L1901
 U 1 1 5AD9ECD6
 P 3250 2500
@@
 VBUS
 $Comp
-L C_Small C1902
+L device:C_Small C1902
 U 1 1 5ADA0DF8
 P 3450 1950
@@
 $EndComp
 $Comp
-L C_Small C1904
+L device:C_Small C1904
 U 1 1 5ADA1011
 P 3750 1950
@@
 $EndComp
 $Comp
-L GND #PWR0252
+L power1:GND #PWR0252
 U 1 1 5ADA11B7
 P 3600 2250
@@
 $EndComp
 $Comp
-L C_Small C1906
+L device:C_Small C1906
 U 1 1 5ADA1247
 P 4150 3350
@@
 $EndComp
 $Comp
-L GND #PWR0253
+L power1:GND #PWR0253
 U 1 1 5ADA1328
 P 4150 3650
@@
 $EndComp
 $Comp
-L R_Small R1901
+L device:R_Small R1901
 U 1 1 5ADA14ED
 P 4150 1950
@@
 	6250 2700 6900 2700
 $Comp
-L SN74LV1T126 U1903
+L sn74lv1t126:SN74LV1T126 U1903
 U 1 1 5AD8BC5F
 P 9250 2550
@@
 	8150 3150 8850 3150
 $Comp
-L +3V3 #PWR0254
+L power1:+3V3 #PWR0254
 U 1 1 5AD8CC08
 P 9750 2350
@@
 	9750 2450 9650 2450
 $Comp
-L GND #PWR0255
+L power1:GND #PWR0255
 U 1 1 5AD8CC90
 P 9700 3450
@@
 	9700 3350 9700 3450
 $Comp
-L GND #PWR0256
+L power1:GND #PWR0256
 U 1 1 5AD8CD22
 P 8750 2750
@@
 	8600 2650 8850 2650
 $Comp
-L R_Small R1905
+L device:R_Small R1905
 U 1 1 5AD8CDB8
 P 9950 3150
@@
 $EndComp
 $Comp
-L +3V3 #PWR0257
+L power1:+3V3 #PWR0257
 U 1 1 5AD8CF57
 P 9750 3050
@@
 	9750 3150 9750 3050
 $Comp
-L R_Small R1904
+L device:R_Small R1904
 U 1 1 5AD8CF83
 P 8500 2650
@@
 VCCIO
 $Comp
-L C_Small C1908
+L device:C_Small C1908
 U 1 1 5AD8D14F
 P 10650 2550
@@
 $EndComp
 $Comp
-L +3V3 #PWR0258
+L power1:+3V3 #PWR0258
 U 1 1 5AD8D3A3
 P 10650 2350
@@
 	10650 2350 10650 2450
 $Comp
-L GND #PWR0259
+L power1:GND #PWR0259
 U 1 1 5AD8D43B
 P 10650 2750
@@
 	10650 2750 10650 2650
 $Comp
-L C_Small C1909
+L device:C_Small C1909
 U 1 1 5AD8D574
 P 10650 3250
@@
 	10650 3050 10650 3150
 $Comp
-L GND #PWR0260
+L power1:GND #PWR0260
 U 1 1 5AD8D581
 P 10650 3450
@@
 	11000 1950 7800 1950
 $Comp
-L SN74LV1T126 U1904
+L sn74lv1t126:SN74LV1T126 U1904
 U 1 1 5AD8DFD6
 P 9250 3250
@@
 Connection ~ 9750 3150
 $Comp
-L GND #PWR0261
+L power1:GND #PWR0261
 U 1 1 5AD8FB0C
 P 10150 3150
@@
 NoConn ~ 6250 3150
 $Comp
-L SMP1255PUTG U1901
+L smp1255putg:SMP1255PUTG U1901
 U 1 1 5ADA96D5
 P 3000 4650
@@
 	3950 4750 3800 4750
 $Comp
-L GND #PWR0262
+L power1:GND #PWR0262
 U 1 1 5ADA9D3F
 P 4100 4700
