File: hardware/10G_clock.sch (KiCad schematic (older format))
At the start: 12 parts

Commit message: Started to route DDR3 Memory.
At first added missing Footprint for Reference- and Terminationvoltage Regulator. Added Powerplanes for GND and VCCO. Added decoupling Network to both DDR3 Memory Chips. There are more small caps, to support Memory from other Manufactors.
Parts:
- gave numbers to parts that had none: 12
Changed lines of the file:
@@
 Clock buffer: Si53340\nDigikey: 336-2499-ND
 $Comp
-L DIFF_OSC U?
+L DIFF_OSC U15
 U 1 1 598A6684
 P 2500 2000
-F 0 "U?" H 2500 1900 60  0000 C CNN
+F 0 "U15" H 2500 1900 60  0000 C CNN
 F 1 "DIFF_OSC" H 2500 2100 60  0000 C CNN
 F 2 "footprints:VDFN_3.2x2.5mm" H 2500 2000 60  0001 C CNN
@@
 $EndComp
 $Comp
-L DIFF_OSC U?
+L DIFF_OSC U16
 U 1 1 598A6719
 P 2500 3700
-F 0 "U?" H 2500 3600 60  0000 C CNN
+F 0 "U16" H 2500 3600 60  0000 C CNN
 F 1 "DIFF_OSC" H 2500 3800 60  0000 C CNN
 F 2 "footprints:VDFN_3.2x2.5mm" H 2500 3700 60  0001 C CNN
@@
 Note: clocks are AC-coupled at receiving device.
 $Comp
-L GND #PWR?
+L GND #PWR082
 U 1 1 598A8A47
 P 1700 2300
-F 0 "#PWR?" H 1700 2050 50  0001 C CNN
+F 0 "#PWR082" H 1700 2050 50  0001 C CNN
 F 1 "GND" H 1700 2150 50  0000 C CNN
 F 2 "" H 1700 2300 50  0000 C CNN
@@
 	1700 2200 1700 2300
 $Comp
-L SI53340 U?
+L SI53340 U17
 U 1 1 598F204D
 P 4700 4300
-F 0 "U?" H 4700 4250 60  0000 C CNN
+F 0 "U17" H 4700 4250 60  0000 C CNN
 F 1 "SI53340" H 4700 4350 60  0000 C CNN
 F 2 "Housings_DFN_QFN:QFN-16-1EP_3x3mm_Pitch0.5mm_ThermalVias" H 4700 4300 60  0001 C CNN
@@
 NoConn ~ 5500 4800
 $Comp
-L C_Small C?
+L C_Small C143
 U 1 1 598F26F6
 P 3500 3900
-F 0 "C?" H 3510 3970 50  0000 L CNN
+F 0 "C143" H 3510 3970 50  0000 L CNN
 F 1 "100n" H 3510 3820 50  0000 L CNN
 F 2 "Capacitors_SMD:C_0402" H 3500 3900 50  0001 C CNN
@@
 $EndComp
 $Comp
-L C_Small C?
+L C_Small C144
 U 1 1 598F2737
 P 3500 4200
-F 0 "C?" H 3510 4270 50  0000 L CNN
+F 0 "C144" H 3510 4270 50  0000 L CNN
 F 1 "100n" H 3510 4120 50  0000 L CNN
 F 2 "Capacitors_SMD:C_0402" H 3500 4200 50  0001 C CNN
@@
 $EndComp
 $Comp
-L R R?
+L R R71
 U 1 1 598F277A
 P 3700 4050
-F 0 "R?" V 3780 4050 50  0000 C CNN
+F 0 "R71" V 3780 4050 50  0000 C CNN
 F 1 "100" V 3700 4050 50  0000 C CNN
 F 2 "Resistors_SMD:R_0402" V 3630 4050 50  0001 C CNN
@@
 Connection ~ 3700 4200
 $Comp
-L C C?
+L C C142
 U 1 1 598F29AD
 P 3350 3250
-F 0 "C?" H 3375 3350 50  0000 L CNN
+F 0 "C142" H 3375 3350 50  0000 L CNN
 F 1 "100n" H 3375 3150 50  0000 L CNN
 F 2 "Capacitors_SMD:C_0402" H 3388 3100 50  0001 C CNN
@@
 $EndComp
 $Comp
-L GND #PWR?
+L GND #PWR083
 U 1 1 598F2A12
 P 3350 3400
-F 0 "#PWR?" H 3350 3150 50  0001 C CNN
+F 0 "#PWR083" H 3350 3150 50  0001 C CNN
 F 1 "GND" H 3350 3250 50  0000 C CNN
 F 2 "" H 3350 3400 50  0000 C CNN
@@
 $EndComp
 $Comp
-L +3V3 #PWR?
+L +3V3 #PWR084
 U 1 1 598F2A6C
 P 3200 3000
-F 0 "#PWR?" H 3200 2850 50  0001 C CNN
+F 0 "#PWR084" H 3200 2850 50  0001 C CNN
 F 1 "+3V3" H 3200 3140 50  0000 C CNN
 F 2 "" H 3200 3000 50  0000 C CNN
@@
 	3300 4200 3400 4200
 $Comp
-L C C?
+L C C145
 U 1 1 598F30AD
 P 4900 3300
-F 0 "C?" H 4925 3400 50  0000 L CNN
+F 0 "C145" H 4925 3400 50  0000 L CNN
 F 1 "1u" H 4925 3200 50  0000 L CNN
 F 2 "Capacitors_SMD:C_0402" H 4938 3150 50  0001 C CNN
@@
 $EndComp
 $Comp
-L GND #PWR?
+L GND #PWR085
 U 1 1 598F3107
 P 4900 3450
-F 0 "#PWR?" H 4900 3200 50  0001 C CNN
+F 0 "#PWR085" H 4900 3200 50  0001 C CNN
 F 1 "GND" H 4900 3300 50  0000 C CNN
 F 2 "" H 4900 3450 50  0000 C CNN
@@
 $EndComp
 $Comp
-L +3V3 #PWR?
+L +3V3 #PWR086
 U 1 1 598F312D
 P 4700 3050
-F 0 "#PWR?" H 4700 2900 50  0001 C CNN
+F 0 "#PWR086" H 4700 2900 50  0001 C CNN
 F 1 "+3V3" H 4700 3190 50  0000 C CNN
 F 2 "" H 4700 3050 50  0000 C CNN
@@
 Connection ~ 4700 3150
 $Comp
-L C C?
+L C C141
 U 1 1 598F396E
 P 3350 1550
-F 0 "C?" H 3375 1650 50  0000 L CNN
+F 0 "C141" H 3375 1650 50  0000 L CNN
 F 1 "100n" H 3375 1450 50  0000 L CNN
 F 2 "Capacitors_SMD:C_0402" H 3388 1400 50  0001 C CNN
@@
 $EndComp
 $Comp
-L GND #PWR?
+L GND #PWR087
 U 1 1 598F3974
 P 3350 1700
-F 0 "#PWR?" H 3350 1450 50  0001 C CNN
+F 0 "#PWR087" H 3350 1450 50  0001 C CNN
 F 1 "GND" H 3350 1550 50  0000 C CNN
 F 2 "" H 3350 1700 50  0000 C CNN
@@
 $EndComp
 $Comp
-L +3V3 #PWR?
+L +3V3 #PWR088
 U 1 1 598F397A
 P 3200 1300
-F 0 "#PWR?" H 3200 1150 50  0001 C CNN
+F 0 "#PWR088" H 3200 1150 50  0001 C CNN
 F 1 "+3V3" H 3200 1440 50  0000 C CNN
 F 2 "" H 3200 1300 50  0000 C CNN
@@
 Connection ~ 3200 1400
 $Comp
-L GND #PWR?
+L GND #PWR089
 U 1 1 598F433B
 P 1700 4000
-F 0 "#PWR?" H 1700 3750 50  0001 C CNN
+F 0 "#PWR089" H 1700 3750 50  0001 C CNN
 F 1 "GND" H 1700 3850 50  0000 C CNN
 F 2 "" H 1700 4000 50  0000 C CNN
@@
 NoConn ~ 1800 3500
 $Comp
-L GND #PWR?
+L GND #PWR090
 U 1 1 598F54B6
 P 4800 5200
-F 0 "#PWR?" H 4800 4950 50  0001 C CNN
+F 0 "#PWR090" H 4800 4950 50  0001 C CNN
 F 1 "GND" H 4800 5050 50  0000 C CNN
 F 2 "" H 4800 5200 50  0000 C CNN
@@
 	3900 3900 3900 4100
 $Comp
-L GND #PWR?
+L GND #PWR091
 U 1 1 598F5D66
 P 2350 4400
-F 0 "#PWR?" H 2350 4150 50  0001 C CNN
+F 0 "#PWR091" H 2350 4150 50  0001 C CNN
 F 1 "GND" H 2350 4250 50  0000 C CNN
 F 2 "" H 2350 4400 50  0000 C CNN
@@
 $EndComp
 $Comp
-L +3V3 #PWR?
+L +3V3 #PWR092
 U 1 1 598F5D8C
 P 2150 4500
-F 0 "#PWR?" H 2150 4350 50  0001 C CNN
+F 0 "#PWR092" H 2150 4350 50  0001 C CNN
 F 1 "+3V3" H 2150 4640 50  0000 C CNN
 F 2 "" H 2150 4500 50  0000 C CNN
@@
 $EndComp
 $Comp
-L GND #PWR?
+L GND #PWR093
 U 1 1 598F5DE1
 P 2350 4700
-F 0 "#PWR?" H 2350 4450 50  0001 C CNN
+F 0 "#PWR093" H 2350 4450 50  0001 C CNN
 F 1 "GND" H 2350 4550 50  0000 C CNN
 F 2 "" H 2350 4700 50  0000 C CNN
@@
 $EndComp
 $Comp
-L R R?
+L R R68
 U 1 1 598F6241
 P 2500 4400
-F 0 "R?" V 2580 4400 50  0000 C CNN
+F 0 "R68" V 2580 4400 50  0000 C CNN
 F 1 "0" V 2500 4400 50  0000 C CNN
 F 2 "Resistors_SMD:R_0402" V 2430 4400 50  0001 C CNN
@@
 $EndComp
 $Comp
-L R R?
+L R R70
 U 1 1 598F6296
 P 2800 4500
-F 0 "R?" V 2880 4500 50  0000 C CNN
+F 0 "R70" V 2880 4500 50  0000 C CNN
 F 1 "0" V 2800 4500 50  0000 C CNN
 F 2 "Resistors_SMD:R_0402" V 2730 4500 50  0001 C CNN
@@
 $EndComp
 $Comp
-L R R?
+L R R69
 U 1 1 598F62E9
 P 2500 4700
-F 0 "R?" V 2580 4700 50  0000 C CNN
+F 0 "R69" V 2580 4700 50  0000 C CNN
 F 1 "0" V 2500 4700 50  0000 C CNN
 F 2 "Resistors_SMD:R_0402" V 2430 4700 50  0001 C CNN

Commit message: Added Power/Protection Circuit
Parts:
- renumbered C141 to C801, C142 to C802, C143 to C803, C144 to C804, C145 to C805, R68 to R801, R69 to R802, R70 to R803, R71 to R804, U15 to U801, U16 to U802, U17 to U803
Changed lines of the file:
@@
 Clock buffer: Si53340\nDigikey: 336-2499-ND
 $Comp
-L DIFF_OSC U15
+L DIFF_OSC U801
 U 1 1 598A6684
 P 2500 2000
-F 0 "U15" H 2500 1900 60  0000 C CNN
+F 0 "U801" H 2500 1900 60  0000 C CNN
 F 1 "DIFF_OSC" H 2500 2100 60  0000 C CNN
 F 2 "footprints:VDFN_3.2x2.5mm" H 2500 2000 60  0001 C CNN
@@
 $EndComp
 $Comp
-L DIFF_OSC U16
+L DIFF_OSC U802
 U 1 1 598A6719
 P 2500 3700
-F 0 "U16" H 2500 3600 60  0000 C CNN
+F 0 "U802" H 2500 3600 60  0000 C CNN
 F 1 "DIFF_OSC" H 2500 3800 60  0000 C CNN
 F 2 "footprints:VDFN_3.2x2.5mm" H 2500 3700 60  0001 C CNN
@@
 	1700 2200 1700 2300
 $Comp
-L SI53340 U17
+L SI53340 U803
 U 1 1 598F204D
 P 4700 4300
-F 0 "U17" H 4700 4250 60  0000 C CNN
+F 0 "U803" H 4700 4250 60  0000 C CNN
 F 1 "SI53340" H 4700 4350 60  0000 C CNN
 F 2 "Housings_DFN_QFN:QFN-16-1EP_3x3mm_Pitch0.5mm_ThermalVias" H 4700 4300 60  0001 C CNN
@@
 NoConn ~ 5500 4800
 $Comp
-L C_Small C143
+L C_Small C803
 U 1 1 598F26F6
 P 3500 3900
-F 0 "C143" H 3510 3970 50  0000 L CNN
+F 0 "C803" H 3510 3970 50  0000 L CNN
 F 1 "100n" H 3510 3820 50  0000 L CNN
 F 2 "Capacitors_SMD:C_0402" H 3500 3900 50  0001 C CNN
@@
 $EndComp
 $Comp
-L C_Small C144
+L C_Small C804
 U 1 1 598F2737
 P 3500 4200
-F 0 "C144" H 3510 4270 50  0000 L CNN
+F 0 "C804" H 3510 4270 50  0000 L CNN
 F 1 "100n" H 3510 4120 50  0000 L CNN
 F 2 "Capacitors_SMD:C_0402" H 3500 4200 50  0001 C CNN
@@
 $EndComp
 $Comp
-L R R71
+L R R804
 U 1 1 598F277A
 P 3700 4050
-F 0 "R71" V 3780 4050 50  0000 C CNN
+F 0 "R804" V 3780 4050 50  0000 C CNN
 F 1 "100" V 3700 4050 50  0000 C CNN
 F 2 "Resistors_SMD:R_0402" V 3630 4050 50  0001 C CNN
@@
 Connection ~ 3700 4200
 $Comp
-L C C142
+L C C802
 U 1 1 598F29AD
 P 3350 3250
-F 0 "C142" H 3375 3350 50  0000 L CNN
+F 0 "C802" H 3375 3350 50  0000 L CNN
 F 1 "100n" H 3375 3150 50  0000 L CNN
 F 2 "Capacitors_SMD:C_0402" H 3388 3100 50  0001 C CNN
@@
 	3300 4200 3400 4200
 $Comp
-L C C145
+L C C805
 U 1 1 598F30AD
 P 4900 3300
-F 0 "C145" H 4925 3400 50  0000 L CNN
+F 0 "C805" H 4925 3400 50  0000 L CNN
 F 1 "1u" H 4925 3200 50  0000 L CNN
 F 2 "Capacitors_SMD:C_0402" H 4938 3150 50  0001 C CNN
@@
 Connection ~ 4700 3150
 $Comp
-L C C141
+L C C801
 U 1 1 598F396E
 P 3350 1550
-F 0 "C141" H 3375 1650 50  0000 L CNN
+F 0 "C801" H 3375 1650 50  0000 L CNN
 F 1 "100n" H 3375 1450 50  0000 L CNN
 F 2 "Capacitors_SMD:C_0402" H 3388 1400 50  0001 C CNN
@@
 $EndComp
 $Comp
-L R R68
+L R R801
 U 1 1 598F6241
 P 2500 4400
-F 0 "R68" V 2580 4400 50  0000 C CNN
+F 0 "R801" V 2580 4400 50  0000 C CNN
 F 1 "0" V 2500 4400 50  0000 C CNN
 F 2 "Resistors_SMD:R_0402" V 2430 4400 50  0001 C CNN
@@
 $EndComp
 $Comp
-L R R70
+L R R803
 U 1 1 598F6296
 P 2800 4500
-F 0 "R70" V 2880 4500 50  0000 C CNN
+F 0 "R803" V 2880 4500 50  0000 C CNN
 F 1 "0" V 2800 4500 50  0000 C CNN
 F 2 "Resistors_SMD:R_0402" V 2730 4500 50  0001 C CNN
@@
 $EndComp
 $Comp
-L R R69
+L R R802
 U 1 1 598F62E9
 P 2500 4700
-F 0 "R69" V 2580 4700 50  0000 C CNN
+F 0 "R802" V 2580 4700 50  0000 C CNN
 F 1 "0" V 2500 4700 50  0000 C CNN
 F 2 "Resistors_SMD:R_0402" V 2430 4700 50  0001 C CNN

Commit message: Length matched DDR3 Memory again.
Forgot to keep enough space between the traces and between the meander waves.

Also, I switched to Kicad 5.0 RC2.

Swaped a few ddr signals.
Parts:
- C801, C802, C805: symbol C -> device:C
- C803, C804: symbol C_Small -> device:C_Small
- R801, R802, R803, R804: symbol R -> device:R
- U801, U802: symbol DIFF_OSC -> diff_osc:DIFF_OSC
- U803: symbol SI53340 -> si53340:SI53340
Changed lines of the file:
@@
-EESchema Schematic File Version 2
-LIBS:zynq_board-rescue
-LIBS:power
-LIBS:device
-LIBS:transistors
-LIBS:conn
-LIBS:linear
-LIBS:regul
-LIBS:74xx
-LIBS:cmos4000
-LIBS:adc-dac
-LIBS:memory
-LIBS:xilinx
-LIBS:microcontrollers
-LIBS:dsp
-LIBS:microchip
-LIBS:analog_switches
-LIBS:motorola
-LIBS:texas
-LIBS:intel
-LIBS:audio
-LIBS:interface
-LIBS:digital-audio
-LIBS:philips
-LIBS:display
-LIBS:cypress
-LIBS:siliconi
-LIBS:opto
-LIBS:atmel
-LIBS:contrib
-LIBS:valves
-LIBS:xilinx_zynq_clg485
-LIBS:SFP_plus
-LIBS:ael2005
-LIBS:diff_osc
-LIBS:si53340
-LIBS:usb3320
-LIBS:nx5p3090
-LIBS:smp1255putg
-LIBS:osc
-LIBS:ddr
-LIBS:misc
-LIBS:tlk10031
-LIBS:lshm-150-xxx-x-dv-a-s
-LIBS:sn74axc8t245
-LIBS:sn74lvc2t45
-LIBS:dmf05lcflp
-LIBS:bss138ps
-LIBS:max14854
-LIBS:switches
-LIBS:ft234xd
-LIBS:sn74lv1t126
-LIBS:emif06-msd02n16
-LIBS:cat24c02tdi-gt3
-LIBS:power_symbols
-LIBS:ti_power_modules
-LIBS:mdr20
-LIBS:dm3cs
-LIBS:lsf0102
-LIBS:dmp3056l
+EESchema Schematic File Version 4
 LIBS:zynq_board-cache
-EELAYER 25 0
+EELAYER 26 0
 EELAYER END
 $Descr A4 11693 8268
@@
 Clock buffer: Si53340\nDigikey: 336-2499-ND
 $Comp
-L DIFF_OSC U801
+L diff_osc:DIFF_OSC U801
 U 1 1 598A6684
 P 2500 2000
@@
 $EndComp
 $Comp
-L DIFF_OSC U802
+L diff_osc:DIFF_OSC U802
 U 1 1 598A6719
 P 2500 3700
@@
 Note: clocks are AC-coupled at receiving device.
 $Comp
-L GND #PWR084
+L power1:GND #PWR084
 U 1 1 598A8A47
 P 1700 2300
@@
 	1700 2200 1700 2300
 $Comp
-L SI53340 U803
+L si53340:SI53340 U803
 U 1 1 598F204D
 P 4700 4300
@@
 NoConn ~ 5500 4800
 $Comp
-L C_Small C803
+L device:C_Small C803
 U 1 1 598F26F6
 P 3500 3900
@@
 $EndComp
 $Comp
-L C_Small C804
+L device:C_Small C804
 U 1 1 598F2737
 P 3500 4200
@@
 $EndComp
 $Comp
-L R R804
+L device:R R804
 U 1 1 598F277A
 P 3700 4050
@@
 Connection ~ 3700 4200
 $Comp
-L C C802
+L device:C C802
 U 1 1 598F29AD
 P 3350 3250
@@
 $EndComp
 $Comp
-L GND #PWR085
+L power1:GND #PWR085
 U 1 1 598F2A12
 P 3350 3400
@@
 $EndComp
 $Comp
-L +3V3 #PWR086
+L power1:+3V3 #PWR086
 U 1 1 598F2A6C
 P 3200 3000
@@
 	3300 4200 3400 4200
 $Comp
-L C C805
+L device:C C805
 U 1 1 598F30AD
 P 4900 3300
@@
 $EndComp
 $Comp
-L GND #PWR087
+L power1:GND #PWR087
 U 1 1 598F3107
 P 4900 3450
@@
 $EndComp
 $Comp
-L +3V3 #PWR088
+L power1:+3V3 #PWR088
 U 1 1 598F312D
 P 4700 3050
@@
 Connection ~ 4700 3150
 $Comp
-L C C801
+L device:C C801
 U 1 1 598F396E
 P 3350 1550
@@
 $EndComp
 $Comp
-L GND #PWR089
+L power1:GND #PWR089
 U 1 1 598F3974
 P 3350 1700
@@
 $EndComp
 $Comp
-L +3V3 #PWR090
+L power1:+3V3 #PWR090
 U 1 1 598F397A
 P 3200 1300
@@
 Connection ~ 3200 1400
 $Comp
-L GND #PWR091
+L power1:GND #PWR091
 U 1 1 598F433B
 P 1700 4000
@@
 NoConn ~ 1800 3500
 $Comp
-L GND #PWR092
+L power1:GND #PWR092
 U 1 1 598F54B6
 P 4800 5200
@@
 	3900 3900 3900 4100
 $Comp
-L GND #PWR093
+L power1:GND #PWR093
 U 1 1 598F5D66
 P 2350 4400
@@
 $EndComp
 $Comp
-L +3V3 #PWR094
+L power1:+3V3 #PWR094
 U 1 1 598F5D8C
 P 2150 4500
@@
 $EndComp
 $Comp
-L GND #PWR095
+L power1:GND #PWR095
 U 1 1 598F5DE1
 P 2350 4700
@@
 $EndComp
 $Comp
-L R R801
+L device:R R801
 U 1 1 598F6241
 P 2500 4400
@@
 $EndComp
 $Comp
-L R R803
+L device:R R803
 U 1 1 598F6296
 P 2800 4500
@@
 $EndComp
 $Comp
-L R R802
+L device:R R802
 U 1 1 598F62E9
 P 2500 4700
