File: hardware/zynq_MGT.sch (KiCad schematic (older format))
At the start: 6 parts

Commit message: Started to route DDR3 Memory.
At first added missing Footprint for Reference- and Terminationvoltage Regulator. Added Powerplanes for GND and VCCO. Added decoupling Network to both DDR3 Memory Chips. There are more small caps, to support Memory from other Manufactors.
Parts:
- gave numbers to parts that had none: 6
Changed lines of the file:
@@
 $EndDescr
 $Comp
-L xc7z030sbg485 U?
+L xc7z030sbg485 U1
 U 5 1 596E7F00
 P 5350 2150
-F 0 "U?" H 5550 2400 60  0000 L CNN
+F 0 "U1" H 5550 2400 60  0000 L CNN
 F 1 "xc7z030sbg485" H 5550 2300 60  0000 L CNN
 F 2 "footprints:SBG485_22x22_19.0x19.0mm_Pitch0.8mm" H 5350 2150 60  0001 C CNN
@@
 MGTREFCLK_1_P
 $Comp
-L C_Small C?
+L C_Small C156
 U 1 1 598A74A2
 P 4250 2550
-F 0 "C?" H 4260 2620 50  0000 L CNN
+F 0 "C156" H 4260 2620 50  0000 L CNN
 F 1 "C_Small" H 4260 2470 50  0000 L CNN
 F 2 "Capacitors_SMD:C_0402" H 4250 2550 50  0001 C CNN
@@
 $EndComp
 $Comp
-L C_Small C?
+L C_Small C155
 U 1 1 598A7543
 P 4000 2450
-F 0 "C?" H 4010 2520 50  0000 L CNN
+F 0 "C155" H 4010 2520 50  0000 L CNN
 F 1 "C_Small" H 4010 2370 50  0000 L CNN
 F 2 "Capacitors_SMD:C_0402" H 4000 2450 50  0001 C CNN
@@
 $EndComp
 $Comp
-L C_Small C?
+L C_Small C153
 U 1 1 598A7566
 P 3500 2250
-F 0 "C?" H 3510 2320 50  0000 L CNN
+F 0 "C153" H 3510 2320 50  0000 L CNN
 F 1 "C_Small" H 3510 2170 50  0000 L CNN
 F 2 "Capacitors_SMD:C_0402" H 3500 2250 50  0001 C CNN
@@
 $EndComp
 $Comp
-L C_Small C?
+L C_Small C154
 U 1 1 598A75B1
 P 3750 2350
-F 0 "C?" H 3760 2420 50  0000 L CNN
+F 0 "C154" H 3760 2420 50  0000 L CNN
 F 1 "C_Small" H 3760 2270 50  0000 L CNN
 F 2 "Capacitors_SMD:C_0402" H 3750 2350 50  0001 C CNN
@@
 MGTX_TX_0_P
 $Comp
-L R_Small R?
+L R_Small R77
 U 1 1 5ADF6841
 P 5100 2150
-F 0 "R?" H 5130 2170 50  0000 L CNN
+F 0 "R77" H 5130 2170 50  0000 L CNN
 F 1 "100Ω, 1%" V 5000 1950 50  0000 L CNN
 F 2 "" H 5100 2150 50  0001 C CNN
@@
 Traces to MGTREF and MGTAVTTRCAL\nhave to be the same length / geometry! \nSee UG476 Figure 5-3.
 $Comp
-L +1V2_MGT #PWR?
+L +1V2_MGT #PWR0117
 U 1 1 5ADF709F
 P 5300 1950
-F 0 "#PWR?" H 5300 1800 50  0001 C CNN
+F 0 "#PWR0117" H 5300 1800 50  0001 C CNN
 F 1 "+1V2_MGT" H 5300 2090 50  0000 C CNN
 F 2 "" H 5300 1950 50  0001 C CNN

Commit message: Added Power/Protection Circuit
Parts:
- renumbered C153 to C1001, C154 to C1002, C155 to C1003, C156 to C1004, R77 to R1001, U1 to U201
Changed lines of the file:
@@
 $EndDescr
 $Comp
-L xc7z030sbg485 U1
+L xc7z030sbg485 U201
 U 5 1 596E7F00
 P 5350 2150
-F 0 "U1" H 5550 2400 60  0000 L CNN
+F 0 "U201" H 5550 2400 60  0000 L CNN
 F 1 "xc7z030sbg485" H 5550 2300 60  0000 L CNN
 F 2 "footprints:SBG485_22x22_19.0x19.0mm_Pitch0.8mm" H 5350 2150 60  0001 C CNN
@@
 MGTREFCLK_1_P
 $Comp
-L C_Small C156
+L C_Small C1004
 U 1 1 598A74A2
 P 4250 2550
-F 0 "C156" H 4260 2620 50  0000 L CNN
+F 0 "C1004" H 4260 2620 50  0000 L CNN
 F 1 "C_Small" H 4260 2470 50  0000 L CNN
 F 2 "Capacitors_SMD:C_0402" H 4250 2550 50  0001 C CNN
@@
 $EndComp
 $Comp
-L C_Small C155
+L C_Small C1003
 U 1 1 598A7543
 P 4000 2450
-F 0 "C155" H 4010 2520 50  0000 L CNN
+F 0 "C1003" H 4010 2520 50  0000 L CNN
 F 1 "C_Small" H 4010 2370 50  0000 L CNN
 F 2 "Capacitors_SMD:C_0402" H 4000 2450 50  0001 C CNN
@@
 $EndComp
 $Comp
-L C_Small C153
+L C_Small C1001
 U 1 1 598A7566
 P 3500 2250
-F 0 "C153" H 3510 2320 50  0000 L CNN
+F 0 "C1001" H 3510 2320 50  0000 L CNN
 F 1 "C_Small" H 3510 2170 50  0000 L CNN
 F 2 "Capacitors_SMD:C_0402" H 3500 2250 50  0001 C CNN
@@
 $EndComp
 $Comp
-L C_Small C154
+L C_Small C1002
 U 1 1 598A75B1
 P 3750 2350
-F 0 "C154" H 3760 2420 50  0000 L CNN
+F 0 "C1002" H 3760 2420 50  0000 L CNN
 F 1 "C_Small" H 3760 2270 50  0000 L CNN
 F 2 "Capacitors_SMD:C_0402" H 3750 2350 50  0001 C CNN
@@
 MGTX_TX_0_P
 $Comp
-L R_Small R77
+L R_Small R1001
 U 1 1 5ADF6841
 P 5100 2150
-F 0 "R77" H 5130 2170 50  0000 L CNN
+F 0 "R1001" H 5130 2170 50  0000 L CNN
 F 1 "100Ω, 1%" V 5000 1950 50  0000 L CNN
 F 2 "" H 5100 2150 50  0001 C CNN

Commit message: Length matched DDR3 Memory again.
Forgot to keep enough space between the traces and between the meander waves.

Also, I switched to Kicad 5.0 RC2.

Swaped a few ddr signals.
Parts:
- C1001, C1002, C1003, C1004: symbol C_Small -> device:C_Small
- R1001: symbol R_Small -> device:R_Small
- U201: symbol xc7z030sbg485 -> xilinx_zynq_clg485:xc7z030sbg485
Changed lines of the file:
@@
-EESchema Schematic File Version 2
-LIBS:zynq_board-rescue
-LIBS:power
-LIBS:device
-LIBS:transistors
-LIBS:conn
-LIBS:linear
-LIBS:regul
-LIBS:74xx
-LIBS:cmos4000
-LIBS:adc-dac
-LIBS:memory
-LIBS:xilinx
-LIBS:microcontrollers
-LIBS:dsp
-LIBS:microchip
-LIBS:analog_switches
-LIBS:motorola
-LIBS:texas
-LIBS:intel
-LIBS:audio
-LIBS:interface
-LIBS:digital-audio
-LIBS:philips
-LIBS:display
-LIBS:cypress
-LIBS:siliconi
-LIBS:opto
-LIBS:atmel
-LIBS:contrib
-LIBS:valves
-LIBS:xilinx_zynq_clg485
-LIBS:SFP_plus
-LIBS:ael2005
-LIBS:diff_osc
-LIBS:si53340
-LIBS:usb3320
-LIBS:nx5p3090
-LIBS:smp1255putg
-LIBS:osc
-LIBS:ddr
-LIBS:misc
-LIBS:tlk10031
-LIBS:lshm-150-xxx-x-dv-a-s
-LIBS:sn74axc8t245
-LIBS:sn74lvc2t45
-LIBS:dmf05lcflp
-LIBS:bss138ps
-LIBS:max14854
-LIBS:switches
-LIBS:ft234xd
-LIBS:sn74lv1t126
-LIBS:emif06-msd02n16
-LIBS:cat24c02tdi-gt3
-LIBS:power_symbols
-LIBS:ti_power_modules
-LIBS:mdr20
-LIBS:dm3cs
-LIBS:lsf0102
-LIBS:dmp3056l
+EESchema Schematic File Version 4
 LIBS:zynq_board-cache
-EELAYER 25 0
+EELAYER 26 0
 EELAYER END
 $Descr A4 11693 8268
@@
 $EndDescr
 $Comp
-L xc7z030sbg485 U201
+L xilinx_zynq_clg485:xc7z030sbg485 U201
 U 5 1 596E7F00
 P 5350 2150
@@
 MGTREFCLK_1_P
 $Comp
-L C_Small C1004
+L device:C_Small C1004
 U 1 1 598A74A2
 P 4250 2550
@@
 $EndComp
 $Comp
-L C_Small C1003
+L device:C_Small C1003
 U 1 1 598A7543
 P 4000 2450
@@
 $EndComp
 $Comp
-L C_Small C1001
+L device:C_Small C1001
 U 1 1 598A7566
 P 3500 2250
@@
 $EndComp
 $Comp
-L C_Small C1002
+L device:C_Small C1002
 U 1 1 598A75B1
 P 3750 2350
@@
 MGTX_TX_0_P
 $Comp
-L R_Small R1001
+L device:R_Small R1001
 U 1 1 5ADF6841
 P 5100 2150
@@
 Traces to MGTREF and MGTAVTTRCAL\nhave to be the same length / geometry! \nSee UG476 Figure 5-3.
 $Comp
-L +1V2_MGT #PWR0119
+L power_symbols:+1V2_MGT #PWR0119
 U 1 1 5ADF709F
 P 5300 1950
